Commit message: [UPD] platform parent

File: sobit_home_description/urdf/base/base.urdf.xacro (robot description, xacro)
@@ -7,5 +7,5 @@
       <parent link="base_footprint" />
       <child link="base_link" />
-      <origin xyz="0 0 0.07555856" rpy="0.0 0.0 0.0" />
+      <origin xyz="0 0 0.0" rpy="0.0 0.0 0.0" />
     </joint>
     <link name="base_link" />
