Commit message: [UPD] prefix for transmissions

File: sobit_home_description/urdf/body/body.transmission.xacro (robot description, xacro)
@@ -1,7 +1,7 @@
-<?xml version="1.0" ?>
+<?xml version="1.0" encoding="UTF-8" ?>
 <robot name="sobit_home"
        xmlns:xacro="http://ros.org/wiki/xacro">
-  <xacro:macro name="body_transmission">
-    <xacro:position_joint_transmission joint="linear_actuator_joint" reduction="1" />
+  <xacro:macro name="body_transmission" params="prefix" >
+    <xacro:SimpleTransmissionPosition joint="${prefix}_lift_joint" reduction="1" />
   </xacro:macro>
 </robot>
