Commit message: [UPD] platform parent

File: sobit_home_description/urdf/body/plate.urdf.xacro (robot description, xacro)
@@ -4,6 +4,6 @@
   <xacro:macro name="plate" params="prefix parent">
     <joint name="${prefix}_bottom_joint" type="fixed">
-      <origin xyz="0 0 0.0225" rpy="0.0 0.0 0.0" />
-      <parent link="${parent}" />
+      <origin xyz="0 0 -0.11" rpy="0.0 0.0 0.0" />
+      <parent link="${prefix}_middle_link" />
       <child link="${prefix}_bottom_link" />
     </joint>
@@ -31,6 +31,6 @@
     </link>
     <joint name="${prefix}_middle_joint" type="fixed">
-      <origin xyz="0.0 0.0 0.1" rpy="0.0 0.0 0.0" />
-      <parent link="${prefix}_bottom_link" />
+      <origin xyz="0.0 0.0 0.271358" rpy="0.0 0.0 0.0" />
+      <parent link="${parent}" />
       <child link="${prefix}_middle_link" />
     </joint>
@@ -58,5 +58,5 @@
     </link>
     <joint name="${prefix}_top_joint" type="fixed">
-      <origin xyz="0.0 0.0 0.03985" rpy="0.0 0.0 0.0" />
+      <origin xyz="0.0 0.0 0.0997" rpy="0.0 0.0 0.0" />
       <parent link="${prefix}_middle_link" />
       <child link="${prefix}_top_link" />

Commit message: [UPD] wheel_base

File: sobit_home_description/urdf/body/plate.urdf.xacro (robot description, xacro)
@@ -58,5 +58,5 @@
     </link>
     <joint name="${prefix}_top_joint" type="fixed">
-      <origin xyz="0.0 0.0 0.0997" rpy="0.0 0.0 0.0" />
+      <origin xyz="0.0 0.0 0.1097" rpy="0.0 0.0 0.0" />
       <parent link="${prefix}_middle_link" />
       <child link="${prefix}_top_link" />

Commit message: [ADD] mobile base cover, [TODO] add colission and inertia

File: sobit_home_description/urdf/body/plate.urdf.xacro (robot description, xacro)
@@ -84,4 +84,32 @@
       </inertial>
     </link>
+    <joint name="${prefix}_cover_joint" type="fixed">
+      <origin xyz="0.0 0.0 ${0.421258 + 0.15/2}" rpy="0.0 0.0 0.0" />
+      <parent link="base_footprint" />
+      <child link="${prefix}_cover_link" />
+    </joint>
+    <link name="${prefix}_cover_link">
+      <visual>
+        <origin xyz="0.0 0.0 0.0" rpy="0.0 0.0 ${M_PI/2.0}" />
+        <geometry>
+          <mesh filename="file://$(find sobit_home_description)/meshes/body/mobile_platform_cover.stl" scale="0.001 0.001 0.001" />
+        </geometry>
+        <material name="black" />
+      </visual>
+      <!-- TODO -->
+      <!-- <collision>
+        <origin xyz="0.0 0.0 0.0" rpy="0.0 0.0 0.0" />
+        <geometry>
+          <box size="0.47 0.47 0.02" />
+        </geometry>
+      </collision> -->
+      <!-- <inertial>
+        <origin xyz="0.0 0.0 0.0" rpy="0.0 0.0 0.0" />
+        <mass value="1.5" />
+        <inertia ixx="${1/12*1.5*(0.47**2+0.02**2)}" ixy="0.0" ixz="0.0"
+                 iyy="${1/12*1.5*(0.02**2+0.47**2)}" iyz="0.0"
+                 izz="${1/12*1.5*(0.47**2+0.47**2)}" />
+      </inertial> -->
+    </link>
   </xacro:macro>
 </robot>

Commit message: [ADD] mobile base cover collisions

File: sobit_home_description/urdf/body/plate.urdf.xacro (robot description, xacro)
@@ -97,18 +97,46 @@
         <material name="black" />
       </visual>
-      <!-- TODO -->
-      <!-- <collision>
+      <!-- top -->
+      <collision>
         <origin xyz="0.0 0.0 0.0" rpy="0.0 0.0 0.0" />
         <geometry>
-          <box size="0.47 0.47 0.02" />
+          <box size="0.575 0.575 0.01" />
         </geometry>
-      </collision> -->
-      <!-- <inertial>
-        <origin xyz="0.0 0.0 0.0" rpy="0.0 0.0 0.0" />
+      </collision>
+      <!-- front -->
+      <collision>
+        <origin xyz="${0.575/2 - 0.01/2} 0.0 ${-0.470/2}" rpy="0.0 0.0 0.0" />
+        <geometry>
+          <box size="0.01 0.575 0.470" />
+        </geometry>
+      </collision>
+      <!-- back -->
+      <collision>
+        <origin xyz="${-(0.575/2 - 0.01/2)} 0.0 ${-0.470/2}" rpy="0.0 0.0 0.0" />
+        <geometry>
+          <box size="0.01 0.575 0.470" />
+        </geometry>
+      </collision>
+      <!-- left -->
+      <collision>
+        <origin xyz="0.0 ${0.575/2 - 0.01/2} ${-0.470/2}" rpy="0.0 0.0 0.0" />
+        <geometry>
+          <box size="0.575 0.01 0.470" />
+        </geometry>
+      </collision>
+      <!-- right -->
+      <collision>
+        <origin xyz="0.0 ${-(0.575/2 - 0.01/2)} ${-0.470/2}" rpy="0.0 0.0 0.0" />
+        <geometry>
+          <box size="0.575 0.01 0.470" />
+        </geometry>
+      </collision>
+      <inertial>
+        <origin xyz="0.0 0.0 ${0.150/2 - 0.0485 - (0.421258 + 0.150/2)/2}" rpy="0.0 0.0 0.0" />
         <mass value="1.5" />
-        <inertia ixx="${1/12*1.5*(0.47**2+0.02**2)}" ixy="0.0" ixz="0.0"
-                 iyy="${1/12*1.5*(0.02**2+0.47**2)}" iyz="0.0"
-                 izz="${1/12*1.5*(0.47**2+0.47**2)}" />
-      </inertial> -->
+        <inertia ixx="${1/12*1.5*(0.575**2+0.470**2)}" ixy="0.0" ixz="0.0"
+                 iyy="${1/12*1.5*(0.470**2+0.575**2)}" iyz="0.0"
+                 izz="${1/12*1.5*(0.575**2+0.575**2)}" />
+      </inertial>
     </link>
   </xacro:macro>
