Commit message: [FIX] yaw of body_link

File: sobit_home_description/urdf/body/body.urdf.xacro (robot description, xacro)
@@ -4,5 +4,5 @@
   <xacro:macro name="body" params="prefix parent" >
     <joint name="${prefix}_joint" type="fixed" >
-      <origin xyz="0.0 0.0 0.0" rpy="0.0 0.0 0.0" />
+      <origin xyz="0.0 0.0 0.565" rpy="0.0 0.0 0.0" />
       <parent link="${parent}" />
       <child link="${prefix}_link" />
@@ -10,5 +10,5 @@
     <link name="${prefix}_link" >
       <visual>
-        <origin xyz="0.0 0.0 0.565" rpy="0.0 0.0 ${M_PI}" />
+        <origin xyz="0.0 0.0 0.0" rpy="0.0 0.0 ${M_PI/2}" />
         <geometry>
           <mesh filename="file://$(find sobit_home_description)/meshes/body/linear_actuator.stl" scale="0.001 0.001 0.001" />

Commit message: [UPD] add linear_actuator

File: sobit_home_description/urdf/body/body.urdf.xacro (robot description, xacro)
@@ -2,11 +2,41 @@
 <robot name="sobit_home"
        xmlns:xacro="http://ros.org/wiki/xacro" >
+  <xacro:include filename="$(find sobit_home_description)/urdf/body/body.transmission.xacro" />
   <xacro:macro name="body" params="prefix parent" >
     <joint name="${prefix}_joint" type="fixed" >
-      <origin xyz="0.0 0.0 0.565" rpy="0.0 0.0 0.0" />
+      <origin xyz="0.0 0.0 0.565" rpy="0.0 0.0 0.0" /> <!-- TODO: height -->
       <parent link="${parent}" />
       <child link="${prefix}_link" />
     </joint>
     <link name="${prefix}_link" >
+      <visual>
+        <origin xyz="0.0 0.0 0.0" rpy="0.0 0.0 ${M_PI/2}" />
+        <geometry>
+          <mesh filename="file://$(find sobit_home_description)/meshes/body/body.stl" scale="0.001 0.001 0.001" />
+        </geometry>
+        <material name="grey" />
+      </visual>
+      <collision>
+        <origin xyz="-${0.02893+0.3/2} 0.0 ${0.034-0.489/2}" rpy="0.0 0.0 0.0" />
+        <geometry>
+          <box size="${(0.02893+0.3/2)*2} 0.3965 0.489"/>
+        </geometry>
+      </collision>
+      <inertial>
+        <origin xyz="-${0.02893+0.3/2} 0.0 ${0.034-0.489/2}" rpy="0.0 0.0 0.0" />
+        <mass value="0.732" />
+        <inertia ixx="${1/12*0.732*(((0.02893+0.3/2)*2)**2+0.489**2)}"  ixy="0.0" ixz="0.0"
+                 iyy="${1/12*0.732*(0.3965**2+0.489**2)}"               iyz="0.0"
+                 izz="${1/12*0.732*(((0.02893+0.3/2)*2)**2+0.3965**2)}" />
+      </inertial>
+    </link>
+    <joint name="linear_actuator_joint" type="prismatic" >
+      <origin xyz="0.0961 0.0425 0.0" rpy="0.0 0.0 0.0" />
+      <parent link="${prefix}_link" />
+      <child link="linear_actuator_link" />
+      <axis xyz="0.0 0.0 1.0" />
+      <limit lower="0.0" upper="0.3" effort="50.0" velocity="0.1" /> <!-- TODO: limit -->
+    </joint>
+    <link name="linear_actuator_link" >
       <visual>
         <origin xyz="0.0 0.0 0.0" rpy="0.0 0.0 ${M_PI/2}" />
@@ -30,4 +60,5 @@
       </inertial>
     </link>
+    <xacro:body_transmission />
   </xacro:macro>
 </robot>

Commit message: [UPD] joint name, prefix

File: sobit_home_description/urdf/body/body.urdf.xacro (robot description, xacro)
@@ -31,12 +31,12 @@
       </inertial>
     </link>
-    <joint name="linear_actuator_joint" type="prismatic" >
+    <joint name="${prefix}_lift_joint" type="prismatic" >
       <origin xyz="0.11275 0.0 0.0" rpy="0.0 0.0 0.0" />
       <parent link="${prefix}_link" />
-      <child link="linear_actuator_link" />
+      <child link="${prefix}_lift_link" />
       <axis xyz="0.0 0.0 1.0" />
       <limit lower="-0.4" upper="0.4" effort="150.0" velocity="0.1" />
     </joint>
-    <link name="linear_actuator_link" >
+    <link name="${prefix}_lift_link" >
       <visual>
         <origin xyz="0.0 0.0 0.0" rpy="0.0 0.0 ${M_PI/2}" />
@@ -60,5 +60,5 @@
       </inertial>
     </link>
-    <xacro:body_transmission />
+    <xacro:body_transmission prefix="${prefix}" />
   </xacro:macro>
 </robot>

Commit message: [UPD] collision of body_link

File: sobit_home_description/urdf/body/body.urdf.xacro (robot description, xacro)
@@ -18,7 +18,7 @@
       </visual>
       <collision>
-        <origin xyz="0.0 -0.053 -0.018" rpy="0.0 0.0 0.0" />
+        <origin xyz="0.0 0.00425 -0.018" rpy="0.0 0.0 0.0" />
         <geometry>
-          <box size="0.0675 0.19 1.07"/>
+          <box size="0.0675 0.085 1.07"/>
         </geometry>
       </collision>

Commit message: [UPD] effort_ratio

File: sobit_home_description/urdf/body/body.urdf.xacro (robot description, xacro)
@@ -36,5 +36,5 @@
       <child link="${prefix}_lift_link" />
       <axis xyz="0.0 0.0 1.0" />
-      <limit lower="-0.4" upper="0.4" effort="150000.0" velocity="0.85" />
+      <limit lower="-0.4" upper="0.4" effort="${150.0 * effort_ratio}" velocity="0.85" />
     </joint>
     <link name="${prefix}_lift_link" >

File: sobit_home_description/urdf/values.urdf.xacro (robot description, xacro)
@@ -3,3 +3,4 @@
        xmlns:xacro="http://www.ros.org/wiki.xacro">
   <xacro:property name="M_PI" value="3.14159265359" />
+  <xacro:property name="effort_ratio" value="100.0" />
 </robot>

Commit message: [UPD] body & linear_actuator

File: sobit_home_description/urdf/body/body.urdf.xacro (robot description, xacro)
@@ -5,5 +5,5 @@
   <xacro:macro name="body" params="prefix parent" >
     <joint name="${prefix}_joint" type="fixed" >
-      <origin xyz="0.0 0.0 0.565" rpy="0.0 0.0 0.0" />
+      <origin xyz="-0.1702 0.0 0.54303" rpy="0.0 0.0 0.0" />
       <parent link="${parent}" />
       <child link="${prefix}_link" />
@@ -11,5 +11,5 @@
     <link name="${prefix}_link" >
       <visual>
-        <origin xyz="0.0 0.0 0.0" rpy="0.0 0.0 ${M_PI/2}" />
+        <origin xyz="0.0152 0.0 -0.53303" rpy="0.0 0.0 ${M_PI/2}" />
         <geometry>
           <mesh filename="file://$(find sobit_home_description)/meshes/body/body.stl" scale="0.001 0.001 0.001" />
@@ -20,5 +20,5 @@
         <origin xyz="0.0 0.00425 -0.018" rpy="0.0 0.0 0.0" />
         <geometry>
-          <box size="0.0675 0.085 1.07"/>
+          <box size="0.13 0.13 1.05"/>
         </geometry>
       </collision>
@@ -32,9 +32,9 @@
     </link>
     <joint name="${prefix}_lift_joint" type="prismatic" >
-      <origin xyz="0.11275 0.0 0.0" rpy="0.0 0.0 0.0" />
+      <origin xyz="0.0 0.0 -0.22613" rpy="0.0 0.0 0.0" />
       <parent link="${prefix}_link" />
       <child link="${prefix}_lift_link" />
       <axis xyz="0.0 0.0 1.0" />
-      <limit lower="-0.4" upper="0.4" effort="150000.0" velocity="0.85" />
+      <limit lower="0" upper="0.69" effort="${150.0 * effort_ratio}" velocity="0.85" />
     </joint>
     <link name="${prefix}_lift_link" >
@@ -47,5 +47,5 @@
       </visual>
       <collision>
-        <origin xyz="0.0 0.0 0.0" rpy="0.0 0.0 0.0" />
+        <origin xyz="0.178 0.0 0.0" rpy="0.0 0.0 0.0" />
         <geometry>
           <box size="0.15 0.35 0.15"/>

File: sobit_home_description/urdf/head/head.urdf.xacro (robot description, xacro)
@@ -7,5 +7,5 @@
       <parent link="${parent}" />
       <child link="${prefix}_base_link" />
-      <origin xyz="0.015 0.0 0.085" rpy="0.0 0.0 0.0" />
+      <origin xyz="0.193 0.0 0.085" rpy="0.0 0.0 0.0" />
     </joint>
     <link name="${prefix}_base_link">

Commit message: [ADD]Upper body cover URDF

File: sobit_home_description/urdf/body/body.urdf.xacro (robot description, xacro)
@@ -46,4 +46,11 @@
         <material name="grey" />
       </visual>
+      <visual>
+        <origin xyz="0.178 0.0 0.0" rpy="0.0 0.0 ${M_PI/2}" />
+        <geometry>
+          <mesh filename="file://$(find sobit_home_description)/meshes/body/body_cover.dae"/>
+        </geometry>
+        <!-- <material name="grey" /> -->
+      </visual>
       <collision>
         <origin xyz="0.178 0.0 0.0" rpy="0.0 0.0 0.0" />

Commit message: [FIX] effor vel values

File: sobit_home_description/urdf/body/body.urdf.xacro (robot description, xacro)
@@ -36,5 +36,5 @@
       <child link="${prefix}_lift_link" />
       <axis xyz="0.0 0.0 1.0" />
-      <limit lower="0" upper="0.69" effort="${150.0 * effort_ratio}" velocity="0.85" />
+      <limit lower="0" upper="0.69" effort="${6.5 * effort_ratio}" velocity="0.5" />
     </joint>
     <link name="${prefix}_lift_link" >

File: sobit_home_description/urdf/wheel/wheel.urdf.xacro (robot description, xacro)
@@ -38,5 +38,5 @@
       <child link="wheel_steer_${id}_link" />
       <axis xyz="0.0 0.0 1.0 " />
-      <limit effort="10.0" velocity="4.817109" />
+      <limit effort="${10.6 * effort_ratio}" velocity="3.14" />
       <!-- <dynamics damping="0.2" friction="0" /> -->
     </joint>
@@ -70,5 +70,5 @@
       <child link="wheel_drive_${id}_link" />
       <axis xyz="0.0 1.0 0.0 " />
-      <limit effort="10.0" velocity="30.0" />
+      <limit effort="${4.5 * effort_ratio}" velocity="50.5" />
     </joint>
     <link name="wheel_drive_${id}_link">

Commit message: [UPD] linear guide with cover (stl), dae is not supported

File: sobit_home_description/urdf/body/body.urdf.xacro (robot description, xacro)
@@ -13,7 +13,9 @@
         <origin xyz="0.0152 0.0 -0.53303" rpy="0.0 0.0 ${M_PI/2}" />
         <geometry>
-          <mesh filename="file://$(find sobit_home_description)/meshes/body/body.stl" scale="0.001 0.001 0.001" />
+          <!-- <mesh filename="file://$(find sobit_home_description)/meshes/body/lift.stl" scale="0.001 0.001 0.001" /> -->
+          <mesh filename="file://$(find sobit_home_description)/meshes/body/lift_w_cover.stl" />
+          <!-- <mesh filename="file://$(find sobit_home_description)/meshes/body/lift_w_cover.dae" /> -->
         </geometry>
-        <material name="grey" />
+        <material name="black" />
       </visual>
       <collision>
