Commit message: [UPD] prefix for transmissions, simplify urdf (todo)

File: sobit_home_description/urdf/hand/hand.urdf.xacro (robot description, xacro)
@@ -3,11 +3,11 @@
        xmlns:xacro="http://ros.org/wiki/xacro" >
   <xacro:include filename="$(find sobit_home_description)/urdf/hand/hand.transmission.xacro" />
-  <xacro:macro name="hand" params="prefix_hand prefix_finger parent">
-    <joint name="${prefix_hand}_base_joint" type="fixed">
+  <xacro:macro name="hand" params="prefix_hand position prefix_finger parent">
+    <joint name="${prefix_hand}_${position}_base_joint" type="fixed">
       <parent link="${parent}" />
       <child link="${prefix_hand}_base_link" />
       <origin xyz="0.0 0.0 0.0" rpy="0.0 0.0 0.0" />
     </joint>
-    <link name="${prefix_hand}_base_link">
+    <link name="${prefix_hand}_${position}_base_link">
       <visual>
         <origin xyz="0.0 0.0 0.0" rpy="${M_PI/2.0} 0.0 ${M_PI/2.0}" />
@@ -31,179 +31,5 @@
       </inertial>
     </link>
-    <joint name="${prefix_hand}_inner_l_joint" type="continuous">
-      <parent link="${prefix_hand}_base_link" />
-      <child link="${prefix_hand}_inner_l_link" />
-      <origin xyz="0.0631932 0.0151495 0.0372231" rpy="0.0 0.0 0.0" />
-      <axis xyz="0.0 0.0 1.0" />
-      <mimic joint="${prefix_hand}_joint" multiplier="-1.0" offset="0" />
-    </joint>
-    <link name="${prefix_hand}_inner_l_link">
-      <visual>
-        <origin xyz="0.0 0.0 0.0" rpy="0.0 0.0 ${M_PI/2.0}" />
-        <geometry>
-          <mesh filename="file://$(find sobit_home_description)/meshes/hand/hand_inner_l.stl" scale="0.001 0.001 0.001" />
-        </geometry>
-        <material name="black" />
-      </visual>
-      <collision>
-        <origin xyz="${0.05408+(0.06006-0.00707)/2} 0.0 -${0.066/2}" rpy="0.0 0.0 0.0" />
-        <geometry>
-          <box size="${0.06006-0.0071} 0.01 0.066" />
-        </geometry>
-      </collision>
-      <inertial>
-        <origin xyz="${0.05408+(0.06006-0.00707)/2} 0.0 -${0.066/2}" rpy="0.0 0.0 ${M_PI/2}" />
-        <mass value="0.08" />
-        <inertia ixx="${1/12*0.08*((0.06006-0.0071)**2+0.066**2)}" ixy="0.0" ixz="0.0"
-                 iyy="${1/12*0.08*(0.01**2+0.066**2)}"             iyz="0.0"
-                 izz="${1/12*0.08*((0.06006-0.0071)**2+0.01**2)}" />
-      </inertial>
-    </link>
-    <joint name="${prefix_hand}_joint" type="revolute">
-      <parent link="${prefix_hand}_base_link" />
-      <child link="${prefix_hand}_link" />
-      <origin xyz="0.0631932 -0.0151495 0.0372231" rpy="0.0 0.0 0.0" />
-      <axis xyz="0.0 0.0 1.0" />
-      <limit lower="${-M_PI/2.0}" upper="0" effort="4.1" velocity="4.796165" />
-    </joint>
-    <link name="${prefix_hand}_link">
-      <visual>
-        <origin xyz="0.0 0.0 0.0" rpy="0.0 0.0 ${M_PI/2.0}" />
-        <geometry>
-          <mesh filename="file://$(find sobit_home_description)/meshes/hand/hand_inner_r.stl" scale="0.001 0.001 0.001" />
-        </geometry>
-        <material name="black" />
-      </visual>
-      <collision>
-        <origin xyz="${0.05408+(0.06006-0.00707)/2} 0.0 -${0.066/2}" rpy="0.0 0.0 0.0" />
-        <geometry>
-          <box size="${0.06006-0.0071} 0.01 0.066" />
-        </geometry>
-      </collision>
-      <inertial>
-        <origin xyz="${0.05408+(0.06006-0.00707)/2} 0.0 -${0.066/2}" rpy="0.0 0.0 ${M_PI/2}" />
-        <mass value="0.08" />
-        <inertia ixx="${1/12*0.08*((0.06006-0.0071)**2+0.066**2)}" ixy="0.0" ixz="0.0"
-                 iyy="${1/12*0.08*(0.01**2+0.066**2)}"             iyz="0.0"
-                 izz="${1/12*0.08*((0.06006-0.0071)**2+0.01**2)}" />
-      </inertial>
-    </link>
-    <joint name="${prefix_hand}_outer_l_joint" type="continuous">
-      <parent link="${prefix_hand}_base_link" />
-      <child link="${prefix_hand}_outer_l_link" />
-      <origin xyz="0.043193 0.04015 0.0282231" rpy="0.0 0.0 0.0" />
-      <axis xyz="0.0 0.0 1.0" />
-      <mimic joint="${prefix_hand}_inner_l_joint" multiplier="1.0" offset="0" />
-    </joint>
-    <link name="${prefix_hand}_outer_l_link">
-      <visual>
-        <origin xyz="0.0 0.0 0.0" rpy="0.0 0.0 ${M_PI/2.0}" />
-        <geometry>
-          <mesh filename="file://$(find sobit_home_description)/meshes/hand/hand_outer_l.stl" scale="0.001 0.001 0.001" />
-        </geometry>
-        <material name="black" />
-      </visual>
-      <collision>
-        <origin xyz="${0.06123+0.04281/2} 0.0 -${0.056/2}" rpy="0.0 0.0 0.0" />
-        <geometry>
-          <box size="0.04281 0.01 0.056" />
-        </geometry>
-      </collision>
-      <inertial>
-        <origin xyz="${0.06123+0.04281/2} 0.0 -${0.056/2}" rpy="0.0 0.0 ${M_PI/2}" />
-        <mass value="0.08" />
-        <inertia ixx="${1/12*0.08*(0.04281**2+0.056**2)}" ixy="0.0" ixz="0.0"
-                 iyy="${1/12*0.08*(0.01**2   +0.056**2)}" iyz="0.0"
-                 izz="${1/12*0.08*(0.04281**2+0.01**2)}" />
-      </inertial>
-    </link>
-    <joint name="${prefix_hand}_outer_r_joint" type="continuous">
-      <parent link="${prefix_hand}_base_link" />
-      <child link="${prefix_hand}_outer_r_link" />
-      <origin xyz="0.043193 -0.04015 0.0282231" rpy="0.0 0.0 0.0" />
-      <axis xyz="0.0 0.0 1.0" />
-      <mimic joint="${prefix_hand}_joint" multiplier="1.0" offset="0" />
-    </joint>
-    <link name="${prefix_hand}_outer_r_link">
-      <visual>
-        <origin xyz="0.0 0.0 0.0" rpy="0.0 0.0 ${M_PI/2.0}" />
-        <geometry>
-          <mesh filename="file://$(find sobit_home_description)/meshes/hand/hand_outer_r.stl" scale="0.001 0.001 0.001" />
-        </geometry>
-        <material name="black" />
-      </visual>
-      <collision>
-        <origin xyz="${0.06123+0.04281/2} 0.0 -${0.056/2}" rpy="0.0 0.0 0.0" />
-        <geometry>
-          <box size="0.04281 0.01 0.056" />
-        </geometry>
-      </collision>
-      <inertial>
-        <origin xyz="${0.06123+0.04281/2} 0.0 -${0.056/2}" rpy="0.0 0.0 ${M_PI/2}" />
-        <mass value="0.08" />
-        <inertia ixx="${1/12*0.08*(0.04281**2+0.056**2)}" ixy="0.0" ixz="0.0"
-                 iyy="${1/12*0.08*(0.01**2   +0.056**2)}" iyz="0.0"
-                 izz="${1/12*0.08*(0.04281**2+0.01**2)}" />
-      </inertial>
-    </link>
-    <joint name="${prefix_hand}_${prefix_finger}_l_joint" type="continuous">
-      <parent link="${prefix_hand}_inner_l_link" />
-      <child link="${prefix_hand}_${prefix_finger}_l_link" />
-      <origin xyz="0.114316 0.0 -0.027729" rpy="0.0 0.0 0.0" />
-      <axis xyz="0.0 0.0 1.0" />
-      <mimic joint="${prefix_hand}_joint" multiplier="1.0" offset="0" />
-    </joint>
-    <link name="${prefix_hand}_${prefix_finger}_l_link">
-      <visual>
-        <origin xyz="-0.029998 0.025 0.0" rpy="0.0 0.0 ${M_PI/2.0}" />
-        <geometry>
-          <mesh filename="file://$(find sobit_home_description)/meshes/hand/hand_finger_l.stl" scale="0.001 0.001 0.001" />
-        </geometry>
-        <material name="black" />
-      </visual>
-      <collision>
-        <origin xyz="${0.007071+(0.012042+0.061128)/2} 0.0 -${0.018/2}" rpy="0.0 0.0 0.0" />
-        <geometry>
-          <box size="${0.012042+0.061128} 0.01137 0.044" />
-        </geometry>
-      </collision>
-      <inertial>
-        <origin xyz="${0.007071+(0.012042+0.061128)/2} 0.0 -${0.018/2}" rpy="0.0 0.0 ${M_PI/2}" />
-        <mass value="0.08" />
-        <inertia ixx="${1/12*0.08*((0.012042+0.061128)**2+0.044**2)}" ixy="0.0" ixz="0.0"
-                 iyy="${1/12*0.08*(0.01137**2+0.044**2)}"             iyz="0.0"
-                 izz="${1/12*0.08*((0.012042+0.061128)**2+0.01137**2)}" />
-      </inertial>
-    </link>
-    <joint name="${prefix_hand}_${prefix_finger}_r_joint" type="continuous">
-      <parent link="${prefix_hand}_link" />
-      <child link="${prefix_hand}_${prefix_finger}_r_link" />
-      <origin xyz="0.114316 0.0 -0.027729" rpy="0.0 0.0 0.0" />
-      <axis xyz="0.0 0.0 1.0" />
-      <mimic joint="${prefix_hand}_joint" multiplier="-1.0" offset="0" />
-    </joint>
-    <link name="${prefix_hand}_${prefix_finger}_r_link">
-      <visual>
-        <origin xyz="-0.029998 -0.025 0.0" rpy="0.0 0.0 ${M_PI/2.0}" />
-        <geometry>
-          <mesh filename="file://$(find sobit_home_description)/meshes/hand/hand_finger_r.stl" scale="0.001 0.001 0.001" />
-        </geometry>
-        <material name="black" />
-      </visual>
-      <collision>
-        <origin xyz="${0.007071+(0.012042+0.061128)/2} 0.0 -${0.018/2}" rpy="0.0 0.0 0.0" />
-        <geometry>
-          <box size="${0.012042+0.061128} 0.01137 0.044" />
-        </geometry>
-      </collision>
-      <inertial>
-        <origin xyz="${0.007071+(0.012042+0.061128)/2} 0.0 -${0.018/2}" rpy="0.0 0.0 ${M_PI/2}" />
-        <mass value="0.08" />
-        <inertia ixx="${1/12*0.08*((0.012042+0.061128)**2+0.044**2)}"   ixy="0.0" ixz="0.0"
-                 iyy="${1/12*0.08*(0.01137**2+0.044**2)}"               iyz="0.0"
-                 izz="${1/12*0.08*((0.012042+0.061128)**2+0.01137**2)}" />
-      </inertial>
-    </link>
-    <xacro:hand_transmission prefix_hand="${prefix_hand}" prefix_finger="${prefix_finger}" />
+    <xacro:hand_transmission prefix_hand="${prefix_hand}" position="${position}" prefix_finger="${prefix_finger}" />
   </xacro:macro>
 </robot>

Commit message: [FIX] toggle mimic

File: sobit_home_description/urdf/hand/hand.urdf.xacro (robot description, xacro)
@@ -130,5 +130,7 @@
       <axis xyz="0.0 1.0 0.0 " />
       <limit lower="${-M_PI/2}" upper="${M_PI/2}" effort="0.52" velocity="11.031179004" />
-      <mimic joint="${prefix_hand}_${position}_${prefix_finger}_l_mcp_joint" multiplier="-1.0" />
+      <xacro:unless value="${$(arg enable_gz)}">
+        <mimic joint="${prefix_hand}_${position}_${prefix_finger}_l_mcp_joint" multiplier="-1.0" />
+      </xacro:unless>
     </joint>
     <link name="${prefix_hand}_${position}_${prefix_finger}_r_mcp_link" >

Commit message: [FIX] mimic direction set in axis

File: sobit_home_description/urdf/hand/hand.urdf.xacro (robot description, xacro)
@@ -128,9 +128,7 @@
       <child link="${prefix_hand}_${position}_${prefix_finger}_r_mcp_link" />
       <origin xyz="-0.002855 ${y_sign * 0.020025} ${-y_sign * 0.024532}" rpy="0.0 0.0 0.0" />
-      <axis xyz="0.0 1.0 0.0 " />
+      <axis xyz="0.0 -1.0 0.0 " />
       <limit lower="${-M_PI/2}" upper="${M_PI/2}" effort="0.52" velocity="11.031179004" />
-      <xacro:unless value="${$(arg enable_gz)}">
-        <mimic joint="${prefix_hand}_${position}_${prefix_finger}_l_mcp_joint" multiplier="-1.0" />
-      </xacro:unless>
+      <mimic joint="${prefix_hand}_${position}_${prefix_finger}_l_mcp_joint" multiplier="1.0" />
     </joint>
     <link name="${prefix_hand}_${position}_${prefix_finger}_r_mcp_link" >

Commit message: [FIX] model name not use '-'

File: sobit_home_description/urdf/hand/hand.urdf.xacro (robot description, xacro)
@@ -136,5 +136,5 @@
         <origin xyz="0.0 0.0 0.0" rpy="${-y_sign * M_PI/2} ${y_sign * M_PI/2} 0.0" />
         <geometry>
-          <mesh filename="file://$(find sobit_home_description)/meshes/hand/switching_gear-m.stl" scale="0.001 0.001 0.001" />
+          <mesh filename="file://$(find sobit_home_description)/meshes/hand/switching_gear_m.stl" scale="0.001 0.001 0.001" />
         </geometry>
         <material name="grey" />
@@ -160,5 +160,5 @@
         <origin xyz="0.0 0.0 0.0" rpy="${-y_sign * M_PI/2} ${-y_sign * M_PI/2} 0.0" />
         <geometry>
-          <mesh filename="file://$(find sobit_home_description)/meshes/hand/middle_pharanx-m.stl" scale="0.001 0.001 0.001" />
+          <mesh filename="file://$(find sobit_home_description)/meshes/hand/middle_pharanx_m.stl" scale="0.001 0.001 0.001" />
         </geometry>
         <material name="grey" />
@@ -190,5 +190,5 @@
         <origin xyz="0.0 0.0 0.0" rpy="${-y_sign * M_PI/2} ${-y_sign * M_PI/2} 0.0" />
         <geometry>
-          <mesh filename="file://$(find sobit_home_description)/meshes/hand/distal_pharanx-m.stl" scale="0.001 0.001 0.001" />
+          <mesh filename="file://$(find sobit_home_description)/meshes/hand/distal_pharanx_m.stl" scale="0.001 0.001 0.001" />
         </geometry>
         <material name="grey" />

Commit message: [ADD] endeffector_link

File: sobit_home_description/urdf/hand/hand.urdf.xacro (robot description, xacro)
@@ -270,4 +270,27 @@
       </inertial>
     </link>
+    <!-- Joint: End Effector -->
+    <joint name="${prefix_hand}_${position}_end_effector_joint" type="fixed">
+      <origin xyz="0.0 ${y_sign*0.13} 0.0" rpy="0 0 0"/>
+      <parent link="${parent}"/>
+      <child link="${prefix_hand}_${position}_end_effector_link"/>
+    </joint>
+    <!-- Link: End Effector -->
+    <link name="${prefix_hand}_${position}_end_effector_link">
+      <visual>
+        <origin xyz="0.0 0.0 0.0" rpy="0 0 0"/>
+        <geometry>
+          <box size="0.01 0.01 0.01" />
+        </geometry>
+        <material name="red"/>
+      </visual>
+      <inertial>
+        <origin xyz="0.0 0.0 0.0" rpy="0 0 0"/>
+        <mass value="0.0001" />
+        <inertia  ixx="${1/12*0.0001*(0.01**2+0.01**2)}" ixy="0.0" ixz="0.0"
+                  iyy="${1/12*0.0001*(0.01**2+0.01**2)}" iyz="0.0"
+                  izz="${1/12*0.0001*(0.01**2+0.01**2)}" />
+      </inertial>
+    </link>
   <xacro:hand_transmission prefix_hand="${prefix_hand}" position="${position}" prefix_finger="${prefix_finger}"/>
   </xacro:macro>

Commit message: [FIX]adjust end_effector_joint orientation

File: sobit_home_description/urdf/hand/hand.urdf.xacro (robot description, xacro)
@@ -272,5 +272,5 @@
     <!-- Joint: End Effector -->
     <joint name="${prefix_hand}_${position}_end_effector_joint" type="fixed">
-      <origin xyz="0.0 ${y_sign*0.13} 0.0" rpy="0 0 0"/>
+      <origin xyz="0.0 ${y_sign*0.13} 0.0" rpy="${y_sign * M_PI/2} 0.0 ${y_sign * M_PI/2}"/>
       <parent link="${parent}"/>
       <child link="${prefix_hand}_${position}_end_effector_link"/>

Commit message: [ADD] Added new function declaration.

File: sobit_home_description/urdf/hand/hand.urdf.xacro (robot description, xacro)
@@ -215,5 +215,5 @@
       <origin xyz="0.036751 ${y_sign * 0.036625} ${y_sign * 0.014550} " rpy="0.0 0.0 0.0" />
       <axis xyz="0.0 0.0 1.0 " />
-      <limit lower="${-M_PI/2}" upper="${M_PI/6}" effort="0.52" velocity="11.031179004" />
+      <limit lower="${-M_PI/2}" upper="${M_PI/2}" effort="0.52" velocity="11.031179004" />
     </joint>
     <link name="${prefix_hand}_${position}_${prefix_finger}_c_mcp_link" >
@@ -245,5 +245,5 @@
       <origin xyz="0.0 ${y_sign * 0.050} 0.0" rpy="0.0 0.0 0.0" />
       <axis xyz="0.0 0.0 1.0 " />
-      <limit lower="${-M_PI/6}" upper="${M_PI/2}" effort="0.52" velocity="11.031179004" />
+      <limit lower="${-M_PI/2}" upper="${M_PI/2}" effort="0.52" velocity="11.031179004" />
     </joint>
     <link name="${prefix_hand}_${position}_${prefix_finger}_c_ip_link" >

Commit message: [UPD] adjust hand urdf

File: sobit_home_description/urdf/hand/hand.urdf.xacro (robot description, xacro)
@@ -18,5 +18,5 @@
       <parent link="${parent}" />
       <child link="${prefix_hand}_${position}_cmc_link" />
-      <origin xyz="0.0 ${y_sign * 0.025375} 0.0" rpy="0.0 0.0 0.0" />
+      <origin xyz="0.0 ${y_sign * 0.025375} 0.0" rpy="0.0 ${M_PI/2} 0.0" />
     </joint>
     <link name="${prefix_hand}_${position}_cmc_link" >
@@ -283,5 +283,5 @@
     <!-- Joint: End Effector -->
     <joint name="${prefix_hand}_${position}_end_effector_joint" type="fixed">
-      <origin xyz="0.0 ${y_sign*0.13} 0.0" rpy="${M_PI} 0.0 ${y_sign * M_PI/2}"/>
+      <origin xyz="0.0 ${y_sign*0.13} 0.0" rpy="${y_sign * M_PI/2} 0.0 ${y_sign * M_PI/2}"/>
       <parent link="${parent}"/>
       <child link="${prefix_hand}_${position}_end_effector_link"/>

Commit message: [FIX] hand orientation

File: sobit_home_description/urdf/hand/hand.urdf.xacro (robot description, xacro)
@@ -18,6 +18,6 @@
       <parent link="${parent}" />
       <child link="${prefix_hand}_${position}_cmc_link" />
-      <origin xyz="0.0 ${y_sign * 0.025375} 0.0" rpy="0.0 0.0 0.0" />
-      <!-- <origin xyz="0.0 ${y_sign * 0.025375} 0.0" rpy="0.0 ${M_PI/2} 0.0" /> -->
+      <!-- <origin xyz="0.0 ${y_sign * 0.025375} 0.0" rpy="0.0 0.0 0.0" /> -->
+      <origin xyz="0.0 ${y_sign * 0.025375} 0.0" rpy="0.0 ${M_PI/2} 0.0" />
     </joint>
     <link name="${prefix_hand}_${position}_cmc_link" >

Commit message: [FIX] add effort ratio param into hand

File: sobit_home_description/urdf/hand/hand.urdf.xacro (robot description, xacro)
@@ -44,5 +44,5 @@
       <origin xyz="-0.002855 ${y_sign * 0.018025} ${y_sign * 0.024532}" rpy="0.0 0.0 0.0" />
       <axis xyz="0.0 1.0 0.0 " />
-      <limit lower="${-M_PI/2}" upper="${M_PI/2}" effort="0.52" velocity="11.031179004" />
+      <limit lower="${-M_PI/2}" upper="${M_PI/2}" effort="${0.52 * effort_ratio}" velocity="11.031179004" />
     </joint>
     <link name="${prefix_hand}_${position}_${prefix_finger}_l_mcp_link" >
@@ -68,5 +68,5 @@
       <origin xyz="-0.02125 ${y_sign * 0.019006} ${y_sign * 0.040125}" rpy="0.0 0.0 0.0" />
       <axis xyz="1.0 0.0 0.0 " />
-      <limit lower="${-M_PI/6}" upper="${M_PI/2}" effort="0.52" velocity="11.031179004" />
+      <limit lower="${-M_PI/6}" upper="${M_PI/2}" effort="${0.52 * effort_ratio}" velocity="11.031179004" />
     </joint>
     <link name="${prefix_hand}_${position}_${prefix_finger}_l_pip_link" >
@@ -99,5 +99,5 @@
       <origin xyz="0.0 ${y_sign * 0.050} 0.0" rpy="0.0 0.0 0.0" />
       <axis xyz="1.0 0.0 0.0 " />
-      <limit lower="${-M_PI/2}" upper="${M_PI/6}" effort="0.52" velocity="11.031179004" />
+      <limit lower="${-M_PI/2}" upper="${M_PI/6}" effort="${0.52 * effort_ratio}" velocity="11.031179004" />
     </joint>
     <link name="${prefix_hand}_${position}_${prefix_finger}_l_dip_link" >
@@ -132,5 +132,5 @@
       <origin xyz="-0.002855 ${y_sign * 0.020025} ${-y_sign * 0.024532}" rpy="0.0 0.0 0.0" />
       <axis xyz="0.0 -1.0 0.0 " />
-      <limit lower="${-M_PI/2}" upper="${M_PI/2}" effort="0.52" velocity="11.031179004" />
+      <limit lower="${-M_PI/2}" upper="${M_PI/2}" effort="${0.52 * effort_ratio}" velocity="11.031179004" />
       <mimic joint="${prefix_hand}_${position}_${prefix_finger}_l_mcp_joint" multiplier="1.0" />
     </joint>
@@ -157,5 +157,5 @@
       <origin xyz="-0.02125 ${y_sign * 0.016750} ${-y_sign * 0.040125}" rpy="0.0 0.0 0.0" />
       <axis xyz="1.0 0.0 0.0 " />
-      <limit lower="${-M_PI/2}" upper="${M_PI/6}" effort="0.52" velocity="11.031179004" />
+      <limit lower="${-M_PI/2}" upper="${M_PI/6}" effort="${0.52 * effort_ratio}" velocity="11.031179004" />
     </joint>
     <link name="${prefix_hand}_${position}_${prefix_finger}_r_pip_link" >
@@ -188,5 +188,5 @@
       <origin xyz="0.0 ${y_sign * 0.050} 0.0" rpy="0.0 0.0 0.0" />
       <axis xyz="1.0 0.0 0.0 " />
-      <limit lower="${-M_PI/6}" upper="${M_PI/2}" effort="0.52" velocity="11.031179004" />
+      <limit lower="${-M_PI/6}" upper="${M_PI/2}" effort="${0.52 * effort_ratio}" velocity="11.031179004" />
     </joint>
     <link name="${prefix_hand}_${position}_${prefix_finger}_r_dip_link" >
@@ -220,10 +220,10 @@
       <origin xyz="0.036751 ${y_sign * 0.036625} ${y_sign * 0.014550} " rpy="0.0 0.0 0.0" />
       <axis xyz="0.0 0.0 1.0 " />
-      <!-- <limit lower="${-M_PI/2}" upper="${M_PI/6}" effort="0.52" velocity="11.031179004" /> -->
+      <!-- <limit lower="${-M_PI/2}" upper="${M_PI/6}" effort="${0.52 * effort_ratio}" velocity="11.031179004" /> -->
       <xacro:if value="${position == 'left'}">
-        <limit lower="${-M_PI/2}" upper="${M_PI/6}" effort="0.52" velocity="11.031" />
+        <limit lower="${-M_PI/2}" upper="${M_PI/6}" effort="${0.52 * effort_ratio}" velocity="11.031" />
       </xacro:if>
       <xacro:if value="${position == 'right'}">
-        <limit lower="${-M_PI/6}" upper="${M_PI/2}" effort="0.52" velocity="11.031" />
+        <limit lower="${-M_PI/6}" upper="${M_PI/2}" effort="${0.52 * effort_ratio}" velocity="11.031" />
       </xacro:if>
     </joint>
@@ -258,8 +258,8 @@
       <axis xyz="0.0 0.0 1.0 " />
       <xacro:if value="${position == 'right'}">
-        <limit lower="${-M_PI/2}" upper="${M_PI/6}" effort="0.52" velocity="11.031" />
+        <limit lower="${-M_PI/2}" upper="${M_PI/6}" effort="${0.52 * effort_ratio}" velocity="11.031" />
       </xacro:if>
       <xacro:if value="${position == 'left'}">
-        <limit lower="${-M_PI/6}" upper="${M_PI/2}" effort="0.52" velocity="11.031" />
+        <limit lower="${-M_PI/6}" upper="${M_PI/2}" effort="${0.52 * effort_ratio}" velocity="11.031" />
       </xacro:if>
     </joint>
