Commit message: Give the fingers their own effort ratio
Finger joints were scaled by effort_ratio (100), giving 52 Nm per finger.
Against stiff object contact that stores huge penetration energy, so
grasped objects stuck to the fingers or were flung on release.
finger_effort_ratio = 1.0 restores the real 0.52 Nm.

File: sobit_home_description/urdf/hand/hand.urdf.xacro (robot description, xacro)
@@ -47,5 +47,5 @@
       <origin xyz="-0.002855 ${y_sign * 0.018025} ${y_sign * 0.024532}" rpy="0.0 0.0 0.0" />
       <axis xyz="0.0 1.0 0.0 " />
-      <limit lower="${-M_PI/2}" upper="${M_PI/2}" effort="${0.52 * effort_ratio}" velocity="11.031179004" />
+      <limit lower="${-M_PI/2}" upper="${M_PI/2}" effort="${0.52 * finger_effort_ratio}" velocity="11.031179004" />
     </joint>
     <link name="${prefix_hand}_${position}_${prefix_finger}_l_mcp_link" >
@@ -71,5 +71,5 @@
       <origin xyz="-0.02125 ${y_sign * 0.019006} ${y_sign * 0.040125}" rpy="0.0 0.0 0.0" />
       <axis xyz="1.0 0.0 0.0 " />
-      <limit lower="${-M_PI/6}" upper="${M_PI/2}" effort="${0.52 * effort_ratio}" velocity="11.031179004" />
+      <limit lower="${-M_PI/6}" upper="${M_PI/2}" effort="${0.52 * finger_effort_ratio}" velocity="11.031179004" />
     </joint>
     <link name="${prefix_hand}_${position}_${prefix_finger}_l_pip_link" >
@@ -102,5 +102,5 @@
       <origin xyz="0.0 ${y_sign * 0.050} 0.0" rpy="0.0 0.0 0.0" />
       <axis xyz="1.0 0.0 0.0 " />
-      <limit lower="${-FINGER_CLOSE}" upper="${M_PI/6}" effort="${0.52 * effort_ratio}" velocity="11.031179004" />
+      <limit lower="${-FINGER_CLOSE}" upper="${M_PI/6}" effort="${0.52 * finger_effort_ratio}" velocity="11.031179004" />
     </joint>
     <link name="${prefix_hand}_${position}_${prefix_finger}_l_dip_link" >
@@ -135,5 +135,5 @@
       <origin xyz="-0.002855 ${y_sign * 0.020025} ${-y_sign * 0.024532}" rpy="0.0 0.0 0.0" />
       <axis xyz="0.0 -1.0 0.0 " />
-      <limit lower="${-M_PI/2}" upper="${M_PI/2}" effort="${0.52 * effort_ratio}" velocity="11.031179004" />
+      <limit lower="${-M_PI/2}" upper="${M_PI/2}" effort="${0.52 * finger_effort_ratio}" velocity="11.031179004" />
       <mimic joint="${prefix_hand}_${position}_${prefix_finger}_l_mcp_joint" multiplier="1.0" />
     </joint>
@@ -160,5 +160,5 @@
       <origin xyz="-0.02125 ${y_sign * 0.016750} ${-y_sign * 0.040125}" rpy="0.0 0.0 0.0" />
       <axis xyz="1.0 0.0 0.0 " />
-      <limit lower="${-M_PI/2}" upper="${M_PI/6}" effort="${0.52 * effort_ratio}" velocity="11.031179004" />
+      <limit lower="${-M_PI/2}" upper="${M_PI/6}" effort="${0.52 * finger_effort_ratio}" velocity="11.031179004" />
     </joint>
     <link name="${prefix_hand}_${position}_${prefix_finger}_r_pip_link" >
@@ -191,5 +191,5 @@
       <origin xyz="0.0 ${y_sign * 0.050} 0.0" rpy="0.0 0.0 0.0" />
       <axis xyz="1.0 0.0 0.0 " />
-      <limit lower="${-M_PI/6}" upper="${FINGER_CLOSE}" effort="${0.52 * effort_ratio}" velocity="11.031179004" />
+      <limit lower="${-M_PI/6}" upper="${FINGER_CLOSE}" effort="${0.52 * finger_effort_ratio}" velocity="11.031179004" />
     </joint>
     <link name="${prefix_hand}_${position}_${prefix_finger}_r_dip_link" >
@@ -223,10 +223,10 @@
       <origin xyz="0.036751 ${y_sign * 0.036625} ${y_sign * 0.014550} " rpy="0.0 0.0 0.0" />
       <axis xyz="0.0 0.0 1.0 " />
-      <!-- <limit lower="${-M_PI/2}" upper="${M_PI/6}" effort="${0.52 * effort_ratio}" velocity="11.031179004" /> -->
+      <!-- <limit lower="${-M_PI/2}" upper="${M_PI/6}" effort="${0.52 * finger_effort_ratio}" velocity="11.031179004" /> -->
       <xacro:if value="${position == 'left'}">
-        <limit lower="${-M_PI/2}" upper="${M_PI/6}" effort="${0.52 * effort_ratio}" velocity="11.031" />
+        <limit lower="${-M_PI/2}" upper="${M_PI/6}" effort="${0.52 * finger_effort_ratio}" velocity="11.031" />
       </xacro:if>
       <xacro:if value="${position == 'right'}">
-        <limit lower="${-M_PI/6}" upper="${M_PI/2}" effort="${0.52 * effort_ratio}" velocity="11.031" />
+        <limit lower="${-M_PI/6}" upper="${M_PI/2}" effort="${0.52 * finger_effort_ratio}" velocity="11.031" />
       </xacro:if>
     </joint>
@@ -261,8 +261,8 @@
       <axis xyz="0.0 0.0 1.0 " />
       <xacro:if value="${position == 'right'}">
-        <limit lower="${-FINGER_CLOSE}" upper="${M_PI/6}" effort="${0.52 * effort_ratio}" velocity="11.031" />
+        <limit lower="${-FINGER_CLOSE}" upper="${M_PI/6}" effort="${0.52 * finger_effort_ratio}" velocity="11.031" />
       </xacro:if>
       <xacro:if value="${position == 'left'}">
-        <limit lower="${-M_PI/6}" upper="${FINGER_CLOSE}" effort="${0.52 * effort_ratio}" velocity="11.031" />
+        <limit lower="${-M_PI/6}" upper="${FINGER_CLOSE}" effort="${0.52 * finger_effort_ratio}" velocity="11.031" />
       </xacro:if>
     </joint>

File: sobit_home_description/urdf/values.urdf.xacro (robot description, xacro)
@@ -4,3 +4,4 @@
   <xacro:property name="M_PI" value="3.14159265359" />
   <xacro:property name="effort_ratio" value="100.0" />
+  <xacro:property name="finger_effort_ratio" value="1.0" />
 </robot>
