Commit message: [UPD] urdf files

File: sobit_home_description/urdf/arm/arm.transmission.xacro (robot description, xacro)
@@ -2,12 +2,10 @@
 <robot name="sobit_home"
        xmlns:xacro="http://ros.org/wiki/xacro">
-  <xacro:macro name="arm_transmission" params="prefix">
-    <xacro:position_joint_transmission joint="${prefix}_shoulder_1_tilt_joint"    reduction="1" />
-    <xacro:position_joint_transmission joint="${prefix}_shoulder_2_tilt_joint"    reduction="1" />
-    <xacro:position_joint_transmission joint="${prefix}_elbow_upper_1_tilt_joint" reduction="1" />
-    <xacro:position_joint_transmission joint="${prefix}_elbow_upper_2_tilt_joint" reduction="1" />
-    <xacro:position_joint_transmission joint="${prefix}_elbow_lower_tilt_joint"   reduction="1" />
-    <xacro:position_joint_transmission joint="${prefix}_elbow_lower_pan_joint"    reduction="1" />
-    <xacro:position_joint_transmission joint="${prefix}_wrist_tilt_joint"         reduction="1" />
+  <xacro:macro name="arm_transmission" params="prefix position" >
+    <xacro:position_joint_transmission joint="${prefix}_${position}_shoulder_tilt_joint"    reduction="1" />
+    <xacro:position_joint_transmission joint="${prefix}_${position}_upper_roll_joint"    reduction="1" />
+    <xacro:position_joint_transmission joint="${prefix}_${position}_uppder_flex_joint"    reduction="1" />
+    <xacro:position_joint_transmission joint="${prefix}_${position}_elbow_joint"    reduction="1" />
+    <xacro:position_joint_transmission joint="${prefix}_${position}_wrist_joint"    reduction="1" />
   </xacro:macro>
 </robot>

File: sobit_home_description/urdf/arm/arm.urdf.xacro (robot description, xacro)
@@ -4,12 +4,24 @@
   <xacro:include filename="$(find sobit_home_description)/urdf/arm/arm.transmission.xacro" />
   <xacro:macro name="arm" params="prefix position parent" >
+    <xacro:if value="${position == 'left'}">
+      <xacro:property name="y_sign" value="1.0" />
+      <xacro:property name="yaw_rot" value="0.0" />
+        <xacro:property name="upper_roll_limit_lower" value="0" />
+        <xacro:property name="upper_roll_limit_upper" value="${M_PI}" />
+    </xacro:if>
+    <xacro:if value="${position == 'right'}">
+      <xacro:property name="y_sign" value="-1.0" />
+      <xacro:property name="yaw_rot" value="${M_PI}" />
+        <xacro:property name="upper_roll_limit_lower" value="${-M_PI}" />
+        <xacro:property name="upper_roll_limit_upper" value="0" />
+    </xacro:if>
     <joint name="${prefix}_${position}_base_joint" type="fixed" >
       <parent link="${parent}" />
       <child link="${prefix}_${position}_base_link" />
-      <origin xyz="0.0 0.079 0.0" rpy="0.0 0.0 0.0" />
+      <origin xyz="0.0 ${y_sign * 0.079} 0.0" rpy="0.0 0.0 0.0" />
     </joint>
     <link name="${prefix}_${position}_base_link" >
       <visual>
-        <origin xyz="0.0 0.0 0.0" rpy="${M_PI/2} 0.0 ${M_PI/2}" />
+        <origin xyz="0.0 0.0 0.0" rpy="${M_PI/2} 0.0 ${M_PI/2+yaw_rot}" />
         <geometry>
           <mesh filename="file://$(find sobit_home_description)/meshes/arm/arm_scapula.stl" scale="0.001 0.001 0.001" />
@@ -34,5 +46,5 @@
       <parent link="${prefix}_${position}_base_link" />
       <child link="${prefix}_${position}_shoulder_tilt_link" />
-      <origin xyz="0.0 0.1355 0.0" rpy="0.0 0.0 0.0" />
+      <origin xyz="0.0 ${y_sign * 0.19875} 0.0" rpy="0.0 0.0 0.0" />
       <axis xyz="0.0 -1.0 0.0 " />
       <limit lower="${-M_PI/2}" upper="${M_PI/2}" effort="${10.6*2}" velocity="11.031179004" />
@@ -40,5 +52,5 @@
     <link name="${prefix}_${position}_shoulder_tilt_link" >
       <visual>
-        <origin xyz="0.0 0.0 0.0" rpy="0.0 0.0 ${M_PI/2}" />
+        <origin xyz="0.0 0.0 0.0" rpy="0.0 0.0 ${M_PI/2+yaw_rot}" />
         <geometry>
           <mesh filename="file://$(find sobit_home_description)/meshes/arm/arm_shoulder.stl" scale="0.001 0.001 0.001" />
@@ -63,7 +75,7 @@
       <parent link="${prefix}_${position}_shoulder_tilt_link" />
       <child link="${prefix}_${position}_upper_roll_link" />
-      <origin xyz="0.0 0.0 -0.09465" rpy="0.0 0.0 0.0" />
-      <axis xyz="0.0 -1.0 0.0 " />
-      <limit lower="${-M_PI/2}" upper="${M_PI/2}" effort="${10.6*2}" velocity="11.031179004" />
+      <origin xyz="0.0 0.0 0.0" rpy="0.0 0.0 0.0" />
+      <axis xyz="1.0 0.0 0.0 " />
+      <limit lower="${upper_roll_limit_lower}" upper="${upper_roll_limit_upper}" effort="${10.6*2}" velocity="11.031179004" />
     </joint>
     <link name="${prefix}_${position}_upper_roll_link" >
@@ -92,11 +104,11 @@
       <parent link="${prefix}_${position}_upper_roll_link" />
       <child link="${prefix}_${position}_upper_flex_link" />
-      <origin xyz="0.0 0.0 -0.209821" rpy="0.0 0.0 0.0" />
-      <axis xyz="0.0 -1.0 0.0 " />
+      <origin xyz="0.0 0.0 -0.215813" rpy="0.0 0.0 0.0" />
+      <axis xyz="0.0 0.0 1.0" />
       <limit lower="${-M_PI/2}" upper="${M_PI/2}" effort="${10.6*2}" velocity="11.031179004" />
     </joint>
     <link name="${prefix}_${position}_upper_flex_link" >
       <visual>
-        <origin xyz="0.0 0.0 0.0" rpy="0.0 0.0 ${M_PI/2}" />
+        <origin xyz="0.0 0.0 0.0" rpy="0.0 0.0 ${-M_PI/2}" />
         <geometry>
           <mesh filename="file://$(find sobit_home_description)/meshes/arm/arm_upper_flex.stl" scale="0.001 0.001 0.001" />
@@ -118,5 +130,63 @@
       </inertial>
     </link>
-    <xacro:arm_transmission prefix="${prefix}" />
+    <joint name="${prefix}_${position}_elbow_joint" type="revolute" >
+      <parent link="${prefix}_${position}_upper_flex_link" />
+      <child link="${prefix}_${position}_elbow_link" />
+      <origin xyz="0.0 0.0 -0.18413635" rpy="0.0 0.0 0.0" />
+      <axis xyz="0.0 -1.0 0.0 " />
+      <limit lower="0" upper="${M_PI/2}" effort="${10.6*2}" velocity="11.031179004" />
+    </joint>
+    <link name="${prefix}_${position}_elbow_link" >
+      <visual>
+        <origin xyz="0.0 0.0 0.0" rpy="0.0 0.0 ${M_PI/2}" />
+        <geometry>
+          <mesh filename="file://$(find sobit_home_description)/meshes/arm/arm_elbow.stl" scale="0.001 0.001 0.001" />
+        </geometry>
+        <material name="grey" />
+      </visual>
+      <collision>
+        <origin xyz="${0.1166/2+0.0224} 0.0 0.0" rpy="0.0 0.0 0.0" />
+        <geometry>
+          <box size="0.1166 0.124 0.043" />
+        </geometry>
+      </collision>
+      <inertial>
+        <origin xyz="${0.1166/2+0.0224} 0.0 0.0" rpy="0.0 0.0 ${M_PI/2}" />
+        <mass value="0.08" />
+        <inertia ixx="${1/12*0.08*(0.1166**2+0.043**2)}" ixy="0.0" ixz="0.0"
+                 iyy="${1/12*0.08*(0.124**2 +0.043**2)}" iyz="0.0"
+                 izz="${1/12*0.08*(0.1166**2+0.124**2)}" />
+      </inertial>
+    </link>
+    <joint name="${prefix}_${position}_wrist_joint" type="revolute" >
+      <parent link="${prefix}_${position}_elbow_link" />
+      <child link="${prefix}_${position}_wrist_link" />
+      <origin xyz="0.0 0.0 -0.5" rpy="0.0 0.0 0.0" />
+      <axis xyz="0.0 -1.0 0.0 " />
+      <limit lower="${-M_PI/2}" upper="${M_PI/2}" effort="${10.6*2}" velocity="11.031179004" />
+    </joint>
+    <link name="${prefix}_${position}_wrist_link" >
+      <visual>
+        <origin xyz="0.0 0.0 0.0" rpy="0.0 0.0 ${M_PI/2}" />
+        <geometry>
+          <mesh filename="file://$(find sobit_home_description)/meshes/arm/arm_wrist.stl" scale="0.001 0.001 0.001" />
+        </geometry>
+        <material name="grey" />
+      </visual>
+      <collision>
+        <origin xyz="${0.1166/2+0.0224} 0.0 0.0" rpy="0.0 0.0 0.0" />
+        <geometry>
+          <box size="0.1166 0.124 0.043" />
+        </geometry>
+      </collision>
+      <inertial>
+        <origin xyz="${0.1166/2+0.0224} 0.0 0.0" rpy="0.0 0.0 ${M_PI/2}" />
+        <mass value="0.08" />
+        <inertia ixx="${1/12*0.08*(0.1166**2+0.043**2)}" ixy="0.0" ixz="0.0"
+                 iyy="${1/12*0.08*(0.124**2 +0.043**2)}" iyz="0.0"
+                 izz="${1/12*0.08*(0.1166**2+0.124**2)}" />
+      </inertial>
+    </link>
+    <xacro:arm_transmission prefix="${prefix}" position="${position}" />
   </xacro:macro>
 </robot>

File: sobit_home_description/urdf/body/body.urdf.xacro (robot description, xacro)
@@ -5,5 +5,5 @@
   <xacro:macro name="body" params="prefix parent" >
     <joint name="${prefix}_joint" type="fixed" >
-      <origin xyz="0.0 -0.0525 0.565" rpy="0.0 0.0 0.0" />
+      <origin xyz="0.0 0.0 0.565" rpy="0.0 0.0 0.0" />
       <parent link="${parent}" />
       <child link="${prefix}_link" />
@@ -32,5 +32,5 @@
     </link>
     <joint name="linear_actuator_joint" type="prismatic" >
-      <origin xyz="0.0961 0.0525 0.0" rpy="0.0 0.0 0.0" />
+      <origin xyz="0.11275 0.0 0.0" rpy="0.0 0.0 0.0" />
       <parent link="${prefix}_link" />
       <child link="linear_actuator_link" />
