Commit message: [UPD] Update for new arm.

File: sobit_home_description/urdf/arm/arm.transmission.xacro (robot description, xacro)
@@ -6,5 +6,6 @@
     <xacro:SimpleTransmissionPosition joint="${prefix}_${position}_upper_roll_joint"     reduction="1" />
     <xacro:SimpleTransmissionPosition joint="${prefix}_${position}_uppder_flex_joint"    reduction="1" />
-    <xacro:SimpleTransmissionPosition joint="${prefix}_${position}_elbow_joint"          reduction="1" />
+    <xacro:SimpleTransmissionPosition joint="${prefix}_${position}_lowe_top_joint"          reduction="1" />
+    <xacro:SimpleTransmissionPosition joint="${prefix}_${position}_lowe_bottom_joint"          reduction="1" />
     <xacro:SimpleTransmissionPosition joint="${prefix}_${position}_wrist_tilt_joint"     reduction="1" />
     <xacro:SimpleTransmissionPosition joint="${prefix}_${position}_wrist_roll_joint"     reduction="1" />

File: sobit_home_description/urdf/arm/arm.urdf.xacro (robot description, xacro)
@@ -37,4 +37,5 @@
       </inertial>
     </link>
+<!-- Shoulder tilt joint -->
     <joint name="${prefix}_${position}_shoulder_tilt_joint" type="revolute" >
       <parent link="${prefix}_${position}_base_link" />
@@ -46,5 +47,5 @@
     <link name="${prefix}_${position}_shoulder_tilt_link" >
       <visual>
-        <origin xyz="0.0 0.0 0.0" rpy="0.0 ${(y_sign+1) * M_PI/2} ${-M_PI/2}" />
+        <origin xyz="0.0 0.0 0.0" rpy="0.0 0.0 ${y_sign * M_PI/2}" />
         <geometry>
           <mesh filename="file://$(find sobit_home_description)/meshes/arm/arm_shoulder.stl" scale="0.001 0.001 0.001" />
@@ -66,8 +67,9 @@
       </inertial>
     </link>
+<!-- Upper roll joint (left) -->
     <joint name="${prefix}_${position}_upper_roll_joint" type="revolute" >
       <parent link="${prefix}_${position}_shoulder_tilt_link" />
       <child link="${prefix}_${position}_upper_roll_link" />
-      <origin xyz="0.0 ${y_sign * 0.0725} 0.0" rpy="0.0 0.0 0.0" />
+      <origin xyz="${y_sign * 0.0510} ${y_sign * 0.100} 0.0" rpy="0.0 0.0 0.0" />
       <axis xyz="1.0 0.0 0.0" />
       <limit lower="${-M_PI/2}" upper="${M_PI/2}" effort="${10.6 * effort_ratio}" velocity="3.14" />
@@ -75,5 +77,10 @@
     <link name="${prefix}_${position}_upper_roll_link" >
       <visual>
-        <origin xyz="0.0 0.0 0.0" rpy="0.0 ${-y_sign * M_PI/2} ${M_PI/2}" />
+        <xacro:if value="${position == 'right'}">
+          <origin xyz="${-y_sign * 0.0510} 0.0 0.0" rpy="${M_PI} 0.0 ${y_sign * M_PI/2}" />
+        </xacro:if>
+        <xacro:unless value="${position == 'right'}">
+          <origin xyz="${-y_sign * 0.0510} 0.0 0.0" rpy="0.0 0.0 ${y_sign * M_PI/2}" />
+        </xacro:unless>
         <geometry>
           <mesh filename="file://$(find sobit_home_description)/meshes/arm/arm_upper_roll.stl" scale="0.001 0.001 0.001" />
@@ -82,5 +89,5 @@
       </visual>
       <collision>
-        <origin xyz="0.0 ${y_sign * 0.13445} 0.0" rpy="0.0 ${y_sign * M_PI/2} ${M_PI/2}" />
+        <origin xyz="${-y_sign * 0.0563} ${y_sign * 0.13445} 0.0" rpy="0.0 ${y_sign * M_PI/2} ${M_PI/2}" />
         <geometry>
           <cylinder length="0.129" radius="${0.076/2}" />
@@ -95,14 +102,33 @@
       </inertial>
     </link>
+<!-- Upper roll sub joint -->
+    <joint name="${prefix}_${position}_upper_roll_sub_joint" type="revolute" >
+      <mimic joint="${prefix}_${position}_upper_roll_joint" multiplier="-1" offset="0"/>
+      <parent link="${prefix}_${position}_shoulder_tilt_link" />
+      <child link="${prefix}_${position}_upper_roll_sub_link" />
+      <origin xyz="${-y_sign * 0.0510} ${y_sign * 0.100} 0.0" rpy="0.0 0.0 0.0" />
+      <axis xyz="-1.0 0.0 0.0" />
+      <limit lower="${-M_PI/2}" upper="${M_PI/2}" effort="${10.6 * effort_ratio}" velocity="3.14" />
+    </joint>
+    <link name="${prefix}_${position}_upper_roll_sub_link" >
+      <inertial>
+        <origin xyz="0.0 ${y_sign * 0.13445} 0.0" rpy="0.0 ${y_sign * M_PI/2} ${M_PI/2}" />
+        <mass value="0.595" />
+        <inertia ixx="${1/12*0.595*(3*0.038**2+0.129**2)}" ixy="0.0" ixz="0.0"
+                 iyy="${1/12*0.595*(3*0.038**2+0.129**2)}" iyz="0.0"
+                 izz="${1/2*0.595*0.038**2}" />
+      </inertial>
+    </link>
+  <!-- Upper flex joint -->
     <joint name="${prefix}_${position}_upper_flex_joint" type="revolute" >
       <parent link="${prefix}_${position}_upper_roll_link" />
       <child link="${prefix}_${position}_upper_flex_link" />
-      <origin xyz="0.0 ${y_sign * 0.2} 0.0" rpy="0.0 0.0 0.0" />
+      <origin xyz="${-y_sign * 0.0510} ${y_sign * 0.1335} 0.0" rpy="0.0 0.0 0.0" />
       <axis xyz="0.0 ${y_sign} 0.0" />
-      <limit lower="${-M_PI}" upper="${M_PI}" effort="${4.1 * effort_ratio}" velocity="4.81" />
+      <limit lower="${-M_PI/2}" upper="${M_PI/2}" effort="${10.6 * effort_ratio}" velocity="4.81" />
     </joint>
     <link name="${prefix}_${position}_upper_flex_link" >
       <visual>
-        <origin xyz="0.0 ${y_sign * 0.2001} 0.0" rpy="${y_sign * M_PI/2} ${-y_sign * M_PI/2} 0.0" />
+          <origin xyz="0.0 ${y_sign * 0.0212} 0.0" rpy="${-y_sign *M_PI/2} 0.0 ${y_sign * M_PI/2}" />
         <geometry>
           <mesh filename="file://$(find sobit_home_description)/meshes/arm/arm_upper_flex.stl" scale="0.001 0.001 0.001" />
@@ -124,36 +150,52 @@
       </inertial>
     </link>
-    <joint name="${prefix}_${position}_elbow_joint" type="revolute" >
+<!-- Upper flex sub joint -->
+    <joint name="${prefix}_${position}_upper_flex_sub_joint" type="revolute" >
+      <mimic joint="${prefix}_${position}_upper_flex_joint" multiplier="1" offset="0"/>
+      <parent link="${prefix}_${position}_upper_roll_link" />
+      <child link="${prefix}_${position}_upper_flex_sub_link" />
+      <origin xyz="${-y_sign * 0.0510} ${y_sign * (0.100+0.0335+0.0510)} 0.0" rpy="0.0 0.0 0.0" />
+      <axis xyz="0.0 ${y_sign} 0.0" />
+      <limit lower="${-M_PI/2}" upper="${M_PI/2}" effort="${10.6 * effort_ratio}" velocity="4.81" />
+    </joint>
+    <link name="${prefix}_${position}_upper_flex_sub_link" >
+      <inertial>
+        <origin xyz="0.0 ${y_sign * 0.06943603} 0.0" rpy="0.0 ${y_sign * M_PI/2} ${-M_PI/2}" />
+        <mass value="0.778" />
+        <inertia ixx="${1/12*0.778*(3*0.038**2+0.171**2)}" ixy="0.0" ixz="0.0"
+                 iyy="${1/12*0.778*(3*0.038**2+0.171**2)}" iyz="0.0"
+                 izz="${1/2*0.778*0.038**2}" />
+      </inertial>
+    </link>
+<!-- Lower top joint -->
+    <joint name="${prefix}_${position}_lower_top_joint" type="revolute" >
       <parent link="${prefix}_${position}_upper_flex_link" />
-      <child link="${prefix}_${position}_elbow_link" />
-      <origin xyz="0.0 ${y_sign * 0.19765} 0.0" rpy="0.0 0.0 0.0" />
+      <child link="${prefix}_${position}_lower_top_link" />
       <axis xyz="0.0 0.0 1.0" />
-        <xacro:if value="${y_sign == -1.0}">
-          <xacro:property name="elbow_lower_limit" value="0.0" />
-          <xacro:property name="elbow_upper_limit" value="${140*M_PI/180}" />
+      <origin xyz="0.05495 ${y_sign * 0.26365} -0.0510" rpy="0.0 0.0 0.0" />
+        <limit lower="${-M_PI/2}" upper="${2/3 * M_PI}" effort="${10.6 * effort_ratio}" velocity="3.14" />
+    </joint>
+    <link name="${prefix}_${position}_lower_top_link" >
+      <visual>
+        <xacro:if value="${position == 'right'}">
+          <origin xyz="0.0 0.0 0.0510" rpy="${M_PI} 0.0 ${-M_PI/2}" />
         </xacro:if>
-        <xacro:if value="${y_sign == 1.0}">
-          <xacro:property name="elbow_lower_limit" value="${-140*M_PI/180}" />
-          <xacro:property name="elbow_upper_limit" value="0.0" />
-        </xacro:if>
-        <limit lower="${elbow_lower_limit}" upper="${elbow_upper_limit}" effort="${10.6 * effort_ratio}" velocity="3.14" />
-    </joint>
-    <link name="${prefix}_${position}_elbow_link" >
-      <visual>
-        <origin xyz="0.0 0.0 0.0" rpy="0.0 ${-y_sign * M_PI/2} ${M_PI/2}" />
-        <geometry>
-          <mesh filename="file://$(find sobit_home_description)/meshes/arm/arm_elbow.stl" scale="0.001 0.001 0.001" />
-        </geometry>
-        <material name="grey" />
-      </visual>
-      <collision>
+        <xacro:unless value="${position == 'right'}">
+          <origin xyz="0.0 0.0 0.0510" rpy="0.0 0.0 ${M_PI/2}" />
+        </xacro:unless>
+        <geometry>
+          <mesh filename="file://$(find sobit_home_description)/meshes/arm/arm_lower_top.stl" scale="0.001 0.001 0.001" />
+        </geometry>
+        <material name="grey" />
+      </visual>
+      <collision>
+        <origin xyz="0.0 0.0 0.0" rpy="0.0 0.0 0.0" />
+        <geometry>
+          <cylinder length="0.386" radius="${0.088156/2}" />
+        </geometry>
+      </collision>
+      <inertial>
         <origin xyz="0.0 ${y_sign * 0.265} 0.0" rpy="0.0 ${-y_sign * M_PI/2} ${M_PI/2}" />
-        <geometry>
-          <cylinder length="0.386" radius="${0.088156/2}" />
-        </geometry>
-      </collision>
-      <inertial>
-        <origin xyz="0.0 ${y_sign * 0.265} 0.0" rpy="0.0 ${-y_sign * M_PI/2} ${M_PI/2}" />
-        <mass value="1.663" /> <!-- mass without FR13-H101K -->
+        <mass value="1.663" /> <!--mass without FR13-H101K -->
         <inertia ixx="${1/12*1.663*(3*0.044**2+0.386**2)}" ixy="0.0" ixz="0.0"
                  iyy="${1/12*1.663*(3*0.044**2+0.386**2)}" iyz="0.0"
@@ -161,16 +203,35 @@
       </inertial>
     </link>
-    <joint name="${prefix}_${position}_wrist_tilt_joint" type="revolute" >
-      <parent link="${prefix}_${position}_elbow_link" />
-      <child link="${prefix}_${position}_wrist_tilt_link" />
-      <origin xyz="0.0 ${y_sign * 0.5} 0.0" rpy="0.0 0.0 0.0" />
-      <axis xyz="0.0 0.0 1.0" />
+<!-- Lower top sub joint -->
+    <joint name="${prefix}_${position}_lower_top_sub_joint" type="revolute" >
+      <mimic joint="${prefix}_${position}_lower_top_joint" multiplier="-1" offset="0"/>
+      <parent link="${prefix}_${position}_upper_flex_link" />
+      <child link="${prefix}_${position}_lower_top_sub_link" />
+      <origin xyz="0.05495 ${y_sign * 0.26365} 0.0510" rpy="0.0 0.0 0.0" />
+      <axis xyz="0.0 0.0 -1.0" />
+      <limit lower="${-M_PI/2}" upper="${M_PI/2}" effort="${10.6 * effort_ratio}" velocity="3.14" />
+    </joint>
+    <link name="${prefix}_${position}_lower_top_sub_link" >
+      <inertial>
+        <origin xyz="0.0 ${y_sign * 0.265} 0.0" rpy="0.0 ${-y_sign * M_PI/2} ${M_PI/2}" />
+        <mass value="1.663" />
+        <inertia ixx="${1/12*1.663*(3*0.044**2+0.386**2)}" ixy="0.0" ixz="0.0"
+                 iyy="${1/12*1.663*(3*0.044**2+0.386**2)}" iyz="0.0"
+                 izz="${1/2*1.663*0.044**2}" />
+      </inertial>
+    </link>
+<!-- Lower bottom joint -->
+    <joint name="${prefix}_${position}_lower_bottom_joint" type="revolute" >
+      <parent link="${prefix}_${position}_lower_top_link" />
+      <child link="${prefix}_${position}_lower_bottom_link" />
+      <origin xyz="0.0 ${y_sign * 0.107} 0.0510" rpy="0.0 0.0 0.0" />
+      <axis xyz="0.0 ${y_sign* 1.0} 0.0" />
       <limit lower="${-M_PI/2}" upper="${M_PI/2}" effort="${4.1 * effort_ratio}" velocity="4.81" />
     </joint>
-    <link name="${prefix}_${position}_wrist_tilt_link" >
-      <visual>
-        <origin xyz="0.0 0.0 0.0" rpy="0.0 ${-y_sign * M_PI/2} ${M_PI/2}" />
-        <geometry>
-          <mesh filename="file://$(find sobit_home_description)/meshes/arm/arm_wrist_tilt.stl" scale="0.001 0.001 0.001" />
+    <link name="${prefix}_${position}_lower_bottom_link" >
+      <visual>
+        <origin xyz="0.0 0.0 0.0" rpy="0.0 0.0 ${y_sign * M_PI/2}" />
+        <geometry>
+          <mesh filename="file://$(find sobit_home_description)/meshes/arm/arm_lower_bottom.stl" scale="0.001 0.001 0.001" />
         </geometry>
         <material name="grey" />
@@ -190,4 +251,36 @@
       </inertial>
     </link>
+<!-- TODO -->
+<!-- Wrist tilt joint -->
+    <joint name="${prefix}_${position}_wrist_tilt_joint" type="revolute" >
+      <parent link="${prefix}_${position}_lower_bottom_link" />
+      <child link="${prefix}_${position}_wrist_tilt_link" />
+      <origin xyz="0.0 ${y_sign * 0.443} 0.0" rpy="0.0 0.0 0.0" />
+      <axis xyz="0.0 0.0 1.0" />
+      <limit lower="${-M_PI/2}" upper="${M_PI/2}" effort="${4.1 * effort_ratio}" velocity="4.81" />
+    </joint>
+    <link name="${prefix}_${position}_wrist_tilt_link" >
+      <visual>
+        <origin xyz="0.0 0.0 0.0" rpy="0.0 ${-y_sign * M_PI/2} ${M_PI/2}" />
+        <geometry>
+          <mesh filename="file://$(find sobit_home_description)/meshes/arm/arm_wrist_tilt.stl" scale="0.001 0.001 0.001" />
+        </geometry>
+        <material name="grey" />
+      </visual>
+      <collision>
+        <origin xyz="0.0 ${y_sign * 0.0462} 0.0" rpy="0.0 ${-y_sign * M_PI/2} ${M_PI/2}" />
+        <geometry>
+          <cylinder length="0.0453" radius="${0.08/2}" />
+        </geometry>
+      </collision>
+      <inertial>
+        <origin xyz="0.0 0.0 0.0" rpy="0.0 ${-y_sign * M_PI/2} ${M_PI/2}" />
+        <mass value="0.341" />
+        <inertia ixx="${1/12*0.341*(3*0.04**2+0.0453**2)}" ixy="0.0" ixz="0.0"
+                 iyy="${1/12*0.341*(3*0.04**2+0.0453**2)}" iyz="0.0"
+                 izz="${1/2*0.341*0.04**2}" />
+      </inertial>
+    </link>
+<!-- Wrist roll joint -->
     <joint name="${prefix}_${position}_wrist_roll_joint" type="revolute" >
       <parent link="${prefix}_${position}_wrist_tilt_link" />
@@ -205,5 +298,5 @@
         <material name="grey" />
       </visual>
-      <!-- <collision>
+      <collision>
         <origin xyz="0.00852612 ${y_sign * 0.07450 / 2} 0.0" rpy="0.0 ${y_sign * M_PI/2} ${y_sign * M_PI/2}" />
         <geometry>
@@ -217,5 +310,5 @@
                  iyy="${1/12*0.016*(0.108**2 +0.0645**2)}" iyz="0.0"
                  izz="${1/12*0.016*(0.108**2+0.0826**2)}" />
-      </inertial> -->
+      </inertial>
     </link>
     <xacro:arm_transmission prefix="${prefix}" position="${position}" />

File: sobit_home_description/urdf/controllers.urdf.xacro (robot description, xacro)
@@ -382,5 +382,24 @@
       <!-- <command_interface name="velocity"/> -->
       <state_interface name="position">
-        <param name="initial_value">-1.5</param>
+        <param name="initial_value">0.0</param>
+      </state_interface>
+      <state_interface name="velocity"/>
+      <state_interface name="effort"/>
+    </joint>
+    <joint name="${prefix}_upper_roll_sub_joint">
+      <xacro:if value="${$(arg enable_gz)}">
+        <command_interface name="position">
+          <param name="min">-${M_PI/2}</param>
+          <param name="max">${M_PI/2}</param>
+        </command_interface>
+      </xacro:if>
+      <xacro:unless value="${$(arg enable_gz)}">
+        <param name="id">33</param>
+        <param name="control_mode">0</param>
+        <param name="interface">rs</param>
+        <param name="Return_Delay_Time">0</param>
+      </xacro:unless>
+      <state_interface name="position">
+        <param name="initial_value">0.0</param>
       </state_interface>
       <state_interface name="velocity"/>
@@ -389,5 +408,5 @@
     <joint name="${prefix}_upper_flex_joint">
       <xacro:unless value="${$(arg enable_gz)}">
-        <param name="id">33</param>
+        <param name="id">34</param>
         <param name="control_mode">0</param>
         <param name="interface">rs</param>
@@ -405,7 +424,26 @@
       <state_interface name="effort"/>
     </joint>
-    <joint name="${prefix}_elbow_joint">
-      <xacro:unless value="${$(arg enable_gz)}">
-        <param name="id">34</param>
+    <joint name="${prefix}_upper_flex_sub_joint">
+      <xacro:if value="${$(arg enable_gz)}">
+        <command_interface name="position">
+          <param name="min">-${M_PI/2}</param>
+          <param name="max">${M_PI/2}</param>
+        </command_interface>
+      </xacro:if>
+      <xacro:unless value="${$(arg enable_gz)}">
+        <param name="id">35</param>
+        <param name="control_mode">0</param>
+        <param name="interface">rs</param>
+        <param name="Return_Delay_Time">0</param>
+      </xacro:unless>
+      <state_interface name="position">
+        <param name="initial_value">0.0</param>
+      </state_interface>
+      <state_interface name="velocity"/>
+      <state_interface name="effort"/>
+    </joint>
+    <joint name="${prefix}_lower_top_joint">
+      <xacro:unless value="${$(arg enable_gz)}">
+        <param name="id">36</param>
         <param name="control_mode">0</param>
         <param name="interface">rs</param>
@@ -418,5 +456,24 @@
       <!-- <command_interface name="velocity"/> -->
       <state_interface name="position">
-        <param name="initial_value">-1.33</param>
+        <param name="initial_value">-1.571</param>
+      </state_interface>
+      <state_interface name="velocity"/>
+      <state_interface name="effort"/>
+    </joint>
+    <joint name="${prefix}_lower_top_sub_joint">
+      <xacro:if value="${$(arg enable_gz)}">
+        <command_interface name="position">
+        <param name="min">${-140*M_PI/180}</param>
+        <param name="max">0</param>
+        </command_interface>
+      </xacro:if>
+      <xacro:unless value="${$(arg enable_gz)}">
+        <param name="id">37</param>
+        <param name="control_mode">0</param>
+        <param name="interface">rs</param>
+        <param name="Return_Delay_Time">0</param>
+      </xacro:unless>
+      <state_interface name="position">
+        <param name="initial_value">1.571</param>
       </state_interface>
       <state_interface name="velocity"/>
@@ -460,5 +517,5 @@
     </joint>
   </xacro:macro>
-  <xacro:macro name="dxl_arm_right_controllers"    params="prefix enable_gz:=False">
+  <xacro:macro name="dxl_arm_right_controllers"     params="prefix enable_gz:=False">
     <joint name="${prefix}_upper_roll_joint">
       <xacro:unless value="${$(arg enable_gz)}">
@@ -474,4 +531,23 @@
       <!-- <command_interface name="velocity"/> -->
       <state_interface name="position">
+        <param name="initial_value">-1.5</param>
+      </state_interface>
+      <state_interface name="velocity"/>
+      <state_interface name="effort"/>
+    </joint>
+    <joint name="${prefix}_upper_roll_sub_joint">
+      <xacro:if value="${$(arg enable_gz)}">
+        <command_interface name="position">
+          <param name="min">-${M_PI/2}</param>
+          <param name="max">${M_PI/2}</param>
+        </command_interface>
+      </xacro:if>
+      <xacro:unless value="${$(arg enable_gz)}">
+        <param name="id">43</param>
+        <param name="control_mode">0</param>
+        <param name="interface">rs</param>
+        <param name="Return_Delay_Time">0</param>
+      </xacro:unless>
+      <state_interface name="position">
         <param name="initial_value">1.5</param>
       </state_interface>
@@ -481,5 +557,5 @@
     <joint name="${prefix}_upper_flex_joint">
       <xacro:unless value="${$(arg enable_gz)}">
-        <param name="id">43</param>
+        <param name="id">44</param>
         <param name="control_mode">0</param>
         <param name="interface">rs</param>
@@ -497,18 +573,74 @@
       <state_interface name="effort"/>
     </joint>
-    <joint name="${prefix}_elbow_joint">
-      <xacro:unless value="${$(arg enable_gz)}">
-        <param name="id">44</param>
-        <param name="control_mode">0</param>
-        <param name="interface">rs</param>
-        <param name="Return_Delay_Time">0</param>
-      </xacro:unless>
-      <command_interface name="position">
-        <param name="min">0.0</param>
-        <param name="max">${140*M_PI/180}</param>
-      </command_interface>
-      <!-- <command_interface name="velocity"/> -->
-      <state_interface name="position">
-        <param name="initial_value">1.33</param>
+    <joint name="${prefix}_upper_flex_sub_joint">
+      <xacro:if value="${$(arg enable_gz)}">
+        <command_interface name="position">
+          <param name="min">-${M_PI/2}</param>
+          <param name="max">${M_PI/2}</param>
+        </command_interface>
+      </xacro:if>
+      <xacro:unless value="${$(arg enable_gz)}">
+        <param name="id">45</param>
+        <param name="control_mode">0</param>
+        <param name="interface">rs</param>
+        <param name="Return_Delay_Time">0</param>
+      </xacro:unless>
+      <state_interface name="position">
+        <param name="initial_value">0.0</param>
+      </state_interface>
+      <state_interface name="velocity"/>
+      <state_interface name="effort"/>
+    </joint>
+    <joint name="${prefix}_lower_top_joint">
+      <xacro:unless value="${$(arg enable_gz)}">
+        <param name="id">46</param>
+        <param name="control_mode">0</param>
+        <param name="interface">rs</param>
+        <param name="Return_Delay_Time">0</param>
+      </xacro:unless>
+      <command_interface name="position">
+        <param name="min">${-140*M_PI/180}</param>
+        <param name="max">0</param>
+      </command_interface>
+      <!-- <command_interface name="velocity"/> -->
+      <state_interface name="position">
+        <param name="initial_value">-1.33</param>
+      </state_interface>
+      <state_interface name="velocity"/>
+      <state_interface name="effort"/>
+    </joint>
+    <joint name="${prefix}_lower_top_sub_joint">
+      <xacro:if value="${$(arg enable_gz)}">
+        <command_interface name="position">
+        <param name="min">${-140*M_PI/180}</param>
+        <param name="max">0</param>
+        </command_interface>
+      </xacro:if>
+      <xacro:unless value="${$(arg enable_gz)}">
+        <param name="id">47</param>
+        <param name="control_mode">0</param>
+        <param name="interface">rs</param>
+        <param name="Return_Delay_Time">0</param>
+      </xacro:unless>
+      <state_interface name="position">
+        <param name="initial_value">-1.33</param>
+      </state_interface>
+      <state_interface name="velocity"/>
+      <state_interface name="effort"/>
+    </joint>
+    <joint name="${prefix}_lower_bottom_joint">
+      <xacro:unless value="${$(arg enable_gz)}">
+        <param name="id">48</param>
+        <param name="control_mode">0</param>
+        <param name="interface">rs</param>
+        <param name="Return_Delay_Time">0</param>
+      </xacro:unless>
+      <command_interface name="position">
+        <param name="min">${-M_PI/2}</param>
+        <param name="max">${M_PI/2}</param>
+      </command_interface>
+      <!-- <command_interface name="velocity"/> -->
+      <state_interface name="position">
+        <param name="initial_value">-1.33</param>
       </state_interface>
       <state_interface name="velocity"/>
