Commit message: [UPD] Update xacro files: Add new joint arm_lower_flex. Update model infomations: mesh files, collision settings and inertials.

File: sobit_home_description/urdf/controllers.urdf.xacro (robot description, xacro)
@@ -414,6 +414,6 @@
       </xacro:unless>
       <command_interface name="position">
-        <param name="min">-${M_PI}</param>
-        <param name="max">${M_PI}</param>
+        <param name="min">-${M_PI/2}</param>
+        <param name="max">${M_P/2}</param>
       </command_interface>
       <!-- <command_interface name="velocity"/> -->
@@ -443,5 +443,5 @@
       <state_interface name="effort"/>
     </joint>
-    <joint name="${prefix}_lower_top_joint">
+    <joint name="${prefix}_elbow_joint">
       <xacro:unless value="${$(arg enable_gz)}">
         <param name="id">36</param>
@@ -451,19 +451,19 @@
       </xacro:unless>
       <command_interface name="position">
-        <param name="min">${-140*M_PI/180}</param>
+        <param name="min">${-8/9 * M_PI}</param>
         <param name="max">0</param>
       </command_interface>
       <!-- <command_interface name="velocity"/> -->
       <state_interface name="position">
-        <param name="initial_value">-1.571</param>
-      </state_interface>
-      <state_interface name="velocity"/>
-      <state_interface name="effort"/>
-    </joint>
-    <joint name="${prefix}_lower_top_sub_joint">
+        <param name="initial_value">1.571</param>
+      </state_interface>
+      <state_interface name="velocity"/>
+      <state_interface name="effort"/>
+    </joint>
+    <joint name="${prefix}_elbow_sub_joint">
       <xacro:if value="${$(arg enable_gz)}">
         <command_interface name="position">
-        <param name="min">${2/3*M_PI}</param>
-        <param name="max">0</param>
+        <param name="min">0</param>
+        <param name="max">${8/9 * M_PI}</param>
         </command_interface>
       </xacro:if>
@@ -475,5 +475,24 @@
       </xacro:unless>
       <state_interface name="position">
-        <param name="initial_value">1.571</param>
+        <param name="initial_value">-1.571</param>
+      </state_interface>
+      <state_interface name="velocity"/>
+      <state_interface name="effort"/>
+    </joint>
+    <joint name="${prefix}_lower_flex_joint">
+      <xacro:if value="${$(arg enable_gz)}">
+        <command_interface name="position">
+        <param name="min">-${M_PI/2}</param>
+        <param name="max">${M_PI/2}</param>
+        </command_interface>
+      </xacro:if>
+      <xacro:unless value="${$(arg enable_gz)}">
+        <param name="id">37</param>
+        <param name="control_mode">0</param>
+        <param name="interface">rs</param>
+        <param name="Return_Delay_Time">0</param>
+      </xacro:unless>
+      <state_interface name="position">
+        <param name="initial_value">0.0</param>
       </state_interface>
       <state_interface name="velocity"/>
@@ -482,5 +501,5 @@
     <joint name="${prefix}_wrist_tilt_joint">
       <xacro:unless value="${$(arg enable_gz)}">
-        <param name="id">35</param>
+        <param name="id">39</param>
         <param name="control_mode">0</param>
         <param name="interface">rs</param>
@@ -500,5 +519,5 @@
     <joint name="${prefix}_wrist_roll_joint">
       <xacro:unless value="${$(arg enable_gz)}">
-        <param name="id">36</param>
+        <param name="id">40</param>
         <param name="control_mode">0</param>
         <param name="interface">rs</param>
@@ -563,6 +582,6 @@
       </xacro:unless>
       <command_interface name="position">
-        <param name="min">-${M_PI}</param>
-        <param name="max">${M_PI}</param>
+        <param name="min">-${M_PI/2}</param>
+        <param name="max">${M_PI/2}</param>
       </command_interface>
       <!-- <command_interface name="velocity"/> -->
@@ -592,5 +611,5 @@
       <state_interface name="effort"/>
     </joint>
-    <joint name="${prefix}_lower_top_joint">
+    <joint name="${prefix}_elbow_joint">
       <xacro:unless value="${$(arg enable_gz)}">
         <param name="id">46</param>
@@ -600,18 +619,18 @@
       </xacro:unless>
       <command_interface name="position">
-        <param name="min">${-140*M_PI/180}</param>
-        <param name="max">0</param>
-      </command_interface>
-      <!-- <command_interface name="velocity"/> -->
-      <state_interface name="position">
-        <param name="initial_value">-1.33</param>
-      </state_interface>
-      <state_interface name="velocity"/>
-      <state_interface name="effort"/>
-    </joint>
-    <joint name="${prefix}_lower_top_sub_joint">
+        <param name="min">0</param>
+        <param name="max">${8/9 * M_PI}</param>
+      </command_interface>
+      <!-- <command_interface name="velocity"/> -->
+      <state_interface name="position">
+        <param name="initial_value">1.571</param>
+      </state_interface>
+      <state_interface name="velocity"/>
+      <state_interface name="effort"/>
+    </joint>
+    <joint name="${prefix}_elbow_sub_joint">
       <xacro:if value="${$(arg enable_gz)}">
         <command_interface name="position">
-        <param name="min">${-140*M_PI/180}</param>
+        <param name="min">-${8/9 * M_PI}</param>
         <param name="max">0</param>
         </command_interface>
@@ -624,10 +643,10 @@
       </xacro:unless>
       <state_interface name="position">
-        <param name="initial_value">-1.33</param>
-      </state_interface>
-      <state_interface name="velocity"/>
-      <state_interface name="effort"/>
-    </joint>
-    <joint name="${prefix}_lower_bottom_joint">
+        <param name="initial_value">-1.571</param>
+      </state_interface>
+      <state_interface name="velocity"/>
+      <state_interface name="effort"/>
+    </joint>
+    <joint name="${prefix}_lower_flex_joint">
       <xacro:unless value="${$(arg enable_gz)}">
         <param name="id">48</param>
@@ -637,10 +656,10 @@
       </xacro:unless>
       <command_interface name="position">
-        <param name="min">${-M_PI/2}</param>
-        <param name="max">${M_PI/2}</param>
-      </command_interface>
-      <!-- <command_interface name="velocity"/> -->
-      <state_interface name="position">
-        <param name="initial_value">-1.33</param>
+        <param name="min">-${M_PI/2}</param>
+        <param name="max">${M_PI/2}</param>
+      </command_interface>
+      <!-- <command_interface name="velocity"/> -->
+      <state_interface name="position">
+        <param name="initial_value">0.0</param>
       </state_interface>
       <state_interface name="velocity"/>
@@ -649,5 +668,5 @@
     <joint name="${prefix}_wrist_tilt_joint">
       <xacro:unless value="${$(arg enable_gz)}">
-        <param name="id">45</param>
+        <param name="id">49</param>
         <param name="control_mode">0</param>
         <param name="interface">rs</param>
@@ -667,5 +686,5 @@
     <joint name="${prefix}_wrist_roll_joint">
       <xacro:unless value="${$(arg enable_gz)}">
-        <param name="id">46</param>
+        <param name="id">50</param>
         <param name="control_mode">0</param>
         <param name="interface">rs</param>
