Commit message: [UPD] urdf files

File: sobit_home_description/urdf/arm/arm.urdf.xacro (robot description, xacro)
@@ -3,17 +3,17 @@
        xmlns:xacro="http://ros.org/wiki/xacro" >
   <xacro:include filename="$(find sobit_home_description)/urdf/arm/arm.transmission.xacro" />
-  <xacro:macro name="arm" params="prefix parent" >
-    <joint name="${prefix}_base_joint" type="fixed" >
+  <xacro:macro name="arm" params="prefix position parent" >
+    <joint name="${prefix}_${position}_base_joint" type="fixed" >
       <parent link="${parent}" />
-      <child link="${prefix}_base_link" />
-      <origin xyz="0.065 0.0 0.0" rpy="0.0 0.0 0.0" />
+      <child link="${prefix}_${position}_base_link" />
+      <origin xyz="0.0 0.079 0.0" rpy="0.0 0.0 0.0" />
     </joint>
-    <link name="${prefix}_base_link" >
+    <link name="${prefix}_${position}_base_link" >
       <visual>
-        <origin xyz="0.0 0.0 0.0" rpy="${M_PI/2} 0.0 0.0" />
+        <origin xyz="0.0 0.0 0.0" rpy="${M_PI/2} 0.0 ${M_PI/2}" />
         <geometry>
-          <mesh filename="file://$(find sobit_home_description)/meshes/arm/arm_base.stl" scale="0.001 0.001 0.001" />
+          <mesh filename="file://$(find sobit_home_description)/meshes/arm/arm_scapula.stl" scale="0.001 0.001 0.001" />
         </geometry>
-        <material name="black" />
+        <material name="grey" />
       </visual>
       <collision>
@@ -31,19 +31,18 @@
       </inertial>
     </link>
-    <joint name="${prefix}_shoulder_1_tilt_joint" type="revolute" >
-      <parent link="${prefix}_base_link" />
-      <child link="${prefix}_shoulder_1_tilt_link" />
-      <origin xyz="0.1560 0.0 0.0215" rpy="0.0 0.0 0.0 " />
+    <joint name="${prefix}_${position}_shoulder_tilt_joint" type="revolute" >
+      <parent link="${prefix}_${position}_base_link" />
+      <child link="${prefix}_${position}_shoulder_tilt_link" />
+      <origin xyz="0.0 0.1355 0.0" rpy="0.0 0.0 0.0" />
       <axis xyz="0.0 -1.0 0.0 " />
       <limit lower="${-M_PI/2}" upper="${M_PI/2}" effort="${10.6*2}" velocity="11.031179004" />
-      <!-- <dynamics damping="0.2" friction="0" /> -->
     </joint>
-    <link name="${prefix}_shoulder_1_tilt_link" >
+    <link name="${prefix}_${position}_shoulder_tilt_link" >
       <visual>
-        <origin xyz="0.0 0.0 0.0" rpy="${M_PI/2} 0.0 ${M_PI/2}" />
+        <origin xyz="0.0 0.0 0.0" rpy="0.0 0.0 ${M_PI/2}" />
         <geometry>
-          <mesh filename="file://$(find sobit_home_description)/meshes/arm/arm_upper.stl" scale="0.001 0.001 0.001" />
+          <mesh filename="file://$(find sobit_home_description)/meshes/arm/arm_shoulder.stl" scale="0.001 0.001 0.001" />
         </geometry>
-        <material name="black" />
+        <material name="grey" />
       </visual>
       <collision>
@@ -61,123 +60,62 @@
       </inertial>
     </link>
-    <joint name="${prefix}_shoulder_2_tilt_joint" type="revolute" >
-      <parent link="${prefix}_base_link" />
-      <child link="${prefix}_shoulder_2_tilt_link" />
-      <origin xyz="0.1560 0.0 0.0215" rpy="0.0 0.0 ${M_PI}" />
-      <axis xyz="0.0 1.0 0.0 " />
-      <mimic joint="${prefix}_shoulder_1_tilt_joint" multiplier="1" offset="0" />
+    <joint name="${prefix}_${position}_upper_roll_joint" type="revolute" >
+      <parent link="${prefix}_${position}_shoulder_tilt_link" />
+      <child link="${prefix}_${position}_upper_roll_link" />
+      <origin xyz="0.0 0.0 -0.09465" rpy="0.0 0.0 0.0" />
+      <axis xyz="0.0 -1.0 0.0 " />
       <limit lower="${-M_PI/2}" upper="${M_PI/2}" effort="${10.6*2}" velocity="11.031179004" />
-      <dynamics damping="0.2" friction="0" />
     </joint>
-    <link name="${prefix}_shoulder_2_tilt_link" />
-    <joint name="${prefix}_elbow_upper_1_tilt_joint" type="revolute" >
-      <parent link="${prefix}_shoulder_1_tilt_link" />
-      <child link="${prefix}_elbow_upper_1_tilt_link" />
-      <origin xyz="0.1500 0.0 0.0" rpy="0.0 0.0 0.0" />
-      <axis xyz="0.0 -1.0 0.0 " />
-      <limit lower="${-M_PI/2}" upper="${M_PI/2}" effort="${4.1*2}" velocity="9.59233" />
-      <!-- <dynamics damping="0.2" friction="0" /> -->
-    </joint>
-    <link name="${prefix}_elbow_upper_1_tilt_link" >
+    <link name="${prefix}_${position}_upper_roll_link" >
       <visual>
-        <origin xyz="0.0 0.0 0.0" rpy="${M_PI/2} 0.0 ${M_PI/2}" />
+        <origin xyz="0.0 0.0 0.0" rpy="0.0 0.0 ${M_PI/2}" />
         <geometry>
-          <mesh filename="file://$(find sobit_home_description)/meshes/arm/arm_inner.stl" scale="0.001 0.001 0.001" />
+          <mesh filename="file://$(find sobit_home_description)/meshes/arm/arm_upper_roll.stl" scale="0.001 0.001 0.001" />
         </geometry>
-        <material name="black" />
+        <material name="grey" />
       </visual>
       <collision>
-        <origin xyz="${0.023+0.127/2} 0.0 0.0" rpy="0.0 0.0 0.0" />
+        <origin xyz="${0.1166/2+0.0224} 0.0 0.0" rpy="0.0 0.0 0.0" />
         <geometry>
-          <box size="0.127 0.048 0.035" />
+          <box size="0.1166 0.124 0.043" />
         </geometry>
       </collision>
       <inertial>
-        <origin xyz="${0.023+0.127/2} 0.0 0.0" rpy="0.0 0.0 ${M_PI/2}" />
+        <origin xyz="${0.1166/2+0.0224} 0.0 0.0" rpy="0.0 0.0 ${M_PI/2}" />
         <mass value="0.08" />
-        <inertia ixx="${1/12*0.08*(0.127**2+0.035**2)}" ixy="0.0" ixz="0.0"
-                 iyy="${1/12*0.08*(0.048**2+0.035**2)}" iyz="0.0"
-                 izz="${1/12*0.08*(0.127**2+0.048**2)}" />
+        <inertia ixx="${1/12*0.08*(0.1166**2+0.043**2)}" ixy="0.0" ixz="0.0"
+                 iyy="${1/12*0.08*(0.124**2 +0.043**2)}" iyz="0.0"
+                 izz="${1/12*0.08*(0.1166**2+0.124**2)}" />
       </inertial>
     </link>
-    <joint name="${prefix}_elbow_upper_2_tilt_joint" type="revolute" >
-      <parent link="${prefix}_shoulder_1_tilt_link" />
-      <child link="${prefix}_elbow_upper_2_tilt_link" />
-      <origin xyz="0.1500 0.0 0.0" rpy="0.0 0.0 ${M_PI}" />
-      <axis xyz="0.0 1.0 0.0 " />
-      <mimic joint="${prefix}_elbow_upper_1_tilt_joint" multiplier="1" offset="0" />
-      <limit lower="${-M_PI/2}" upper="${M_PI/2}" effort="${4.1*2}" velocity="9.59233" />
-      <dynamics damping="0.2" friction="0" />
+    <joint name="${prefix}_${position}_upper_flex_joint" type="revolute" >
+      <parent link="${prefix}_${position}_upper_roll_link" />
+      <child link="${prefix}_${position}_upper_flex_link" />
+      <origin xyz="0.0 0.0 -0.209821" rpy="0.0 0.0 0.0" />
+      <axis xyz="0.0 -1.0 0.0 " />
+      <limit lower="${-M_PI/2}" upper="${M_PI/2}" effort="${10.6*2}" velocity="11.031179004" />
     </joint>
-    <link name="${prefix}_elbow_upper_2_tilt_link" />
-    <joint name="${prefix}_elbow_lower_tilt_joint" type="revolute" >
-      <parent link="${prefix}_elbow_upper_1_tilt_link" />
-      <child link="${prefix}_elbow_lower_tilt_link" />
-      <origin xyz="0.1500 0.0 0.0" rpy="0.0 0.0 0.0" />
-      <axis xyz="0.0 -1.0 0.0 " />
-      <limit lower="${-M_PI/2}" upper="${M_PI/2}" effort="4.1" velocity="4.796165" />
-      <!-- <dynamics damping="0.2" friction="0" /> -->
-    </joint>
-    <link name="${prefix}_elbow_lower_tilt_link" >
+    <link name="${prefix}_${position}_upper_flex_link" >
       <visual>
-        <origin xyz="0.0 0.0 0.0" rpy="${M_PI/2} 0.0 ${M_PI/2}" />
+        <origin xyz="0.0 0.0 0.0" rpy="0.0 0.0 ${M_PI/2}" />
         <geometry>
-          <mesh filename="file://$(find sobit_home_description)/meshes/arm/arm_elbow_lower_tilt.stl" scale="0.001 0.001 0.001" />
+          <mesh filename="file://$(find sobit_home_description)/meshes/arm/arm_upper_flex.stl" scale="0.001 0.001 0.001" />
         </geometry>
-        <material name="black" />
+        <material name="grey" />
       </visual>
       <collision>
-        <origin xyz="${0.028-0.005/2} 0.0 -${(0.0215-0.01825)/2}" rpy="0.0 0.0 0.0" />
+        <origin xyz="${0.1166/2+0.0224} 0.0 0.0" rpy="0.0 0.0 0.0" />
         <geometry>
-          <box size="0.005 0.041 0.024" />
+          <box size="0.1166 0.124 0.043" />
         </geometry>
       </collision>
       <inertial>
-        <origin xyz="${0.028-0.005/2} 0.0 -${(0.0215-0.01825)/2}" rpy="0.0 0.0 ${M_PI/2}" />
+        <origin xyz="${0.1166/2+0.0224} 0.0 0.0" rpy="0.0 0.0 ${M_PI/2}" />
         <mass value="0.08" />
-        <inertia ixx="${1/12*0.08*(0.005**2+0.024**2)}" ixy="0.0" ixz="0.0"
-                 iyy="${1/12*0.08*(0.041**2+0.024**2)}" iyz="0.0"
-                 izz="${1/12*0.08*(0.005**2+0.041**2)}" />
+        <inertia ixx="${1/12*0.08*(0.1166**2+0.043**2)}" ixy="0.0" ixz="0.0"
+                 iyy="${1/12*0.08*(0.124**2 +0.043**2)}" iyz="0.0"
+                 izz="${1/12*0.08*(0.1166**2+0.124**2)}" />
       </inertial>
     </link>
-    <joint name="${prefix}_elbow_lower_pan_joint" type="revolute" >
-      <parent link="${prefix}_elbow_lower_tilt_link" />
-      <child link="${prefix}_elbow_lower_pan_link" />
-      <origin xyz="0.028 0.0 0.0" rpy="0.0 0.0 0.0" />
-      <axis xyz="1.0 0.0 0.0 " />
-      <limit lower="${-M_PI/2}" upper="${M_PI/2}" effort="4.1" velocity="4.796165" />
-      <!-- <dynamics damping="0.2" friction="0" /> -->
-    </joint>
-    <link name="${prefix}_elbow_lower_pan_link" >
-      <visual>
-        <origin xyz="0.0 0.0 0.0" rpy="${M_PI/2} 0.0 ${M_PI/2}" />
-        <geometry>
-          <mesh filename="file://$(find sobit_home_description)/meshes/arm/arm_elbow_lower_pan.stl" scale="0.001 0.001 0.001" />
-        </geometry>
-        <material name="black" />
-      </visual>
-      <collision>
-        <origin xyz="${0.002+0.120/2} 0.0 -${(0.0215-0.01825)/2}" rpy="0.0 0.0 0.0" />
-        <geometry>
-          <box size="0.120 0.048 0.03975" />
-        </geometry>
-      </collision>
-      <inertial>
-        <origin xyz="${0.002+0.120/2} 0.0 -${(0.0215-0.01825)/2}" rpy="0.0 0.0 ${M_PI/2}" />
-        <mass value="0.08" />
-        <inertia ixx="${1/12*0.08*(0.120**2+0.03975**2)}" ixy="0.0" ixz="0.0"
-                 iyy="${1/12*0.08*(0.048**2+0.03975**2)}" iyz="0.0"
-                 izz="${1/12*0.08*(0.120**2+0.048**2)}" />
-      </inertial>
-    </link>
-    <joint name="${prefix}_wrist_tilt_joint" type="revolute" >
-      <parent link="${prefix}_elbow_lower_pan_link" />
-      <child link="${prefix}_wrist_tilt_link" />
-      <origin xyz="0.122009 0.0 0.0" rpy="0.0 0.0 0.0" />
-      <axis xyz="0.0 -1.0 0.0" />
-      <limit lower="${-M_PI/2}" upper="${M_PI/2}" effort="4.1" velocity="4.796165" />
-      <!-- <dynamics damping="0.2" friction="0" /> -->
-    </joint>
-    <link name="${prefix}_wrist_tilt_link" />
     <xacro:arm_transmission prefix="${prefix}" />
   </xacro:macro>

File: sobit_home_description/urdf/body/body.urdf.xacro (robot description, xacro)
@@ -5,5 +5,5 @@
   <xacro:macro name="body" params="prefix parent" >
     <joint name="${prefix}_joint" type="fixed" >
-      <origin xyz="0.0 0.0 0.565" rpy="0.0 0.0 0.0" /> <!-- TODO: height -->
+      <origin xyz="0.0 -0.0525 0.565" rpy="0.0 0.0 0.0" />
       <parent link="${parent}" />
       <child link="${prefix}_link" />
@@ -32,9 +32,9 @@
     </link>
     <joint name="linear_actuator_joint" type="prismatic" >
-      <origin xyz="0.0961 0.0425 0.0" rpy="0.0 0.0 0.0" />
+      <origin xyz="0.0961 0.0525 0.0" rpy="0.0 0.0 0.0" />
       <parent link="${prefix}_link" />
       <child link="linear_actuator_link" />
       <axis xyz="0.0 0.0 1.0" />
-      <limit lower="0.0" upper="0.3" effort="50.0" velocity="0.1" /> <!-- TODO: limit -->
+      <limit lower="-0.4" upper="0.4" effort="50.0" velocity="0.1" />
     </joint>
     <link name="linear_actuator_link" >
