Commit message: [UPD] update arm controller definitions and adjust joint parameters

File: sobit_home_description/urdf/arm/arm.urdf.xacro (robot description, xacro)
@@ -46,5 +46,5 @@
       <parent link="${prefix}_${position}_base_link" />
       <child link="${prefix}_${position}_shoulder_tilt_link" />
-      <origin xyz="0.0 ${y_sign * 0.19875} 0.0" rpy="0.0 0.0 0.0" />
+      <origin xyz="0.0 ${y_sign * 0.126} 0.0" rpy="0.0 0.0 0.0" />
       <axis xyz="0.0 -1.0 0.0 " />
       <limit lower="${-M_PI/2}" upper="${M_PI/2}" effort="${10.6*2}" velocity="11.031179004" />
@@ -52,5 +52,5 @@
     <link name="${prefix}_${position}_shoulder_tilt_link" >
       <visual>
-        <origin xyz="0.0 0.0 0.0" rpy="0.0 0.0 ${M_PI/2+yaw_rot}" />
+        <origin xyz="0.0 ${y_sign * 0.07275} 0.0" rpy="0.0 0.0 ${M_PI/2+yaw_rot}" />
         <geometry>
           <mesh filename="file://$(find sobit_home_description)/meshes/arm/arm_shoulder.stl" scale="0.001 0.001 0.001" />
@@ -75,5 +75,5 @@
       <parent link="${prefix}_${position}_shoulder_tilt_link" />
       <child link="${prefix}_${position}_upper_roll_link" />
-      <origin xyz="0.0 0.0 0.0" rpy="0.0 0.0 0.0" />
+      <origin xyz="0.0 ${y_sign * 0.0725} 0.0" rpy="0.0 0.0 0.0" />
       <axis xyz="1.0 0.0 0.0 " />
       <limit lower="${upper_roll_limit_lower}" upper="${upper_roll_limit_upper}" effort="${10.6*2}" velocity="11.031179004" />

File: sobit_home_description/urdf/controllers.urdf.xacro (robot description, xacro)
@@ -156,6 +156,41 @@
         </xacro:unless>
       </hardware>
-      <joint name="arm_left_shoulder_tilt_joint">
-      <joint name="${name}_joint">
+      <xacro:arm_controllers position="left"/>
+      <xacro:arm_controllers position="right"/>
+      <joint name="head_pan_joint">
+        <xacro:unless value="${$(arg enable_gz)}">
+          <param name="id">21</param>
+          <param name="control_mode">3</param>
+          <param name="interface">rp</param>
+        </xacro:unless>
+        <command_interface name="position">
+          <param name="min">-0.4</param>
+          <param name="max">0.4</param>
+        </command_interface>
+        <!-- <command_interface name="velocity"/> -->
+        <state_interface name="position">
+          <param name="initial_value">0.0</param>
+        </state_interface>
+        <state_interface name="velocity"/>
+        <state_interface name="effort"/>
+      </joint>
+      <joint name="head_tilt_joint">
+        <xacro:unless value="${$(arg enable_gz)}">
+          <param name="id">21</param>
+          <param name="control_mode">3</param>
+          <param name="interface">rp</param>
+        </xacro:unless>
+        <command_interface name="position">
+          <param name="min">-0.4</param>
+          <param name="max">0.4</param>
+        </command_interface>
+        <!-- <command_interface name="velocity"/> -->
+        <state_interface name="position">
+          <param name="initial_value">0.0</param>
+        </state_interface>
+        <state_interface name="velocity"/>
+        <state_interface name="effort"/>
+      </joint>
+      <joint name="linear_actuator_joint">
         <xacro:unless value="${$(arg enable_gz)}">
           <param name="id">20</param>
@@ -167,80 +202,14 @@
           <param name="max">0.4</param>
         </command_interface>
-        <!-- <command_interface name="velocity"/> -->
-        <state_interface name="position">
-          <param name="initial_value">0.0</param>
-        </state_interface>
-        <state_interface name="velocity"/>
-        <state_interface name="effort"/>
-      </joint>
-      <joint name="arm_left_upper_roll_joint">
-        <xacro:unless value="${$(arg enable_gz)}">
-          <param name="id">21</param>
-          <param name="control_mode">3</param>
-          <param name="interface">rp</param>
-        </xacro:unless>
-        <command_interface name="position">
-          <param name="min">-0.4</param>
-          <param name="max">0.4</param>
-        </command_interface>
-        <!-- <command_interface name="velocity"/> -->
-        <state_interface name="position">
-          <param name="initial_value">0.0</param>
-        </state_interface>
-        <state_interface name="velocity"/>
-        <state_interface name="effort"/>
-      </joint>
-      <joint name="arm_left_upper_flex_joint">
-        <xacro:unless value="${$(arg enable_gz)}">
-          <param name="id">21</param>
-          <param name="control_mode">3</param>
-          <param name="interface">rp</param>
-        </xacro:unless>
-        <command_interface name="position">
-          <param name="min">-0.4</param>
-          <param name="max">0.4</param>
-        </command_interface>
-        <!-- <command_interface name="velocity"/> -->
-        <state_interface name="position">
-          <param name="initial_value">0.0</param>
-        </state_interface>
-        <state_interface name="velocity"/>
-        <state_interface name="effort"/>
-      </joint>
-      <joint name="arm_left_elbow_joint">
-        <xacro:unless value="${$(arg enable_gz)}">
-          <param name="id">21</param>
-          <param name="control_mode">3</param>
-          <param name="interface">rp</param>
-        </xacro:unless>
-        <command_interface name="position">
-          <param name="min">-0.4</param>
-          <param name="max">0.4</param>
-        </command_interface>
-        <!-- <command_interface name="velocity"/> -->
-        <state_interface name="position">
-          <param name="initial_value">0.0</param>
-        </state_interface>
-        <state_interface name="velocity"/>
-        <state_interface name="effort"/>
-      </joint>
-      <joint name="arm_left_wrist_joint">
-        <xacro:unless value="${$(arg enable_gz)}">
-          <param name="id">21</param>
-          <param name="control_mode">3</param>
-          <param name="interface">rp</param>
-        </xacro:unless>
-        <command_interface name="position">
-          <param name="min">-0.4</param>
-          <param name="max">0.4</param>
-        </command_interface>
-        <!-- <command_interface name="velocity"/> -->
-        <state_interface name="position">
-          <param name="initial_value">0.0</param>
-        </state_interface>
-        <state_interface name="velocity"/>
-        <state_interface name="effort"/>
-      </joint>
-      <joint name="arm_right_shoulder_tilt_joint">
+        <state_interface name="position">
+          <param name="initial_value">0.0</param>
+        </state_interface>
+        <state_interface name="velocity"/>
+        <state_interface name="effort"/>
+      </joint>
+    </ros2_control>
+  </xacro:macro>
+  <xacro:macro name="arm_controllers" params="position">
+      <joint name="arm_${position}_shoulder_tilt_joint">
         <xacro:unless value="${$(arg enable_gz)}">
           <param name="id">20</param>
@@ -259,124 +228,72 @@
         <state_interface name="effort"/>
       </joint>
-      <joint name="arm_right_upper_roll_joint">
-        <xacro:unless value="${$(arg enable_gz)}">
-          <param name="id">21</param>
-          <param name="control_mode">3</param>
-          <param name="interface">rp</param>
-        </xacro:unless>
-        <command_interface name="position">
-          <param name="min">-0.4</param>
-          <param name="max">0.4</param>
-        </command_interface>
-        <!-- <command_interface name="velocity"/> -->
-        <state_interface name="position">
-          <param name="initial_value">0.0</param>
-        </state_interface>
-        <state_interface name="velocity"/>
-        <state_interface name="effort"/>
-      </joint>
-      <joint name="arm_right_upper_flex_joint">
-        <xacro:unless value="${$(arg enable_gz)}">
-          <param name="id">21</param>
-          <param name="control_mode">3</param>
-          <param name="interface">rp</param>
-        </xacro:unless>
-        <command_interface name="position">
-          <param name="min">-0.4</param>
-          <param name="max">0.4</param>
-        </command_interface>
-        <!-- <command_interface name="velocity"/> -->
-        <state_interface name="position">
-          <param name="initial_value">0.0</param>
-        </state_interface>
-        <state_interface name="velocity"/>
-        <state_interface name="effort"/>
-      </joint>
-      <joint name="arm_right_elbow_joint">
-        <xacro:unless value="${$(arg enable_gz)}">
-          <param name="id">21</param>
-          <param name="control_mode">3</param>
-          <param name="interface">rp</param>
-        </xacro:unless>
-        <command_interface name="position">
-          <param name="min">-0.4</param>
-          <param name="max">0.4</param>
-        </command_interface>
-        <!-- <command_interface name="velocity"/> -->
-        <state_interface name="position">
-          <param name="initial_value">0.0</param>
-        </state_interface>
-        <state_interface name="velocity"/>
-        <state_interface name="effort"/>
-      </joint>
-      <joint name="arm_right_wrist_joint">
-        <xacro:unless value="${$(arg enable_gz)}">
-          <param name="id">21</param>
-          <param name="control_mode">3</param>
-          <param name="interface">rp</param>
-        </xacro:unless>
-        <command_interface name="position">
-          <param name="min">-0.4</param>
-          <param name="max">0.4</param>
-        </command_interface>
-        <!-- <command_interface name="velocity"/> -->
-        <state_interface name="position">
-          <param name="initial_value">0.0</param>
-        </state_interface>
-        <state_interface name="velocity"/>
-        <state_interface name="effort"/>
-      </joint>
-      <joint name="head_pan_joint">
-        <xacro:unless value="${$(arg enable_gz)}">
-          <param name="id">21</param>
-          <param name="control_mode">3</param>
-          <param name="interface">rp</param>
-        </xacro:unless>
-        <command_interface name="position">
-          <param name="min">-0.4</param>
-          <param name="max">0.4</param>
-        </command_interface>
-        <!-- <command_interface name="velocity"/> -->
-        <state_interface name="position">
-          <param name="initial_value">0.0</param>
-        </state_interface>
-        <state_interface name="velocity"/>
-        <state_interface name="effort"/>
-      </joint>
-      <joint name="head_tilt_joint">
-        <xacro:unless value="${$(arg enable_gz)}">
-          <param name="id">21</param>
-          <param name="control_mode">3</param>
-          <param name="interface">rp</param>
-        </xacro:unless>
-        <command_interface name="position">
-          <param name="min">-0.4</param>
-          <param name="max">0.4</param>
-        </command_interface>
-        <!-- <command_interface name="velocity"/> -->
-        <state_interface name="position">
-          <param name="initial_value">0.0</param>
-        </state_interface>
-        <state_interface name="velocity"/>
-        <state_interface name="effort"/>
-      </joint>
-      <joint name="linear_actuator_joint">
-        <xacro:unless value="${$(arg enable_gz)}">
-          <param name="id">20</param>
-          <param name="control_mode">3</param>
-          <param name="interface">rp</param>
-        </xacro:unless>
-        <command_interface name="position">
-          <param name="min">-0.4</param>
-          <param name="max">0.4</param>
-        </command_interface>
-        <!-- <command_interface name="velocity"/> -->
-        <state_interface name="position">
-          <param name="initial_value">0.0</param>
-        </state_interface>
-        <state_interface name="velocity"/>
-        <state_interface name="effort"/>
-      </joint>
-    </ros2_control>
+      <joint name="arm_${position}_upper_roll_joint">
+        <xacro:unless value="${$(arg enable_gz)}">
+          <param name="id">21</param>
+          <param name="control_mode">3</param>
+          <param name="interface">rp</param>
+        </xacro:unless>
+        <command_interface name="position">
+          <param name="min">-0.4</param>
+          <param name="max">0.4</param>
+        </command_interface>
+        <!-- <command_interface name="velocity"/> -->
+        <state_interface name="position">
+          <param name="initial_value">0.0</param>
+        </state_interface>
+        <state_interface name="velocity"/>
+        <state_interface name="effort"/>
+      </joint>
+      <joint name="arm_${position}_upper_flex_joint">
+        <xacro:unless value="${$(arg enable_gz)}">
+          <param name="id">21</param>
+          <param name="control_mode">3</param>
+          <param name="interface">rp</param>
+        </xacro:unless>
+        <command_interface name="position">
+          <param name="min">-0.4</param>
+          <param name="max">0.4</param>
+        </command_interface>
+        <!-- <command_interface name="velocity"/> -->
+        <state_interface name="position">
+          <param name="initial_value">0.0</param>
+        </state_interface>
+        <state_interface name="velocity"/>
+        <state_interface name="effort"/>
+      </joint>
+      <joint name="arm_${position}_elbow_joint">
+        <xacro:unless value="${$(arg enable_gz)}">
+          <param name="id">21</param>
+          <param name="control_mode">3</param>
+          <param name="interface">rp</param>
+        </xacro:unless>
+        <command_interface name="position">
+          <param name="min">-0.4</param>
+          <param name="max">0.4</param>
+        </command_interface>
+        <!-- <command_interface name="velocity"/> -->
+        <state_interface name="position">
+          <param name="initial_value">0.0</param>
+        </state_interface>
+        <state_interface name="velocity"/>
+        <state_interface name="effort"/>
+      </joint>
+      <joint name="arm_${position}_wrist_joint">
+        <xacro:unless value="${$(arg enable_gz)}">
+          <param name="id">21</param>
+          <param name="control_mode">3</param>
+          <param name="interface">rp</param>
+        </xacro:unless>
+        <command_interface name="position">
+          <param name="min">-0.4</param>
+          <param name="max">0.4</param>
+        </command_interface>
+        <!-- <command_interface name="velocity"/> -->
+        <state_interface name="position">
+          <param name="initial_value">0.0</param>
+        </state_interface>
+        <state_interface name="velocity"/>
+        <state_interface name="effort"/>
+      </joint>
   </xacro:macro>
   <xacro:macro name="ros2_controllers" params="enable_gz:=False robot_name:=sobit_home">
