Commit message: [UPD] collision properties

File: sobit_home_description/urdf/arm/arm.urdf.xacro (robot description, xacro)
@@ -30,7 +30,7 @@
       </visual>
       <collision>
-        <origin xyz="${0.140/2} 0.0 ${0.043/2}" rpy="0.0 0.0 0.0" />
+        <origin xyz="0.0 ${y_sign * 0.124/2} 0.0" rpy="0.0 0.0 0.0" />
         <geometry>
-          <box size="0.140 0.156 0.043" />
+          <box size="0.054 0.124 0.054" />
         </geometry>
       </collision>
@@ -52,5 +52,5 @@
     <link name="${prefix}_${position}_shoulder_tilt_link" >
       <visual>
-        <origin xyz="0.0 ${y_sign * 0.07275} 0.0" rpy="0.0 0.0 ${M_PI/2+yaw_rot}" />
+        <origin xyz="0.0 0.0  0.0" rpy="0.0 0.0 ${M_PI/2+yaw_rot}" />
         <geometry>
           <mesh filename="file://$(find sobit_home_description)/meshes/arm/arm_shoulder.stl" scale="0.001 0.001 0.001" />
@@ -59,7 +59,8 @@
       </visual>
       <collision>
-        <origin xyz="${0.1166/2+0.0224} 0.0 0.0" rpy="0.0 0.0 0.0" />
+        <origin xyz="0 ${y_sign * 0.104/2} 0.0" rpy="0.0 0.0 0.0" />
         <geometry>
-          <box size="0.1166 0.124 0.043" />
+          <!-- <cylinder length="0.104" radius="${0.08/2}" /> -->
+          <box size="0.0535 0.104 0.045" />
         </geometry>
       </collision>
@@ -87,10 +88,10 @@
         <material name="grey" />
       </visual>
-      <collision>
-        <origin xyz="${0.1166/2+0.0224} 0.0 0.0" rpy="0.0 0.0 0.0" />
+      <!-- <collision>
+        <origin xyz="0.0 0.0 0.0" rpy="0.0 0.0 0.0" />
         <geometry>
           <box size="0.1166 0.124 0.043" />
         </geometry>
-      </collision>
+      </collision> -->
       <inertial>
         <origin xyz="${0.1166/2+0.0224} 0.0 0.0" rpy="0.0 0.0 ${M_PI/2}" />
@@ -101,5 +102,5 @@
       </inertial>
     </link>
-    <joint name="${prefix}_${position}_upper_flex_joint" type="revolute" >
+    <!-- <joint name="${prefix}_${position}_upper_flex_joint" type="revolute" >
       <parent link="${prefix}_${position}_upper_roll_link" />
       <child link="${prefix}_${position}_upper_flex_link" />
@@ -187,5 +188,5 @@
                  izz="${1/12*0.08*(0.1166**2+0.124**2)}" />
       </inertial>
-    </link>
+    </link> -->
     <xacro:arm_transmission prefix="${prefix}" position="${position}" />
   </xacro:macro>

File: sobit_home_description/urdf/body/body.urdf.xacro (robot description, xacro)
@@ -18,7 +18,7 @@
       </visual>
       <collision>
-        <origin xyz="-${0.02893+0.3/2} 0.0 ${0.034-0.489/2}" rpy="0.0 0.0 0.0" />
+        <origin xyz="0.0 -0.053 -0.018" rpy="0.0 0.0 0.0" />
         <geometry>
-          <box size="${(0.02893+0.3/2)*2} 0.3965 0.489"/>
+          <box size="0.0675 0.19 1.07"/>
         </geometry>
       </collision>
@@ -47,7 +47,7 @@
       </visual>
       <collision>
-        <origin xyz="-${0.02893+0.3/2} 0.0 ${0.034-0.489/2}" rpy="0.0 0.0 0.0" />
+        <origin xyz="0.0 0.0 0.0" rpy="0.0 0.0 0.0" />
         <geometry>
-          <box size="${(0.02893+0.3/2)*2} 0.3965 0.489"/>
+          <box size="0.15 0.35 0.15"/>
         </geometry>
       </collision>

File: sobit_home_description/urdf/body/plate.urdf.xacro (robot description, xacro)
@@ -17,7 +17,7 @@
       </visual>
       <collision>
-        <origin xyz="0.0 0.0 -${0.009/2}" rpy="0.0 0.0 0.0" />
+        <origin xyz="0.0 0.0 0.0" rpy="0.0 0.0 0.0" />
         <geometry>
-          <box size="0.3 0.3 0.009" />
+          <box size="0.47 0.19 0.20" />
         </geometry>
       </collision>
@@ -44,7 +44,7 @@
       </visual>
       <collision>
-        <origin xyz="0.0 0.0 -${0.009/2}" rpy="0.0 0.0 0.0" />
+        <origin xyz="0.0 0.0 0.0" rpy="0.0 0.0 0.0" />
         <geometry>
-          <box size="0.3 0.3 0.009" />
+          <box size="0.47 0.47 0.02" />
         </geometry>
       </collision>
@@ -71,7 +71,7 @@
       </visual>
       <collision>
-        <origin xyz="0.0 0.0 -${0.009/2}" rpy="0.0 0.0 0.0" />
+        <origin xyz="0.0 0.0 0.0" rpy="0.0 0.0 0.0" />
         <geometry>
-          <box size="0.3 0.3 0.009" />
+          <box size="0.47 0.47 0.02" />
         </geometry>
       </collision>

File: sobit_home_description/urdf/head/head.urdf.xacro (robot description, xacro)
@@ -18,7 +18,7 @@
       </visual>
       <collision>
-        <origin xyz="${0.05125-0.15125/2} 0.0 0.0" rpy="0.0 0.0 0.0" />
+        <origin xyz="-0.015 0.0 -${0.01/2}" rpy="0.0 0.0 0.0" />
         <geometry>
-          <box size="0.15125 0.0285 0.044"/>
+          <box size="0.15 0.125 0.01"/>
         </geometry>
       </collision>
@@ -46,10 +46,10 @@
         <material name="black" />
       </visual>
-      <collision>
+      <!-- <collision>
         <origin xyz="0.0 0.0 ${0.00525+0.03525/2}" rpy="0.0 0.0 0.0" />
         <geometry>
           <box size="0.0285 0.037 0.03525"/>
         </geometry>
-      </collision>
+      </collision> -->
       <inertial>
         <origin xyz="0.0 0.0 ${0.00525+0.03525/2}" rpy="0.0 0.0 ${M_PI/2}" />
@@ -76,7 +76,7 @@
       </visual>
       <collision>
-        <origin xyz="0.0 0.0 ${0.028+0.0115/2}" rpy="0.0 0.0 0.0" />
+        <origin xyz="-0.01 0.0 0.00943" rpy="0.0 0.0 0.0" />
         <geometry>
-          <box size="0.046 0.0466 0.0115"/>
+          <box size="0.155 0.278 0.2"/>
         </geometry>
       </collision>

File: sobit_home_description/urdf/sensor/lidar.urdf.xacro (robot description, xacro)
@@ -17,7 +17,7 @@
       </visual>
       <collision>
-        <origin xyz="${0.092/2} 0.0 -${0.007/2}" rpy="0.0 0.0 0.0" />
+        <origin xyz="0.0236 0.0 -0.066" rpy="0.0 0.0 0.0" />
         <geometry>
-          <box size="0.092 0.184 0.007"/>
+          <box size="0.141 0.05 0.158"/>
         </geometry>
       </collision>

File: sobit_home_description/urdf/sensor/mic.urdf.xacro (robot description, xacro)
@@ -16,5 +16,5 @@
         <material name="black" />
       </visual>
-      <collision>
+      <!-- <collision>
         <origin xyz="0.0 ${(0.02-0.1146-0.0146)/2} -${0.02/2}" rpy="0.0 0.0 0.0" />
         <geometry>
@@ -22,5 +22,5 @@
         </geometry>
         <material name="black" />
-      </collision>
+      </collision> -->
       <inertial>
         <origin xyz="0.0 ${(0.02-0.1146-0.0146)/2} -${0.02/2}" rpy="0.0 0.0 0.0" />
@@ -45,5 +45,5 @@
         <material name="black" />
       </visual>
-      <collision>
+      <!-- <collision>
         <origin xyz="${0.0+0.04911} -${0.0112/2} ${0.035+0.0266}" rpy="0.0 ${M_PI/2-25*M_PI/180} 0.0" />
         <geometry>
@@ -51,5 +51,5 @@
         </geometry>
         <material name="black" />
-      </collision>
+      </collision> -->
       <inertial>
         <origin xyz="${0.0+0.04911} -${0.0112/2} ${0.035+0.0266}" rpy="0.0 ${M_PI/2-25*M_PI/180} 0.0" />

File: sobit_home_description/urdf/wheel/wheel.urdf.xacro (robot description, xacro)
@@ -17,10 +17,10 @@
         <material name="black" />
       </visual>
-      <collision>
+      <!-- <collision>
         <origin xyz="${0.01388-0.05525/2} 0.0 -${0.005+0.034/2+0.02/2}" rpy="0.0 0.0 0.0" />
         <geometry>
           <box size="0.05525 0.0285 0.084" />
         </geometry>
-      </collision>
+      </collision> -->
       <inertial>
         <origin xyz="${0.01388-0.05525/2} 0.0 -${0.005+0.034/2+0.02/2}" rpy="0.0 0.0 0.0" />
@@ -49,10 +49,10 @@
         <material name="black" />
       </visual>
-      <collision>
+      <!-- <collision>
         <origin xyz="${0.0244+0.0436/2} 0.0 ${0.034/2+0.0149-0.1766/2}" rpy="0.0 0.0 0.0" />
         <geometry>
           <box size="0.0436 0.0495 0.1766" />
         </geometry>
-      </collision>
+      </collision> -->
       <inertial>
         <origin xyz="${0.0244+0.0436/2} 0.0 ${0.034/2+0.0149-0.1766/2}" rpy="0.0 0.0 0.0" />
@@ -81,15 +81,15 @@
       </visual>
       <collision>
-        <origin xyz="-${0.0055+0.029/2} 0.0 0.0" rpy="${M_PI/2} 0.0 ${M_PI+M_PI/2.0}" />
+        <origin xyz="0.0 0.0 0.0" rpy="${M_PI/2.0} 0.0 ${M_PI}" />
         <geometry>
-          <cylinder radius="${0.144/2}" length="0.029"/>
+          <cylinder radius="0.075" length="0.017"/>
         </geometry>
       </collision>
       <inertial>
-        <origin xyz="-${0.0055+0.029/2} 0.0 0.0" rpy="0.0 0.0 0.0" />
+        <origin xyz="-${0.0055+0.017/2} 0.0 0.0" rpy="0.0 0.0 0.0" />
         <mass value="1" />
         <inertia ixx="${1/2 *1*(0.144/2)**2}"              ixy="0.0" ixz="0.0"
-                 iyy="${1/12*1*(3*(0.144/2)**2+0.029**2)}" iyz="0.0"
-                 izz="${1/12*1*(3*(0.144/2)**2+0.029**2)}" />
+                 iyy="${1/12*1*(3*(0.144/2)**2+0.017**2)}" iyz="0.0"
+                 izz="${1/12*1*(3*(0.144/2)**2+0.017**2)}" />
       </inertial>
     </link>

Commit message: [UPD] collision

File: sobit_home_description/urdf/arm/arm.urdf.xacro (robot description, xacro)
@@ -59,8 +59,7 @@
       </visual>
       <collision>
-        <origin xyz="0 ${y_sign * 0.104/2} 0.0" rpy="0.0 0.0 0.0" />
+        <origin xyz="0 ${y_sign * 0.104/2} 0.0" rpy="${M_PI/2+yaw_rot} 0.0 0.0" />
         <geometry>
-          <!-- <cylinder length="0.104" radius="${0.08/2}" /> -->
-          <box size="0.0535 0.104 0.045" />
+          <cylinder length="0.104" radius="${0.08/2}" />
         </geometry>
       </collision>
@@ -88,10 +87,10 @@
         <material name="grey" />
       </visual>
-      <!-- <collision>
-        <origin xyz="0.0 0.0 0.0" rpy="0.0 0.0 0.0" />
+      <collision>
+        <origin xyz="0.0 0.0 -0.13445" rpy="0.0 0.0 0.0" />
         <geometry>
-          <box size="0.1166 0.124 0.043" />
+          <cylinder length="0.129" radius="${0.076/2}" />
         </geometry>
-      </collision> -->
+      </collision>
       <inertial>
         <origin xyz="${0.1166/2+0.0224} 0.0 0.0" rpy="0.0 0.0 ${M_PI/2}" />
@@ -102,5 +101,5 @@
       </inertial>
     </link>
-    <!-- <joint name="${prefix}_${position}_upper_flex_joint" type="revolute" >
+    <joint name="${prefix}_${position}_upper_flex_joint" type="revolute" >
       <parent link="${prefix}_${position}_upper_roll_link" />
       <child link="${prefix}_${position}_upper_flex_link" />
@@ -118,7 +117,7 @@
       </visual>
       <collision>
-        <origin xyz="${0.1166/2+0.0224} 0.0 0.0" rpy="0.0 0.0 0.0" />
+        <origin xyz="0.0 0.0 -0.06943603" rpy="0.0 0.0 0.0" />
         <geometry>
-          <box size="0.1166 0.124 0.043" />
+          <cylinder length="0.171" radius="${0.076/2}" />
         </geometry>
       </collision>
@@ -147,7 +146,7 @@
       </visual>
       <collision>
-        <origin xyz="${0.1166/2+0.0224} 0.0 0.0" rpy="0.0 0.0 0.0" />
+        <origin xyz="0.0 0.0 -0.265" rpy="0.0 0.0 0.0" />
         <geometry>
-          <box size="0.1166 0.124 0.043" />
+          <cylinder length="0.38679886" radius="${0.088156/2}" />
         </geometry>
       </collision>
@@ -176,7 +175,7 @@
       </visual>
       <collision>
-        <origin xyz="${0.1166/2+0.0224} 0.0 0.0" rpy="0.0 0.0 0.0" />
+        <origin xyz="0.0 0.0 -0.0462" rpy="0.0 0.0 0.0" />
         <geometry>
-          <box size="0.1166 0.124 0.043" />
+          <cylinder length="0.04529731" radius="${0.08/2}" />
         </geometry>
       </collision>
@@ -188,5 +187,5 @@
                  izz="${1/12*0.08*(0.1166**2+0.124**2)}" />
       </inertial>
-    </link> -->
+    </link>
     <xacro:arm_transmission prefix="${prefix}" position="${position}" />
   </xacro:macro>
