Commit message: [UPD] inertial

File: sobit_home_description/urdf/arm/arm.urdf.xacro (robot description, xacro)
@@ -6,13 +6,11 @@
     <xacro:if value="${position == 'left'}">
       <xacro:property name="y_sign" value="1.0" />
-      <xacro:property name="yaw_rot" value="0.0" />
-        <xacro:property name="upper_roll_limit_lower" value="0" />
-        <xacro:property name="upper_roll_limit_upper" value="${M_PI}" />
+        <xacro:property name="upper_roll_limit_lower" value="${-M_PI/2}" />
+        <xacro:property name="upper_roll_limit_upper" value="${M_PI/2}" />
     </xacro:if>
     <xacro:if value="${position == 'right'}">
       <xacro:property name="y_sign" value="-1.0" />
-      <xacro:property name="yaw_rot" value="${M_PI}" />
-        <xacro:property name="upper_roll_limit_lower" value="${-M_PI}" />
-        <xacro:property name="upper_roll_limit_upper" value="0" />
+        <xacro:property name="upper_roll_limit_lower" value="${M_PI/2}" />
+        <xacro:property name="upper_roll_limit_upper" value="${-M_PI/2}" />
     </xacro:if>
     <joint name="${prefix}_${position}_base_joint" type="fixed" >
@@ -23,5 +21,5 @@
     <link name="${prefix}_${position}_base_link" >
       <visual>
-        <origin xyz="0.0 0.0 0.0" rpy="${M_PI/2} 0.0 ${M_PI/2+yaw_rot}" />
+        <origin xyz="0.0 0.0 0.0" rpy="${M_PI/2} 0.0 ${y_sign * M_PI/2}" />
         <geometry>
           <mesh filename="file://$(find sobit_home_description)/meshes/arm/arm_scapula.stl" scale="0.001 0.001 0.001" />
@@ -36,9 +34,9 @@
       </collision>
       <inertial>
-        <origin xyz="${0.140/2} 0.0 ${0.043/2}" rpy="0.0 0.0 ${M_PI/2}" />
+        <origin xyz="0.0 ${y_sign * 0.124/2} 0.0" rpy="0.0 0.0 0.0" />
         <mass value="0.08" />
-        <inertia ixx="${1/12*0.08*(0.140**2+0.043**2)}" ixy="0.0" ixz="0.0"
-                 iyy="${1/12*0.08*(0.156**2+0.043**2)}" iyz="0.0"
-                 izz="${1/12*0.08*(0.140**2+0.156**2)}" />
+        <inertia ixx="${1/12*0.08*(0.124**2+0.054**2)}" ixy="0.0" ixz="0.0"
+                 iyy="${1/12*0.08*(0.054**2+0.054**2)}" iyz="0.0"
+                 izz="${1/12*0.08*(0.054**2+0.124**2)}" />
       </inertial>
     </link>
@@ -47,10 +45,10 @@
       <child link="${prefix}_${position}_shoulder_tilt_link" />
       <origin xyz="0.0 ${y_sign * 0.126} 0.0" rpy="0.0 0.0 0.0" />
-      <axis xyz="0.0 -1.0 0.0 " />
+      <axis xyz="0.0 1.0 0.0 " />
       <limit lower="${-M_PI/2}" upper="${M_PI/2}" effort="${10.6*2}" velocity="11.031179004" />
     </joint>
     <link name="${prefix}_${position}_shoulder_tilt_link" >
       <visual>
-        <origin xyz="0.0 0.0  0.0" rpy="0.0 0.0 ${M_PI/2+yaw_rot}" />
+        <origin xyz="0.0 0.0 0.0" rpy="0.0 0.0 ${y_sign * M_PI/2}" />
         <geometry>
           <mesh filename="file://$(find sobit_home_description)/meshes/arm/arm_shoulder.stl" scale="0.001 0.001 0.001" />
@@ -59,5 +57,5 @@
       </visual>
       <collision>
-        <origin xyz="0 ${y_sign * 0.104/2} 0.0" rpy="${M_PI/2+yaw_rot} 0.0 0.0" />
+        <origin xyz="0.0 ${y_sign * 0.104/2} 0.0" rpy="${y_sign * M_PI/2} 0.0 0.0" />
         <geometry>
           <cylinder length="0.104" radius="${0.08/2}" />
@@ -65,9 +63,9 @@
       </collision>
       <inertial>
-        <origin xyz="${0.1166/2+0.0224} 0.0 0.0" rpy="0.0 0.0 ${M_PI/2}" />
+        <origin xyz="0 ${y_sign * 0.104/2} 0.0" rpy="${y_sign * M_PI/2} 0.0 0.0" />
         <mass value="0.08" />
-        <inertia ixx="${1/12*0.08*(0.1166**2+0.043**2)}" ixy="0.0" ixz="0.0"
-                 iyy="${1/12*0.08*(0.124**2 +0.043**2)}" iyz="0.0"
-                 izz="${1/12*0.08*(0.1166**2+0.124**2)}" />
+        <inertia ixx="${1/12*0.08*(3*0.04**2+0.104**2)}" ixy="0.0" ixz="0.0"
+                 iyy="${1/12*0.08*(3*0.04**2+0.104**2)}" iyz="0.0"
+                 izz="${1/2*0.08*0.04**2}" />
       </inertial>
     </link>
@@ -81,5 +79,5 @@
     <link name="${prefix}_${position}_upper_roll_link" >
       <visual>
-        <origin xyz="0.0 0.0 0.0" rpy="0.0 0.0 ${M_PI/2}" />
+        <origin xyz="0.0 0.0 0.0" rpy="0.0 ${-y_sign * M_PI/2} ${M_PI/2}" />
         <geometry>
           <mesh filename="file://$(find sobit_home_description)/meshes/arm/arm_upper_roll.stl" scale="0.001 0.001 0.001" />
@@ -88,5 +86,5 @@
       </visual>
       <collision>
-        <origin xyz="0.0 0.0 -0.13445" rpy="0.0 0.0 0.0" />
+        <origin xyz="0.0 ${y_sign * 0.13445} 0.0" rpy="0.0 ${y_sign * M_PI/2} ${M_PI/2}" />
         <geometry>
           <cylinder length="0.129" radius="${0.076/2}" />
@@ -94,9 +92,9 @@
       </collision>
       <inertial>
-        <origin xyz="${0.1166/2+0.0224} 0.0 0.0" rpy="0.0 0.0 ${M_PI/2}" />
+        <origin xyz="0.0 ${y_sign * 0.13445} 0.0" rpy="0.0 ${y_sign * M_PI/2} ${M_PI/2}" />
         <mass value="0.08" />
-        <inertia ixx="${1/12*0.08*(0.1166**2+0.043**2)}" ixy="0.0" ixz="0.0"
-                 iyy="${1/12*0.08*(0.124**2 +0.043**2)}" iyz="0.0"
-                 izz="${1/12*0.08*(0.1166**2+0.124**2)}" />
+        <inertia ixx="${1/12*0.08*(3*0.038**2+0.129**2)}" ixy="0.0" ixz="0.0"
+                 iyy="${1/12*0.08*(3*0.038**2+0.129**2)}" iyz="0.0"
+                 izz="${1/2*0.08*0.038**2}" />
       </inertial>
     </link>
@@ -104,11 +102,11 @@
       <parent link="${prefix}_${position}_upper_roll_link" />
       <child link="${prefix}_${position}_upper_flex_link" />
-      <origin xyz="0.0 0.0 -0.215813" rpy="0.0 0.0 0.0" />
-      <axis xyz="0.0 0.0 1.0" />
+      <origin xyz="0.0 ${y_sign * 0.215813} 0.0" rpy="0.0 0.0 0.0" />
+      <axis xyz="0.0 1.0 0.0" />
       <limit lower="${-M_PI/2}" upper="${M_PI/2}" effort="${10.6*2}" velocity="11.031179004" />
     </joint>
     <link name="${prefix}_${position}_upper_flex_link" >
       <visual>
-        <origin xyz="0.0 0.0 0.0" rpy="0.0 0.0 ${-M_PI/2}" />
+        <origin xyz="0.0 0.0 0.0" rpy="0.0 ${y_sign * M_PI/2} ${-M_PI/2}" />
         <geometry>
           <mesh filename="file://$(find sobit_home_description)/meshes/arm/arm_upper_flex.stl" scale="0.001 0.001 0.001" />
@@ -117,5 +115,5 @@
       </visual>
       <collision>
-        <origin xyz="0.0 0.0 -0.06943603" rpy="0.0 0.0 0.0" />
+        <origin xyz="0.0 ${y_sign * 0.06943603} 0.0" rpy="0.0 ${y_sign * M_PI/2} ${-M_PI/2}" />
         <geometry>
           <cylinder length="0.171" radius="${0.076/2}" />
@@ -123,9 +121,9 @@
       </collision>
       <inertial>
-        <origin xyz="${0.1166/2+0.0224} 0.0 0.0" rpy="0.0 0.0 ${M_PI/2}" />
+        <origin xyz="0.0 ${y_sign * 0.06943603} 0.0" rpy="0.0 ${y_sign * M_PI/2} ${-M_PI/2}" />
         <mass value="0.08" />
-        <inertia ixx="${1/12*0.08*(0.1166**2+0.043**2)}" ixy="0.0" ixz="0.0"
-                 iyy="${1/12*0.08*(0.124**2 +0.043**2)}" iyz="0.0"
-                 izz="${1/12*0.08*(0.1166**2+0.124**2)}" />
+        <inertia ixx="${1/12*0.08*(3*0.038**2+0.171**2)}" ixy="0.0" ixz="0.0"
+                 iyy="${1/12*0.08*(3*0.038**2+0.171**2)}" iyz="0.0"
+                 izz="${1/2*0.08*0.038**2}" />
       </inertial>
     </link>
@@ -133,11 +131,11 @@
       <parent link="${prefix}_${position}_upper_flex_link" />
       <child link="${prefix}_${position}_elbow_link" />
-      <origin xyz="0.0 0.0 -0.18413635" rpy="0.0 0.0 0.0" />
-      <axis xyz="0.0 -1.0 0.0 " />
+      <origin xyz="0.0 ${y_sign * 0.18413635} 0.0" rpy="0.0 0.0 0.0" />
+      <axis xyz="0.0 0.0 -1.0" />
       <limit lower="0" upper="${M_PI/2}" effort="${10.6*2}" velocity="11.031179004" />
     </joint>
     <link name="${prefix}_${position}_elbow_link" >
       <visual>
-        <origin xyz="0.0 0.0 0.0" rpy="0.0 0.0 ${M_PI/2}" />
+        <origin xyz="0.0 0.0 0.0" rpy="0.0 ${-y_sign * M_PI/2} ${M_PI/2}" />
         <geometry>
           <mesh filename="file://$(find sobit_home_description)/meshes/arm/arm_elbow.stl" scale="0.001 0.001 0.001" />
@@ -146,15 +144,15 @@
       </visual>
       <collision>
-        <origin xyz="0.0 0.0 -0.265" rpy="0.0 0.0 0.0" />
+        <origin xyz="0.0 ${y_sign * 0.265} 0.0" rpy="0.0 ${-y_sign * M_PI/2} ${M_PI/2}" />
         <geometry>
-          <cylinder length="0.38679886" radius="${0.088156/2}" />
+          <cylinder length="0.386" radius="${0.088156/2}" />
         </geometry>
       </collision>
       <inertial>
-        <origin xyz="${0.1166/2+0.0224} 0.0 0.0" rpy="0.0 0.0 ${M_PI/2}" />
+        <origin xyz="0.0 ${y_sign * 0.265} 0.0" rpy="0.0 ${-y_sign * M_PI/2} ${M_PI/2}" />
         <mass value="0.08" />
-        <inertia ixx="${1/12*0.08*(0.1166**2+0.043**2)}" ixy="0.0" ixz="0.0"
-                 iyy="${1/12*0.08*(0.124**2 +0.043**2)}" iyz="0.0"
-                 izz="${1/12*0.08*(0.1166**2+0.124**2)}" />
+        <inertia ixx="${1/12*0.08*(3*0.044**2+0.386**2)}" ixy="0.0" ixz="0.0"
+                 iyy="${1/12*0.08*(3*0.044**2+0.386**2)}" iyz="0.0"
+                 izz="${1/2*0.08*0.044**2}" />
       </inertial>
     </link>
@@ -162,11 +160,11 @@
       <parent link="${prefix}_${position}_elbow_link" />
       <child link="${prefix}_${position}_wrist_link" />
-      <origin xyz="0.0 0.0 -0.5" rpy="0.0 0.0 0.0" />
-      <axis xyz="0.0 -1.0 0.0 " />
+      <origin xyz="0.0 ${y_sign * 0.5} 0.0" rpy="0.0 0.0 0.0" />
+      <axis xyz="0.0 0.0 -1.0 " />
       <limit lower="${-M_PI/2}" upper="${M_PI/2}" effort="${10.6*2}" velocity="11.031179004" />
     </joint>
     <link name="${prefix}_${position}_wrist_link" >
       <visual>
-        <origin xyz="0.0 0.0 0.0" rpy="0.0 0.0 ${M_PI/2}" />
+        <origin xyz="0.0 0.0 0.0" rpy="0.0 ${-y_sign * M_PI/2} ${M_PI/2}" />
         <geometry>
           <mesh filename="file://$(find sobit_home_description)/meshes/arm/arm_wrist.stl" scale="0.001 0.001 0.001" />
@@ -175,15 +173,15 @@
       </visual>
       <collision>
-        <origin xyz="0.0 0.0 -0.0462" rpy="0.0 0.0 0.0" />
+        <origin xyz="0.0 ${y_sign * 0.0462} 0.0" rpy="0.0 ${-y_sign * M_PI/2} ${M_PI/2}" />
         <geometry>
-          <cylinder length="0.04529731" radius="${0.08/2}" />
+          <cylinder length="0.0453" radius="${0.08/2}" />
         </geometry>
       </collision>
       <inertial>
-        <origin xyz="${0.1166/2+0.0224} 0.0 0.0" rpy="0.0 0.0 ${M_PI/2}" />
+        <origin xyz="0.0 ${y_sign * 0.0462} 0.0" rpy="0.0 ${-y_sign * M_PI/2} ${M_PI/2}" />
         <mass value="0.08" />
-        <inertia ixx="${1/12*0.08*(0.1166**2+0.043**2)}" ixy="0.0" ixz="0.0"
-                 iyy="${1/12*0.08*(0.124**2 +0.043**2)}" iyz="0.0"
-                 izz="${1/12*0.08*(0.1166**2+0.124**2)}" />
+        <inertia ixx="${1/12*0.08*(3*0.04**2+0.0453**2)}" ixy="0.0" ixz="0.0"
+                 iyy="${1/12*0.08*(3*0.04**2+0.0453**2)}" iyz="0.0"
+                 izz="${1/2*0.08*0.04**2}" />
       </inertial>
     </link>

File: sobit_home_description/urdf/body/body.urdf.xacro (robot description, xacro)
@@ -24,9 +24,9 @@
       </collision>
       <inertial>
-        <origin xyz="-${0.02893+0.3/2} 0.0 ${0.034-0.489/2}" rpy="0.0 0.0 0.0" />
+        <origin xyz="0.0 0.00425 -0.018" rpy="0.0 0.0 0.0" />
         <mass value="0.732" />
-        <inertia ixx="${1/12*0.732*(((0.02893+0.3/2)*2)**2+0.489**2)}"  ixy="0.0" ixz="0.0"
-                 iyy="${1/12*0.732*(0.3965**2+0.489**2)}"               iyz="0.0"
-                 izz="${1/12*0.732*(((0.02893+0.3/2)*2)**2+0.3965**2)}" />
+        <inertia ixx="${1/12*0.732*(0.085**2+1.07**2)}"  ixy="0.0" ixz="0.0"
+                 iyy="${1/12*0.732*(1.07**2+0.0675**2)}" iyz="0.0"
+                 izz="${1/12*0.732*(0.0675**2+0.085**2)}" />
       </inertial>
     </link>
@@ -36,5 +36,5 @@
       <child link="${prefix}_lift_link" />
       <axis xyz="0.0 0.0 1.0" />
-      <limit lower="-0.4" upper="0.4" effort="150.0" velocity="0.1" />
+      <limit lower="-0.4" upper="0.4" effort="150000.0" velocity="0.1" />
     </joint>
     <link name="${prefix}_lift_link" >
@@ -53,9 +53,9 @@
       </collision>
       <inertial>
-        <origin xyz="-${0.02893+0.3/2} 0.0 ${0.034-0.489/2}" rpy="0.0 0.0 0.0" />
+        <origin xyz="0.0 0.0 0.0" rpy="0.0 0.0 0.0" />
         <mass value="0.732" />
-        <inertia ixx="${1/12*0.732*(((0.02893+0.3/2)*2)**2+0.489**2)}"  ixy="0.0" ixz="0.0"
-                 iyy="${1/12*0.732*(0.3965**2+0.489**2)}"               iyz="0.0"
-                 izz="${1/12*0.732*(((0.02893+0.3/2)*2)**2+0.3965**2)}" />
+        <inertia ixx="${1/12*0.732*(0.35**2+0.15**2)}"  ixy="0.0" ixz="0.0"
+                 iyy="${1/12*0.732*(0.15**2+0.15**2)}"  iyz="0.0"
+                 izz="${1/12*0.732*(0.15**2+0.35**2)}" />
       </inertial>
     </link>

File: sobit_home_description/urdf/body/plate.urdf.xacro (robot description, xacro)
@@ -23,9 +23,9 @@
       </collision>
       <inertial>
-        <origin xyz="0.0 0.0 -${0.009/2}" rpy="0.0 0.0 0.0" />
+        <origin xyz="0.0 0.0 0.0" rpy="0.0 0.0 0.0" />
         <mass value="0.08" />
-        <inertia ixx="${1/12*0.08*(0.3**2+0.009**2)}" ixy="0.0" ixz="0.0"
-                 iyy="${1/12*0.08*(0.3**2+0.009**2)}" iyz="0.0"
-                 izz="${1/12*0.08*(0.3**2+0.3**2)}" />
+        <inertia ixx="${1/12*0.08*(0.19**2+0.20**2)}" ixy="0.0" ixz="0.0"
+                 iyy="${1/12*0.08*(0.20**2+0.47**2)}" iyz="0.0"
+                 izz="${1/12*0.08*(0.47**2+0.19**2)}" />
       </inertial>
     </link>
@@ -50,9 +50,9 @@
       </collision>
       <inertial>
-        <origin xyz="0.0 0.0 -${0.009/2}" rpy="0.0 0.0 0.0" />
+        <origin xyz="0.0 0.0 0.0" rpy="0.0 0.0 0.0" />
         <mass value="0.08" />
-        <inertia ixx="${1/12*0.08*(0.3**2+0.009**2)}" ixy="0.0" ixz="0.0"
-                 iyy="${1/12*0.08*(0.3**2+0.009**2)}" iyz="0.0"
-                 izz="${1/12*0.08*(0.3**2+0.3**2)}" />
+        <inertia ixx="${1/12*0.08*(0.47**2+0.02**2)}" ixy="0.0" ixz="0.0"
+                 iyy="${1/12*0.08*(0.02**2+0.47**2)}" iyz="0.0"
+                 izz="${1/12*0.08*(0.47**2+0.47**2)}" />
       </inertial>
     </link>
@@ -77,9 +77,9 @@
       </collision>
       <inertial>
-        <origin xyz="0.0 0.0 -${0.009/2}" rpy="0.0 0.0 0.0" />
+        <origin xyz="0.0 0.0 0.0" rpy="0.0 0.0 0.0" />
         <mass value="0.08" />
-        <inertia ixx="${1/12*0.08*(0.3**2+0.009**2)}" ixy="0.0" ixz="0.0"
-                 iyy="${1/12*0.08*(0.3**2+0.009**2)}" iyz="0.0"
-                 izz="${1/12*0.08*(0.3**2+0.3**2)}" />
+        <inertia ixx="${1/12*0.08*(0.47**2+0.02**2)}" ixy="0.0" ixz="0.0"
+                 iyy="${1/12*0.08*(0.02**2+0.47**2)}" iyz="0.0"
+                 izz="${1/12*0.08*(0.47**2+0.47**2)}" />
       </inertial>
     </link>

File: sobit_home_description/urdf/head/head.urdf.xacro (robot description, xacro)
@@ -24,9 +24,9 @@
       </collision>
       <inertial>
-        <origin xyz="${0.05125-0.15125/2} 0.0 0.0" rpy="0.0 0.0 0.0" />
+        <origin xyz="-0.015 0.0 -${0.01/2}" rpy="0.0 0.0 0.0" />
         <mass value="0.08" />
-        <inertia ixx="${1/12*0.08*(0.15125**2+0.044**2)}" ixy="0.0" ixz="0.0"
-                 iyy="${1/12*0.08*(0.0285**2 +0.044**2)}" iyz="0.0"
-                 izz="${1/12*0.08*(0.15125**2+0.0285**2)}" />
+        <inertia ixx="${1/12*0.08*(0.125**2+0.01**2)}" ixy="0.0" ixz="0.0"
+                 iyy="${1/12*0.08*(0.01**2 +0.15**2)}" iyz="0.0"
+                 izz="${1/12*0.08*(0.15**2+0.125**2)}" />
       </inertial>
     </link>
@@ -46,16 +46,16 @@
         <material name="black" />
       </visual>
-      <!-- <collision>
-        <origin xyz="0.0 0.0 ${0.00525+0.03525/2}" rpy="0.0 0.0 0.0" />
+      <collision>
+        <origin xyz="0.0 0.0 0.0046" rpy="0.0 0.0 0.0" />
         <geometry>
-          <box size="0.0285 0.037 0.03525"/>
+          <cylinder length="0.0092" radius="${0.065/2}"/>
         </geometry>
-      </collision> -->
+      </collision>
       <inertial>
-        <origin xyz="0.0 0.0 ${0.00525+0.03525/2}" rpy="0.0 0.0 ${M_PI/2}" />
+        <origin xyz="0.0 0.0 0.0046" rpy="0.0 0.0 0.0" />
         <mass value="0.08" />
-        <inertia ixx="${1/12*0.08*(0.0285**2+0.03525**2)}" ixy="0.0" ixz="0.0"
-                 iyy="${1/12*0.08*(0.037**2 +0.03525**2)}" iyz="0.0"
-                 izz="${1/12*0.08*(0.0285**2+0.037**2)}" />
+        <inertia ixx="${1/12*0.08*(3*0.0325**2+0.0092**2)}"     ixy="0.0" ixz="0.0"
+                 iyy="${1/12*0.08*(3*0.0325**2+0.04009253**2)}" iyz="0.0"
+                 izz="${1/2*0.08*0.0325**2}" />
       </inertial>
     </link>
@@ -82,9 +82,9 @@
       </collision>
       <inertial>
-        <origin xyz="0.0 0.0 ${0.028+0.0115/2}" rpy="0.0 0.0 0.0" />
+        <origin xyz="-0.01 0.0 0.00943" rpy="0.0 0.0 0.0" />
         <mass value="0.08" />
-        <inertia ixx="${1/12*0.08*(0.046**2 +0.0115**2)}" ixy="0.0" ixz="0.0"
-                 iyy="${1/12*0.08*(0.0466**2+0.0115**2)}" iyz="0.0"
-                 izz="${1/12*0.08*(0.046**2 +0.0466**2)}" />
+        <inertia ixx="${1/12*0.08*(0.278**2 +0.2**2)}" ixy="0.0" ixz="0.0"
+                 iyy="${1/12*0.08*(0.2**2+0.155**2)}"  iyz="0.0"
+                 izz="${1/12*0.08*(0.155**2 +0.278**2)}" />
       </inertial>
     </link>

File: sobit_home_description/urdf/sensor/lidar.urdf.xacro (robot description, xacro)
@@ -17,7 +17,7 @@
       </visual>
       <collision>
-        <origin xyz="0.0236 0.0 -0.066" rpy="0.0 0.0 0.0" />
+        <origin xyz="0.0705 0.0 -0.071" rpy="0.0 0.0 0.0" />
         <geometry>
-          <box size="0.141 0.05 0.158"/>
+          <box size="0.0941 0.05 0.158"/>
         </geometry>
       </collision>

File: sobit_home_description/urdf/wheel/wheel.urdf.xacro (robot description, xacro)
@@ -17,16 +17,16 @@
         <material name="black" />
       </visual>
-      <!-- <collision>
-        <origin xyz="${0.01388-0.05525/2} 0.0 -${0.005+0.034/2+0.02/2}" rpy="0.0 0.0 0.0" />
+      <collision>
+        <origin xyz="0.0 0.0 0.0" rpy="0.0 0.0 ${M_PI/2.0}" />
         <geometry>
-          <box size="0.05525 0.0285 0.084" />
+          <cylinder length="0.0797" radius="0.075"/>
         </geometry>
-      </collision> -->
+      </collision>
       <inertial>
-        <origin xyz="${0.01388-0.05525/2} 0.0 -${0.005+0.034/2+0.02/2}" rpy="0.0 0.0 0.0" />
+        <origin xyz="0.0 0.0 0.0" rpy="0.0 0.0 ${M_PI/2.0}" />
         <mass value="1" />
-        <inertia ixx="${1/12*1*(0.05525**2+0.084**2)}" ixy="0.0" ixz="0.0"
-                 iyy="${1/12*1*(0.0285**2 +0.084**2)}" iyz="0.0"
-                 izz="${1/12*1*(0.05525**2+0.0285**2)}" />
+        <inertia ixx="${1/12*0.08*(3*0.075**2+0.0797**2)}" ixy="0.0" ixz="0.0"
+                 iyy="${1/12*0.08*(3*0.075**2+0.0797**2)}" iyz="0.0"
+                 izz="${1/2*0.08*0.075**2}" />
       </inertial>
     </link>
@@ -49,16 +49,16 @@
         <material name="black" />
       </visual>
-      <!-- <collision>
-        <origin xyz="${0.0244+0.0436/2} 0.0 ${0.034/2+0.0149-0.1766/2}" rpy="0.0 0.0 0.0" />
+      <collision>
+        <origin xyz="0.0 0.0 -0.030925" rpy="0.0 0.0 ${M_PI/2}" />
         <geometry>
-          <box size="0.0436 0.0495 0.1766" />
+          <box size="0.1 0.1 0.06185" />
         </geometry>
-      </collision> -->
+      </collision>
       <inertial>
-        <origin xyz="${0.0244+0.0436/2} 0.0 ${0.034/2+0.0149-0.1766/2}" rpy="0.0 0.0 0.0" />
+        <origin xyz="0.0 0.0 -0.030925" rpy="0.0 0.0 ${M_PI/2}" />
         <mass value="1" />
-        <inertia ixx="${1/12*1*(0.0436**2+0.1766**2)}" ixy="0.0" ixz="0.0"
-                 iyy="${1/12*1*(0.0495**2+0.1766**2)}" iyz="0.0"
-                 izz="${1/12*1*(0.0436**2+0.0495**2)}" />
+        <inertia ixx="${1/12*1*(0.1**2+0.06185**2)}" ixy="0.0" ixz="0.0"
+                 iyy="${1/12*1*(0.06185**2+0.1**2)}" iyz="0.0"
+                 izz="${1/12*1*(0.1**2+0.1**2)}" />
       </inertial>
     </link>
@@ -83,13 +83,13 @@
         <origin xyz="0.0 0.0 0.0" rpy="${M_PI/2.0} 0.0 ${M_PI}" />
         <geometry>
-          <cylinder radius="0.075" length="0.017"/>
+          <cylinder length="0.017" radius="0.075"/>
         </geometry>
       </collision>
       <inertial>
-        <origin xyz="-${0.0055+0.017/2} 0.0 0.0" rpy="0.0 0.0 0.0" />
+        <origin xyz="0.0 0.0 0.0" rpy="${M_PI/2.0} 0.0 ${M_PI}" />
         <mass value="1" />
-        <inertia ixx="${1/2 *1*(0.144/2)**2}"              ixy="0.0" ixz="0.0"
-                 iyy="${1/12*1*(3*(0.144/2)**2+0.017**2)}" iyz="0.0"
-                 izz="${1/12*1*(3*(0.144/2)**2+0.017**2)}" />
+        <inertia ixx="${1/12*1*(3*0.075**2+0.017**2)}" ixy="0.0" ixz="0.0"
+                 iyy="${1/12*1*(3*0.075**2+0.017**2)}" iyz="0.0"
+                 izz="${1/2*1*0.075**2}" />
       </inertial>
     </link>
