Commit message: [UPD] update mass

File: sobit_home_description/urdf/arm/arm.urdf.xacro (robot description, xacro)
@@ -35,8 +35,8 @@
       <inertial>
         <origin xyz="0.0 ${y_sign * 0.124/2} 0.0" rpy="0.0 0.0 0.0" />
-        <mass value="0.08" />
-        <inertia ixx="${1/12*0.08*(0.124**2+0.054**2)}" ixy="0.0" ixz="0.0"
-                 iyy="${1/12*0.08*(0.054**2+0.054**2)}" iyz="0.0"
-                 izz="${1/12*0.08*(0.054**2+0.124**2)}" />
+        <mass value="0.855" /> <!-- mass without FRP54-A110K -->
+        <inertia ixx="${1/12*0.855*(0.124**2+0.054**2)}" ixy="0.0" ixz="0.0"
+                 iyy="${1/12*0.855*(0.054**2+0.054**2)}" iyz="0.0"
+                 izz="${1/12*0.855*(0.054**2+0.124**2)}" />
       </inertial>
     </link>
@@ -46,5 +46,5 @@
       <origin xyz="0.0 ${y_sign * 0.126} 0.0" rpy="0.0 0.0 0.0" />
       <axis xyz="0.0 1.0 0.0 " />
-      <limit lower="${-M_PI/2}" upper="${M_PI/2}" effort="${10.6*2}" velocity="11.031179004" />
+      <limit lower="${-M_PI/2}" upper="${M_PI/2}" effort="44.7" velocity="3.0" />
     </joint>
     <link name="${prefix}_${position}_shoulder_tilt_link" >
@@ -64,8 +64,8 @@
       <inertial>
         <origin xyz="0 ${y_sign * 0.104/2} 0.0" rpy="${y_sign * M_PI/2} 0.0 0.0" />
-        <mass value="0.08" />
-        <inertia ixx="${1/12*0.08*(3*0.04**2+0.104**2)}" ixy="0.0" ixz="0.0"
-                 iyy="${1/12*0.08*(3*0.04**2+0.104**2)}" iyz="0.0"
-                 izz="${1/2*0.08*0.04**2}" />
+        <mass value="0.504" />
+        <inertia ixx="${1/12*0.504*(3*0.04**2+0.104**2)}" ixy="0.0" ixz="0.0"
+                 iyy="${1/12*0.504*(3*0.04**2+0.104**2)}" iyz="0.0"
+                 izz="${1/2*0.504*0.04**2}" />
       </inertial>
     </link>
@@ -75,5 +75,5 @@
       <origin xyz="0.0 ${y_sign * 0.0725} 0.0" rpy="0.0 0.0 0.0" />
       <axis xyz="1.0 0.0 0.0 " />
-      <limit lower="${upper_roll_limit_lower}" upper="${upper_roll_limit_upper}" effort="${10.6*2}" velocity="11.031179004" />
+      <limit lower="${upper_roll_limit_lower}" upper="${upper_roll_limit_upper}" effort="1060.0" velocity="3.14" />
     </joint>
     <link name="${prefix}_${position}_upper_roll_link" >
@@ -93,8 +93,8 @@
       <inertial>
         <origin xyz="0.0 ${y_sign * 0.13445} 0.0" rpy="0.0 ${y_sign * M_PI/2} ${M_PI/2}" />
-        <mass value="0.08" />
-        <inertia ixx="${1/12*0.08*(3*0.038**2+0.129**2)}" ixy="0.0" ixz="0.0"
-                 iyy="${1/12*0.08*(3*0.038**2+0.129**2)}" iyz="0.0"
-                 izz="${1/2*0.08*0.038**2}" />
+        <mass value="0.595" />
+        <inertia ixx="${1/12*0.595*(3*0.038**2+0.129**2)}" ixy="0.0" ixz="0.0"
+                 iyy="${1/12*0.595*(3*0.038**2+0.129**2)}" iyz="0.0"
+                 izz="${1/2*0.595*0.038**2}" />
       </inertial>
     </link>
@@ -104,5 +104,5 @@
       <origin xyz="0.0 ${y_sign * 0.215813} 0.0" rpy="0.0 0.0 0.0" />
       <axis xyz="0.0 1.0 0.0" />
-      <limit lower="${-M_PI/2}" upper="${M_PI/2}" effort="${10.6*2}" velocity="11.031179004" />
+      <limit lower="${-M_PI/2}" upper="${M_PI/2}" effort="4.1" velocity="4.81" />
     </joint>
     <link name="${prefix}_${position}_upper_flex_link" >
@@ -122,8 +122,8 @@
       <inertial>
         <origin xyz="0.0 ${y_sign * 0.06943603} 0.0" rpy="0.0 ${y_sign * M_PI/2} ${-M_PI/2}" />
-        <mass value="0.08" />
-        <inertia ixx="${1/12*0.08*(3*0.038**2+0.171**2)}" ixy="0.0" ixz="0.0"
-                 iyy="${1/12*0.08*(3*0.038**2+0.171**2)}" iyz="0.0"
-                 izz="${1/2*0.08*0.038**2}" />
+        <mass value="0.778" />
+        <inertia ixx="${1/12*0.778*(3*0.038**2+0.171**2)}" ixy="0.0" ixz="0.0"
+                 iyy="${1/12*0.778*(3*0.038**2+0.171**2)}" iyz="0.0"
+                 izz="${1/2*0.778*0.038**2}" />
       </inertial>
     </link>
@@ -133,5 +133,5 @@
       <origin xyz="0.0 ${y_sign * 0.18413635} 0.0" rpy="0.0 0.0 0.0" />
       <axis xyz="0.0 0.0 -1.0" />
-      <limit lower="0" upper="${M_PI/2}" effort="${10.6*2}" velocity="11.031179004" />
+      <limit lower="0" upper="${M_PI/2}" effort="10.6" velocity="3.14" />
     </joint>
     <link name="${prefix}_${position}_elbow_link" >
@@ -151,8 +151,8 @@
       <inertial>
         <origin xyz="0.0 ${y_sign * 0.265} 0.0" rpy="0.0 ${-y_sign * M_PI/2} ${M_PI/2}" />
-        <mass value="0.08" />
-        <inertia ixx="${1/12*0.08*(3*0.044**2+0.386**2)}" ixy="0.0" ixz="0.0"
-                 iyy="${1/12*0.08*(3*0.044**2+0.386**2)}" iyz="0.0"
-                 izz="${1/2*0.08*0.044**2}" />
+        <mass value="1.663" /> <!-- mass without FR13-H101K -->
+        <inertia ixx="${1/12*1.663*(3*0.044**2+0.386**2)}" ixy="0.0" ixz="0.0"
+                 iyy="${1/12*1.663*(3*0.044**2+0.386**2)}" iyz="0.0"
+                 izz="${1/2*1.663*0.044**2}" />
       </inertial>
     </link>
@@ -162,5 +162,5 @@
       <origin xyz="0.0 ${y_sign * 0.5} 0.0" rpy="0.0 0.0 0.0" />
       <axis xyz="0.0 0.0 -1.0 " />
-      <limit lower="${-M_PI/2}" upper="${M_PI/2}" effort="${10.6*2}" velocity="11.031179004" />
+      <limit lower="${-M_PI/2}" upper="${M_PI/2}" effort="4.1" velocity="4.81" />
     </joint>
     <link name="${prefix}_${position}_wrist_link" >
@@ -180,8 +180,8 @@
       <inertial>
         <origin xyz="0.0 ${y_sign * 0.0462} 0.0" rpy="0.0 ${-y_sign * M_PI/2} ${M_PI/2}" />
-        <mass value="0.08" />
-        <inertia ixx="${1/12*0.08*(3*0.04**2+0.0453**2)}" ixy="0.0" ixz="0.0"
-                 iyy="${1/12*0.08*(3*0.04**2+0.0453**2)}" iyz="0.0"
-                 izz="${1/2*0.08*0.04**2}" />
+        <mass value="0.341" />
+        <inertia ixx="${1/12*0.341*(3*0.04**2+0.0453**2)}" ixy="0.0" ixz="0.0"
+                 iyy="${1/12*0.341*(3*0.04**2+0.0453**2)}" iyz="0.0"
+                 izz="${1/2*0.341*0.04**2}" />
       </inertial>
     </link>

File: sobit_home_description/urdf/body/body.urdf.xacro (robot description, xacro)
@@ -25,8 +25,8 @@
       <inertial>
         <origin xyz="0.0 0.00425 -0.018" rpy="0.0 0.0 0.0" />
-        <mass value="0.732" />
-        <inertia ixx="${1/12*0.732*(0.085**2+1.07**2)}"  ixy="0.0" ixz="0.0"
-                 iyy="${1/12*0.732*(1.07**2+0.0675**2)}" iyz="0.0"
-                 izz="${1/12*0.732*(0.0675**2+0.085**2)}" />
+        <mass value="9.6" />
+        <inertia ixx="${1/12*9.6*(0.085**2+1.07**2)}"  ixy="0.0" ixz="0.0"
+                 iyy="${1/12*9.6*(1.07**2+0.0675**2)}" iyz="0.0"
+                 izz="${1/12*9.6*(0.0675**2+0.085**2)}" />
       </inertial>
     </link>
@@ -36,5 +36,5 @@
       <child link="${prefix}_lift_link" />
       <axis xyz="0.0 0.0 1.0" />
-      <limit lower="-0.4" upper="0.4" effort="150000.0" velocity="0.1" />
+      <limit lower="-0.4" upper="0.4" effort="150000.0" velocity="0.85" />
     </joint>
     <link name="${prefix}_lift_link" >
@@ -54,8 +54,8 @@
       <inertial>
         <origin xyz="0.0 0.0 0.0" rpy="0.0 0.0 0.0" />
-        <mass value="0.732" />
-        <inertia ixx="${1/12*0.732*(0.35**2+0.15**2)}"  ixy="0.0" ixz="0.0"
-                 iyy="${1/12*0.732*(0.15**2+0.15**2)}"  iyz="0.0"
-                 izz="${1/12*0.732*(0.15**2+0.35**2)}" />
+        <mass value="0.678" /> <!-- mass without wood plate and aluminum frame -->
+        <inertia ixx="${1/12*0.678*(0.35**2+0.15**2)}"  ixy="0.0" ixz="0.0"
+                 iyy="${1/12*0.678*(0.15**2+0.15**2)}"  iyz="0.0"
+                 izz="${1/12*0.678*(0.15**2+0.35**2)}" />
       </inertial>
     </link>

File: sobit_home_description/urdf/body/plate.urdf.xacro (robot description, xacro)
@@ -24,8 +24,8 @@
       <inertial>
         <origin xyz="0.0 0.0 0.0" rpy="0.0 0.0 0.0" />
-        <mass value="0.08" />
-        <inertia ixx="${1/12*0.08*(0.19**2+0.20**2)}" ixy="0.0" ixz="0.0"
-                 iyy="${1/12*0.08*(0.20**2+0.47**2)}" iyz="0.0"
-                 izz="${1/12*0.08*(0.47**2+0.19**2)}" />
+        <mass value="5.0" /> <!-- TODO -->
+        <inertia ixx="${1/12*5.0*(0.19**2+0.20**2)}" ixy="0.0" ixz="0.0"
+                 iyy="${1/12*5.0*(0.20**2+0.47**2)}" iyz="0.0"
+                 izz="${1/12*5.0*(0.47**2+0.19**2)}" />
       </inertial>
     </link>
@@ -51,8 +51,8 @@
       <inertial>
         <origin xyz="0.0 0.0 0.0" rpy="0.0 0.0 0.0" />
-        <mass value="0.08" />
-        <inertia ixx="${1/12*0.08*(0.47**2+0.02**2)}" ixy="0.0" ixz="0.0"
-                 iyy="${1/12*0.08*(0.02**2+0.47**2)}" iyz="0.0"
-                 izz="${1/12*0.08*(0.47**2+0.47**2)}" />
+        <mass value="1.0" /> <!-- TODO -->
+        <inertia ixx="${1/12*1.0*(0.47**2+0.02**2)}" ixy="0.0" ixz="0.0"
+                 iyy="${1/12*1.0*(0.02**2+0.47**2)}" iyz="0.0"
+                 izz="${1/12*1.0*(0.47**2+0.47**2)}" />
       </inertial>
     </link>
@@ -78,8 +78,8 @@
       <inertial>
         <origin xyz="0.0 0.0 0.0" rpy="0.0 0.0 0.0" />
-        <mass value="0.08" />
-        <inertia ixx="${1/12*0.08*(0.47**2+0.02**2)}" ixy="0.0" ixz="0.0"
-                 iyy="${1/12*0.08*(0.02**2+0.47**2)}" iyz="0.0"
-                 izz="${1/12*0.08*(0.47**2+0.47**2)}" />
+        <mass value="1.5" /> <!-- TODO -->
+        <inertia ixx="${1/12*1.5*(0.47**2+0.02**2)}" ixy="0.0" ixz="0.0"
+                 iyy="${1/12*1.5*(0.02**2+0.47**2)}" iyz="0.0"
+                 izz="${1/12*1.5*(0.47**2+0.47**2)}" />
       </inertial>
     </link>

File: sobit_home_description/urdf/head/head.urdf.xacro (robot description, xacro)
@@ -25,8 +25,8 @@
       <inertial>
         <origin xyz="-0.015 0.0 -${0.01/2}" rpy="0.0 0.0 0.0" />
-        <mass value="0.08" />
-        <inertia ixx="${1/12*0.08*(0.125**2+0.01**2)}" ixy="0.0" ixz="0.0"
-                 iyy="${1/12*0.08*(0.01**2 +0.15**2)}" iyz="0.0"
-                 izz="${1/12*0.08*(0.15**2+0.125**2)}" />
+        <mass value="0.424" />
+        <inertia ixx="${1/12*0.424*(0.125**2+0.01**2)}" ixy="0.0" ixz="0.0"
+                 iyy="${1/12*0.424*(0.01**2 +0.15**2)}" iyz="0.0"
+                 izz="${1/12*0.424*(0.15**2+0.125**2)}" />
       </inertial>
     </link>
@@ -36,5 +36,5 @@
       <origin xyz="0.0 0.0 0.0" rpy="0.0 0.0 0.0" />
       <axis xyz="0 0 1" />
-      <limit lower="${-M_PI/4.0}" upper="${M_PI/4.0}" effort="4.1" velocity="4.796165" />
+      <limit lower="${-M_PI/4.0}" upper="${M_PI/4.0}" effort="4.1" velocity="4.81" />
     </joint>
     <link name="${prefix}_pan_link">
@@ -54,8 +54,8 @@
       <inertial>
         <origin xyz="0.0 0.0 0.0046" rpy="0.0 0.0 0.0" />
-        <mass value="0.08" />
-        <inertia ixx="${1/12*0.08*(3*0.0325**2+0.0092**2)}"     ixy="0.0" ixz="0.0"
-                 iyy="${1/12*0.08*(3*0.0325**2+0.04009253**2)}" iyz="0.0"
-                 izz="${1/2*0.08*0.0325**2}" />
+        <mass value="0.457" />
+        <inertia ixx="${1/12*0.457*(3*0.0325**2+0.0092**2)}"     ixy="0.0" ixz="0.0"
+                 iyy="${1/12*0.457*(3*0.0325**2+0.04009253**2)}" iyz="0.0"
+                 izz="${1/2*0.457*0.0325**2}" />
       </inertial>
     </link>
@@ -65,5 +65,5 @@
       <origin xyz="0.05 0.0 0.131" rpy="0.0 0.0 0.0" />
       <axis xyz="0 -1 0" />
-      <limit lower="${-M_PI/4.0}" upper="${M_PI/6.0}" effort="4.1" velocity="4.796165" />
+      <limit lower="${-M_PI/4.0}" upper="${M_PI/6.0}" effort="4.1" velocity="4.81" />
     </joint>
     <link name="${prefix}_tilt_link">
@@ -83,8 +83,8 @@
       <inertial>
         <origin xyz="-0.01 0.0 0.00943" rpy="0.0 0.0 0.0" />
-        <mass value="0.08" />
-        <inertia ixx="${1/12*0.08*(0.278**2 +0.2**2)}" ixy="0.0" ixz="0.0"
-                 iyy="${1/12*0.08*(0.2**2+0.155**2)}"  iyz="0.0"
-                 izz="${1/12*0.08*(0.155**2 +0.278**2)}" />
+        <mass value="1.88" /> <!-- mass without camera and display-->
+        <inertia ixx="${1/12*1.88*(0.278**2 +0.2**2)}" ixy="0.0" ixz="0.0"
+                 iyy="${1/12*1.88*(0.2**2+0.155**2)}"  iyz="0.0"
+                 izz="${1/12*1.88*(0.155**2 +0.278**2)}" />
       </inertial>
     </link>

File: sobit_home_description/urdf/sensor/lidar.urdf.xacro (robot description, xacro)
@@ -24,8 +24,8 @@
       <inertial>
         <origin xyz="${0.092/2} 0.0 -${0.007/2}" rpy="0.0 0.0 0.0" />
-        <mass value="0.08" />
-        <inertia ixx="${1/12*0.08*(0.092**2+0.007**2)}" ixy="0.0" ixz="0.0"
-                 iyy="${1/12*0.08*(0.184**2+0.007**2)}" iyz="0.0"
-                 izz="${1/12*0.08*(0.092**2+0.184**2)}" />
+        <mass value="0.172" />
+        <inertia ixx="${1/12*0.172*(0.092**2+0.007**2)}" ixy="0.0" ixz="0.0"
+                 iyy="${1/12*0.172*(0.184**2+0.007**2)}" iyz="0.0"
+                 izz="${1/12*0.172*(0.092**2+0.184**2)}" />
       </inertial>
     </link>
@@ -35,6 +35,6 @@
   </xacro:macro>
   <xacro:macro name="lidar" params="parent prefix robot_name">
-    <xacro:lidar_edge parent="${parent}" prefix="${prefix}_front" robot_name="${robot_name}" stand_x= " 0.2357767" stand_y=" 0.2357767" stand_z="0.01" hokuyo_x="0.06914214" hokuyo_y="0.0" hokuyo_z="-0.142" yaw="${M_PI-M_PI/4}"/>
-    <xacro:lidar_edge parent="${parent}" prefix="${prefix}_back"  robot_name="${robot_name}" stand_x= "-0.2357767" stand_y="-0.2357767" stand_z="0.01" hokuyo_x="0.06914214" hokuyo_y="0.0" hokuyo_z="-0.142" yaw="${-M_PI/4}"/>
+    <xacro:lidar_edge prefix="${prefix}_front" parent="${parent}" robot_name="${robot_name}" stand_x= " 0.2357767" stand_y=" 0.2357767" stand_z="0.01" hokuyo_x="0.06914214" hokuyo_y="0.0" hokuyo_z="-0.142" yaw="${M_PI-M_PI/4}"/>
+    <xacro:lidar_edge prefix="${prefix}_back"  parent="${parent}" robot_name="${robot_name}" stand_x= "-0.2357767" stand_y="-0.2357767" stand_z="0.01" hokuyo_x="0.06914214" hokuyo_y="0.0" hokuyo_z="-0.142" yaw="${-M_PI/4}"/>
   </xacro:macro>
 </robot>

File: sobit_home_description/urdf/wheel/wheel.urdf.xacro (robot description, xacro)
@@ -25,8 +25,8 @@
       <inertial>
         <origin xyz="0.0 0.0 0.0" rpy="0.0 0.0 ${M_PI/2.0}" />
-        <mass value="1" />
-        <inertia ixx="${1/12*0.08*(3*0.075**2+0.0797**2)}" ixy="0.0" ixz="0.0"
-                 iyy="${1/12*0.08*(3*0.075**2+0.0797**2)}" iyz="0.0"
-                 izz="${1/2*0.08*0.075**2}" />
+        <mass value="0.877" /> <!-- mass without frame and robomaster -->
+        <inertia ixx="${1/12*0.877*(3*0.075**2+0.0797**2)}" ixy="0.0" ixz="0.0"
+                 iyy="${1/12*0.877*(3*0.075**2+0.0797**2)}" iyz="0.0"
+                 izz="${1/2*0.877*0.075**2}" />
       </inertial>
     </link>
@@ -57,8 +57,8 @@
       <inertial>
         <origin xyz="0.0 0.0 -0.030925" rpy="0.0 0.0 ${M_PI/2}" />
-        <mass value="1" />
-        <inertia ixx="${1/12*1*(0.1**2+0.06185**2)}" ixy="0.0" ixz="0.0"
-                 iyy="${1/12*1*(0.06185**2+0.1**2)}" iyz="0.0"
-                 izz="${1/12*1*(0.1**2+0.1**2)}" />
+        <mass value="0.889" /> <!-- mass without timing belt and others -->
+        <inertia ixx="${1/12*0.889*(0.1**2+0.06185**2)}" ixy="0.0" ixz="0.0"
+                 iyy="${1/12*0.889*(0.06185**2+0.1**2)}" iyz="0.0"
+                 izz="${1/12*0.889*(0.1**2+0.1**2)}" />
       </inertial>
     </link>
@@ -88,8 +88,8 @@
       <inertial>
         <origin xyz="0.0 0.0 0.0" rpy="${M_PI/2.0} 0.0 ${M_PI}" />
-        <mass value="1" />
-        <inertia ixx="${1/12*1*(3*0.075**2+0.017**2)}" ixy="0.0" ixz="0.0"
-                 iyy="${1/12*1*(3*0.075**2+0.017**2)}" iyz="0.0"
-                 izz="${1/2*1*0.075**2}" />
+        <mass value="0.5" /> <!-- TODO -->
+        <inertia ixx="${1/12*0.5*(3*0.075**2+0.017**2)}" ixy="0.0" ixz="0.0"
+                 iyy="${1/12*0.5*(3*0.075**2+0.017**2)}" iyz="0.0"
+                 izz="${1/2*0.5*0.075**2}" />
       </inertial>
     </link>

Commit message: [FIX] joint limits

File: sobit_home_description/urdf/arm/arm.urdf.xacro (robot description, xacro)
@@ -11,6 +11,6 @@
     <xacro:if value="${position == 'right'}">
       <xacro:property name="y_sign" value="-1.0" />
-        <xacro:property name="upper_roll_limit_lower" value="${M_PI/2}" />
-        <xacro:property name="upper_roll_limit_upper" value="${-M_PI/2}" />
+        <xacro:property name="upper_roll_limit_lower" value="${-M_PI/2}" />
+        <xacro:property name="upper_roll_limit_upper" value="${M_PI/2}" />
     </xacro:if>
     <joint name="${prefix}_${position}_base_joint" type="fixed" >
