Commit message: add hand collision box, addjust arm_wrist collision box, update hand .stl files

File: sobit_home_description/urdf/arm/arm.urdf.xacro (robot description, xacro)
@@ -160,7 +160,7 @@
       <parent link="${prefix}_${position}_elbow_link" />
       <child link="${prefix}_${position}_wrist_tilt_link" />
-      <origin xyz="0.0 0.0 -0.5" rpy="0.0 0.0 0.0" />
-      <axis xyz="0.0 -1.0 0.0 " />
-      <limit lower="${-M_PI/2}" upper="${M_PI/2}" effort="${10.6*2}" velocity="11.031179004" />
+      <origin xyz="0.0 ${y_sign * 0.5} 0.0" rpy="0.0 0.0 0.0" />
+      <axis xyz="0.0 0.0 -1.0 " />
+      <limit lower="${-M_PI/2}" upper="${M_PI/2}" effort="4.1" velocity="4.81" />
     </joint>
     <link name="${prefix}_${position}_wrist_tilt_link" >
@@ -168,10 +168,10 @@
         <origin xyz="0.0 0.0 0.0" rpy="0.0 ${-y_sign * M_PI/2} ${M_PI/2}" />
         <geometry>
-          <mesh filename="file://$(find sobit_home_description)/meshes/arm/arm_wrist.stl" scale="0.001 0.001 0.001" />
-        </geometry>
-        <material name="grey" />
-      </visual>
-      <collision>
-        <origin xyz="0.0 ${y_sign * 0.0462} 0.0" rpy="0.0 ${-y_sign * M_PI/2} ${M_PI/2}" />
+          <mesh filename="file://$(find sobit_home_description)/meshes/arm/arm_wrist_tilt.stl" scale="0.001 0.001 0.001" />
+        </geometry>
+        <material name="grey" />
+      </visual>
+      <collision>
+        <origin xyz="0.0 0.0 0.0" rpy="0.0 ${-y_sign * M_PI/2} ${M_PI/2}" />
         <geometry>
           <cylinder length="0.0453" radius="${0.08/2}" />
@@ -179,5 +179,5 @@
       </collision>
       <inertial>
-        <origin xyz="0.0 ${y_sign * 0.0462} 0.0" rpy="0.0 ${-y_sign * M_PI/2} ${M_PI/2}" />
+        <origin xyz="0.0 0.0 0.0" rpy="0.0 ${-y_sign * M_PI/2} ${M_PI/2}" />
         <mass value="0.341" />
         <inertia ixx="${1/12*0.341*(3*0.04**2+0.0453**2)}" ixy="0.0" ixz="0.0"
@@ -189,11 +189,11 @@
       <parent link="${prefix}_${position}_wrist_tilt_link" />
       <child link="${prefix}_${position}_wrist_roll_link" />
-      <origin xyz="0.0 0.0 -0.06648176" rpy="0.0 0.0 0.0" />
-      <axis xyz="0.0 0.0 1.0 " />
+      <origin xyz="0.0 ${y_sign * 0.06648202} 0.0" rpy="0.0 0.0 0.0" />
+      <axis xyz="0.0 1.0 0.0 " />
       <limit lower="${-M_PI/2}" upper="${M_PI/2}" effort="${10.6*2}" velocity="11.031179004" />
     </joint>
     <link name="${prefix}_${position}_wrist_roll_link" >
       <visual>
-        <origin xyz="0.0 0.0 0.0" rpy="0.0 ${M_PI} 0.0" />
+        <origin xyz="0.0 0.0 0.0" rpy="${-y_sign * M_PI/2} ${M_PI} 0.0" />
         <geometry>
           <mesh filename="file://$(find sobit_home_description)/meshes/arm/arm_wrist_roll.stl" scale="0.001 0.001 0.001" />
@@ -201,11 +201,11 @@
         <material name="grey" />
       </visual>
-      <!-- 後でコメントアウト -->
-      <collision>
-        <origin xyz="${0.1166/2+0.0224} 0.0 0.0" rpy="0.0 0.0 0.0" />
-        <geometry>
-          <box size="0.1166 0.124 0.043" />
-        </geometry>
-      </collision>
+      <collision>
+        <origin xyz="0.0 0.0 0.0" rpy="${-y_sign * M_PI/2} ${M_PI} 0.0" />
+        <geometry>
+          <cylinder length="0.0" radius="0.0" />
+          <!-- <box size="0.0 0.0 0.0" /> -->
+        </geometry>
+      </collision>"
       <inertial>
         <origin xyz="${0.1166/2+0.0224} 0.0 0.0" rpy="0.0 0.0 ${M_PI/2}" />

File: sobit_home_description/urdf/hand/hand.urdf.xacro (robot description, xacro)
@@ -6,5 +6,4 @@
     <xacro:if value="${position == 'left'}">
       <xacro:property name="y_sign" value="1.0" />
-      <xacro:property name="yaw_rot" value="0.0" />
         <xacro:property name="upper_roll_limit_lower" value="0" />
         <xacro:property name="upper_roll_limit_upper" value="${M_PI}" />
@@ -12,5 +11,4 @@
     <xacro:if value="${position == 'right'}">
       <xacro:property name="y_sign" value="-1.0" />
-      <xacro:property name="yaw_rot" value="${M_PI}" />
         <xacro:property name="upper_roll_limit_lower" value="${-M_PI}" />
         <xacro:property name="upper_roll_limit_upper" value="0" />
@@ -20,9 +18,9 @@
       <parent link="${parent}" />
       <child link="${prefix_hand}_${position}_cmc_link" />
-      <origin xyz="0.0 0.0 0.0" rpy="0.0 0.0 0.0" />
+      <origin xyz="0.0 ${y_sign * 0.025375} 0.0" rpy="0.0 0.0 0.0" />
     </joint>
     <link name="${prefix_hand}_${position}_cmc_link" >
       <visual>
-        <origin xyz="0.0 0.0 0.0" rpy="${M_PI} 0.0 ${-M_PI/2}" />
+        <origin xyz="0.0 0.0 0.0" rpy="${-y_sign * M_PI/2} ${y_sign * M_PI/2} 0.0" />
         <geometry>
           <mesh filename="file://$(find sobit_home_description)/meshes/hand/hand_base.stl" scale="0.001 0.001 0.001" />
@@ -31,11 +29,11 @@
       </visual>
       <collision>
-        <origin xyz="${0.140/2} 0.0 ${0.043/2}" rpy="0.0 0.0 0.0" />
-        <geometry>
-          <box size="0.140 0.156 0.043" />
-        </geometry>
-      </collision>
-      <inertial>
-        <origin xyz="${0.140/2} 0.0 ${0.043/2}" rpy="0.0 0.0 ${M_PI/2}" />
+        <origin xyz="0.00852612 ${y_sign * 0.008875} 0.0" rpy="${-y_sign * M_PI/2} ${y_sign * M_PI/2} 0.0" />
+        <geometry>
+          <box size="0.108064 0.08255 0.06450" />
+        </geometry>
+      </collision>
+      <inertial>
+        <origin xyz="0.0 0.0 0.0" rpy="${-y_sign * M_PI/2} ${y_sign * M_PI/2} 0.0" />
         <mass value="0.08" />
         <inertia ixx="${1/12*0.08*(0.140**2+0.043**2)}" ixy="0.0" ixz="0.0"
@@ -48,11 +46,11 @@
       <parent link="${prefix_hand}_${position}_cmc_link" />
       <child link="${prefix_hand}_${position}_${prefix_finger}_l_mcp_link" />
-      <origin xyz="-0.003249 0.024532 -0.046" rpy="0.0 0.0 0.0" />
-      <axis xyz="0.0 0.0 1.0 " />
+      <origin xyz="-0.002855 ${y_sign * 0.018025} ${y_sign * 0.024532}" rpy="0.0 0.0 0.0" />
+      <axis xyz="0.0 1.0 0.0 " />
       <limit lower="${-M_PI/2}" upper="${M_PI/2}" effort="0.52" velocity="11.031179004" />
     </joint>
     <link name="${prefix_hand}_${position}_${prefix_finger}_l_mcp_link" >
       <visual>
-        <origin xyz="0.0 0.0 0.0" rpy="${M_PI} 0.0 ${-(2*M_PI/15+M_PI/2)}" />
+        <origin xyz="0.0 0.0 0.0" rpy="${-y_sign * M_PI/2} ${y_sign * (2*M_PI/15 + M_PI/2)} 0.0" />
         <geometry>
           <mesh filename="file://$(find sobit_home_description)/meshes/hand/switching_gear.stl" scale="0.001 0.001 0.001" />
@@ -61,11 +59,11 @@
       </visual>
       <collision>
-        <origin xyz="${0.140/2} 0.0 ${0.043/2}" rpy="0.0 0.0 0.0" />
-        <geometry>
-          <box size="0.140 0.156 0.043" />
-        </geometry>
-      </collision>
-      <inertial>
-        <origin xyz="${0.140/2} 0.0 ${0.043/2}" rpy="0.0 0.0 ${M_PI/2}" />
+        <origin xyz="0.0 0.0 0.0" rpy="${-y_sign * M_PI/2} ${y_sign * (2*M_PI/15 + M_PI/2)} 0.0" />
+        <geometry>
+          <box size="0.0 0.0 0.0" />
+        </geometry>
+      </collision>
+      <inertial>
+        <origin xyz="0.0 0.0 0.0" rpy="${-y_sign * M_PI/2} ${y_sign * (2*M_PI/15 + M_PI/2)} 0.0" />
         <mass value="0.08" />
         <inertia ixx="${1/12*0.08*(0.140**2+0.043**2)}" ixy="0.0" ixz="0.0"
@@ -77,5 +75,5 @@
       <parent link="${prefix_hand}_${position}_${prefix_finger}_l_mcp_link" />
       <child link="${prefix_hand}_${position}_${prefix_finger}_l_pip_link" />
-      <origin xyz="-0.02125 0.040125 -0.018575" rpy="0.0 0.0 0.0" />
+      <origin xyz="-0.02125 ${y_sign * 0.019006} ${y_sign * 0.040125}" rpy="0.0 0.0 0.0" />
       <axis xyz="1.0 0.0 0.0 " />
       <limit lower="${-M_PI/6}" upper="${M_PI/2}" effort="0.52" velocity="11.031179004" />
@@ -83,5 +81,5 @@
     <link name="${prefix_hand}_${position}_${prefix_finger}_l_pip_link" >
       <visual>
-        <origin xyz="0.0 0.0 0.0" rpy="0.0 ${M_PI} ${M_PI/2}" />
+        <origin xyz="0.0 0.0 0.0" rpy="${-y_sign * M_PI/2} ${y_sign * M_PI/2} 0.0" />
         <geometry>
           <mesh filename="file://$(find sobit_home_description)/meshes/hand/middle_pharanx.stl" scale="0.001 0.001 0.001" />
@@ -90,11 +88,11 @@
       </visual>
       <collision>
-        <origin xyz="${0.140/2} 0.0 ${0.043/2}" rpy="0.0 0.0 0.0" />
-        <geometry>
-          <box size="0.140 0.156 0.043" />
-        </geometry>
-      </collision>
-      <inertial>
-        <origin xyz="${0.140/2} 0.0 ${0.043/2}" rpy="0.0 0.0 ${M_PI/2}" />
+        <origin xyz="0.01445 ${y_sign * 0.027375} 0.0" rpy="${-y_sign * M_PI/2} ${y_sign * M_PI/2} 0.0" />
+        <geometry>
+          <box size="0.022 0.031 0.030" />
+        </geometry>
+      </collision>
+      <inertial>
+        <origin xyz="0.0 0.0 0.0" rpy="${-y_sign * M_PI/2} ${y_sign * M_PI/2} 0.0" />
         <mass value="0.08" />
         <inertia ixx="${1/12*0.08*(0.140**2+0.043**2)}" ixy="0.0" ixz="0.0"
@@ -106,5 +104,5 @@
       <parent link="${prefix_hand}_${position}_${prefix_finger}_l_pip_link" />
       <child link="${prefix_hand}_${position}_${prefix_finger}_l_dip_link" />
-      <origin xyz="0.0 0.0 -0.050" rpy="0.0 0.0 0.0" />
+      <origin xyz="0.0 ${y_sign * 0.050} 0.0" rpy="0.0 0.0 0.0" />
       <axis xyz="1.0 0.0 0.0 " />
       <limit lower="${-M_PI/2}" upper="${M_PI/6}" effort="0.52" velocity="11.031179004" />
@@ -112,18 +110,18 @@
     <link name="${prefix_hand}_${position}_${prefix_finger}_l_dip_link" >
       <visual>
-        <origin xyz="0.0 0.0 0.0" rpy="0.0 ${M_PI} ${M_PI/2}" />
+        <origin xyz="0.0 0.0 0.0" rpy="${-y_sign * M_PI/2} ${y_sign * M_PI/2} 0.0" />
         <geometry>
           <mesh filename="file://$(find sobit_home_description)/meshes/hand/distal_pharanx.stl" scale="0.001 0.001 0.001" />
         </geometry>
-        <material name="blue" />
-      </visual>
-      <collision>
-        <origin xyz="${0.140/2} 0.0 ${0.043/2}" rpy="0.0 0.0 0.0" />
-        <geometry>
-          <box size="0.140 0.156 0.043" />
-        </geometry>
-      </collision>
-      <inertial>
-        <origin xyz="${0.140/2} 0.0 ${0.043/2}" rpy="0.0 0.0 ${M_PI/2}" />
+        <material name="grey" />
+      </visual>
+      <collision>
+        <origin xyz="0.01445 ${y_sign * 0.032375} ${-y_sign * 0.001}" rpy="${-y_sign * M_PI/2} ${y_sign * M_PI/2} 0.0" />
+        <geometry>
+          <box size="0.022 0.031 0.035" />
+        </geometry>
+      </collision>
+      <inertial>
+        <origin xyz="0.0 0.0 0.0" rpy="${-y_sign * M_PI/2} ${y_sign * M_PI/2} 0.0" />
         <mass value="0.08" />
         <inertia ixx="${1/12*0.08*(0.140**2+0.043**2)}" ixy="0.0" ixz="0.0"
@@ -137,6 +135,6 @@
       <parent link="${prefix_hand}_${position}_cmc_link" />
       <child link="${prefix_hand}_${position}_${prefix_finger}_r_mcp_link" />
-      <origin xyz="-0.003249 -0.024532 -0.046" rpy="0.0 0.0 0.0" />
-      <axis xyz="0.0 0.0 1.0 " />
+      <origin xyz="-0.002855 ${y_sign * 0.020025} ${-y_sign * 0.024532}" rpy="0.0 0.0 0.0" />
+      <axis xyz="0.0 1.0 0.0 " />
       <limit lower="${-M_PI/2}" upper="${M_PI/2}" effort="0.52" velocity="11.031179004" />
       <mimic joint="${prefix_hand}_${position}_${prefix_finger}_l_mcp_joint" multiplier="-1.0" />
@@ -144,5 +142,5 @@
     <link name="${prefix_hand}_${position}_${prefix_finger}_r_mcp_link" >
       <visual>
-        <origin xyz="0.0 0.0 -0.002006" rpy="${M_PI} 0.0 ${-M_PI/2}" />
+        <origin xyz="0.0 0.0 0.0" rpy="${-y_sign * M_PI/2} ${y_sign * M_PI/2} 0.0" />
         <geometry>
           <mesh filename="file://$(find sobit_home_description)/meshes/hand/switching_gear-m.stl" scale="0.001 0.001 0.001" />
@@ -151,11 +149,11 @@
       </visual>
       <collision>
-        <origin xyz="${0.140/2} 0.0 ${0.043/2}" rpy="0.0 0.0 0.0" />
-        <geometry>
-          <box size="0.140 0.156 0.043" />
-        </geometry>
-      </collision>
-      <inertial>
-        <origin xyz="${0.140/2} 0.0 ${0.043/2}" rpy="0.0 0.0 ${M_PI/2}" />
+        <origin xyz="0.0 0.0 -0.002006" rpy="${-y_sign * M_PI/2} ${y_sign * M_PI/2} 0.0" />
+        <geometry>
+          <box size="0.0 0.0 0.0" />
+        </geometry>
+      </collision>
+      <inertial>
+        <origin xyz="0.0 0.0 -0.002006" rpy="${-y_sign * M_PI/2} ${y_sign * M_PI/2} 0.0" />
         <mass value="0.08" />
         <inertia ixx="${1/12*0.08*(0.140**2+0.043**2)}" ixy="0.0" ixz="0.0"
@@ -167,5 +165,5 @@
       <parent link="${prefix_hand}_${position}_${prefix_finger}_r_mcp_link" />
       <child link="${prefix_hand}_${position}_${prefix_finger}_r_pip_link" />
-      <origin xyz="-0.02125 -0.040125 -0.018575" rpy="0.0 0.0 0.0" />
+      <origin xyz="-0.02125 ${y_sign * 0.016750} ${-y_sign * 0.040125}" rpy="0.0 0.0 0.0" />
       <axis xyz="1.0 0.0 0.0 " />
       <limit lower="${-M_PI/2}" upper="${M_PI/6}" effort="0.52" velocity="11.031179004" />
@@ -173,5 +171,5 @@
     <link name="${prefix_hand}_${position}_${prefix_finger}_r_pip_link" >
       <visual>
-        <origin xyz="0.0 0.0 0.0" rpy="0.0 ${M_PI} ${-M_PI/2}" />
+        <origin xyz="0.0 0.0 0.0" rpy="${-y_sign * M_PI/2} ${-y_sign * M_PI/2} 0.0" />
         <geometry>
           <mesh filename="file://$(find sobit_home_description)/meshes/hand/middle_pharanx-m.stl" scale="0.001 0.001 0.001" />
@@ -180,11 +178,11 @@
       </visual>
       <collision>
-        <origin xyz="${0.140/2} 0.0 ${0.043/2}" rpy="0.0 0.0 0.0" />
-        <geometry>
-          <box size="0.140 0.156 0.043" />
-        </geometry>
-      </collision>
-      <inertial>
-        <origin xyz="${0.140/2} 0.0 ${0.043/2}" rpy="0.0 0.0 ${M_PI/2}" />
+        <origin xyz="0.01445 ${y_sign * 0.027375} 0.0" rpy="${-y_sign * M_PI/2} ${y_sign * M_PI/2} 0.0" />
+        <geometry>
+          <box size="0.022 0.031 0.030" />
+        </geometry>
+      </collision>
+      <inertial>
+        <origin xyz="0.0 0.0 0.0" rpy="${-y_sign * M_PI/2} ${-y_sign * M_PI/2} 0.0" />
         <mass value="0.08" />
         <inertia ixx="${1/12*0.08*(0.140**2+0.043**2)}" ixy="0.0" ixz="0.0"
@@ -196,5 +194,5 @@
       <parent link="${prefix_hand}_${position}_${prefix_finger}_r_pip_link" />
       <child link="${prefix_hand}_${position}_${prefix_finger}_r_dip_link" />
-      <origin xyz="0.0 0.0 -0.050" rpy="0.0 0.0 0.0" />
+      <origin xyz="0.0 ${y_sign * 0.050} 0.0" rpy="0.0 0.0 0.0" />
       <axis xyz="1.0 0.0 0.0 " />
       <limit lower="${-M_PI/6}" upper="${M_PI/2}" effort="0.52" velocity="11.031179004" />
@@ -202,18 +200,18 @@
     <link name="${prefix_hand}_${position}_${prefix_finger}_r_dip_link" >
       <visual>
-        <origin xyz="0.0 0.0 0.0" rpy="0.0 ${M_PI} ${-M_PI/2}" />
+        <origin xyz="0.0 0.0 0.0" rpy="${-y_sign * M_PI/2} ${-y_sign * M_PI/2} 0.0" />
         <geometry>
           <mesh filename="file://$(find sobit_home_description)/meshes/hand/distal_pharanx-m.stl" scale="0.001 0.001 0.001" />
         </geometry>
-        <material name="green" />
-      </visual>
-      <collision>
-        <origin xyz="${0.140/2} 0.0 ${0.043/2}" rpy="0.0 0.0 0.0" />
-        <geometry>
-          <box size="0.140 0.156 0.043" />
-        </geometry>
-      </collision>
-      <inertial>
-        <origin xyz="${0.140/2} 0.0 ${0.043/2}" rpy="0.0 0.0 ${M_PI/2}" />
+        <material name="grey" />
+      </visual>
+      <collision>
+        <origin xyz="0.01445 ${y_sign * 0.032375} ${y_sign * 0.001}" rpy="${-y_sign * M_PI/2} ${y_sign * M_PI/2} 0.0" />
+        <geometry>
+          <box size="0.022 0.031 0.035" />
+        </geometry>
+      </collision>
+      <inertial>
+        <origin xyz="0.0 0.0 0.0" rpy="${-y_sign * M_PI/2} ${-y_sign * M_PI/2} 0.0" />
         <mass value="0.08" />
         <inertia ixx="${1/12*0.08*(0.140**2+0.043**2)}" ixy="0.0" ixz="0.0"
@@ -226,11 +224,11 @@
       <parent link="${prefix_hand}_${position}_cmc_link" />
       <child link="${prefix_hand}_${position}_${prefix_finger}_c_mcp_link" />
-      <origin xyz="0.036751 0.01435 -0.062" rpy="0.0 0.0 0.0" />
-      <axis xyz="0.0 1.0 0.0 " />
+      <origin xyz="0.036751 ${y_sign * 0.036625} ${y_sign * 0.014550} " rpy="0.0 0.0 0.0" />
+      <axis xyz="0.0 0.0 1.0 " />
       <limit lower="${-M_PI/2}" upper="${M_PI/6}" effort="0.52" velocity="11.031179004" />
     </joint>
     <link name="${prefix_hand}_${position}_${prefix_finger}_c_mcp_link" >
       <visual>
-        <origin xyz="0.0 0.0 0.0" rpy="0.0 ${M_PI} ${M_PI}" />
+        <origin xyz="0.0 0.0 0.0" rpy="${-y_sign * M_PI/2} 0.0 0.0" />
         <geometry>
           <mesh filename="file://$(find sobit_home_description)/meshes/hand/thumb_middle_pharanx.stl" scale="0.001 0.001 0.001" />
@@ -239,11 +237,11 @@
       </visual>
       <collision>
-        <origin xyz="${0.140/2} 0.0 ${0.043/2}" rpy="0.0 0.0 0.0" />
-        <geometry>
-          <box size="0.140 0.156 0.043" />
-        </geometry>
-      </collision>
-      <inertial>
-        <origin xyz="${0.140/2} 0.0 ${0.043/2}" rpy="0.0 0.0 ${M_PI/2}" />
+        <origin xyz="-0.001 ${y_sign * 0.027375} ${-y_sign * 0.01445}" rpy="0.0 0.0 0.0" />
+        <geometry>
+          <box size="0.022 0.0334 0.030" />
+        </geometry>
+      </collision>
+      <inertial>
+        <origin xyz="0.0 0.0 0.0" rpy="${-y_sign * M_PI/2} 0.0 0.0" />
         <mass value="0.08" />
         <inertia ixx="${1/12*0.08*(0.140**2+0.043**2)}" ixy="0.0" ixz="0.0"
@@ -255,5 +253,5 @@
       <parent link="${prefix_hand}_${position}_${prefix_finger}_c_mcp_link" />
       <child link="${prefix_hand}_${position}_${prefix_finger}_c_ip_link" />
-      <origin xyz="0.0 0.0 -0.050" rpy="0.0 0.0 0.0" />
+      <origin xyz="0.0 ${y_sign * 0.050} 0.0" rpy="0.0 0.0 0.0" />
       <axis xyz="0.0 1.0 0.0 " />
       <limit lower="${-M_PI/6}" upper="${M_PI/2}" effort="0.52" velocity="11.031179004" />
@@ -261,18 +259,18 @@
     <link name="${prefix_hand}_${position}_${prefix_finger}_c_ip_link" >
       <visual>
-        <origin xyz="0.0 0.0 0.0" rpy="0.0 ${M_PI} ${M_PI}" />
+        <origin xyz="0.0 0.0 0.0" rpy="${-y_sign * M_PI/2} 0.0 0.0" />
         <geometry>
           <mesh filename="file://$(find sobit_home_description)/meshes/hand/thumb_distal_pharanx.stl" scale="0.001 0.001 0.001" />
         </geometry>
-        <material name="red" />
-      </visual>
-      <collision>
-        <origin xyz="${0.140/2} 0.0 ${0.043/2}" rpy="0.0 0.0 0.0" />
-        <geometry>
-          <box size="0.140 0.156 0.043" />
-        </geometry>
-      </collision>
-      <inertial>
-        <origin xyz="${0.140/2} 0.0 ${0.043/2}" rpy="0.0 0.0 ${M_PI/2}" />
+        <material name="green" />
+      </visual>
+      <collision>
+        <origin xyz="-0.001 ${y_sign * 0.034375} ${-y_sign * 0.01445}" rrpy="${-y_sign * M_PI/2} ${y_sign * M_PI/2} 0.0" />
+        <geometry>
+          <box size="0.022 0.031 0.035" />
+        </geometry>
+      </collision>
+      <inertial>
+        <origin xyz="0.0 0.0 0.0" rpy="${-y_sign * M_PI/2} 0.0 0.0" />
         <mass value="0.08" />
         <inertia ixx="${1/12*0.08*(0.140**2+0.043**2)}" ixy="0.0" ixz="0.0"
