Commit message: addjust wrist collision box, add collision and inertial to hand parts

File: sobit_home_description/urdf/arm/arm.urdf.xacro (robot description, xacro)
@@ -173,5 +173,5 @@
       </visual>
       <collision>
-        <origin xyz="0.0 0.0 0.0" rpy="0.0 ${-y_sign * M_PI/2} ${M_PI/2}" />
+        <origin xyz="0.0 ${y_sign * 0.0462} 0.0" rpy="0.0 ${-y_sign * M_PI/2} ${M_PI/2}" />
         <geometry>
           <cylinder length="0.0453" radius="${0.08/2}" />
@@ -195,5 +195,5 @@
     <link name="${prefix}_${position}_wrist_roll_link" >
       <visual>
-        <origin xyz="0.0 0.0 0.0" rpy="${-y_sign * M_PI/2} ${M_PI} 0.0" />
+        <origin xyz="0.0 0.0 0.0" rpy="0.0 0.0 0.0" />
         <geometry>
           <mesh filename="file://$(find sobit_home_description)/meshes/arm/arm_wrist_roll.stl" scale="0.001 0.001 0.001" />
@@ -202,16 +202,17 @@
       </visual>
       <collision>
-        <origin xyz="0.0 0.0 0.0" rpy="${-y_sign * M_PI/2} ${M_PI} 0.0" />
-        <geometry>
-          <cylinder length="0.0" radius="0.0" />
-          <!-- <box size="0.0 0.0 0.0" /> -->
-        </geometry>
-      </collision>"
-      <inertial>
-        <origin xyz="${0.1166/2+0.0224} 0.0 0.0" rpy="0.0 0.0 ${M_PI/2}" />
-        <mass value="0.08" />
-        <inertia ixx="${1/12*0.08*(0.1166**2+0.043**2)}" ixy="0.0" ixz="0.0"
-                 iyy="${1/12*0.08*(0.124**2 +0.043**2)}" iyz="0.0"
-                 izz="${1/12*0.08*(0.1166**2+0.124**2)}" />
+        <origin xyz="0.00852612 ${y_sign * 0.07450 / 2} 0.0" rpy="0.0 ${y_sign * M_PI/2} ${y_sign * M_PI/2}" />
+        <geometry>
+          <!-- <box size="0.108064 0.08255 0.0645" /> -->
+          <box size="0.108 0.0826 0.0645" />
+        </geometry>
+      </collision>
+      <inertial>
+        <origin xyz="0.0 0.0 0.0" rpy="0.0 0.0 0.0" />
+        <!-- <mass value="0.0160103055903" /> -->
+        <mass value="0.016" />
+        <inertia ixx="${1/12*0.016*(0.0645**2+0.0826**2)}" ixy="0.0" ixz="0.0"
+                 iyy="${1/12*0.016*(0.108**2 +0.0645**2)}" iyz="0.0"
+                 izz="${1/12*0.016*(0.108**2+0.0826**2)}" />
       </inertial>
     </link>

File: sobit_home_description/urdf/hand/hand.urdf.xacro (robot description, xacro)
@@ -28,16 +28,11 @@
         <material name="grey" />
       </visual>
-      <collision>
+      <inertial>
         <origin xyz="0.00852612 ${y_sign * 0.008875} 0.0" rpy="${-y_sign * M_PI/2} ${y_sign * M_PI/2} 0.0" />
-        <geometry>
-          <box size="0.108064 0.08255 0.06450" />
-        </geometry>
-      </collision>
-      <inertial>
-        <origin xyz="0.0 0.0 0.0" rpy="${-y_sign * M_PI/2} ${y_sign * M_PI/2} 0.0" />
-        <mass value="0.08" />
-        <inertia ixx="${1/12*0.08*(0.140**2+0.043**2)}" ixy="0.0" ixz="0.0"
-                 iyy="${1/12*0.08*(0.156**2+0.043**2)}" iyz="0.0"
-                 izz="${1/12*0.08*(0.140**2+0.156**2)}" />
+        <!-- <mass value="0.1814929213426" /> -->
+        <mass value="0.181" />
+        <inertia ixx="${1/12*0.181*(0.0645**2+0.0826**2)}" ixy="0.0" ixz="0.0"
+                 iyy="${1/12*0.181*(0.108**2+0.0645**2)}" iyz="0.0"
+                 izz="${1/12*0.181*(0.108**2+0.0826**2)}" />
       </inertial>
     </link>
@@ -58,16 +53,11 @@
         <material name="grey" />
       </visual>
-      <collision>
+      <inertial>
         <origin xyz="0.0 0.0 0.0" rpy="${-y_sign * M_PI/2} ${y_sign * (2*M_PI/15 + M_PI/2)} 0.0" />
-        <geometry>
-          <box size="0.0 0.0 0.0" />
-        </geometry>
-      </collision>
-      <inertial>
-        <origin xyz="0.0 0.0 0.0" rpy="${-y_sign * M_PI/2} ${y_sign * (2*M_PI/15 + M_PI/2)} 0.0" />
-        <mass value="0.08" />
-        <inertia ixx="${1/12*0.08*(0.140**2+0.043**2)}" ixy="0.0" ixz="0.0"
-                 iyy="${1/12*0.08*(0.156**2+0.043**2)}" iyz="0.0"
-                 izz="${1/12*0.08*(0.140**2+0.156**2)}" />
+        <!-- <mass value="0.022421331012" /> -->
+        <mass value="0.0224" />
+        <inertia ixx="${1/12*0.0224*(0.0645**2+0.0826**2)}" ixy="0.0" ixz="0.0"
+                 iyy="${1/12*0.0224*(0.108**2 +0.0645**2)}" iyz="0.0"
+                 izz="${1/12*0.0224*(0.108**2+0.0826**2)}" />
       </inertial>
     </link>
@@ -88,5 +78,5 @@
       </visual>
       <collision>
-        <origin xyz="0.01445 ${y_sign * 0.027375} 0.0" rpy="${-y_sign * M_PI/2} ${y_sign * M_PI/2} 0.0" />
+        <origin xyz="0.01445 ${y_sign * 0.030375} 0.0" rpy="${-y_sign * M_PI/2} ${y_sign * M_PI/2} 0.0" />
         <geometry>
           <box size="0.022 0.031 0.030" />
@@ -95,8 +85,9 @@
       <inertial>
         <origin xyz="0.0 0.0 0.0" rpy="${-y_sign * M_PI/2} ${y_sign * M_PI/2} 0.0" />
-        <mass value="0.08" />
-        <inertia ixx="${1/12*0.08*(0.140**2+0.043**2)}" ixy="0.0" ixz="0.0"
-                 iyy="${1/12*0.08*(0.156**2+0.043**2)}" iyz="0.0"
-                 izz="${1/12*0.08*(0.140**2+0.156**2)}" />
+        <!-- <mass value="0.036103135757000006" /> -->
+        <mass value="0.0361" />
+        <inertia ixx="${1/12*0.0361*(0.031**2+0.030**2)}" ixy="0.0" ixz="0.0"
+                 iyy="${1/12*0.0361*(0.022**2+0.031**2)}" iyz="0.0"
+                 izz="${1/12*0.0361*(0.022**2+0.031**2)}" />
       </inertial>
     </link>
@@ -124,8 +115,9 @@
       <inertial>
         <origin xyz="0.0 0.0 0.0" rpy="${-y_sign * M_PI/2} ${y_sign * M_PI/2} 0.0" />
-        <mass value="0.08" />
-        <inertia ixx="${1/12*0.08*(0.140**2+0.043**2)}" ixy="0.0" ixz="0.0"
-                 iyy="${1/12*0.08*(0.156**2+0.043**2)}" iyz="0.0"
-                 izz="${1/12*0.08*(0.140**2+0.156**2)}" />
+        <!-- <mass value="0.0371972081495" /> -->
+        <mass value="0.0372" />
+        <inertia ixx="${1/12*0.0372*(0.035**2+0.031**2)}" ixy="0.0" ixz="0.0"
+                 iyy="${1/12*0.0372*(0.022**2+0.035**2)}" iyz="0.0"
+                 izz="${1/12*0.0372*(0.022**2+0.031**2)}" />
       </inertial>
     </link>
@@ -148,16 +140,11 @@
         <material name="grey" />
       </visual>
-      <collision>
-        <origin xyz="0.0 0.0 -0.002006" rpy="${-y_sign * M_PI/2} ${y_sign * M_PI/2} 0.0" />
-        <geometry>
-          <box size="0.0 0.0 0.0" />
-        </geometry>
-      </collision>
-      <inertial>
-        <origin xyz="0.0 0.0 -0.002006" rpy="${-y_sign * M_PI/2} ${y_sign * M_PI/2} 0.0" />
-        <mass value="0.08" />
-        <inertia ixx="${1/12*0.08*(0.140**2+0.043**2)}" ixy="0.0" ixz="0.0"
-                 iyy="${1/12*0.08*(0.156**2+0.043**2)}" iyz="0.0"
-                 izz="${1/12*0.08*(0.140**2+0.156**2)}" />
+      <inertial>
+        <origin xyz="0.0 0.0 0.0" rpy="${-y_sign * M_PI/2} ${y_sign * (2*M_PI/15 + M_PI/2)} 0.0" />
+        <!-- <mass value="0.0216864236256" /> -->
+        <mass value="0.0217" />
+        <inertia ixx="${1/12*0.0217*(0.0645**2+0.0826**2)}" ixy="0.0" ixz="0.0"
+                 iyy="${1/12*0.0217*(0.108**2 +0.0645**2)}" iyz="0.0"
+                 izz="${1/12*0.0217*(0.108**2+0.0826**2)}" />
       </inertial>
     </link>
@@ -178,5 +165,5 @@
       </visual>
       <collision>
-        <origin xyz="0.01445 ${y_sign * 0.027375} 0.0" rpy="${-y_sign * M_PI/2} ${y_sign * M_PI/2} 0.0" />
+        <origin xyz="0.01445 ${y_sign * 0.030375} 0.0" rpy="${-y_sign * M_PI/2} ${y_sign * M_PI/2} 0.0" />
         <geometry>
           <box size="0.022 0.031 0.030" />
@@ -185,8 +172,9 @@
       <inertial>
         <origin xyz="0.0 0.0 0.0" rpy="${-y_sign * M_PI/2} ${-y_sign * M_PI/2} 0.0" />
-        <mass value="0.08" />
-        <inertia ixx="${1/12*0.08*(0.140**2+0.043**2)}" ixy="0.0" ixz="0.0"
-                 iyy="${1/12*0.08*(0.156**2+0.043**2)}" iyz="0.0"
-                 izz="${1/12*0.08*(0.140**2+0.156**2)}" />
+        <!-- <mass value="0.0361032786215" /> -->
+        <mass value="0.0361" />
+        <inertia ixx="${1/12*0.0361*(0.0031**2+0.030**2)}" ixy="0.0" ixz="0.0"
+                 iyy="${1/12*0.0361*(0.01445**2+0.0031**2)}" iyz="0.0"
+                 izz="${1/12*0.0361*(0.01445**2+0.030**2)}" />
       </inertial>
     </link>
@@ -214,8 +202,9 @@
       <inertial>
         <origin xyz="0.0 0.0 0.0" rpy="${-y_sign * M_PI/2} ${-y_sign * M_PI/2} 0.0" />
-        <mass value="0.08" />
-        <inertia ixx="${1/12*0.08*(0.140**2+0.043**2)}" ixy="0.0" ixz="0.0"
-                 iyy="${1/12*0.08*(0.156**2+0.043**2)}" iyz="0.0"
-                 izz="${1/12*0.08*(0.140**2+0.156**2)}" />
+        <!-- <mass value="0.0371997477059" /> -->
+        <mass value="0.0372" />
+        <inertia ixx="${1/12*0.0372*(0.035**2+0.031**2)}" ixy="0.0" ixz="0.0"
+                 iyy="${1/12*0.0372*(0.022**2+0.035**2)}" iyz="0.0"
+                 izz="${1/12*0.0372*(0.022**2+0.031**2)}" />
       </inertial>
     </link>
@@ -237,15 +226,16 @@
       </visual>
       <collision>
-        <origin xyz="-0.001 ${y_sign * 0.027375} ${-y_sign * 0.01445}" rpy="0.0 0.0 0.0" />
-        <geometry>
-          <box size="0.022 0.0334 0.030" />
-        </geometry>
-      </collision>
-      <inertial>
-        <origin xyz="0.0 0.0 0.0" rpy="${-y_sign * M_PI/2} 0.0 0.0" />
-        <mass value="0.08" />
-        <inertia ixx="${1/12*0.08*(0.140**2+0.043**2)}" ixy="0.0" ixz="0.0"
-                 iyy="${1/12*0.08*(0.156**2+0.043**2)}" iyz="0.0"
-                 izz="${1/12*0.08*(0.140**2+0.156**2)}" />
+        <origin xyz="-0.001 ${y_sign * 0.032375} ${-y_sign * 0.01445}" rpy="0.0 0.0 0.0" />
+        <geometry>
+          <box size="0.022 0.031 0.034" />
+        </geometry>
+      </collision>
+      <inertial>
+        <origin xyz="0.0 0.0 0.0" rpy="${-y_sign * M_PI/2} 0.0 0.0" />
+        <!-- <mass value="0.0377428526807" /> -->
+        <mass value="0.0377" />
+        <inertia ixx="${1/12*0.0377*(0.034**2+0.031**2)}" ixy="0.0" ixz="0.0"
+                 iyy="${1/12*0.0377*(0.022**2+0.034**2)}" iyz="0.0"
+                 izz="${1/12*0.0377*(0.022**2+0.031**2)}" />
       </inertial>
     </link>
@@ -254,5 +244,5 @@
       <child link="${prefix_hand}_${position}_${prefix_finger}_c_ip_link" />
       <origin xyz="0.0 ${y_sign * 0.050} 0.0" rpy="0.0 0.0 0.0" />
-      <axis xyz="0.0 1.0 0.0 " />
+      <axis xyz="0.0 0.0 1.0 " />
       <limit lower="${-M_PI/6}" upper="${M_PI/2}" effort="0.52" velocity="11.031179004" />
     </joint>
@@ -263,18 +253,19 @@
           <mesh filename="file://$(find sobit_home_description)/meshes/hand/thumb_distal_pharanx.stl" scale="0.001 0.001 0.001" />
         </geometry>
-        <material name="green" />
+        <material name="grey" />
       </visual>
       <collision>
         <origin xyz="-0.001 ${y_sign * 0.034375} ${-y_sign * 0.01445}" rrpy="${-y_sign * M_PI/2} ${y_sign * M_PI/2} 0.0" />
         <geometry>
-          <box size="0.022 0.031 0.035" />
-        </geometry>
-      </collision>
-      <inertial>
-        <origin xyz="0.0 0.0 0.0" rpy="${-y_sign * M_PI/2} 0.0 0.0" />
-        <mass value="0.08" />
-        <inertia ixx="${1/12*0.08*(0.140**2+0.043**2)}" ixy="0.0" ixz="0.0"
-                 iyy="${1/12*0.08*(0.156**2+0.043**2)}" iyz="0.0"
-                 izz="${1/12*0.08*(0.140**2+0.156**2)}" />
+          <box size="0.022 0.031 0.0334" />
+        </geometry>
+      </collision>
+      <inertial>
+        <origin xyz="0.0 0.0 0.0" rpy="${-y_sign * M_PI/2} 0.0 0.0" />
+        <!-- <mass value="0.017059696584599996" /> -->
+        <mass value="0.0171" />
+        <inertia ixx="${1/12*0.0171*(0.0334**2+0.031**2)}" ixy="0.0" ixz="0.0"
+                 iyy="${1/12*0.0171*(0.022**2+0.0334**2)}" iyz="0.0"
+                 izz="${1/12*0.0171*(0.022**2+0.031**2)}" />
       </inertial>
     </link>
@@ -282,2 +273,12 @@
   </xacro:macro>
 </robot>
+<!--
+<<tsukada no memo>> =============================================================================
+この順序はパーツのvisualやcollisionのオリジンが回転することに依存しない...らしい？？？
+ただし、.stlをインポートする際の原点に対するパーツの軸方向が影響している可能性があるような気が...
+<box size = "w"  "d"  "h" >
+  w: x方向の大きさ(幅)
+  d: y方向の大きさ（奥行き）
+  h: z方向の大きさ（高さ）
+======================================================================================
+-->

Commit message: [FIX] joint limits for arm and controllers

File: sobit_home_description/urdf/arm/arm.urdf.xacro (robot description, xacro)
@@ -6,11 +6,7 @@
     <xacro:if value="${position == 'left'}">
       <xacro:property name="y_sign" value="1.0" />
-        <xacro:property name="upper_roll_limit_lower" value="${-M_PI/2}" />
-        <xacro:property name="upper_roll_limit_upper" value="${M_PI/2}" />
     </xacro:if>
     <xacro:if value="${position == 'right'}">
       <xacro:property name="y_sign" value="-1.0" />
-        <xacro:property name="upper_roll_limit_lower" value="${-M_PI/2}" />
-        <xacro:property name="upper_roll_limit_upper" value="${M_PI/2}" />
     </xacro:if>
     <joint name="${prefix}_${position}_base_joint" type="fixed" >
@@ -21,5 +17,5 @@
     <link name="${prefix}_${position}_base_link" >
       <visual>
-        <origin xyz="0.0 0.0 0.0" rpy="${M_PI/2} 0.0 ${y_sign * M_PI/2}" />
+        <origin xyz="0.0 0.0 0.0" rpy="0.0 ${(y_sign+1) * M_PI/2} ${-M_PI/2}" />
         <geometry>
           <mesh filename="file://$(find sobit_home_description)/meshes/arm/arm_scapula.stl" scale="0.001 0.001 0.001" />
@@ -45,10 +41,10 @@
       <child link="${prefix}_${position}_shoulder_tilt_link" />
       <origin xyz="0.0 ${y_sign * 0.126} 0.0" rpy="0.0 0.0 0.0" />
-      <axis xyz="0.0 1.0 0.0 " />
-      <limit lower="${-M_PI/2}" upper="${M_PI/2}" effort="44.7" velocity="3.0" />
+      <axis xyz="0.0 ${y_sign} 0.0" />
+      <limit lower="${-M_PI/2}" upper="${M_PI/2}" effort="${44.7 * effort_ratio}" velocity="3.0" />
     </joint>
     <link name="${prefix}_${position}_shoulder_tilt_link" >
       <visual>
-        <origin xyz="0.0 0.0 0.0" rpy="0.0 0.0 ${y_sign * M_PI/2}" />
+        <origin xyz="0.0 0.0 0.0" rpy="0.0 ${(y_sign+1) * M_PI/2} ${-M_PI/2}" />
         <geometry>
           <mesh filename="file://$(find sobit_home_description)/meshes/arm/arm_shoulder.stl" scale="0.001 0.001 0.001" />
@@ -74,6 +70,6 @@
       <child link="${prefix}_${position}_upper_roll_link" />
       <origin xyz="0.0 ${y_sign * 0.0725} 0.0" rpy="0.0 0.0 0.0" />
-      <axis xyz="1.0 0.0 0.0 " />
-      <limit lower="${upper_roll_limit_lower}" upper="${upper_roll_limit_upper}" effort="1060.0" velocity="3.14" />
+      <axis xyz="1.0 0.0 0.0" />
+      <limit lower="${-M_PI/2}" upper="${M_PI/2}" effort="${10.6 * effort_ratio}" velocity="3.14" />
     </joint>
     <link name="${prefix}_${position}_upper_roll_link" >
@@ -103,10 +99,10 @@
       <child link="${prefix}_${position}_upper_flex_link" />
       <origin xyz="0.0 ${y_sign * 0.215813} 0.0" rpy="0.0 0.0 0.0" />
-      <axis xyz="0.0 1.0 0.0" />
-      <limit lower="${-M_PI/2}" upper="${M_PI/2}" effort="4.1" velocity="4.81" />
+      <axis xyz="0.0 ${y_sign} 0.0" />
+      <limit lower="${-y_sign * M_PI/2}" upper="${y_sign * M_PI/2}" effort="${4.1 * effort_ratio}" velocity="4.81" />
     </joint>
     <link name="${prefix}_${position}_upper_flex_link" >
       <visual>
-        <origin xyz="0.0 0.0 0.0" rpy="0.0 ${y_sign * M_PI/2} ${-M_PI/2}" />
+        <origin xyz="0.0 0.0 0.0" rpy="${y_sign * M_PI/2} ${-y_sign * M_PI/2} 0.0" />
         <geometry>
           <mesh filename="file://$(find sobit_home_description)/meshes/arm/arm_upper_flex.stl" scale="0.001 0.001 0.001" />
@@ -132,6 +128,14 @@
       <child link="${prefix}_${position}_elbow_link" />
       <origin xyz="0.0 ${y_sign * 0.18413635} 0.0" rpy="0.0 0.0 0.0" />
-      <axis xyz="0.0 0.0 -1.0" />
-      <limit lower="0" upper="${M_PI/2}" effort="10.6" velocity="3.14" />
+      <axis xyz="0.0 0.0 1.0" />
+        <xacro:if value="${y_sign == -1.0}">
+          <xacro:property name="elbow_lower_limit" value="0.0" />
+          <xacro:property name="elbow_upper_limit" value="${M_PI/2}" />
+        </xacro:if>
+        <xacro:if value="${y_sign == 1.0}">
+          <xacro:property name="elbow_lower_limit" value="${-M_PI/2}" />
+          <xacro:property name="elbow_upper_limit" value="0.0" />
+        </xacro:if>
+        <limit lower="${elbow_lower_limit}" upper="${elbow_upper_limit}" effort="${10.6 * effort_ratio}" velocity="3.14" />
     </joint>
     <link name="${prefix}_${position}_elbow_link" >
@@ -161,6 +165,6 @@
       <child link="${prefix}_${position}_wrist_tilt_link" />
       <origin xyz="0.0 ${y_sign * 0.5} 0.0" rpy="0.0 0.0 0.0" />
-      <axis xyz="0.0 0.0 -1.0 " />
-      <limit lower="${-M_PI/2}" upper="${M_PI/2}" effort="4.1" velocity="4.81" />
+      <axis xyz="0.0 0.0 1.0" />
+      <limit lower="${-y_sign * M_PI/2}" upper="${y_sign * M_PI/2}" effort="${4.1 * effort_ratio}" velocity="4.81" />
     </joint>
     <link name="${prefix}_${position}_wrist_tilt_link" >
@@ -190,6 +194,6 @@
       <child link="${prefix}_${position}_wrist_roll_link" />
       <origin xyz="0.0 ${y_sign * 0.06648202} 0.0" rpy="0.0 0.0 0.0" />
-      <axis xyz="0.0 1.0 0.0 " />
-      <limit lower="${-M_PI/2}" upper="${M_PI/2}" effort="${10.6*2}" velocity="11.031179004" />
+      <axis xyz="0.0 ${y_sign} 0.0" />
+      <limit lower="${-y_sign * M_PI/2}" upper="${y_sign * M_PI/2}" effort="${10.6 * effort_ratio}" velocity="11.031179004" />
     </joint>
     <link name="${prefix}_${position}_wrist_roll_link" >

File: sobit_home_description/urdf/controllers.urdf.xacro (robot description, xacro)
@@ -365,6 +365,6 @@
       </xacro:unless>
       <command_interface name="position">
-        <param name="min">0</param>
-        <param name="max">${M_PI/2}</param>
+        <param name="min">-${M_PI/2}</param>
+        <param name="max">0</param>
       </command_interface>
       <!-- <command_interface name="velocity"/> -->
@@ -399,6 +399,6 @@
       </xacro:unless>
       <command_interface name="position">
-        <param name="min">-1.570796327</param>
-        <param name="max">1.570796327</param>
+        <param name="min">-${M_PI/2}</param>
+        <param name="max">${M_PI/2}</param>
       </command_interface>
       <!-- <command_interface name="velocity"/> -->
@@ -452,5 +452,5 @@
       </xacro:unless>
       <command_interface name="position">
-        <param name="min">-${M_PI/2}</param>
+        <param name="min">0</param>
         <param name="max">${M_PI/2}</param>
       </command_interface>
