Commit message: [UPD] arm upper & elbow

File: sobit_home_description/urdf/arm/arm.urdf.xacro (robot description, xacro)
@@ -6,20 +6,16 @@
     <xacro:if value="${position == 'left'}">
       <xacro:property name="y_sign" value="1.0" />
-        <xacro:property name="upper_roll_limit_lower" value="${-M_PI/2}" />
-        <xacro:property name="upper_roll_limit_upper" value="${M_PI/2}" />
     </xacro:if>
     <xacro:if value="${position == 'right'}">
       <xacro:property name="y_sign" value="-1.0" />
-        <xacro:property name="upper_roll_limit_lower" value="${-M_PI/2}" />
-        <xacro:property name="upper_roll_limit_upper" value="${M_PI/2}" />
     </xacro:if>
     <joint name="${prefix}_${position}_base_joint" type="fixed" >
       <parent link="${parent}" />
       <child link="${prefix}_${position}_base_link" />
-      <origin xyz="0.0 ${y_sign * 0.079} 0.0" rpy="0.0 0.0 0.0" />
+      <origin xyz="0.178 ${y_sign * 0.079} 0.0" rpy="0.0 0.0 0.0" />
     </joint>
     <link name="${prefix}_${position}_base_link" >
       <visual>
-        <origin xyz="0.0 0.0 0.0" rpy="${M_PI/2} 0.0 ${y_sign * M_PI/2}" />
+        <origin xyz="0.0 0.0 0.0" rpy="0.0 ${(y_sign+1) * M_PI/2} ${-M_PI/2}" />
         <geometry>
           <mesh filename="file://$(find sobit_home_description)/meshes/arm/arm_scapula.stl" scale="0.001 0.001 0.001" />
@@ -45,10 +41,10 @@
       <child link="${prefix}_${position}_shoulder_tilt_link" />
       <origin xyz="0.0 ${y_sign * 0.126} 0.0" rpy="0.0 0.0 0.0" />
-      <axis xyz="0.0 1.0 0.0 " />
-      <limit lower="${-M_PI/2}" upper="${M_PI/2}" effort="44.7" velocity="3.0" />
+      <axis xyz="0.0 ${y_sign} 0.0" />
+      <limit lower="${-M_PI/2}" upper="${M_PI/2}" effort="${44.7 * effort_ratio}" velocity="3.0" />
     </joint>
     <link name="${prefix}_${position}_shoulder_tilt_link" >
       <visual>
-        <origin xyz="0.0 0.0 0.0" rpy="0.0 0.0 ${y_sign * M_PI/2}" />
+        <origin xyz="0.0 0.0 0.0" rpy="0.0 ${(y_sign+1) * M_PI/2} ${-M_PI/2}" />
         <geometry>
           <mesh filename="file://$(find sobit_home_description)/meshes/arm/arm_shoulder.stl" scale="0.001 0.001 0.001" />
@@ -74,6 +70,6 @@
       <child link="${prefix}_${position}_upper_roll_link" />
       <origin xyz="0.0 ${y_sign * 0.0725} 0.0" rpy="0.0 0.0 0.0" />
-      <axis xyz="1.0 0.0 0.0 " />
-      <limit lower="${upper_roll_limit_lower}" upper="${upper_roll_limit_upper}" effort="1060.0" velocity="3.14" />
+      <axis xyz="1.0 0.0 0.0" />
+      <limit lower="${-M_PI/2}" upper="${M_PI/2}" effort="${10.6 * effort_ratio}" velocity="3.14" />
     </joint>
     <link name="${prefix}_${position}_upper_roll_link" >
@@ -102,11 +98,11 @@
       <parent link="${prefix}_${position}_upper_roll_link" />
       <child link="${prefix}_${position}_upper_flex_link" />
-      <origin xyz="0.0 ${y_sign * 0.215813} 0.0" rpy="0.0 0.0 0.0" />
-      <axis xyz="0.0 1.0 0.0" />
-      <limit lower="${-M_PI/2}" upper="${M_PI/2}" effort="4.1" velocity="4.81" />
+      <origin xyz="0.0 ${y_sign * 0.2} 0.0" rpy="0.0 0.0 0.0" />
+      <axis xyz="0.0 ${y_sign} 0.0" />
+      <limit lower="${-y_sign * M_PI/2}" upper="${y_sign * M_PI/2}" effort="${4.1 * effort_ratio}" velocity="4.81" />
     </joint>
     <link name="${prefix}_${position}_upper_flex_link" >
       <visual>
-        <origin xyz="0.0 0.0 0.0" rpy="0.0 ${y_sign * M_PI/2} ${-M_PI/2}" />
+        <origin xyz="0.0 ${y_sign * 0.2001} 0.0" rpy="${y_sign * M_PI/2} ${-y_sign * M_PI/2} 0.0" />
         <geometry>
           <mesh filename="file://$(find sobit_home_description)/meshes/arm/arm_upper_flex.stl" scale="0.001 0.001 0.001" />
@@ -131,7 +127,15 @@
       <parent link="${prefix}_${position}_upper_flex_link" />
       <child link="${prefix}_${position}_elbow_link" />
-      <origin xyz="0.0 ${y_sign * 0.18413635} 0.0" rpy="0.0 0.0 0.0" />
-      <axis xyz="0.0 0.0 -1.0" />
-      <limit lower="0" upper="${M_PI/2}" effort="10.6" velocity="3.14" />
+      <origin xyz="0.0 ${y_sign * 0.19765} 0.0" rpy="0.0 0.0 0.0" />
+      <axis xyz="0.0 0.0 1.0" />
+        <xacro:if value="${y_sign == -1.0}">
+          <xacro:property name="elbow_lower_limit" value="0.0" />
+          <xacro:property name="elbow_upper_limit" value="${140*M_PI/180}" />
+        </xacro:if>
+        <xacro:if value="${y_sign == 1.0}">
+          <xacro:property name="elbow_lower_limit" value="${-140*M_PI/180}" />
+          <xacro:property name="elbow_upper_limit" value="0.0" />
+        </xacro:if>
+        <limit lower="${elbow_lower_limit}" upper="${elbow_upper_limit}" effort="${10.6 * effort_ratio}" velocity="3.14" />
     </joint>
     <link name="${prefix}_${position}_elbow_link" >
@@ -161,6 +165,6 @@
       <child link="${prefix}_${position}_wrist_tilt_link" />
       <origin xyz="0.0 ${y_sign * 0.5} 0.0" rpy="0.0 0.0 0.0" />
-      <axis xyz="0.0 0.0 -1.0 " />
-      <limit lower="${-M_PI/2}" upper="${M_PI/2}" effort="4.1" velocity="4.81" />
+      <axis xyz="0.0 0.0 1.0" />
+      <limit lower="${-y_sign * M_PI/2}" upper="${y_sign * M_PI/2}" effort="${4.1 * effort_ratio}" velocity="4.81" />
     </joint>
     <link name="${prefix}_${position}_wrist_tilt_link" >
@@ -190,6 +194,6 @@
       <child link="${prefix}_${position}_wrist_roll_link" />
       <origin xyz="0.0 ${y_sign * 0.06648202} 0.0" rpy="0.0 0.0 0.0" />
-      <axis xyz="0.0 1.0 0.0 " />
-      <limit lower="${-M_PI/2}" upper="${M_PI/2}" effort="${10.6*2}" velocity="11.031179004" />
+      <axis xyz="0.0 ${y_sign} 0.0" />
+      <limit lower="${-y_sign * M_PI/2}" upper="${y_sign * M_PI/2}" effort="${10.6 * effort_ratio}" velocity="11.031179004" />
     </joint>
     <link name="${prefix}_${position}_wrist_roll_link" >

Commit message: [UPD] adjust joint limit angles

File: sobit_home_description/urdf/arm/arm.urdf.xacro (robot description, xacro)
@@ -42,5 +42,5 @@
       <origin xyz="0.0 ${y_sign * 0.126} 0.0" rpy="0.0 0.0 0.0" />
       <axis xyz="0.0 ${y_sign} 0.0" />
-      <limit lower="${-M_PI/2}" upper="${M_PI/2}" effort="${44.7 * effort_ratio}" velocity="3.0" />
+      <limit lower="${-M_PI}" upper="${M_PI}" effort="${44.7 * effort_ratio}" velocity="3.0" />
     </joint>
     <link name="${prefix}_${position}_shoulder_tilt_link" >
@@ -100,5 +100,5 @@
       <origin xyz="0.0 ${y_sign * 0.2} 0.0" rpy="0.0 0.0 0.0" />
       <axis xyz="0.0 ${y_sign} 0.0" />
-      <limit lower="${-y_sign * M_PI/2}" upper="${y_sign * M_PI/2}" effort="${4.1 * effort_ratio}" velocity="4.81" />
+      <limit lower="${-y_sign * M_PI}" upper="${y_sign * M_PI}" effort="${4.1 * effort_ratio}" velocity="4.81" />
     </joint>
     <link name="${prefix}_${position}_upper_flex_link" >
@@ -195,5 +195,5 @@
       <origin xyz="0.0 ${y_sign * 0.06648202} 0.0" rpy="0.0 0.0 0.0" />
       <axis xyz="0.0 ${y_sign} 0.0" />
-      <limit lower="${-y_sign * M_PI/2}" upper="${y_sign * M_PI/2}" effort="${10.6 * effort_ratio}" velocity="11.031179004" />
+      <limit lower="${-y_sign * M_PI}" upper="${y_sign * M_PI}" effort="${10.6 * effort_ratio}" velocity="11.031179004" />
     </joint>
     <link name="${prefix}_${position}_wrist_roll_link" >

File: sobit_home_description/urdf/controllers.urdf.xacro (robot description, xacro)
@@ -300,6 +300,6 @@
       </xacro:unless>
       <command_interface name="position">
-        <param name="min">-${M_PI/2}</param>
-        <param name="max">${M_PI/2}</param>
+        <param name="min">-${M_PI}</param>
+        <param name="max">${M_PI}</param>
       </command_interface>
       <!-- <command_interface name="velocity"/> -->
@@ -320,6 +320,6 @@
       </xacro:unless>
       <command_interface name="position">
-        <param name="min">-${M_PI/2}</param>
-        <param name="max">${M_PI/2}</param>
+        <param name="min">-${M_PI}</param>
+        <param name="max">${M_PI}</param>
       </command_interface>
       <!-- <command_interface name="velocity"/> -->
@@ -358,4 +358,40 @@
       </xacro:unless>
       <command_interface name="position">
+        <param name="min">-${M_PI}</param>
+        <param name="max">${M_PI}</param>
+      </command_interface>
+      <!-- <command_interface name="velocity"/> -->
+      <state_interface name="position">
+        <param name="initial_value">0.0</param>
+      </state_interface>
+      <state_interface name="velocity"/>
+      <state_interface name="effort"/>
+    </joint>
+    <joint name="${prefix}_elbow_joint">
+      <xacro:unless value="${$(arg enable_gz)}">
+        <param name="id">34</param>
+        <param name="control_mode">0</param>
+        <param name="interface">rs</param>
+        <param name="Return_Delay_Time">0</param>
+      </xacro:unless>
+      <command_interface name="position">
+        <param name="min">${-140*M_PI/180}</param>
+        <param name="max">0</param>
+      </command_interface>
+      <!-- <command_interface name="velocity"/> -->
+      <state_interface name="position">
+        <param name="initial_value">-1.33</param>
+      </state_interface>
+      <state_interface name="velocity"/>
+      <state_interface name="effort"/>
+    </joint>
+    <joint name="${prefix}_wrist_tilt_joint">
+      <xacro:unless value="${$(arg enable_gz)}">
+        <param name="id">35</param>
+        <param name="control_mode">0</param>
+        <param name="interface">rs</param>
+        <param name="Return_Delay_Time">0</param>
+      </xacro:unless>
+      <command_interface name="position">
         <param name="min">-${M_PI/2}</param>
         <param name="max">${M_PI/2}</param>
@@ -368,40 +404,4 @@
       <state_interface name="effort"/>
     </joint>
-    <joint name="${prefix}_elbow_joint">
-      <xacro:unless value="${$(arg enable_gz)}">
-        <param name="id">34</param>
-        <param name="control_mode">0</param>
-        <param name="interface">rs</param>
-        <param name="Return_Delay_Time">0</param>
-      </xacro:unless>
-      <command_interface name="position">
-        <param name="min">-${M_PI/2}</param>
-        <param name="max">0</param>
-      </command_interface>
-      <!-- <command_interface name="velocity"/> -->
-      <state_interface name="position">
-        <param name="initial_value">-1.33</param>
-      </state_interface>
-      <state_interface name="velocity"/>
-      <state_interface name="effort"/>
-    </joint>
-    <joint name="${prefix}_wrist_tilt_joint">
-      <xacro:unless value="${$(arg enable_gz)}">
-        <param name="id">35</param>
-        <param name="control_mode">0</param>
-        <param name="interface">rs</param>
-        <param name="Return_Delay_Time">0</param>
-      </xacro:unless>
-      <command_interface name="position">
-        <param name="min">-${M_PI/2}</param>
-        <param name="max">${M_PI/2}</param>
-      </command_interface>
-      <!-- <command_interface name="velocity"/> -->
-      <state_interface name="position">
-        <param name="initial_value">0.0</param>
-      </state_interface>
-      <state_interface name="velocity"/>
-      <state_interface name="effort"/>
-    </joint>
     <joint name="${prefix}_wrist_roll_joint">
       <xacro:unless value="${$(arg enable_gz)}">
@@ -412,6 +412,6 @@
       </xacro:unless>
       <command_interface name="position">
-        <param name="min">-${M_PI/2}</param>
-        <param name="max">${M_PI/2}</param>
+        <param name="min">-${M_PI}</param>
+        <param name="max">${M_PI}</param>
       </command_interface>
       <!-- <command_interface name="velocity"/> -->
@@ -450,4 +450,40 @@
       </xacro:unless>
       <command_interface name="position">
+        <param name="min">-${M_PI}</param>
+        <param name="max">${M_PI}</param>
+      </command_interface>
+      <!-- <command_interface name="velocity"/> -->
+      <state_interface name="position">
+        <param name="initial_value">0.0</param>
+      </state_interface>
+      <state_interface name="velocity"/>
+      <state_interface name="effort"/>
+    </joint>
+    <joint name="${prefix}_elbow_joint">
+      <xacro:unless value="${$(arg enable_gz)}">
+        <param name="id">44</param>
+        <param name="control_mode">0</param>
+        <param name="interface">rs</param>
+        <param name="Return_Delay_Time">0</param>
+      </xacro:unless>
+      <command_interface name="position">
+        <param name="min">0.0</param>
+        <param name="max">${140*M_PI/180}</param>
+      </command_interface>
+      <!-- <command_interface name="velocity"/> -->
+      <state_interface name="position">
+        <param name="initial_value">1.33</param>
+      </state_interface>
+      <state_interface name="velocity"/>
+      <state_interface name="effort"/>
+    </joint>
+    <joint name="${prefix}_wrist_tilt_joint">
+      <xacro:unless value="${$(arg enable_gz)}">
+        <param name="id">45</param>
+        <param name="control_mode">0</param>
+        <param name="interface">rs</param>
+        <param name="Return_Delay_Time">0</param>
+      </xacro:unless>
+      <command_interface name="position">
         <param name="min">-${M_PI/2}</param>
         <param name="max">${M_PI/2}</param>
@@ -460,40 +496,4 @@
       <state_interface name="effort"/>
     </joint>
-    <joint name="${prefix}_elbow_joint">
-      <xacro:unless value="${$(arg enable_gz)}">
-        <param name="id">44</param>
-        <param name="control_mode">0</param>
-        <param name="interface">rs</param>
-        <param name="Return_Delay_Time">0</param>
-      </xacro:unless>
-      <command_interface name="position">
-        <param name="min">0</param>
-        <param name="max">${M_PI/2}</param>
-      </command_interface>
-      <!-- <command_interface name="velocity"/> -->
-      <state_interface name="position">
-        <param name="initial_value">1.33</param>
-      </state_interface>
-      <state_interface name="velocity"/>
-      <state_interface name="effort"/>
-    </joint>
-    <joint name="${prefix}_wrist_tilt_joint">
-      <xacro:unless value="${$(arg enable_gz)}">
-        <param name="id">45</param>
-        <param name="control_mode">0</param>
-        <param name="interface">rs</param>
-        <param name="Return_Delay_Time">0</param>
-      </xacro:unless>
-      <command_interface name="position">
-        <param name="min">-${M_PI/2}</param>
-        <param name="max">${M_PI/2}</param>
-      </command_interface>
-      <!-- <command_interface name="velocity"/> -->
-      <state_interface name="position">
-        <param name="initial_value">0.0</param>
-      </state_interface>
-      <state_interface name="velocity"/>
-      <state_interface name="effort"/>
-    </joint>
     <joint name="${prefix}_wrist_roll_joint">
       <xacro:unless value="${$(arg enable_gz)}">
@@ -504,6 +504,6 @@
       </xacro:unless>
       <command_interface name="position">
-        <param name="min">-1.570796327</param>
-        <param name="max">1.570796327</param>
+        <param name="min">-${M_PI}</param>
+        <param name="max">${M_PI}</param>
       </command_interface>
       <!-- <command_interface name="velocity"/> -->
@@ -525,5 +525,5 @@
       </xacro:unless>
       <command_interface name="position">
-        <param name="min">-${M_PI/2}</param>
+        <param name="min">${-M_PI/2}</param>
         <param name="max">${M_PI/2}</param>
       </command_interface>
@@ -553,5 +553,5 @@
       </xacro:unless>
       <command_interface name="position">
-        <param name="min">-${M_PI/2}</param>
+        <param name="min">${-M_PI/2}</param>
         <param name="max">${M_PI/2}</param>
       </command_interface>
@@ -572,6 +572,6 @@
       </xacro:unless>
       <command_interface name="position">
-        <param name="min">-${M_PI/2}</param>
-        <param name="max">${M_PI/2}</param>
+        <param name="min">${-M_PI/2}</param>
+        <param name="max">${M_PI/6}</param>
       </command_interface>
       <!-- <command_interface name="velocity"/> -->
@@ -591,6 +591,6 @@
       </xacro:unless>
       <command_interface name="position">
-        <param name="min">-${M_PI/2}</param>
-        <param name="max">${M_PI/2}</param>
+        <param name="min">${-M_PI/2}</param>
+        <param name="max">${M_PI/6}</param>
       </command_interface>
       <!-- <command_interface name="velocity"/> -->
@@ -610,5 +610,5 @@
       </xacro:unless>
       <command_interface name="position">
-        <param name="min">-${M_PI/2}</param>
+        <param name="min">${-M_PI/6}</param>
         <param name="max">${M_PI/2}</param>
       </command_interface>
@@ -629,6 +629,6 @@
       </xacro:unless>
       <command_interface name="position">
-        <param name="min">-${M_PI/2}</param>
-        <param name="max">${M_PI/2}</param>
+        <param name="min">${-M_PI/2}</param>
+        <param name="max">${M_PI/6}</param>
       </command_interface>
       <!-- <command_interface name="velocity"/> -->
@@ -648,5 +648,5 @@
       </xacro:unless>
       <command_interface name="position">
-        <param name="min">-${M_PI/2}</param>
+        <param name="min">${-M_PI/6}</param>
         <param name="max">${M_PI/2}</param>
       </command_interface>
@@ -716,6 +716,6 @@
       </xacro:unless>
       <command_interface name="position">
-        <param name="min">-2.0</param>
-        <param name="max">0.5</param>
+        <param name="min">${-M_PI/2}</param>
+        <param name="max">${M_PI/6}</param>
       </command_interface>
       <!-- <command_interface name="velocity"/> -->
@@ -735,5 +735,5 @@
       </xacro:unless>
       <command_interface name="position">
-        <param name="min">-0.9</param>
+        <param name="min">${-M_PI/6}</param>
         <param name="max">${M_PI/2}</param>
       </command_interface>
@@ -754,6 +754,6 @@
       </xacro:unless>
       <command_interface name="position">
-        <param name="min">-2.0</param>
-        <param name="max">0.5</param>
+        <param name="min">${-M_PI/2}</param>
+        <param name="max">${M_PI/6}</param>
       </command_interface>
       <!-- <command_interface name="velocity"/> -->
@@ -773,6 +773,6 @@
       </xacro:unless>
       <command_interface name="position">
-        <param name="min">-${M_PI/2}</param>
-        <param name="max">0.5</param>
+        <param name="min">${-M_PI/2}</param>
+        <param name="max">${M_PI/6}</param>
       </command_interface>
       <!-- <command_interface name="velocity"/> -->
@@ -792,6 +792,6 @@
       </xacro:unless>
       <command_interface name="position">
-        <param name="min">-0.5</param>
-        <param name="max">2.0</param>
+        <param name="min">${-M_PI/6}</param>
+        <param name="max">${M_PI/2}</param>
       </command_interface>
       <!-- <command_interface name="velocity"/> -->

File: sobit_home_description/urdf/hand/hand.urdf.xacro (robot description, xacro)
@@ -251,5 +251,10 @@
       <origin xyz="0.0 ${y_sign * 0.050} 0.0" rpy="0.0 0.0 0.0" />
       <axis xyz="0.0 0.0 1.0 " />
-      <limit lower="${-M_PI/6}" upper="${M_PI/2}" effort="0.52" velocity="11.031179004" />
+      <xacro:if value="${position == 'right'}">
+        <limit lower="${-M_PI/2}" upper="${M_PI/6}" effort="0.52" velocity="11.031" />
+      </xacro:if>
+      <xacro:if value="${position == 'left'}">
+        <limit lower="${-M_PI/6}" upper="${M_PI/2}" effort="0.52" velocity="11.031" />
+      </xacro:if>
     </joint>
     <link name="${prefix_hand}_${position}_${prefix_finger}_c_ip_link" >
@@ -278,5 +283,5 @@
     <!-- Joint: End Effector -->
     <joint name="${prefix_hand}_${position}_end_effector_joint" type="fixed">
-      <origin xyz="0.0 ${y_sign*0.13} 0.0" rpy="${y_sign * M_PI/2} 0.0 ${y_sign * M_PI/2}"/>
+      <origin xyz="0.0 ${y_sign*0.13} 0.0" rpy="${M_PI} 0.0 ${y_sign * M_PI/2}"/>
       <parent link="${parent}"/>
       <child link="${prefix_hand}_${position}_end_effector_link"/>

Commit message: [FIX] wrist roll mesh orientation

File: sobit_home_description/urdf/arm/arm.urdf.xacro (robot description, xacro)
@@ -199,5 +199,5 @@
     <link name="${prefix}_${position}_wrist_roll_link" >
       <visual>
-        <origin xyz="0.0 0.0 0.0" rpy="0.0 0.0 0.0" />
+        <origin xyz="0.0 0.0 0.0" rpy="0.0 ${y_sign * M_PI/2} ${y_sign * M_PI/2}" />
         <geometry>
           <mesh filename="file://$(find sobit_home_description)/meshes/arm/arm_wrist_roll.stl" scale="0.001 0.001 0.001" />
@@ -205,19 +205,17 @@
         <material name="grey" />
       </visual>
-      <collision>
+      <!-- <collision>
         <origin xyz="0.00852612 ${y_sign * 0.07450 / 2} 0.0" rpy="0.0 ${y_sign * M_PI/2} ${y_sign * M_PI/2}" />
         <geometry>
-          <!-- <box size="0.108064 0.08255 0.0645" /> -->
           <box size="0.108 0.0826 0.0645" />
         </geometry>
       </collision>
       <inertial>
-        <origin xyz="0.0 0.0 0.0" rpy="0.0 0.0 0.0" />
-        <!-- <mass value="0.0160103055903" /> -->
+        <origin xyz="0.0 0.0 0.0" rpy="0.0 ${y_sign * M_PI/2} ${y_sign * M_PI/2}" />
         <mass value="0.016" />
         <inertia ixx="${1/12*0.016*(0.0645**2+0.0826**2)}" ixy="0.0" ixz="0.0"
                  iyy="${1/12*0.016*(0.108**2 +0.0645**2)}" iyz="0.0"
                  izz="${1/12*0.016*(0.108**2+0.0826**2)}" />
-      </inertial>
+      </inertial> -->
     </link>
     <xacro:arm_transmission prefix="${prefix}" position="${position}" />

Commit message: [FIX] adjust joint lower and upper limits in URDF

File: sobit_home_description/urdf/arm/arm.urdf.xacro (robot description, xacro)
@@ -100,5 +100,5 @@
       <origin xyz="0.0 ${y_sign * 0.2} 0.0" rpy="0.0 0.0 0.0" />
       <axis xyz="0.0 ${y_sign} 0.0" />
-      <limit lower="${-y_sign * M_PI}" upper="${y_sign * M_PI}" effort="${4.1 * effort_ratio}" velocity="4.81" />
+      <limit lower="${-M_PI}" upper="${M_PI}" effort="${4.1 * effort_ratio}" velocity="4.81" />
     </joint>
     <link name="${prefix}_${position}_upper_flex_link" >
@@ -166,5 +166,5 @@
       <origin xyz="0.0 ${y_sign * 0.5} 0.0" rpy="0.0 0.0 0.0" />
       <axis xyz="0.0 0.0 1.0" />
-      <limit lower="${-y_sign * M_PI/2}" upper="${y_sign * M_PI/2}" effort="${4.1 * effort_ratio}" velocity="4.81" />
+      <limit lower="${-M_PI/2}" upper="${M_PI/2}" effort="${4.1 * effort_ratio}" velocity="4.81" />
     </joint>
     <link name="${prefix}_${position}_wrist_tilt_link" >
@@ -195,5 +195,5 @@
       <origin xyz="0.0 ${y_sign * 0.06648202} 0.0" rpy="0.0 0.0 0.0" />
       <axis xyz="0.0 ${y_sign} 0.0" />
-      <limit lower="${-y_sign * M_PI}" upper="${y_sign * M_PI}" effort="${10.6 * effort_ratio}" velocity="11.031179004" />
+      <limit lower="${-M_PI}" upper="${M_PI}" effort="${10.6 * effort_ratio}" velocity="11.031179004" />
     </joint>
     <link name="${prefix}_${position}_wrist_roll_link" >
