Commit message: [UPD] Modified urdf settings.

File: sobit_home_description/urdf/arm/arm.urdf.xacro (robot description, xacro)
@@ -71,5 +71,5 @@
       <parent link="${prefix}_${position}_shoulder_tilt_link" />
       <child link="${prefix}_${position}_upper_roll_link" />
-      <origin xyz="${y_sign * 0.0510} ${y_sign * 0.100} 0.0" rpy="0.0 0.0 0.0" />
+      <origin xyz="${-y_sign * 0.0510} ${y_sign * 0.100} 0.0" rpy="0.0 0.0 0.0" />
       <axis xyz="1.0 0.0 0.0" />
       <limit lower="${-M_PI/2}" upper="${M_PI/2}" effort="${10.6 * effort_ratio}" velocity="3.14" />
@@ -78,8 +78,8 @@
       <visual>
         <xacro:if value="${position == 'right'}">
-          <origin xyz="${-y_sign * 0.0510} 0.0 0.0" rpy="${M_PI} 0.0 ${y_sign * M_PI/2}" />
+          <origin xyz="${y_sign * 0.0510} 0.0 0.0" rpy="${M_PI} 0.0 ${y_sign * M_PI/2}" />
         </xacro:if>
         <xacro:unless value="${position == 'right'}">
-          <origin xyz="${-y_sign * 0.0510} 0.0 0.0" rpy="0.0 0.0 ${y_sign * M_PI/2}" />
+          <origin xyz="${y_sign * 0.0510} 0.0 0.0" rpy="0.0 0.0 ${y_sign * M_PI/2}" />
         </xacro:unless>
         <geometry>
@@ -107,5 +107,5 @@
       <parent link="${prefix}_${position}_shoulder_tilt_link" />
       <child link="${prefix}_${position}_upper_roll_sub_link" />
-      <origin xyz="${-y_sign * 0.0510} ${y_sign * 0.100} 0.0" rpy="0.0 0.0 0.0" />
+      <origin xyz="${y_sign * 0.0510} ${y_sign * 0.100} 0.0" rpy="0.0 0.0 0.0" />
       <axis xyz="-1.0 0.0 0.0" />
       <limit lower="${-M_PI/2}" upper="${M_PI/2}" effort="${10.6 * effort_ratio}" velocity="3.14" />
@@ -124,5 +124,5 @@
       <parent link="${prefix}_${position}_upper_roll_link" />
       <child link="${prefix}_${position}_upper_flex_link" />
-      <origin xyz="${-y_sign * 0.0510} ${y_sign * 0.1335} 0.0" rpy="0.0 0.0 0.0" />
+      <origin xyz="${y_sign * 0.0510} ${y_sign * 0.1335} 0.0" rpy="0.0 0.0 0.0" />
       <axis xyz="0.0 ${y_sign} 0.0" />
       <limit lower="${-M_PI/2}" upper="${M_PI/2}" effort="${10.6 * effort_ratio}" velocity="4.81" />
@@ -155,5 +155,5 @@
       <parent link="${prefix}_${position}_upper_roll_link" />
       <child link="${prefix}_${position}_upper_flex_sub_link" />
-      <origin xyz="${-y_sign * 0.0510} ${y_sign * (0.100+0.0335+0.0510)} 0.0" rpy="0.0 0.0 0.0" />
+      <origin xyz="${y_sign * 0.0510} ${y_sign * (0.100+0.0335+0.0510)} 0.0" rpy="0.0 0.0 0.0" />
       <axis xyz="0.0 ${y_sign} 0.0" />
       <limit lower="${-M_PI/2}" upper="${M_PI/2}" effort="${10.6 * effort_ratio}" velocity="4.81" />
@@ -173,5 +173,5 @@
       <child link="${prefix}_${position}_lower_top_link" />
       <axis xyz="0.0 0.0 1.0" />
-      <origin xyz="0.05495 ${y_sign * 0.26365} -0.0510" rpy="0.0 0.0 0.0" />
+      <origin xyz="0.05495 ${y_sign * 0.26365} ${y_sign * 0.0510}" rpy="0.0 0.0 0.0" />
         <limit lower="${-M_PI/2}" upper="${2/3 * M_PI}" effort="${10.6 * effort_ratio}" velocity="3.14" />
     </joint>
@@ -179,8 +179,8 @@
       <visual>
         <xacro:if value="${position == 'right'}">
-          <origin xyz="0.0 0.0 0.0510" rpy="${M_PI} 0.0 ${-M_PI/2}" />
+          <origin xyz="0.0 0.0 ${y_sign * -0.0510}" rpy="${M_PI} 0.0 ${-M_PI/2}" />
         </xacro:if>
         <xacro:unless value="${position == 'right'}">
-          <origin xyz="0.0 0.0 0.0510" rpy="0.0 0.0 ${M_PI/2}" />
+          <origin xyz="0.0 0.0 ${-y_sign * 0.0510}" rpy="0.0 0.0 ${M_PI/2}" />
         </xacro:unless>
         <geometry>
@@ -208,5 +208,5 @@
       <parent link="${prefix}_${position}_upper_flex_link" />
       <child link="${prefix}_${position}_lower_top_sub_link" />
-      <origin xyz="0.05495 ${y_sign * 0.26365} 0.0510" rpy="0.0 0.0 0.0" />
+      <origin xyz="0.05495 ${y_sign * 0.26365} ${-y_sign * 0.0510}" rpy="0.0 0.0 0.0" />
       <axis xyz="0.0 0.0 -1.0" />
       <limit lower="${-M_PI/2}" upper="${M_PI/2}" effort="${10.6 * effort_ratio}" velocity="3.14" />
@@ -225,5 +225,5 @@
       <parent link="${prefix}_${position}_lower_top_link" />
       <child link="${prefix}_${position}_lower_bottom_link" />
-      <origin xyz="0.0 ${y_sign * 0.107} 0.0510" rpy="0.0 0.0 0.0" />
+      <origin xyz="0.0 ${y_sign * 0.107} ${-y_sign * 0.0510}" rpy="0.0 0.0 0.0" />
       <axis xyz="0.0 ${y_sign* 1.0} 0.0" />
       <limit lower="${-M_PI/2}" upper="${M_PI/2}" effort="${4.1 * effort_ratio}" velocity="4.81" />

File: sobit_home_description/urdf/controllers.urdf.xacro (robot description, xacro)
@@ -464,5 +464,5 @@
       <xacro:if value="${$(arg enable_gz)}">
         <command_interface name="position">
-        <param name="min">${-140*M_PI/180}</param>
+        <param name="min">${2/3*M_PI}</param>
         <param name="max">0</param>
         </command_interface>

File: sobit_home_description/urdf/hand/hand.urdf.xacro (robot description, xacro)
@@ -18,5 +18,6 @@
       <parent link="${parent}" />
       <child link="${prefix_hand}_${position}_cmc_link" />
-      <origin xyz="0.0 ${y_sign * 0.025375} 0.0" rpy="0.0 ${M_PI/2} 0.0" />
+      <origin xyz="0.0 ${y_sign * 0.025375} 0.0" rpy="0.0 0.0 0.0" />
+      <!-- <origin xyz="0.0 ${y_sign * 0.025375} 0.0" rpy="0.0 ${M_PI/2} 0.0" /> -->
     </joint>
     <link name="${prefix_hand}_${position}_cmc_link" >

Commit message: [FIX] Fixed mimic settings and command_interface settings.

File: sobit_home_description/urdf/arm/arm.urdf.xacro (robot description, xacro)
@@ -92,5 +92,4 @@
         <geometry>
           <cylinder length="0.1285" radius="${0.142/2}" />
-          <!-- <cylinder length="0.1285" radius="${0.142/2}" /> -->
         </geometry>
       </collision>

File: sobit_home_description/urdf/controllers.urdf.xacro (robot description, xacro)
@@ -382,5 +382,5 @@
       <!-- <command_interface name="velocity"/> -->
       <state_interface name="position">
-        <param name="initial_value">0.0</param>
+        <param name="initial_value">1.5</param>
       </state_interface>
       <state_interface name="velocity"/>
@@ -388,10 +388,10 @@
     </joint>
     <joint name="${prefix}_upper_roll_sub_joint">
-      <xacro:if value="${$(arg enable_gz)}">
+      <!-- <xacro:if value="${$(arg enable_gz)}">
         <command_interface name="position">
           <param name="min">-${M_PI/2}</param>
           <param name="max">${M_PI/2}</param>
         </command_interface>
-      </xacro:if>
+      </xacro:if> -->
       <xacro:unless value="${$(arg enable_gz)}">
         <param name="id">33</param>
@@ -401,5 +401,5 @@
       </xacro:unless>
       <state_interface name="position">
-        <param name="initial_value">0.0</param>
+        <param name="initial_value">-1.5</param>
       </state_interface>
       <state_interface name="velocity"/>
@@ -425,10 +425,10 @@
     </joint>
     <joint name="${prefix}_upper_flex_sub_joint">
-      <xacro:if value="${$(arg enable_gz)}">
+      <!-- <xacro:if value="${$(arg enable_gz)}">
         <command_interface name="position">
           <param name="min">-${M_PI/2}</param>
           <param name="max">${M_PI/2}</param>
         </command_interface>
-      </xacro:if>
+      </xacro:if> -->
       <xacro:unless value="${$(arg enable_gz)}">
         <param name="id">35</param>
@@ -456,5 +456,5 @@
       <!-- <command_interface name="velocity"/> -->
       <state_interface name="position">
-        <param name="initial_value">1.571</param>
+        <param name="initial_value">-1.571</param>
       </state_interface>
       <state_interface name="velocity"/>
@@ -462,10 +462,10 @@
     </joint>
     <joint name="${prefix}_elbow_sub_joint">
-      <xacro:if value="${$(arg enable_gz)}">
+      <!-- <xacro:if value="${$(arg enable_gz)}">
         <command_interface name="position">
         <param name="min">0</param>
         <param name="max">${8/9 * M_PI}</param>
         </command_interface>
-      </xacro:if>
+      </xacro:if> -->
       <xacro:unless value="${$(arg enable_gz)}">
         <param name="id">37</param>
@@ -475,5 +475,5 @@
       </xacro:unless>
       <state_interface name="position">
-        <param name="initial_value">-1.571</param>
+        <param name="initial_value">1.571</param>
       </state_interface>
       <state_interface name="velocity"/>
@@ -556,10 +556,10 @@
     </joint>
     <joint name="${prefix}_upper_roll_sub_joint">
-      <xacro:if value="${$(arg enable_gz)}">
+      <!-- <xacro:if value="${$(arg enable_gz)}">
         <command_interface name="position">
           <param name="min">-${M_PI/2}</param>
           <param name="max">${M_PI/2}</param>
         </command_interface>
-      </xacro:if>
+      </xacro:if> -->
       <xacro:unless value="${$(arg enable_gz)}">
         <param name="id">43</param>
@@ -593,10 +593,10 @@
     </joint>
     <joint name="${prefix}_upper_flex_sub_joint">
-      <xacro:if value="${$(arg enable_gz)}">
+      <!-- <xacro:if value="${$(arg enable_gz)}">
         <command_interface name="position">
           <param name="min">-${M_PI/2}</param>
           <param name="max">${M_PI/2}</param>
         </command_interface>
-      </xacro:if>
+      </xacro:if> -->
       <xacro:unless value="${$(arg enable_gz)}">
         <param name="id">45</param>
@@ -630,10 +630,10 @@
     </joint>
     <joint name="${prefix}_elbow_sub_joint">
-      <xacro:if value="${$(arg enable_gz)}">
+      <!-- <xacro:if value="${$(arg enable_gz)}">
         <command_interface name="position">
         <param name="min">-${8/9 * M_PI}</param>
         <param name="max">0</param>
         </command_interface>
-      </xacro:if>
+      </xacro:if> -->
       <xacro:unless value="${$(arg enable_gz)}">
         <param name="id">47</param>

Commit message: [UPD] Remove old mesh file and arrange TF origin of some joints.

File: sobit_home_description/urdf/arm/arm.urdf.xacro (robot description, xacro)
@@ -71,5 +71,5 @@
       <parent link="${prefix}_${position}_shoulder_tilt_link" />
       <child link="${prefix}_${position}_upper_roll_link" />
-        <origin xyz="${-y_sign * 0.0510} ${y_sign * 0.100} 0.0" rpy="0.0 0.0 0.0" />
+        <origin xyz="0.0510 ${y_sign * 0.100} 0.0" rpy="0.0 0.0 0.0" />
       <axis xyz="-1.0 0.0 0.0" />
       <limit lower="${-M_PI/2}" upper="${M_PI/2}" effort="${10.6 * effort_ratio}" velocity="3.14" />
@@ -81,5 +81,5 @@
         </xacro:if>
         <xacro:unless value="${position == 'right'}">
-          <origin xyz="${y_sign * 0.0510} 0.0 0.0" rpy="0.0 0.0 ${y_sign * M_PI/2}" />
+          <origin xyz="${-y_sign * 0.0510} 0.0 0.0" rpy="0.0 0.0 ${y_sign * M_PI/2}" />
         </xacro:unless>
         <geometry>
@@ -107,5 +107,5 @@
       <parent link="${prefix}_${position}_shoulder_tilt_link" />
       <child link="${prefix}_${position}_upper_roll_sub_link" />
-      <origin xyz="${y_sign * 0.0510} ${y_sign * 0.100} 0.0" rpy="0.0 0.0 0.0" />
+      <origin xyz="-0.0510 ${y_sign * 0.100} 0.0" rpy="0.0 0.0 0.0" />
       <axis xyz="1.0 0.0 0.0" />
       <limit lower="${-M_PI/2}" upper="${M_PI/2}" effort="${10.6 * effort_ratio}" velocity="3.14" />
@@ -124,5 +124,5 @@
       <parent link="${prefix}_${position}_upper_roll_link" />
       <child link="${prefix}_${position}_upper_flex_link" />
-      <origin xyz="${y_sign * 0.0510} ${y_sign * 0.1135} 0.0" rpy="0.0 0.0 0.0" />
+      <origin xyz="-0.0510 ${y_sign * 0.1135} 0.0" rpy="0.0 0.0 0.0" />
       <axis xyz="0.0 ${y_sign} 0.0" />
       <limit lower="${-M_PI/2}" upper="${M_PI/2}" effort="${10.6 * effort_ratio}" velocity="4.81" />
@@ -160,5 +160,5 @@
       <parent link="${prefix}_${position}_upper_roll_link" />
       <child link="${prefix}_${position}_upper_flex_sub_link" />
-      <origin xyz="${y_sign * 0.0510} ${y_sign * (0.1135+0.0510)} 0.0" rpy="0.0 0.0 0.0" />
+      <origin xyz="-0.0510 ${y_sign * (0.1135+0.0510)} 0.0" rpy="0.0 0.0 0.0" />
       <axis xyz="0.0 ${y_sign} 0.0" />
       <limit lower="${-M_PI/2}" upper="${M_PI/2}" effort="${10.6 * effort_ratio}" velocity="4.81" />
@@ -178,5 +178,5 @@
       <child link="${prefix}_${position}_elbow_link" />
       <axis xyz="0.0 0.0 1.0" />
-      <origin xyz="0.05495 ${y_sign * (0.28865-0.00765)} ${y_sign * 0.0510}" rpy="0.0 0.0 0.0" />
+      <origin xyz="0.05495 ${y_sign * (0.28865-0.00765)} 0.0510" rpy="0.0 0.0 0.0" />
       <xacro:if value="${position == 'right'}">
         <limit lower="0.0" upper="${8/9 * M_PI}" effort="${10.6 * effort_ratio}" velocity="3.14" />
@@ -188,10 +188,11 @@
     <link name="${prefix}_${position}_elbow_link" >
       <visual>
-        <xacro:if value="${position == 'right'}">
-          <origin xyz="0.0 0.0 ${-y_sign * 0.0510}" rpy="${M_PI} 0.0 ${-M_PI/2}" />
+        <!-- <xacro:if value="${position == 'right'}">
+          <origin xyz="0.0 0.0 0.0510" rpy="${M_PI} 0.0 ${-M_PI/2}" />
         </xacro:if>
         <xacro:unless value="${position == 'right'}">
-          <origin xyz="0.0 0.0 ${-y_sign * 0.0510}" rpy="0.0 0.0 ${M_PI/2}" />
-        </xacro:unless>
+          <origin xyz="0.0 0.0 -0.0510" rpy="0.0 0.0 ${M_PI/2}" />
+        </xacro:unless> -->
+        <origin xyz="0.0 0.0 -0.0510" rpy="0.0 0.0 ${y_sign * M_PI/2}" />
         <geometry>
           <mesh filename="file://$(find sobit_home_description)/meshes/arm/arm_elbow.stl" scale="0.001 0.001 0.001" />
@@ -213,10 +214,10 @@
       </inertial>
     </link>
-<!-- Lower top sub joint -->
+<!-- Elbow sub joint -->
     <joint name="${prefix}_${position}_elbow_sub_joint" type="revolute" >
       <mimic joint="${prefix}_${position}_elbow_joint" multiplier="-1" offset="0"/>
       <parent link="${prefix}_${position}_upper_flex_link" />
       <child link="${prefix}_${position}_elbow_sub_link" />
-      <origin xyz="0.05495 ${y_sign * (0.28865-0.00765)} ${-y_sign * 0.0510}" rpy="0.0 0.0 0.0" />
+      <origin xyz="0.05495 ${y_sign * (0.28865-0.00765)} -0.0510" rpy="0.0 0.0 0.0" />
       <axis xyz="0.0 0.0 -1.0" />
       <limit lower="${-M_PI/2}" upper="${M_PI/2}" effort="${10.6 * effort_ratio}" velocity="3.14" />
@@ -235,5 +236,5 @@
       <parent link="${prefix}_${position}_elbow_link" />
       <child link="${prefix}_${position}_lower_flex_link" />
-      <origin xyz="0.0 ${y_sign * 0.107} ${-y_sign * 0.0510}" rpy="0.0 0.0 0.0" />
+      <origin xyz="0.0 ${y_sign * 0.107} -0.0510" rpy="0.0 0.0 0.0" />
       <axis xyz="0.0 ${y_sign* 1.0} 0.0" />
       <limit lower="${-M_PI/2}" upper="${M_PI/2}" effort="${4.1 * effort_ratio}" velocity="4.81" />

Commit message: [UPD] Remove commentout.

File: sobit_home_description/urdf/arm/arm.urdf.xacro (robot description, xacro)
@@ -188,10 +188,4 @@
     <link name="${prefix}_${position}_elbow_link" >
       <visual>
-        <!-- <xacro:if value="${position == 'right'}">
-          <origin xyz="0.0 0.0 0.0510" rpy="${M_PI} 0.0 ${-M_PI/2}" />
-        </xacro:if>
-        <xacro:unless value="${position == 'right'}">
-          <origin xyz="0.0 0.0 -0.0510" rpy="0.0 0.0 ${M_PI/2}" />
-        </xacro:unless> -->
         <origin xyz="0.0 0.0 -0.0510" rpy="0.0 0.0 ${y_sign * M_PI/2}" />
         <geometry>

Commit message: [FIX] collisions

File: sobit_home_description/urdf/arm/arm.urdf.xacro (robot description, xacro)
@@ -89,5 +89,5 @@
       </visual>
       <collision>
-        <origin xyz="${y_sign * 0.0510} ${y_sign * (0.1285)/2 + y_sign * 0.05} 0.0" rpy="${y_sign * M_PI/2} 0.0 0.0" />
+        <origin xyz="-0.0510 ${y_sign * (0.1285)/2 + y_sign * 0.05} 0.0" rpy="${y_sign * M_PI/2} 0.0 0.0" />
         <geometry>
           <cylinder length="0.1285" radius="${0.142/2}" />
@@ -95,5 +95,5 @@
       </collision>
       <inertial>
-        <origin xyz="${y_sign * 0.0510} ${y_sign * (0.1285)/2 + y_sign * 0.05} 0.0" rpy="${y_sign * M_PI/2} 0.0 0.0" />
+        <origin xyz="-0.0510 ${y_sign * (0.1285)/2 + y_sign * 0.05} 0.0" rpy="${y_sign * M_PI/2} 0.0 0.0" />
         <mass value="1.31" />
         <inertia ixx="${1/12*1.31*(3*0.0875**2+0.1285**2)}" ixy="0.0" ixz="0.0"
@@ -195,5 +195,5 @@
       </visual>
       <collision>
-        <origin xyz="0.0 ${y_sign * 0.12/2 + y_sign * 0.09} ${-y_sign * 0.051}" rpy="${y_sign * M_PI/2} 0.0 0.0" />
+        <origin xyz="0.0 ${y_sign * 0.12/2 + y_sign * 0.09} -0.0510" rpy="${y_sign * M_PI/2} 0.0 0.0" />
         <geometry>
           <cylinder length="0.12" radius="${0.110/2}" />
@@ -201,5 +201,5 @@
       </collision>
       <inertial>
-        <origin xyz="0.0 ${y_sign * 0.12/2 + y_sign * 0.09} ${-y_sign * 0.051}" rpy="${y_sign * M_PI/2} 0.0 0.0" />
+        <origin xyz="0.0 ${y_sign * 0.12/2 + y_sign * 0.09} -0.0510" rpy="${y_sign * M_PI/2} 0.0 0.0" />
         <mass value="0.466"/>
         <inertia ixx="${1/12*0.466*(3*0.055**2+0.12**2)}" ixy="0.0" ixz="0.0"

Commit message: [FIX] joint effort

File: sobit_home_description/urdf/arm/arm.urdf.xacro (robot description, xacro)
@@ -292,5 +292,5 @@
       <origin xyz="0.0 ${y_sign * 0.06648202} 0.0" rpy="0.0 0.0 0.0" />
       <axis xyz="0.0 ${y_sign} 0.0" />
-      <limit lower="${-M_PI}" upper="${M_PI}" effort="${10.6 * effort_ratio}" velocity="11.031179004" />
+      <limit lower="${-M_PI}" upper="${M_PI}" effort="${4.1 * effort_ratio}" velocity="11.031179004" />
     </joint>
     <link name="${prefix}_${position}_wrist_roll_link" >

Commit message: [FIX] effort value

File: sobit_home_description/urdf/arm/arm.urdf.xacro (robot description, xacro)
@@ -126,5 +126,5 @@
       <origin xyz="-0.0510 ${y_sign * 0.1135} 0.0" rpy="0.0 0.0 0.0" />
       <axis xyz="0.0 ${y_sign} 0.0" />
-      <limit lower="${-M_PI/2}" upper="${M_PI/2}" effort="${10.6 * effort_ratio}" velocity="4.81" />
+      <limit lower="${-M_PI/2}" upper="${M_PI/2}" effort="${10.6 * effort_ratio}" velocity="3.14" />
     </joint>
     <link name="${prefix}_${position}_upper_flex_link" >
@@ -162,5 +162,5 @@
       <origin xyz="-0.0510 ${y_sign * (0.1135+0.0510)} 0.0" rpy="0.0 0.0 0.0" />
       <axis xyz="0.0 ${y_sign} 0.0" />
-      <limit lower="${-M_PI/2}" upper="${M_PI/2}" effort="${10.6 * effort_ratio}" velocity="4.81" />
+      <limit lower="${-M_PI/2}" upper="${M_PI/2}" effort="${10.6 * effort_ratio}" velocity="3.14" />
     </joint>
     <link name="${prefix}_${position}_upper_flex_sub_link" >
@@ -232,5 +232,5 @@
       <origin xyz="0.0 ${y_sign * 0.107} -0.0510" rpy="0.0 0.0 0.0" />
       <axis xyz="0.0 ${y_sign* 1.0} 0.0" />
-      <limit lower="${-M_PI/2}" upper="${M_PI/2}" effort="${4.1 * effort_ratio}" velocity="4.81" />
+      <limit lower="${-M_PI/2}" upper="${M_PI/2}" effort="${10.6 * effort_ratio}" velocity="3.14" />
     </joint>
     <link name="${prefix}_${position}_lower_flex_link" >
@@ -262,5 +262,5 @@
       <origin xyz="0.0 ${y_sign * 0.443} 0.0" rpy="0.0 0.0 0.0" />
       <axis xyz="0.0 0.0 1.0" />
-      <limit lower="${-M_PI/2}" upper="${M_PI/2}" effort="${4.1 * effort_ratio}" velocity="4.81" />
+      <limit lower="${-M_PI/2}" upper="${M_PI/2}" effort="${4.1 * effort_ratio}" velocity="4.82" />
     </joint>
     <link name="${prefix}_${position}_wrist_tilt_link" >
@@ -292,5 +292,5 @@
       <origin xyz="0.0 ${y_sign * 0.06648202} 0.0" rpy="0.0 0.0 0.0" />
       <axis xyz="0.0 ${y_sign} 0.0" />
-      <limit lower="${-M_PI}" upper="${M_PI}" effort="${4.1 * effort_ratio}" velocity="11.031179004" />
+      <limit lower="${-M_PI}" upper="${M_PI}" effort="${4.1 * effort_ratio}" velocity="4.82" />
     </joint>
     <link name="${prefix}_${position}_wrist_roll_link" >
