Commit message: [UPD] visual color

File: sobit_home_description/urdf/arm/arm.urdf.xacro (robot description, xacro)
@@ -21,5 +21,5 @@
           <mesh filename="file://$(find sobit_home_description)/meshes/arm/arm_scapula.stl" scale="0.001 0.001 0.001" />
         </geometry>
-        <material name="grey" />
+        <material name="black" />
       </visual>
       <collision>
@@ -51,5 +51,5 @@
           <mesh filename="file://$(find sobit_home_description)/meshes/arm/arm_shoulder.stl" scale="0.001 0.001 0.001" />
         </geometry>
-        <material name="grey" />
+        <material name="black" />
       </visual>
       <collision>
@@ -86,5 +86,5 @@
           <mesh filename="file://$(find sobit_home_description)/meshes/arm/arm_upper_roll.stl" scale="0.001 0.001 0.001" />
         </geometry>
-        <material name="grey" />
+        <material name="black" />
       </visual>
       <collision>
@@ -139,5 +139,5 @@
           <mesh filename="file://$(find sobit_home_description)/meshes/arm/arm_upper_flex.stl" scale="0.001 0.001 0.001" />
         </geometry>
-        <material name="grey" />
+        <material name="black" />
       </visual>
       <collision>
@@ -192,5 +192,5 @@
           <mesh filename="file://$(find sobit_home_description)/meshes/arm/arm_elbow.stl" scale="0.001 0.001 0.001" />
         </geometry>
-        <material name="grey" />
+        <material name="black" />
       </visual>
       <collision>
@@ -240,5 +240,5 @@
           <mesh filename="file://$(find sobit_home_description)/meshes/arm/arm_lower_bottom.stl" scale="0.001 0.001 0.001" />
         </geometry>
-        <material name="grey" />
+        <material name="black" />
       </visual>
       <collision>
@@ -270,5 +270,5 @@
           <mesh filename="file://$(find sobit_home_description)/meshes/arm/arm_wrist_tilt.stl" scale="0.001 0.001 0.001" />
         </geometry>
-        <material name="grey"/>
+        <material name="black"/>
       </visual>
       <collision>
@@ -300,5 +300,5 @@
           <mesh filename="file://$(find sobit_home_description)/meshes/arm/arm_wrist_roll.stl" scale="0.001 0.001 0.001" />
         </geometry>
-        <material name="grey" />
+        <material name="black" />
       </visual>
       <collision>

File: sobit_home_description/urdf/body/body.urdf.xacro (robot description, xacro)
@@ -51,5 +51,4 @@
           <mesh filename="file://$(find sobit_home_description)/meshes/body/body_cover.dae"/>
         </geometry>
-        <!-- <material name="grey" /> -->
       </visual>
       <collision>

File: sobit_home_description/urdf/hand/hand.urdf.xacro (robot description, xacro)
@@ -27,5 +27,5 @@
           <mesh filename="file://$(find sobit_home_description)/meshes/hand/hand_base.stl" scale="0.001 0.001 0.001" />
         </geometry>
-        <material name="grey" />
+        <material name="black" />
       </visual>
       <inertial>
@@ -52,5 +52,5 @@
           <mesh filename="file://$(find sobit_home_description)/meshes/hand/switching_gear.stl" scale="0.001 0.001 0.001" />
         </geometry>
-        <material name="grey" />
+        <material name="black" />
       </visual>
       <inertial>
@@ -76,5 +76,5 @@
           <mesh filename="file://$(find sobit_home_description)/meshes/hand/middle_pharanx.stl" scale="0.001 0.001 0.001" />
         </geometry>
-        <material name="grey" />
+        <material name="black" />
       </visual>
       <collision>
@@ -106,5 +106,5 @@
           <mesh filename="file://$(find sobit_home_description)/meshes/hand/distal_pharanx.stl" scale="0.001 0.001 0.001" />
         </geometry>
-        <material name="grey" />
+        <material name="black" />
       </visual>
       <collision>
@@ -139,5 +139,5 @@
           <mesh filename="file://$(find sobit_home_description)/meshes/hand/switching_gear_m.stl" scale="0.001 0.001 0.001" />
         </geometry>
-        <material name="grey" />
+        <material name="black" />
       </visual>
       <inertial>
@@ -163,5 +163,5 @@
           <mesh filename="file://$(find sobit_home_description)/meshes/hand/middle_pharanx_m.stl" scale="0.001 0.001 0.001" />
         </geometry>
-        <material name="grey" />
+        <material name="black" />
       </visual>
       <collision>
@@ -193,5 +193,5 @@
           <mesh filename="file://$(find sobit_home_description)/meshes/hand/distal_pharanx_m.stl" scale="0.001 0.001 0.001" />
         </geometry>
-        <material name="grey" />
+        <material name="black" />
       </visual>
       <collision>
@@ -230,5 +230,5 @@
           <mesh filename="file://$(find sobit_home_description)/meshes/hand/thumb_middle_pharanx.stl" scale="0.001 0.001 0.001" />
         </geometry>
-        <material name="grey" />
+        <material name="black" />
       </visual>
       <collision>
@@ -265,5 +265,5 @@
           <mesh filename="file://$(find sobit_home_description)/meshes/hand/thumb_distal_pharanx.stl" scale="0.001 0.001 0.001" />
         </geometry>
-        <material name="grey" />
+        <material name="black" />
       </visual>
       <collision>

Commit message: [FIX] arm joints rotation axis

File: sobit_home_description/urdf/arm/arm.urdf.xacro (robot description, xacro)
@@ -42,5 +42,5 @@
       <child link="${prefix}_${position}_shoulder_tilt_link" />
       <origin xyz="0.0 ${y_sign * 0.126} 0.0" rpy="0.0 0.0 0.0" />
-      <axis xyz="0.0 ${y_sign} 0.0" />
+      <axis xyz="0.0 -1.0 0.0" />
       <limit lower="${-M_PI}" upper="${M_PI}" effort="${44.7 * effort_ratio}" velocity="3.0" />
     </joint>
@@ -72,5 +72,5 @@
       <child link="${prefix}_${position}_upper_roll_link" />
         <origin xyz="0.0510 ${y_sign * 0.100} 0.0" rpy="0.0 0.0 0.0" />
-      <axis xyz="-1.0 0.0 0.0" />
+      <axis xyz="${y_sign} 0.0 0.0" />
       <limit lower="${-M_PI/2}" upper="${M_PI/2}" effort="${10.6 * effort_ratio}" velocity="3.14" />
     </joint>
@@ -108,5 +108,5 @@
       <child link="${prefix}_${position}_upper_roll_sub_link" />
       <origin xyz="-0.0510 ${y_sign * 0.100} 0.0" rpy="0.0 0.0 0.0" />
-      <axis xyz="1.0 0.0 0.0" />
+      <axis xyz="${y_sign * -1} 0.0 0.0" />
       <limit lower="${-M_PI/2}" upper="${M_PI/2}" effort="${10.6 * effort_ratio}" velocity="3.14" />
     </joint>
@@ -125,5 +125,5 @@
       <child link="${prefix}_${position}_upper_flex_link" />
       <origin xyz="-0.0510 ${y_sign * 0.1135} 0.0" rpy="0.0 0.0 0.0" />
-      <axis xyz="0.0 ${y_sign} 0.0" />
+      <axis xyz="0.0 -1.0 0.0" />
       <limit lower="${-M_PI/2}" upper="${M_PI/2}" effort="${10.6 * effort_ratio}" velocity="3.14" />
     </joint>
@@ -161,5 +161,5 @@
       <child link="${prefix}_${position}_upper_flex_sub_link" />
       <origin xyz="-0.0510 ${y_sign * (0.1135+0.0510)} 0.0" rpy="0.0 0.0 0.0" />
-      <axis xyz="0.0 ${y_sign} 0.0" />
+      <axis xyz="0.0 -1.0 0.0" />
       <limit lower="${-M_PI/2}" upper="${M_PI/2}" effort="${10.6 * effort_ratio}" velocity="3.14" />
     </joint>
@@ -177,12 +177,7 @@
       <parent link="${prefix}_${position}_upper_flex_link" />
       <child link="${prefix}_${position}_elbow_link" />
-      <axis xyz="0.0 0.0 1.0" />
+      <axis xyz="0.0 0.0 ${y_sign * -1}" />
       <origin xyz="0.05495 ${y_sign * (0.28865-0.00765)} 0.0510" rpy="0.0 0.0 0.0" />
-      <xacro:if value="${position == 'right'}">
-        <limit lower="0.0" upper="${8/9 * M_PI}" effort="${10.6 * effort_ratio}" velocity="3.14" />
-      </xacro:if>
-      <xacro:unless value="${position == 'right'}">
-        <limit lower="${-8/9 * M_PI}" upper="0.0" effort="${10.6 * effort_ratio}" velocity="3.14" />
-      </xacro:unless>
+      <limit lower="0.0" upper="${8/9 * M_PI}" effort="${10.6 * effort_ratio}" velocity="3.14" />
     </joint>
     <link name="${prefix}_${position}_elbow_link" >
@@ -214,5 +209,5 @@
       <child link="${prefix}_${position}_elbow_sub_link" />
       <origin xyz="0.05495 ${y_sign * (0.28865-0.00765)} -0.0510" rpy="0.0 0.0 0.0" />
-      <axis xyz="0.0 0.0 -1.0" />
+      <axis xyz="0.0 0.0 ${y_sign}" />
       <limit lower="${-M_PI/2}" upper="${M_PI/2}" effort="${10.6 * effort_ratio}" velocity="3.14" />
     </joint>
@@ -231,5 +226,5 @@
       <child link="${prefix}_${position}_lower_flex_link" />
       <origin xyz="0.0 ${y_sign * 0.107} -0.0510" rpy="0.0 0.0 0.0" />
-      <axis xyz="0.0 ${y_sign* 1.0} 0.0" />
+      <axis xyz="0.0 -1.0 0.0" />
       <limit lower="${-M_PI/2}" upper="${M_PI/2}" effort="${10.6 * effort_ratio}" velocity="3.14" />
     </joint>
@@ -261,5 +256,5 @@
       <child link="${prefix}_${position}_wrist_tilt_link" />
       <origin xyz="0.0 ${y_sign * 0.443} 0.0" rpy="0.0 0.0 0.0" />
-      <axis xyz="0.0 0.0 1.0" />
+      <axis xyz="0.0 0.0 ${y_sign * -1}" />
       <limit lower="${-M_PI/2}" upper="${M_PI/2}" effort="${4.1 * effort_ratio}" velocity="4.82" />
     </joint>
@@ -291,5 +286,5 @@
       <child link="${prefix}_${position}_wrist_roll_link" />
       <origin xyz="0.0 ${y_sign * 0.06648202} 0.0" rpy="0.0 0.0 0.0" />
-      <axis xyz="0.0 ${y_sign} 0.0" />
+      <axis xyz="0.0 -1.0 0.0" />
       <limit lower="${-M_PI}" upper="${M_PI}" effort="${4.1 * effort_ratio}" velocity="4.82" />
     </joint>

Commit message: [FIX] inertia values

File: sobit_home_description/urdf/arm/arm.urdf.xacro (robot description, xacro)
@@ -62,7 +62,7 @@
         <origin xyz="0.0 ${y_sign * 0.075} 0.0" rpy="${M_PI/2} 0.0 0.0" />
         <mass value="0.600" />
-        <inertia ixx="${1/12*0.600*(3*0.89**2+0.100**2)}" ixy="0.0" ixz="0.0"
-                 iyy="${1/12*0.600*(3*0.89**2+0.100**2)}" iyz="0.0"
-                 izz="${1/2*0.600*0.89**2}" />
+        <inertia ixx="${1/12*0.600*(3*0.089**2+0.100**2)}" ixy="0.0" ixz="0.0"
+                 iyy="${1/12*0.600*(3*0.089**2+0.100**2)}" iyz="0.0"
+                 izz="${1/2*0.600*0.089**2}" />
       </inertial>
     </link>
@@ -112,11 +112,11 @@
     </joint>
     <link name="${prefix}_${position}_upper_roll_sub_link" >
-      <inertial>
+      <!-- <inertial>
         <origin xyz="${y_sign * 0.0510} ${y_sign * (0.1285)/2 + y_sign * 0.10} 0.0" rpy="${y_sign * M_PI/2} 0.0 0.0" />
-        <mass value="1.73" />
+        <mass value="1.31" />
         <inertia ixx="${1/12*1.31*(3*0.0875**2+0.1285**2)}" ixy="0.0" ixz="0.0"
                  iyy="${1/12*1.31*(3*0.0875**2+0.1285**2)}" iyz="0.0"
                  izz="${1/2*1.31*0.0875**2}" />
-      </inertial>
+      </inertial> -->
     </link>
   <!-- Upper flex joint -->
@@ -165,5 +165,5 @@
     </joint>
     <link name="${prefix}_${position}_upper_flex_sub_link" >
-      <inertial>
+      <!-- <inertial>
         <origin xyz="0.0 ${y_sign * 0.170/2 + y_sign * (0.095+0.01)} 0.0" rpy="${y_sign * M_PI/2} 0.0 0.0" />
         <mass value="1.006" />
@@ -171,5 +171,5 @@
                  iyy="${1/12*1.006*(3*0.038**2+0.170**2)}" iyz="0.0"
                  izz="${1/2*1.006*0.038**2}" />
-      </inertial>
+      </inertial> -->
     </link>
 <!-- Elbow joint -->
@@ -213,5 +213,5 @@
     </joint>
     <link name="${prefix}_${position}_elbow_sub_link" >
-      <inertial>
+      <!-- <inertial>
         <origin xyz="0.0 ${y_sign * 0.12/2 + y_sign * 0.09} ${-y_sign * 0.051}" rpy="${y_sign * M_PI/2} 0.0 0.0" />
         <mass value="0.466"/>
@@ -219,5 +219,5 @@
                  iyy="${1/12*0.466*(3*0.055**2+0.12**2)}" iyz="0.0"
                  izz="${1/2*0.466*0.055**2}" />
-      </inertial>
+      </inertial> -->
     </link>
 <!-- Lower bottom joint -->

File: sobit_home_description/urdf/hand/hand.urdf.xacro (robot description, xacro)
@@ -85,5 +85,6 @@
       </collision>
       <inertial>
-        <origin xyz="0.0 0.0 0.0" rpy="${-y_sign * M_PI/2} ${y_sign * M_PI/2} 0.0" />
+        <origin xyz="0.01445 ${y_sign * 0.030375} 0.0" rpy="${-y_sign * M_PI/2} ${y_sign * M_PI/2} 0.0" />
+        <!-- <origin xyz="0.0 0.0 0.0" rpy="${-y_sign * M_PI/2} ${y_sign * M_PI/2} 0.0" /> -->
         <!-- <mass value="0.036103135757000006" /> -->
         <mass value="0.0361" />
@@ -115,5 +116,6 @@
       </collision>
       <inertial>
-        <origin xyz="0.0 0.0 0.0" rpy="${-y_sign * M_PI/2} ${y_sign * M_PI/2} 0.0" />
+        <origin xyz="0.01445 ${y_sign * 0.032375} ${-y_sign * 0.001}" rpy="${-y_sign * M_PI/2} ${y_sign * M_PI/2} 0.0" />
+        <!-- <origin xyz="0.0 0.0 0.0" rpy="${-y_sign * M_PI/2} ${y_sign * M_PI/2} 0.0" /> -->
         <!-- <mass value="0.0371972081495" /> -->
         <mass value="0.0372" />
@@ -172,10 +174,11 @@
       </collision>
       <inertial>
-        <origin xyz="0.0 0.0 0.0" rpy="${-y_sign * M_PI/2} ${-y_sign * M_PI/2} 0.0" />
+        <origin xyz="0.01445 ${y_sign * 0.030375} 0.0" rpy="${-y_sign * M_PI/2} ${y_sign * M_PI/2} 0.0" />
+        <!-- <origin xyz="0.0 0.0 0.0" rpy="${-y_sign * M_PI/2} ${-y_sign * M_PI/2} 0.0" /> -->
         <!-- <mass value="0.0361032786215" /> -->
         <mass value="0.0361" />
-        <inertia ixx="${1/12*0.0361*(0.0031**2+0.030**2)}" ixy="0.0" ixz="0.0"
-                 iyy="${1/12*0.0361*(0.01445**2+0.0031**2)}" iyz="0.0"
-                 izz="${1/12*0.0361*(0.01445**2+0.030**2)}" />
+        <inertia ixx="${1/12*0.0361*(0.031**2+0.030**2)}" ixy="0.0" ixz="0.0"
+                 iyy="${1/12*0.0361*(0.022**2+0.030**2)}" iyz="0.0"
+                 izz="${1/12*0.0361*(0.022**2+0.031**2)}" />
       </inertial>
     </link>
@@ -202,5 +205,6 @@
       </collision>
       <inertial>
-        <origin xyz="0.0 0.0 0.0" rpy="${-y_sign * M_PI/2} ${-y_sign * M_PI/2} 0.0" />
+        <origin xyz="0.01445 ${y_sign * 0.032375} ${y_sign * 0.001}" rpy="${-y_sign * M_PI/2} ${y_sign * M_PI/2} 0.0" />
+        <!-- <origin xyz="0.0 0.0 0.0" rpy="${-y_sign * M_PI/2} ${-y_sign * M_PI/2} 0.0" /> -->
         <!-- <mass value="0.0371997477059" /> -->
         <mass value="0.0372" />
@@ -239,5 +243,6 @@
       </collision>
       <inertial>
-        <origin xyz="0.0 0.0 0.0" rpy="${-y_sign * M_PI/2} 0.0 0.0" />
+        <origin xyz="-0.001 ${y_sign * 0.032375} ${-y_sign * 0.01445}" rpy="0.0 0.0 0.0" />
+        <!-- <origin xyz="0.0 0.0 0.0" rpy="${-y_sign * M_PI/2} 0.0 0.0" /> -->
         <!-- <mass value="0.0377428526807" /> -->
         <mass value="0.0377" />
@@ -274,5 +279,6 @@
       </collision>
       <inertial>
-        <origin xyz="0.0 0.0 0.0" rpy="${-y_sign * M_PI/2} 0.0 0.0" />
+        <origin xyz="-0.001 ${y_sign * 0.034375} ${-y_sign * 0.01445}" rrpy="${-y_sign * M_PI/2} ${y_sign * M_PI/2} 0.0" />
+        <!-- <origin xyz="0.0 0.0 0.0" rpy="${-y_sign * M_PI/2} 0.0 0.0" /> -->
         <!-- <mass value="0.017059696584599996" /> -->
         <mass value="0.0171" />
@@ -290,5 +296,5 @@
     <!-- Link: End Effector -->
     <link name="${prefix_hand}_${position}_end_effector_link">
-      <visual>
+      <!-- <visual>
         <origin xyz="0.0 0.0 0.0" rpy="0 0 0"/>
         <geometry>
@@ -296,6 +302,6 @@
         </geometry>
         <material name="red"/>
-      </visual>
-      <inertial>
+      </visual> -->
+      <!-- <inertial>
         <origin xyz="0.0 0.0 0.0" rpy="0 0 0"/>
         <mass value="0.0001" />
@@ -303,17 +309,7 @@
                   iyy="${1/12*0.0001*(0.01**2+0.01**2)}" iyz="0.0"
                   izz="${1/12*0.0001*(0.01**2+0.01**2)}" />
-      </inertial>
+      </inertial> -->
     </link>
   <xacro:hand_transmission prefix_hand="${prefix_hand}" position="${position}" prefix_finger="${prefix_finger}"/>
   </xacro:macro>
 </robot>
-<!--
-<<tsukada no memo>> =============================================================================
-この順序はパーツのvisualやcollisionのオリジンが回転することに依存しない...らしい？？？
-ただし、.stlをインポートする際の原点に対するパーツの軸方向が影響している可能性があるような気が...
-<box size = "w"  "d"  "h" >
-  w: x方向の大きさ(幅)
-  d: y方向の大きさ（奥行き）
-  h: z方向の大きさ（高さ）
-======================================================================================
--->

Commit message: [UNDO] sublinks inertia

File: sobit_home_description/urdf/arm/arm.urdf.xacro (robot description, xacro)
@@ -112,5 +112,5 @@
     </joint>
     <link name="${prefix}_${position}_upper_roll_sub_link" >
-      <!-- <inertial>
+      <inertial>
         <origin xyz="${y_sign * 0.0510} ${y_sign * (0.1285)/2 + y_sign * 0.10} 0.0" rpy="${y_sign * M_PI/2} 0.0 0.0" />
         <mass value="1.31" />
@@ -118,5 +118,5 @@
                  iyy="${1/12*1.31*(3*0.0875**2+0.1285**2)}" iyz="0.0"
                  izz="${1/2*1.31*0.0875**2}" />
-      </inertial> -->
+      </inertial>
     </link>
   <!-- Upper flex joint -->
@@ -165,5 +165,5 @@
     </joint>
     <link name="${prefix}_${position}_upper_flex_sub_link" >
-      <!-- <inertial>
+      <inertial>
         <origin xyz="0.0 ${y_sign * 0.170/2 + y_sign * (0.095+0.01)} 0.0" rpy="${y_sign * M_PI/2} 0.0 0.0" />
         <mass value="1.006" />
@@ -171,5 +171,5 @@
                  iyy="${1/12*1.006*(3*0.038**2+0.170**2)}" iyz="0.0"
                  izz="${1/2*1.006*0.038**2}" />
-      </inertial> -->
+      </inertial>
     </link>
 <!-- Elbow joint -->
@@ -213,5 +213,5 @@
     </joint>
     <link name="${prefix}_${position}_elbow_sub_link" >
-      <!-- <inertial>
+      <inertial>
         <origin xyz="0.0 ${y_sign * 0.12/2 + y_sign * 0.09} ${-y_sign * 0.051}" rpy="${y_sign * M_PI/2} 0.0 0.0" />
         <mass value="0.466"/>
@@ -219,5 +219,5 @@
                  iyy="${1/12*0.466*(3*0.055**2+0.12**2)}" iyz="0.0"
                  izz="${1/2*0.466*0.055**2}" />
-      </inertial> -->
+      </inertial>
     </link>
 <!-- Lower bottom joint -->
