Commit message: Remove arm sub-linkage mimic joints from URDF, ros2_control and SRDF

File: sobit_home_description/urdf/arm/arm.urdf.xacro (robot description, xacro)
@@ -102,22 +102,4 @@
       </inertial>
     </link>
-<!-- Upper roll sub joint -->
-    <joint name="${prefix}_${position}_upper_roll_sub_joint" type="revolute" >
-      <mimic joint="${prefix}_${position}_upper_roll_joint" multiplier="-1" offset="0"/>
-      <parent link="${prefix}_${position}_shoulder_tilt_link" />
-      <child link="${prefix}_${position}_upper_roll_sub_link" />
-      <origin xyz="-0.0510 ${y_sign * 0.100} 0.0" rpy="0.0 0.0 0.0" />
-      <axis xyz="${y_sign * -1} 0.0 0.0" />
-      <limit lower="${-M_PI/2}" upper="${M_PI/2}" effort="${10.6 * effort_ratio}" velocity="3.14" />
-    </joint>
-    <link name="${prefix}_${position}_upper_roll_sub_link" >
-      <inertial>
-        <origin xyz="${y_sign * 0.0510} ${y_sign * (0.1285)/2 + y_sign * 0.10} 0.0" rpy="${y_sign * M_PI/2} 0.0 0.0" />
-        <mass value="1.31" />
-        <inertia ixx="${1/12*1.31*(3*0.0875**2+0.1285**2)}" ixy="0.0" ixz="0.0"
-                 iyy="${1/12*1.31*(3*0.0875**2+0.1285**2)}" iyz="0.0"
-                 izz="${1/2*1.31*0.0875**2}" />
-      </inertial>
-    </link>
   <!-- Upper flex joint -->
     <joint name="${prefix}_${position}_upper_flex_joint" type="revolute" >
@@ -149,22 +131,4 @@
       <inertial>
         <origin xyz="0.0 ${y_sign * 0.170/2 + y_sign * (0.095+0.025)} 0.0" rpy="${y_sign * M_PI/2} 0.0 0.0" />
-        <mass value="1.006" />
-        <inertia ixx="${1/12*1.006*(3*0.038**2+0.170**2)}" ixy="0.0" ixz="0.0"
-                 iyy="${1/12*1.006*(3*0.038**2+0.170**2)}" iyz="0.0"
-                 izz="${1/2*1.006*0.038**2}" />
-      </inertial>
-    </link>
-<!-- Upper flex sub joint -->
-    <joint name="${prefix}_${position}_upper_flex_sub_joint" type="revolute" >
-      <mimic joint="${prefix}_${position}_upper_flex_joint" multiplier="1" offset="0"/>
-      <parent link="${prefix}_${position}_upper_roll_link" />
-      <child link="${prefix}_${position}_upper_flex_sub_link" />
-      <origin xyz="-0.0510 ${y_sign * (0.1135+0.0510)} 0.0" rpy="0.0 0.0 0.0" />
-      <axis xyz="0.0 -1.0 0.0" />
-      <limit lower="${-M_PI/2}" upper="${M_PI/2}" effort="${10.6 * effort_ratio}" velocity="3.14" />
-    </joint>
-    <link name="${prefix}_${position}_upper_flex_sub_link" >
-      <inertial>
-        <origin xyz="0.0 ${y_sign * 0.170/2 + y_sign * (0.095+0.01)} 0.0" rpy="${y_sign * M_PI/2} 0.0 0.0" />
         <mass value="1.006" />
         <inertia ixx="${1/12*1.006*(3*0.038**2+0.170**2)}" ixy="0.0" ixz="0.0"
@@ -203,22 +167,4 @@
       </inertial>
     </link>
-<!-- Elbow sub joint -->
-    <joint name="${prefix}_${position}_elbow_sub_joint" type="revolute" >
-      <mimic joint="${prefix}_${position}_elbow_joint" multiplier="-1" offset="0"/>
-      <parent link="${prefix}_${position}_upper_flex_link" />
-      <child link="${prefix}_${position}_elbow_sub_link" />
-      <origin xyz="0.05495 ${y_sign * (0.28865-0.00765)} -0.0510" rpy="0.0 0.0 0.0" />
-      <axis xyz="0.0 0.0 ${y_sign}" />
-      <limit lower="${-M_PI/2}" upper="${M_PI/2}" effort="${10.6 * effort_ratio}" velocity="3.14" />
-    </joint>
-    <link name="${prefix}_${position}_elbow_sub_link" >
-      <inertial>
-        <origin xyz="0.0 ${y_sign * 0.12/2 + y_sign * 0.09} ${-y_sign * 0.051}" rpy="${y_sign * M_PI/2} 0.0 0.0" />
-        <mass value="0.466"/>
-        <inertia ixx="${1/12*0.466*(3*0.055**2+0.12**2)}" ixy="0.0" ixz="0.0"
-                 iyy="${1/12*0.466*(3*0.055**2+0.12**2)}" iyz="0.0"
-                 izz="${1/2*0.466*0.055**2}" />
-      </inertial>
-    </link>
 <!-- Lower bottom joint -->
     <joint name="${prefix}_${position}_lower_flex_joint" type="revolute" >

File: sobit_home_description/urdf/controllers.urdf.xacro (robot description, xacro)
@@ -389,19 +389,4 @@
       <state_interface name="effort"/>
     </joint>
-    <joint name="${prefix}_upper_roll_sub_joint">
-      <param name="mimic">${prefix}_upper_roll_joint</param>
-      <param name="multiplier">-1</param>
-      <xacro:unless value="${$(arg enable_gz)}">
-        <param name="id">33</param>
-        <param name="control_mode">0</param>
-        <param name="interface">rs</param>
-        <param name="Return_Delay_Time">0</param>
-      </xacro:unless>
-      <state_interface name="position">
-        <param name="initial_value">1.571</param>
-      </state_interface>
-      <state_interface name="velocity"/>
-      <state_interface name="effort"/>
-    </joint>
     <joint name="${prefix}_upper_flex_joint">
       <xacro:unless value="${$(arg enable_gz)}">
@@ -416,19 +401,4 @@
         <param name="max">${M_PI/2}</param>
       </command_interface>
-      <state_interface name="position">
-        <param name="initial_value">0.0</param>
-      </state_interface>
-      <state_interface name="velocity"/>
-      <state_interface name="effort"/>
-    </joint>
-    <joint name="${prefix}_upper_flex_sub_joint">
-      <param name="mimic">${prefix}_upper_flex_joint</param>
-      <param name="multiplier">1</param>
-      <xacro:unless value="${$(arg enable_gz)}">
-        <param name="id">35</param>
-        <param name="control_mode">0</param>
-        <param name="interface">rs</param>
-        <param name="Return_Delay_Time">0</param>
-      </xacro:unless>
       <state_interface name="position">
         <param name="initial_value">0.0</param>
@@ -455,19 +425,4 @@
       <state_interface name="effort"/>
     </joint>
-    <joint name="${prefix}_elbow_sub_joint">
-      <param name="mimic">${prefix}_elbow_joint</param>
-      <param name="multiplier">-1</param>
-      <xacro:unless value="${$(arg enable_gz)}">
-        <param name="id">37</param>
-        <param name="control_mode">0</param>
-        <param name="interface">rs</param>
-        <param name="Return_Delay_Time">0</param>
-      </xacro:unless>
-      <state_interface name="position">
-        <param name="initial_value">-1.571</param>
-      </state_interface>
-      <state_interface name="velocity"/>
-      <state_interface name="effort"/>
-    </joint>
     <joint name="${prefix}_lower_flex_joint">
       <xacro:unless value="${$(arg enable_gz)}">
@@ -543,19 +498,4 @@
       <state_interface name="effort"/>
     </joint>
-    <joint name="${prefix}_upper_roll_sub_joint">
-      <param name="mimic">${prefix}_upper_roll_joint</param>
-      <param name="multiplier">-1</param>
-      <xacro:unless value="${$(arg enable_gz)}">
-        <param name="id">43</param>
-        <param name="control_mode">0</param>
-        <param name="interface">rs</param>
-        <param name="Return_Delay_Time">0</param>
-      </xacro:unless>
-      <state_interface name="position">
-        <param name="initial_value">1.571</param>
-      </state_interface>
-      <state_interface name="velocity"/>
-      <state_interface name="effort"/>
-    </joint>
     <joint name="${prefix}_upper_flex_joint">
       <xacro:unless value="${$(arg enable_gz)}">
@@ -575,19 +515,4 @@
       <state_interface name="effort"/>
     </joint>
-    <joint name="${prefix}_upper_flex_sub_joint">
-      <param name="mimic">${prefix}_upper_flex_joint</param>
-      <param name="multiplier">1</param>
-      <xacro:unless value="${$(arg enable_gz)}">
-        <param name="id">45</param>
-        <param name="control_mode">0</param>
-        <param name="interface">rs</param>
-        <param name="Return_Delay_Time">0</param>
-      </xacro:unless>
-      <state_interface name="position">
-        <param name="initial_value">0.0</param>
-      </state_interface>
-      <state_interface name="velocity"/>
-      <state_interface name="effort"/>
-    </joint>
     <joint name="${prefix}_elbow_joint">
       <xacro:unless value="${$(arg enable_gz)}">
@@ -603,19 +528,4 @@
       <state_interface name="position">
         <param name="initial_value">1.571</param>
-      </state_interface>
-      <state_interface name="velocity"/>
-      <state_interface name="effort"/>
-    </joint>
-    <joint name="${prefix}_elbow_sub_joint">
-      <param name="mimic">${prefix}_elbow_joint</param>
-      <param name="multiplier">-1</param>
-      <xacro:unless value="${$(arg enable_gz)}">
-        <param name="id">47</param>
-        <param name="control_mode">0</param>
-        <param name="interface">rs</param>
-        <param name="Return_Delay_Time">0</param>
-      </xacro:unless>
-      <state_interface name="position">
-        <param name="initial_value">-1.571</param>
       </state_interface>
       <state_interface name="velocity"/>
