Commit message: [RM] lidar already implemented in urg pkg

File: sobit_home_description/urdf/gazebo.urdf.xacro (robot description, xacro)
@@ -129,42 +129,4 @@
       </gazebo>
     </xacro:if>
-    <!-- Sensor - LiDAR -->
-    <xacro:macro name="gz_lidar" params="frame topic enable_gz_lidar update_rate sample_rate min_angle max_angle min_range max_range">
-      <xacro:if value="${enable_gz_lidar}">
-        <gazebo reference="${frame}">
-          <sensor name='${frame}_sensor' type='gpu_lidar'>
-            <pose>0 0 0 0 0 0</pose>
-            <gz_frame_id>${robot_name}/${frame}</gz_frame_id>
-            <topic>${robot_name}/${topic}</topic>
-            <update_rate>${update_rate}</update_rate>
-            <ray>
-              <scan>
-                <horizontal>
-                  <samples>${sample_rate}</samples>
-                  <resolution>1</resolution>
-                  <min_angle>${min_angle}</min_angle>
-                  <max_angle>${max_angle}</max_angle>
-                </horizontal>
-                <vertical>
-                  <samples>1</samples>
-                  <resolution>0.01</resolution>
-                  <min_angle>0</min_angle>
-                  <max_angle>0</max_angle>
-                </vertical>
-                </scan>
-              <range>
-                <min>${min_range}</min>
-                <max>${max_range}</max>
-                <resolution>0.01</resolution>
-              </range>
-            </ray>
-            <always_on>1</always_on>
-            <visualize>true</visualize>
-          </sensor>
-        </gazebo>
-      </xacro:if>
-    </xacro:macro>
-    <xacro:gz_lidar frame="lidar_front_laser" topic="lidar_front/scan" enable_gz_lidar="${enable_gz_lidar_front}" update_rate="50" sample_rate="720" min_angle="-2.35619" max_angle="2.35619" min_range="0.1" max_range="60.0" />
-    <xacro:gz_lidar frame="lidar_back_laser"  topic="lidar_back/scan"  enable_gz_lidar="${enable_gz_lidar_back}"  update_rate="50" sample_rate="720" min_angle="-2.35619" max_angle="2.35619" min_range="0.1" max_range="60.0" />
     <gazebo reference="base_link">
       <self_collide>0</self_collide>

Commit message: [FIX] Head Camera Depth gz_frame_id

File: sobit_home_description/urdf/gazebo.urdf.xacro (robot description, xacro)
@@ -2,5 +2,5 @@
 <!-- SOBIT HOME (Gazebo) -->
 <robot name="sobit_home_gazebo" xmlns:xacro="http://ros.org/wiki/xacro">
-  <xacro:macro name="gazebo_sensors" params="robot_name enable_gz_head_cam_color:=True enable_gz_head_cam_depth:=True enable_gz_hand_left_cam_color:=True enable_gz_hand_left_cam_depth:=True enable_gz_hand_right_cam_color:=True enable_gz_hand_right_cam_depth:=True enable_gz_lidar_front:=True enable_gz_lidar_back:=True">
+  <xacro:macro name="gazebo_sensors" params="robot_name enable_gz_head_cam_color:=True enable_gz_head_cam_depth:=True enable_gz_hand_left_cam_color:=True enable_gz_hand_left_cam_depth:=True enable_gz_hand_right_cam_color:=True enable_gz_hand_right_cam_depth:=True">
     <!-- Sensor - Head Camera (Color) -->
     <xacro:if value="${enable_gz_head_cam_color}">
@@ -41,5 +41,5 @@
           <pose>0 0 0 ${M_PI/2} -${M_PI/2} 0 </pose>
           <!-- <ignition_frame_id>${robot_name}/head_camera_depth_optical_frame</ignition_frame_id> -->
-          <gz_frame_id>${robot_name}/head_camera_depth_optical_frame</gz_frame_id>
+          <gz_frame_id>${robot_name}/head_camera_depth_frame</gz_frame_id>
           <topic>${robot_name}/head_camera/depth</topic>
           <always_on>1</always_on>
@@ -51,5 +51,4 @@
               <width>640</width>
               <height>480</height>
-              <format>R_FLOAT32</format>
             </image>
             <clip>

Commit message: [DEL] not used friction settings

File: sobit_home_description/urdf/gazebo.urdf.xacro (robot description, xacro)
@@ -129,20 +129,4 @@
       </gazebo>
     </xacro:if>
-    <gazebo reference="base_link">
-      <self_collide>0</self_collide>
-      <collision>
-        <surface>
-          <friction>
-            <ode>
-              <mu>0.0</mu>
-              <mu2>0.0</mu2>
-              <fdir1>0 0 0</fdir1>
-              <slip1>0.0</slip1>
-              <slip2>0.0</slip2>
-            </ode>
-          </friction>
-        </surface>
-      </collision>
-    </gazebo>
     <!-- Publish Joint States -->
     <gazebo>

Commit message: [UPD] gemini 336L model

File: sobit_home_description/urdf/gazebo.urdf.xacro (robot description, xacro)
@@ -37,8 +37,9 @@
     <!-- Sensor - Head Camera (Depth) -->
     <xacro:if value="${enable_head_cam_depth}">
-      <gazebo reference="head_camera_depth_optical_frame">
+      <!-- <gazebo reference="head_camera_depth_optical_frame"> -->
+      <gazebo reference="head_camera_depth_frame">
         <sensor name="head_camera_depth" type="depth_camera">
-          <pose>0 0 0 ${M_PI/2} -${M_PI/2} 0 </pose>
-          <!-- <ignition_frame_id>${robot_name}/head_camera_depth_optical_frame</ignition_frame_id> -->
+          <!-- <pose>0 0 0 ${M_PI/2} -${M_PI/2} 0 </pose> -->
+          <pose>0 0 0 0 0 0 </pose>
           <gz_frame_id>head_camera_depth_frame</gz_frame_id>
           <topic>${robot_name}/head_camera/depth</topic>

File: sobit_home_description/urdf/sensor/camera_head.urdf.xacro (robot description, xacro)
@@ -2,5 +2,6 @@
 <robot name="sobit_home"
        xmlns:xacro="http://ros.org/wiki/xacro">
-  <xacro:include filename="$(find orbbec_description)/urdf/gemini_336.urdf.xacro" />
+  <!-- <xacro:include filename="$(find orbbec_description)/urdf/gemini_336.urdf.xacro" /> -->
+  <xacro:include filename="$(find orbbec_description)/urdf/gemini_335_L_336_L_macro.urdf.xacro" />
   <xacro:macro name="camera_head" params="prefix parent">
     <joint name="${prefix}_camera_base_joint" type="fixed">
@@ -10,7 +11,10 @@
     </joint>
     <link name="${prefix}_camera_base_link"/>
-    <xacro:gemini_336 parent="${prefix}_camera_base_link" tf_prefix="${prefix}_">
+    <!-- <xacro:gemini_336 parent="${prefix}_camera_base_link" tf_prefix="${prefix}_">
       <origin xyz="0.01 0 -0.0125" rpy="0 0 0"/>
-    </xacro:gemini_336>
+    </xacro:gemini_336> -->
+    <xacro:gemini_335_L_336_L parent="${prefix}_camera_base_link" tf_prefix="${prefix}_">
+      <origin xyz="0.01120544 0.0 -0.01411253" rpy="0 0 0"/>
+    </xacro:gemini_335_L_336_L>
   </xacro:macro>
 </robot>
