Commit message: [UPD] robomaster, dynamixel ros2 control

File: sobit_home_description/urdf/controllers.urdf.xacro (robot description, xacro)
@@ -3,18 +3,26 @@
 <robot name="sobit_home_controllers" xmlns:xacro="http://www.ros.org/wiki/xacro">
   <xacro:macro name="controllers_Dx" params="name enable_gz:=False robot_name:=sobit_pro">
-    <ros2_control name="${name}" type="system">
+    <ros2_control name="${name}_steer_control" type="system">
       <hardware>
-        <plugin>dynamixel_hardware/DynamixelHardware</plugin>
-        <param name="usb_port">/dev/ttyUSB1</param>
-        <param name="baud_rate">1000000</param>
-        <!-- <param name="use_dummy">true</param> -->
+        <xacro:if value="${$(arg enable_gz)}">
+          <plugin>gz_ros2_control/GazeboSimSystem</plugin>
+        </xacro:if>
+        <xacro:unless value="${$(arg enable_gz)}">
+          <plugin>dynamixel_hardware/DynamixelHardware</plugin>
+          <param name="usb_port">/dev/ttyUSB1</param>
+          <param name="baud_rate">1000000</param>
+        </xacro:unless>
       </hardware>
-      <joint name="wheel_f_l_steer_joint">
-        <param name="id">5</param>
+      <joint name="${name}_steer_f_l_joint">
+        <xacro:unless value="${$(arg enable_gz)}">
+          <param name="id">11</param>
+          <param name="control_mode">0</param>
+          <param name="interface">rs</param>
+        </xacro:unless>
         <command_interface name="position">
-          <param name="min">-1.57</param>
-          <param name="max">1.57</param>  <!-- 1.57 -->
+          <param name="min">-3.141592654</param>
+          <param name="max">3.141592654</param>
         </command_interface>
-        <command_interface name="velocity"/>
+        <!-- <command_interface name="velocity"/> -->
         <state_interface name="position">
           <param name="initial_value">0.0</param>
@@ -23,11 +31,15 @@
         <state_interface name="effort"/>
       </joint>
-      <joint name="wheel_f_r_steer_joint">
-        <param name="id">6</param>
+      <joint name="${name}_steer_f_r_joint">
+        <xacro:unless value="${$(arg enable_gz)}">
+          <param name="id">12</param>
+          <param name="control_mode">0</param>
+          <param name="interface">rs</param>
+        </xacro:unless>
         <command_interface name="position">
-          <param name="min">-1.57</param>
-          <param name="max">1.57</param>  <!-- 1.57 -->
+          <param name="min">-3.141592654</param>
+          <param name="max">3.141592654</param>
         </command_interface>
-        <command_interface name="velocity"/>
+        <!-- <command_interface name="velocity"/> -->
         <state_interface name="position">
           <param name="initial_value">0.0</param>
@@ -36,11 +48,15 @@
         <state_interface name="effort"/>
       </joint>
-      <joint name="wheel_b_l_steer_joint">
-        <param name="id">7</param>
+      <joint name="${name}_steer_b_l_joint">
+        <xacro:unless value="${$(arg enable_gz)}">
+          <param name="id">13</param>
+          <param name="control_mode">0</param>
+          <param name="interface">rs</param>
+        </xacro:unless>
         <command_interface name="position">
-          <param name="min">-1.57</param>
-          <param name="max">1.57</param>  <!-- 1.57 -->
+          <param name="min">-3.141592654</param>
+          <param name="max">3.141592654</param>
         </command_interface>
-        <command_interface name="velocity"/>
+        <!-- <command_interface name="velocity"/> -->
         <state_interface name="position">
           <param name="initial_value">0.0</param>
@@ -49,11 +65,15 @@
         <state_interface name="effort"/>
       </joint>
-      <joint name="wheel_b_r_steer_joint">
-        <param name="id">8</param>
+      <joint name="${name}_steer_b_r_joint">
+        <xacro:unless value="${$(arg enable_gz)}">
+          <param name="id">14</param>
+          <param name="control_mode">0</param>
+          <param name="interface">rs</param>
+        </xacro:unless>
         <command_interface name="position">
-          <param name="min">-1.57</param>
-          <param name="max">1.57</param>  <!-- 1.57 -->
+          <param name="min">-3.141592654</param>
+          <param name="max">3.141592654</param>
         </command_interface>
-        <command_interface name="velocity"/>
+        <!-- <command_interface name="velocity"/> -->
         <state_interface name="position">
           <param name="initial_value">0.0</param>
@@ -62,29 +82,69 @@
         <state_interface name="effort"/>
       </joint>
-      <joint name="wheel_f_r_drive_joint">
-        <param name="id">1</param>
-        <command_interface name="velocity"/>
+    </ros2_control>
+    <ros2_control name="${name}_drive_control" type="system">
+      <hardware>
+        <xacro:if value="${$(arg enable_gz)}">
+          <plugin>gz_ros2_control/GazeboSimSystem</plugin>
+        </xacro:if>
+        <xacro:unless value="${$(arg enable_gz)}">
+          <plugin>rm_motors_hw/RmMotorsSystemHardware</plugin>
+          <param name="can_interface">can0</param>
+          <param name="simulate">false</param>
+        </xacro:unless>
+      </hardware>
+      <joint name="${name}_drive_f_l_joint">
+        <param name="motor_id">1</param>
+        <param name="motor_type">m3508</param>
+        <command_interface name="velocity">
+          <param name="min">-10</param>
+          <param name="max">10</param>
+        </command_interface>
+        <state_interface name="position"/>
         <state_interface name="velocity"/>
+        <state_interface name="effort"/>
+        <state_interface name="temperature"/>
       </joint>
-      <joint name="wheel_f_l_drive_joint">
-        <param name="id">2</param>
-        <command_interface name="velocity"/>
+      <joint name="${name}_drive_f_r_joint">
+        <param name="motor_id">2</param>
+        <param name="motor_type">m3508</param>
+        <command_interface name="velocity">
+          <param name="min">-10</param>
+          <param name="max">10</param>
+        </command_interface>
+        <state_interface name="position"/>
         <state_interface name="velocity"/>
+        <state_interface name="effort"/>
+        <state_interface name="temperature"/>
       </joint>
-      <joint name="wheel_b_r_drive_joint">
-        <param name="id">3</param>
-        <command_interface name="velocity"/>
+      <joint name="${name}_drive_b_l_joint">
+        <param name="motor_id">3</param>
+        <param name="motor_type">m3508</param>
+        <command_interface name="velocity">
+          <param name="min">-10</param>
+          <param name="max">10</param>
+        </command_interface>
+        <state_interface name="position"/>
         <state_interface name="velocity"/>
+        <state_interface name="effort"/>
+        <state_interface name="temperature"/>
       </joint>
-      <joint name="wheel_b_l_drive_joint">
-        <param name="id">4</param>
-        <command_interface name="velocity"/>
+      <joint name="${name}_drive_b_r_joint">
+        <param name="motor_id">4</param>
+        <param name="motor_type">m3508</param>
+        <command_interface name="velocity">
+          <param name="min">-10</param>
+          <param name="max">10</param>
+        </command_interface>
+        <state_interface name="position"/>
         <state_interface name="velocity"/>
+        <state_interface name="effort"/>
+        <state_interface name="temperature"/>
       </joint>
     </ros2_control>
-    <!-- Ignition ROS2 Control -->
+    <!-- Gazebo Sim ROS2 Control -->
     <xacro:if value="${$(arg enable_gz)}">
       <gazebo>
-        <plugin filename="ign_ros2_control-system" name="ign_ros2_control::IgnitionROS2ControlPlugin">
+        <plugin filename="gz_ros2_control-system" name="gz_ros2_control::GazeboSimROS2ControlPlugin">
           <ros>
             <namespace>${robot_name}</namespace>

Commit message: [FIX] port name

File: sobit_home_description/urdf/controllers.urdf.xacro (robot description, xacro)
@@ -2,5 +2,5 @@
 <!-- SOBIT home (Dynamixel Control) -->
 <robot name="sobit_home_controllers" xmlns:xacro="http://www.ros.org/wiki/xacro">
-  <xacro:macro name="controllers_Dx" params="name enable_gz:=False robot_name:=sobit_pro">
+  <xacro:macro name="wheel_controllers" params="name enable_gz:=False robot_name:=sobit_pro">
     <ros2_control name="${name}_steer_control" type="system">
       <hardware>
@@ -10,5 +10,5 @@
         <xacro:unless value="${$(arg enable_gz)}">
           <plugin>dynamixel_hardware/DynamixelHardware</plugin>
-          <param name="usb_port">/dev/ttyUSB1</param>
+          <param name="port_name">/dev/ttyUSB0</param>
           <param name="baud_rate">1000000</param>
         </xacro:unless>
