Commit message: [UPD] controllers based on real robot

File: sobit_home_description/urdf/controllers.urdf.xacro (robot description, xacro)
@@ -1,7 +1,7 @@
 <?xml version="1.0" encoding="UTF-8" ?>
-<!-- SOBIT home (Dynamixel Control) -->
+<!-- SOBIT HOME (Controllers) -->
 <robot name="sobit_home_controllers" xmlns:xacro="http://www.ros.org/wiki/xacro">
-  <xacro:macro name="wheel_controllers" params="name enable_gz:=False robot_name:=sobit_home">
-    <ros2_control name="${name}_steer_control" type="system">
+  <xacro:macro name="controllers" params="enable_gz:=False robot_name:=sobit_home">
+    <ros2_control name="dynamixel_control" type="system">
       <hardware>
         <xacro:if value="${$(arg enable_gz)}">
@@ -14,74 +14,12 @@
         </xacro:unless>
       </hardware>
-      <joint name="${name}_steer_f_l_joint">
-        <xacro:unless value="${$(arg enable_gz)}">
-          <param name="id">11</param>
-          <param name="control_mode">0</param>
-          <param name="interface">rs</param>
-        </xacro:unless>
-        <command_interface name="position">
-          <param name="min">-3.141592654</param>
-          <param name="max">3.141592654</param>
-        </command_interface>
-        <!-- <command_interface name="velocity"/> -->
-        <state_interface name="position">
-          <param name="initial_value">0.0</param>
-        </state_interface>
-        <state_interface name="velocity"/>
-        <state_interface name="effort"/>
-      </joint>
-      <joint name="${name}_steer_f_r_joint">
-        <xacro:unless value="${$(arg enable_gz)}">
-          <param name="id">12</param>
-          <param name="control_mode">0</param>
-          <param name="interface">rs</param>
-        </xacro:unless>
-        <command_interface name="position">
-          <param name="min">-3.141592654</param>
-          <param name="max">3.141592654</param>
-        </command_interface>
-        <!-- <command_interface name="velocity"/> -->
-        <state_interface name="position">
-          <param name="initial_value">0.0</param>
-        </state_interface>
-        <state_interface name="velocity"/>
-        <state_interface name="effort"/>
-      </joint>
-      <joint name="${name}_steer_b_l_joint">
-        <xacro:unless value="${$(arg enable_gz)}">
-          <param name="id">13</param>
-          <param name="control_mode">0</param>
-          <param name="interface">rs</param>
-        </xacro:unless>
-        <command_interface name="position">
-          <param name="min">-3.141592654</param>
-          <param name="max">3.141592654</param>
-        </command_interface>
-        <!-- <command_interface name="velocity"/> -->
-        <state_interface name="position">
-          <param name="initial_value">0.0</param>
-        </state_interface>
-        <state_interface name="velocity"/>
-        <state_interface name="effort"/>
-      </joint>
-      <joint name="${name}_steer_b_r_joint">
-        <xacro:unless value="${$(arg enable_gz)}">
-          <param name="id">14</param>
-          <param name="control_mode">0</param>
-          <param name="interface">rs</param>
-        </xacro:unless>
-        <command_interface name="position">
-          <param name="min">-3.141592654</param>
-          <param name="max">3.141592654</param>
-        </command_interface>
-        <!-- <command_interface name="velocity"/> -->
-        <state_interface name="position">
-          <param name="initial_value">0.0</param>
-        </state_interface>
-        <state_interface name="velocity"/>
-        <state_interface name="effort"/>
-      </joint>
+      <xacro:dx_head_controllers        prefix="head"       enable_gz="${$(arg enable_gz)}"/>
+      <xacro:dx_arm_left_controllers    prefix="arm_left"   enable_gz="${$(arg enable_gz)}"/>
+      <xacro:dx_arm_right_controllers   prefix="arm_right"  enable_gz="${$(arg enable_gz)}"/>
+      <!-- <xacro:dx_hand_left_controllers   prefix="hand_left"  enable_gz="${$(arg enable_gz)}"/> -->
+      <!-- <xacro:dx_hand_right_controllers  prefix="hand_right" enable_gz="${$(arg enable_gz)}"/> -->
+      <xacro:dx_wheel_steer_controllers prefix="wheel"      enable_gz="${$(arg enable_gz)}"/>
     </ros2_control>
-    <ros2_control name="${name}_drive_control" type="system">
+    <ros2_control name="robomaster_control" type="system">
       <hardware>
         <xacro:if value="${$(arg enable_gz)}">
@@ -94,208 +32,20 @@
         </xacro:unless>
       </hardware>
-      <joint name="${name}_drive_f_l_joint">
-        <param name="motor_id">1</param>
-        <param name="motor_type">m3508</param>
-        <command_interface name="effort">
-          <param name="min">-10</param>
-          <param name="max">10</param>
-        </command_interface>
-        <state_interface name="position"/>
-        <state_interface name="velocity"/>
-        <state_interface name="effort"/>
-        <state_interface name="temperature"/>
-      </joint>
-      <joint name="${name}_drive_f_r_joint">
-        <param name="motor_id">2</param>
-        <param name="motor_type">m3508</param>
-        <command_interface name="effort">
-          <param name="min">-10</param>
-          <param name="max">10</param>
-        </command_interface>
-        <state_interface name="position"/>
-        <state_interface name="velocity"/>
-        <state_interface name="effort"/>
-        <state_interface name="temperature"/>
-      </joint>
-      <joint name="${name}_drive_b_l_joint">
-        <param name="motor_id">3</param>
-        <param name="motor_type">m3508</param>
-        <command_interface name="effort">
-          <param name="min">-10</param>
-          <param name="max">10</param>
-        </command_interface>
-        <state_interface name="position"/>
-        <state_interface name="velocity"/>
-        <state_interface name="effort"/>
-        <state_interface name="temperature"/>
-      </joint>
-      <joint name="${name}_drive_b_r_joint">
-        <param name="motor_id">4</param>
-        <param name="motor_type">m3508</param>
-        <command_interface name="effort">
-          <param name="min">-10</param>
-          <param name="max">10</param>
-        </command_interface>
-        <state_interface name="position"/>
-        <state_interface name="velocity"/>
-        <state_interface name="effort"/>
-        <state_interface name="temperature"/>
-      </joint>
+      <xacro:rm_wheel_drive_controllers prefix="wheel" enable_gz="${$(arg enable_gz)}"/>
     </ros2_control>
-  </xacro:macro>
-  <xacro:macro name="joint_controllers" params="name enable_gz:=False robot_name:=sobit_home">
-    <ros2_control name="${name}_position_control" type="system">
+    <ros2_control name="iai_control" type="system">
       <hardware>
         <xacro:if value="${$(arg enable_gz)}">
           <plugin>gz_ros2_control/GazeboSimSystem</plugin>
         </xacro:if>
-        <xacro:unless value="${$(arg enable_gz)}">
-          <plugin>dynamixel_hardware/DynamixelHardware</plugin>
-          <param name="port_name">/dev/ttyUSB0</param>
-          <param name="baud_rate">1000000</param>
-        </xacro:unless>
+        <!-- TODO - Develop IAI controller -->
+        <!-- <xacro:unless value="${$(arg enable_gz)}">
+          <plugin>iai_hardware/IaiHardware</plugin>
+          <param name="port_name">/dev/ttyUSB1</param>
+          <param name="baud_rate">115200</param>
+        </xacro:unless> -->
       </hardware>
-      <xacro:arm_controllers position="left"/>
-      <xacro:arm_controllers position="right"/>
-      <joint name="head_pan_joint">
-        <xacro:unless value="${$(arg enable_gz)}">
-          <param name="id">21</param>
-          <param name="control_mode">3</param>
-          <param name="interface">rp</param>
-        </xacro:unless>
-        <command_interface name="position">
-          <param name="min">-0.4</param>
-          <param name="max">0.4</param>
-        </command_interface>
-        <!-- <command_interface name="velocity"/> -->
-        <state_interface name="position">
-          <param name="initial_value">0.0</param>
-        </state_interface>
-        <state_interface name="velocity"/>
-        <state_interface name="effort"/>
-      </joint>
-      <joint name="head_tilt_joint">
-        <xacro:unless value="${$(arg enable_gz)}">
-          <param name="id">21</param>
-          <param name="control_mode">3</param>
-          <param name="interface">rp</param>
-        </xacro:unless>
-        <command_interface name="position">
-          <param name="min">-0.4</param>
-          <param name="max">0.4</param>
-        </command_interface>
-        <!-- <command_interface name="velocity"/> -->
-        <state_interface name="position">
-          <param name="initial_value">0.0</param>
-        </state_interface>
-        <state_interface name="velocity"/>
-        <state_interface name="effort"/>
-      </joint>
-      <joint name="linear_actuator_joint">
-        <xacro:unless value="${$(arg enable_gz)}">
-          <param name="id">20</param>
-          <param name="control_mode">3</param>
-          <param name="interface">rp</param>
-        </xacro:unless>
-        <command_interface name="position">
-          <param name="min">-0.4</param>
-          <param name="max">0.4</param>
-        </command_interface>
-        <state_interface name="position">
-          <param name="initial_value">0.0</param>
-        </state_interface>
-        <state_interface name="velocity"/>
-        <state_interface name="effort"/>
-      </joint>
+      <xacro:iai_body_controllers prefix="body" enable_gz="${$(arg enable_gz)}"/>
     </ros2_control>
-  </xacro:macro>
-  <xacro:macro name="arm_controllers" params="position">
-      <joint name="arm_${position}_shoulder_tilt_joint">
-        <xacro:unless value="${$(arg enable_gz)}">
-          <param name="id">20</param>
-          <param name="control_mode">3</param>
-          <param name="interface">rp</param>
-        </xacro:unless>
-        <command_interface name="position">
-          <param name="min">-0.4</param>
-          <param name="max">0.4</param>
-        </command_interface>
-        <!-- <command_interface name="velocity"/> -->
-        <state_interface name="position">
-          <param name="initial_value">0.0</param>
-        </state_interface>
-        <state_interface name="velocity"/>
-        <state_interface name="effort"/>
-      </joint>
-      <joint name="arm_${position}_upper_roll_joint">
-        <xacro:unless value="${$(arg enable_gz)}">
-          <param name="id">21</param>
-          <param name="control_mode">3</param>
-          <param name="interface">rp</param>
-        </xacro:unless>
-        <command_interface name="position">
-          <param name="min">-0.4</param>
-          <param name="max">0.4</param>
-        </command_interface>
-        <!-- <command_interface name="velocity"/> -->
-        <state_interface name="position">
-          <param name="initial_value">0.0</param>
-        </state_interface>
-        <state_interface name="velocity"/>
-        <state_interface name="effort"/>
-      </joint>
-      <joint name="arm_${position}_upper_flex_joint">
-        <xacro:unless value="${$(arg enable_gz)}">
-          <param name="id">21</param>
-          <param name="control_mode">3</param>
-          <param name="interface">rp</param>
-        </xacro:unless>
-        <command_interface name="position">
-          <param name="min">-0.4</param>
-          <param name="max">0.4</param>
-        </command_interface>
-        <!-- <command_interface name="velocity"/> -->
-        <state_interface name="position">
-          <param name="initial_value">0.0</param>
-        </state_interface>
-        <state_interface name="velocity"/>
-        <state_interface name="effort"/>
-      </joint>
-      <joint name="arm_${position}_elbow_joint">
-        <xacro:unless value="${$(arg enable_gz)}">
-          <param name="id">21</param>
-          <param name="control_mode">3</param>
-          <param name="interface">rp</param>
-        </xacro:unless>
-        <command_interface name="position">
-          <param name="min">-0.4</param>
-          <param name="max">0.4</param>
-        </command_interface>
-        <!-- <command_interface name="velocity"/> -->
-        <state_interface name="position">
-          <param name="initial_value">0.0</param>
-        </state_interface>
-        <state_interface name="velocity"/>
-        <state_interface name="effort"/>
-      </joint>
-      <joint name="arm_${position}_wrist_joint">
-        <xacro:unless value="${$(arg enable_gz)}">
-          <param name="id">21</param>
-          <param name="control_mode">3</param>
-          <param name="interface">rp</param>
-        </xacro:unless>
-        <command_interface name="position">
-          <param name="min">-0.4</param>
-          <param name="max">0.4</param>
-        </command_interface>
-        <!-- <command_interface name="velocity"/> -->
-        <state_interface name="position">
-          <param name="initial_value">0.0</param>
-        </state_interface>
-        <state_interface name="velocity"/>
-        <state_interface name="effort"/>
-      </joint>
-  </xacro:macro>
-  <xacro:macro name="ros2_controllers" params="enable_gz:=False robot_name:=sobit_home">
     <!-- Gazebo Sim ROS2 Control -->
     <xacro:if value="${$(arg enable_gz)}">
@@ -305,8 +55,600 @@
             <namespace>${robot_name}</namespace>
           </ros>
-          <parameters>$(find ${robot_name}_control)/config/gz_controllers.yaml</parameters>
+          <parameters>$(find sobit_home_control)/config/gz_controllers.yaml</parameters>
         </plugin>
       </gazebo>
     </xacro:if>
   </xacro:macro>
+  <xacro:macro name="rm_wheel_drive_controllers"  params="prefix enable_gz:=False">
+    <joint name="${prefix}_drive_f_l_joint">
+      <param name="motor_id">1</param>
+      <param name="motor_type">m3508</param>
+      <command_interface name="effort">
+        <param name="min">-10</param>
+        <param name="max">10</param>
+      </command_interface>
+      <state_interface name="position"/>
+      <state_interface name="velocity"/>
+      <state_interface name="effort"/>
+      <state_interface name="temperature"/>
+    </joint>
+    <joint name="${prefix}_drive_f_r_joint">
+      <param name="motor_id">2</param>
+      <param name="motor_type">m3508</param>
+      <command_interface name="effort">
+        <param name="min">-10</param>
+        <param name="max">10</param>
+      </command_interface>
+      <state_interface name="position"/>
+      <state_interface name="velocity"/>
+      <state_interface name="effort"/>
+      <state_interface name="temperature"/>
+    </joint>
+    <joint name="${prefix}_drive_b_l_joint">
+      <param name="motor_id">3</param>
+      <param name="motor_type">m3508</param>
+      <command_interface name="effort">
+        <param name="min">-10</param>
+        <param name="max">10</param>
+      </command_interface>
+      <state_interface name="position"/>
+      <state_interface name="velocity"/>
+      <state_interface name="effort"/>
+      <state_interface name="temperature"/>
+    </joint>
+    <joint name="${prefix}_drive_b_r_joint">
+      <param name="motor_id">4</param>
+      <param name="motor_type">m3508</param>
+      <command_interface name="effort">
+        <param name="min">-10</param>
+        <param name="max">10</param>
+      </command_interface>
+      <state_interface name="position"/>
+      <state_interface name="velocity"/>
+      <state_interface name="effort"/>
+      <state_interface name="temperature"/>
+    </joint>
+  </xacro:macro>
+  <xacro:macro name="dx_wheel_steer_controllers"  params="prefix enable_gz:=False">
+    <joint name="${prefix}_steer_f_l_joint">
+      <xacro:unless value="${$(arg enable_gz)}">
+        <param name="id">11</param>
+        <param name="control_mode">0</param>
+        <param name="interface">rs</param>
+      </xacro:unless>
+      <command_interface name="position">
+        <param name="min">-3.141592654</param>
+        <param name="max">3.141592654</param>
+      </command_interface>
+      <!-- <command_interface name="velocity"/> -->
+      <state_interface name="position">
+        <param name="initial_value">0.0</param>
+      </state_interface>
+      <state_interface name="velocity"/>
+      <state_interface name="effort"/>
+    </joint>
+    <joint name="${prefix}_steer_f_r_joint">
+      <xacro:unless value="${$(arg enable_gz)}">
+        <param name="id">12</param>
+        <param name="control_mode">0</param>
+        <param name="interface">rs</param>
+      </xacro:unless>
+      <command_interface name="position">
+        <param name="min">-3.141592654</param>
+        <param name="max">3.141592654</param>
+      </command_interface>
+      <!-- <command_interface name="velocity"/> -->
+      <state_interface name="position">
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
Commit message: [ADD] add mimic joint for sim

File: sobit_home_description/urdf/controllers.urdf.xacro (robot description, xacro)
@@ -85,5 +85,5 @@
             <namespace>$(arg robot_name)</namespace>
           </ros>
-          <parameters>$(find sobit_home_control)/config/controllers.yaml</parameters>
+          <parameters>$(find sobit_home_control)/config/gz_controllers.yaml</parameters>
         </plugin>
       </gazebo>
@@ -488,4 +488,23 @@
       <state_interface name="effort"/>
     </joint>
+    <xacro:if value="${$(arg enable_gz)}">
+      <joint name="${prefix}_finger_r_mcp_joint">
+        <xacro:unless value="${$(arg enable_gz)}">
+          <param name="id">50</param>
+          <param name="control_mode">6</param>
+          <param name="interface">ttl</param>
+        </xacro:unless>
+        <command_interface name="position">
+          <param name="min">-${M_PI/2}</param>
+          <param name="max">${M_PI/2}</param>
+        </command_interface>
+        <!-- <command_interface name="velocity"/> -->
+        <state_interface name="position">
+          <param name="initial_value">0.0</param>
+        </state_interface>
+        <state_interface name="velocity"/>
+        <state_interface name="effort"/>
+      </joint>
+    </xacro:if>
     <joint name="${prefix}_finger_l_dip_joint">
       <xacro:unless value="${$(arg enable_gz)}">
@@ -609,4 +628,23 @@
       <state_interface name="effort"/>
     </joint>
+    <xacro:if value="${$(arg enable_gz)}">
+      <joint name="${prefix}_finger_r_mcp_joint">
+        <xacro:unless value="${$(arg enable_gz)}">
+          <param name="id">60</param>
+          <param name="control_mode">6</param>
+          <param name="interface">ttl</param>
+        </xacro:unless>
+        <command_interface name="position">
+          <param name="min">-${M_PI/2}</param>
+          <param name="max">${M_PI/2}</param>
+        </command_interface>
+        <!-- <command_interface name="velocity"/> -->
+        <state_interface name="position">
+          <param name="initial_value">0.0</param>
+        </state_interface>
+        <state_interface name="velocity"/>
+        <state_interface name="effort"/>
+      </joint>
+    </xacro:if>
     <joint name="${prefix}_finger_l_dip_joint">
       <xacro:unless value="${$(arg enable_gz)}">
