Commit message: [Fix] Joint names and motor IDs.

File: sobit_home_description/urdf/controllers.urdf.xacro (robot description, xacro)
@@ -503,23 +503,23 @@
       </joint>
     </xacro:if>
+    <joint name="${prefix}_finger_l_pip_joint">
+      <xacro:unless value="${$(arg enable_gz)}">
+        <param name="id">51</param>
+        <param name="control_mode">6</param>
+        <param name="interface">ttl</param>
+      </xacro:unless>
+      <command_interface name="position">
+        <param name="min">-${M_PI/2}</param>
+        <param name="max">${M_PI/2}</param>
+      </command_interface>
+      <!-- <command_interface name="velocity"/> -->
+      <state_interface name="position">
+        <param name="initial_value">0.0</param>
+      </state_interface>
+      <state_interface name="velocity"/>
+      <state_interface name="effort"/>
+    </joint>
     <joint name="${prefix}_finger_l_dip_joint">
       <xacro:unless value="${$(arg enable_gz)}">
-        <param name="id">51</param>
-        <param name="control_mode">6</param>
-        <param name="interface">ttl</param>
-      </xacro:unless>
-      <command_interface name="position">
-        <param name="min">-${M_PI/2}</param>
-        <param name="max">${M_PI/2}</param>
-      </command_interface>
-      <!-- <command_interface name="velocity"/> -->
-      <state_interface name="position">
-        <param name="initial_value">0.0</param>
-      </state_interface>
-      <state_interface name="velocity"/>
-      <state_interface name="effort"/>
-    </joint>
-    <joint name="${prefix}_finger_l_pip_joint">
-      <xacro:unless value="${$(arg enable_gz)}">
         <param name="id">52</param>
         <param name="control_mode">6</param>
@@ -571,5 +571,5 @@
       <state_interface name="effort"/>
     </joint>
-    <joint name="${prefix}_finger_r_dip_joint">
+    <joint name="${prefix}_finger_r_pip_joint">
       <xacro:unless value="${$(arg enable_gz)}">
         <param name="id">55</param>
@@ -588,5 +588,5 @@
       <state_interface name="effort"/>
     </joint>
-      <joint name="${prefix}_finger_r_pip_joint">
+      <joint name="${prefix}_finger_r_dip_joint">
       <xacro:unless value="${$(arg enable_gz)}">
         <param name="id">56</param>
@@ -635,23 +635,23 @@
       </joint>
     </xacro:if>
+    <joint name="${prefix}_finger_l_pip_joint">
+      <xacro:unless value="${$(arg enable_gz)}">
+        <param name="id">61</param>
+        <param name="control_mode">6</param>
+        <param name="interface">ttl</param>
+      </xacro:unless>
+      <command_interface name="position">
+        <param name="min">-${M_PI/2}</param>
+        <param name="max">${M_PI/2}</param>
+      </command_interface>
+      <!-- <command_interface name="velocity"/> -->
+      <state_interface name="position">
+        <param name="initial_value">0.0</param>
+      </state_interface>
+      <state_interface name="velocity"/>
+      <state_interface name="effort"/>
+    </joint>
     <joint name="${prefix}_finger_l_dip_joint">
       <xacro:unless value="${$(arg enable_gz)}">
-        <param name="id">61</param>
-        <param name="control_mode">6</param>
-        <param name="interface">ttl</param>
-      </xacro:unless>
-      <command_interface name="position">
-        <param name="min">-${M_PI/2}</param>
-        <param name="max">${M_PI/2}</param>
-      </command_interface>
-      <!-- <command_interface name="velocity"/> -->
-      <state_interface name="position">
-        <param name="initial_value">0.0</param>
-      </state_interface>
-      <state_interface name="velocity"/>
-      <state_interface name="effort"/>
-    </joint>
-    <joint name="${prefix}_finger_l_pip_joint">
-      <xacro:unless value="${$(arg enable_gz)}">
         <param name="id">62</param>
         <param name="control_mode">6</param>
@@ -703,22 +703,22 @@
       <state_interface name="effort"/>
     </joint>
+    <joint name="${prefix}_finger_r_pip_joint">
+      <xacro:unless value="${$(arg enable_gz)}">
+        <param name="id">65</param>
+        <param name="control_mode">6</param>
+        <param name="interface">ttl</param>
+      </xacro:unless>
+      <command_interface name="position">
+        <param name="min">-${M_PI/2}</param>
+        <param name="max">${M_PI/2}</param>
+      </command_interface>
+      <!-- <command_interface name="velocity"/> -->
+      <state_interface name="position">
+        <param name="initial_value">0.0</param>
+      </state_interface>
+      <state_interface name="velocity"/>
+      <state_interface name="effort"/>
+    </joint>
     <joint name="${prefix}_finger_r_dip_joint">
-      <xacro:unless value="${$(arg enable_gz)}">
-        <param name="id">65</param>
-        <param name="control_mode">6</param>
-        <param name="interface">ttl</param>
-      </xacro:unless>
-      <command_interface name="position">
-        <param name="min">-${M_PI/2}</param>
-        <param name="max">${M_PI/2}</param>
-      </command_interface>
-      <!-- <command_interface name="velocity"/> -->
-      <state_interface name="position">
-        <param name="initial_value">0.0</param>
-      </state_interface>
-      <state_interface name="velocity"/>
-      <state_interface name="effort"/>
-    </joint>
-    <joint name="${prefix}_finger_r_pip_joint">
       <xacro:unless value="${$(arg enable_gz)}">
         <param name="id">66</param>

Commit message: [FIX] get arg value as property

File: sobit_home_description/urdf/controllers.urdf.xacro (robot description, xacro)
@@ -10,6 +10,7 @@
           </xacro:if>
           <xacro:unless value="${$(arg enable_gz)}">
+            <xacro:property name="dxl_lower_body_port" value="$(arg dxl_lower_body_port)"/>
             <plugin>dynamixel_hardware/DynamixelHardware</plugin>
-            <param name="port_name">"${arg dxl_lower_body_port}"</param>
+            <param name="port_name">${dxl_lower_body_port}</param>
             <param name="baud_rate">1000000</param>
           </xacro:unless>
@@ -25,6 +26,7 @@
           </xacro:if>
           <xacro:unless value="${$(arg enable_gz)}">
+            <xacro:property name="dxl_upper_body_port" value="$(arg dxl_upper_body_port)"/>
             <plugin>dynamixel_hardware/DynamixelHardware</plugin>
-            <param name="port_name">"${arg dxl_upper_body_port}"</param>
+            <param name="port_name">${dxl_upper_body_port}</param>
             <param name="baud_rate">1000000</param>
           </xacro:unless>

Commit message: update anction server

File: sobit_home_description/urdf/controllers.urdf.xacro (robot description, xacro)
@@ -502,5 +502,5 @@
         <param name="id">50</param>
         <param name="control_mode">6</param>
-        <param name="Goal_Current">50</param>
+        <param name="Goal_Current">300</param>
         <param name="interface">ttl</param>
       </xacro:unless>
@@ -531,5 +531,5 @@
         <param name="id">51</param>
         <param name="control_mode">6</param>
-        <param name="Goal_Current">50</param>
+        <param name="Goal_Current">150</param>
         <param name="interface">ttl</param>
       </xacro:unless>
@@ -549,5 +549,5 @@
         <param name="id">52</param>
         <param name="control_mode">6</param>
-        <param name="Goal_Current">50</param>
+        <param name="Goal_Current">100</param>
         <param name="interface">ttl</param>
       </xacro:unless>
@@ -567,5 +567,5 @@
         <param name="id">53</param>
         <param name="control_mode">6</param>
-        <param name="Goal_Current">50</param>
+        <param name="Goal_Current">225</param>
         <param name="interface">ttl</param>
       </xacro:unless>
@@ -585,5 +585,5 @@
         <param name="id">54</param>
         <param name="control_mode">6</param>
-        <param name="Goal_Current">50</param>
+        <param name="Goal_Current">150</param>
         <param name="interface">ttl</param>
       </xacro:unless>
@@ -603,5 +603,5 @@
         <param name="id">55</param>
         <param name="control_mode">6</param>
-        <param name="Goal_Current">50</param>
+        <param name="Goal_Current">150</param>
         <param name="interface">ttl</param>
       </xacro:unless>
@@ -621,5 +621,5 @@
         <param name="id">56</param>
         <param name="control_mode">6</param>
-        <param name="Goal_Current">50</param>
+        <param name="Goal_Current">100</param>
         <param name="interface">ttl</param>
       </xacro:unless>
@@ -641,10 +641,10 @@
         <param name="id">60</param>
         <param name="control_mode">6</param>
-        <param name="Goal_Current">50</param>
-        <param name="interface">ttl</param>
-      </xacro:unless>
-      <command_interface name="position">
-        <param name="min">-${M_PI/2}</param>
-        <param name="max">${M_PI/2}</param>
+        <param name="Goal_Current">300</param>
+        <param name="interface">ttl</param>
+      </xacro:unless>
+      <command_interface name="position">
+        <param name="min">-1.7</param>
+        <param name="max">1.70</param>
       </command_interface>
       <!-- <command_interface name="velocity"/> -->
@@ -670,21 +670,39 @@
         <param name="id">61</param>
         <param name="control_mode">6</param>
+        <param name="Goal_Current">200</param>
+        <param name="interface">ttl</param>
+      </xacro:unless>
+      <command_interface name="position">
+        <param name="min">-0.5</param>
+        <param name="max">${M_PI/2}</param>
+      </command_interface>
+      <!-- <command_interface name="velocity"/> -->
+      <state_interface name="position">
+        <param name="initial_value">0.0</param>
+      </state_interface>
+      <state_interface name="velocity"/>
+      <state_interface name="effort"/>
+    </joint>
+    <joint name="${prefix}_finger_l_dip_joint">
+      <xacro:unless value="${$(arg enable_gz)}">
+        <param name="id">62</param>
+        <param name="control_mode">6</param>
         <param name="Goal_Current">50</param>
         <param name="interface">ttl</param>
       </xacro:unless>
       <command_interface name="position">
-        <param name="min">-${M_PI/2}</param>
-        <param name="max">${M_PI/2}</param>
-      </command_interface>
-      <!-- <command_interface name="velocity"/> -->
-      <state_interface name="position">
-        <param name="initial_value">0.0</param>
-      </state_interface>
-      <state_interface name="velocity"/>
-      <state_interface name="effort"/>
-    </joint>
-    <joint name="${prefix}_finger_l_dip_joint">
-      <xacro:unless value="${$(arg enable_gz)}">
-        <param name="id">62</param>
+        <param name="min">-2.0</param>
+        <param name="max">0.5</param>
+      </command_interface>
+      <!-- <command_interface name="velocity"/> -->
+      <state_interface name="position">
+        <param name="initial_value">0.0</param>
+      </state_interface>
+      <state_interface name="velocity"/>
+      <state_interface name="effort"/>
+    </joint>
+    <joint name="${prefix}_finger_c_mcp_joint">
+      <xacro:unless value="${$(arg enable_gz)}">
+        <param name="id">63</param>
         <param name="control_mode">6</param>
         <param name="Goal_Current">50</param>
@@ -692,17 +710,17 @@
       </xacro:unless>
       <command_interface name="position">
-        <param name="min">-${M_PI/2}</param>
-        <param name="max">${M_PI/2}</param>
-      </command_interface>
-      <!-- <command_interface name="velocity"/> -->
-      <state_interface name="position">
-        <param name="initial_value">0.0</param>
-      </state_interface>
-      <state_interface name="velocity"/>
-      <state_interface name="effort"/>
-    </joint>
-    <joint name="${prefix}_finger_c_mcp_joint">
-      <xacro:unless value="${$(arg enable_gz)}">
-        <param name="id">63</param>
+        <param name="min">-0.9</param>
+        <param name="max">${M_PI/2}</param>
+      </command_interface>
+      <!-- <command_interface name="velocity"/> -->
+      <state_interface name="position">
+        <param name="initial_value">0.0</param>
+      </state_interface>
+      <state_interface name="velocity"/>
+      <state_interface name="effort"/>
+    </joint>
+    <joint name="${prefix}_finger_c_ip_joint">
+      <xacro:unless value="${$(arg enable_gz)}">
+        <param name="id">64</param>
         <param name="control_mode">6</param>
         <param name="Goal_Current">50</param>
@@ -710,17 +728,17 @@
       </xacro:unless>
       <command_interface name="position">
-        <param name="min">-${M_PI/2}</param>
-        <param name="max">${M_PI/2}</param>
-      </command_interface>
-      <!-- <command_interface name="velocity"/> -->
-      <state_interface name="position">
-        <param name="initial_value">0.0</param>
-      </state_interface>
-      <state_interface name="velocity"/>
-      <state_interface name="effort"/>
-    </joint>
-    <joint name="${prefix}_finger_c_ip_joint">
-      <xacro:unless value="${$(arg enable_gz)}">
-        <param name="id">64</param>
+        <param name="min">-2.0</param>
+        <param name="max">0.5</param>
+      </command_interface>
+      <!-- <command_interface name="velocity"/> -->
+      <state_interface name="position">
+        <param name="initial_value">0.0</param>
+      </state_interface>
+      <state_interface name="velocity"/>
+      <state_interface name="effort"/>
+    </joint>
+    <joint name="${prefix}_finger_r_pip_joint">
+      <xacro:unless value="${$(arg enable_gz)}">
+        <param name="id">65</param>
         <param name="control_mode">6</param>
         <param name="Goal_Current">50</param>
@@ -729,16 +747,16 @@
       <command_interface name="position">
         <param name="min">-${M_PI/2}</param>
-        <param name="max">${M_PI/2}</param>
-      </command_interface>
-      <!-- <command_interface name="velocity"/> -->
-      <state_interface name="position">
-        <param name="initial_value">0.0</param>
-      </state_interface>
-      <state_interface name="velocity"/>
-      <state_interface name="effort"/>
-    </joint>
-    <joint name="${prefix}_finger_r_pip_joint">
-      <xacro:unless value="${$(arg enable_gz)}">
-        <param name="id">65</param>
+        <param name="max">0.5</param>
+      </command_interface>
+      <!-- <command_interface name="velocity"/> -->
+      <state_interface name="position">
+        <param name="initial_value">0.0</param>
+      </state_interface>
+      <state_interface name="velocity"/>
+      <state_interface name="effort"/>
+    </joint>
+    <joint name="${prefix}_finger_r_dip_joint">
+      <xacro:unless value="${$(arg enable_gz)}">
+        <param name="id">66</param>
         <param name="control_mode">6</param>
         <param name="Goal_Current">50</param>
@@ -746,24 +764,6 @@
       </xacro:unless>
       <command_interface name="position">
-        <param name="min">-${M_PI/2}</param>
-        <param name="max">${M_PI/2}</param>
-      </command_interface>
-      <!-- <command_interface name="velocity"/> -->
-      <state_interface name="position">
-        <param name="initial_value">0.0</param>
-      </state_interface>
-      <state_interface name="velocity"/>
-      <state_interface name="effort"/>
-    </joint>
-    <joint name="${prefix}_finger_r_dip_joint">
-      <xacro:unless value="${$(arg enable_gz)}">
-        <param name="id">66</param>
-        <param name="control_mode">6</param>
-        <param name="Goal_Current">50</param>
-        <param name="interface">ttl</param>
-      </xacro:unless>
-      <command_interface name="position">
-        <param name="min">-${M_PI/2}</param>
-        <param name="max">${M_PI/2}</param>
+        <param name="min">-0.5</param>
+        <param name="max">2.0</param>
       </command_interface>
       <!-- <command_interface name="velocity"/> -->

Commit message: [UPD] Modified some limitation parameters.

File: sobit_home_description/urdf/controllers.urdf.xacro (robot description, xacro)
@@ -669,6 +669,6 @@
       </xacro:unless>
       <command_interface name="position">
-        <param name="min">-1.7</param>
-        <param name="max">1.70</param>
+        <param name="min">${-M_PI/2}</param>
+        <param name="max">${M_PI/2}</param>
       </command_interface>
       <!-- <command_interface name="velocity"/> -->
@@ -697,5 +697,5 @@
       </xacro:unless>
       <command_interface name="position">
-        <param name="min">-0.5</param>
+        <param name="min">${-M_PI/2}</param>
         <param name="max">${M_PI/2}</param>
       </command_interface>

File: sobit_home_description/urdf/hand/hand.urdf.xacro (robot description, xacro)
@@ -215,5 +215,11 @@
       <origin xyz="0.036751 ${y_sign * 0.036625} ${y_sign * 0.014550} " rpy="0.0 0.0 0.0" />
       <axis xyz="0.0 0.0 1.0 " />
-      <limit lower="${-M_PI/2}" upper="${M_PI/6}" effort="0.52" velocity="11.031179004" />
+      <!-- <limit lower="${-M_PI/2}" upper="${M_PI/6}" effort="0.52" velocity="11.031179004" /> -->
+      <xacro:if value="${position == 'left'}">
+        <limit lower="${-M_PI/2}" upper="${M_PI/6}" effort="0.52" velocity="11.031" />
+      </xacro:if>
+      <xacro:if value="${position == 'right'}">
+        <limit lower="${-M_PI/6}" upper="${M_PI/2}" effort="0.52" velocity="11.031" />
+      </xacro:if>
     </joint>
     <link name="${prefix_hand}_${position}_${prefix_finger}_c_mcp_link" >

Commit message: [FIX] async only with real robot

File: sobit_home_description/urdf/controllers.urdf.xacro (robot description, xacro)
@@ -3,4 +3,8 @@
 <robot name="sobit_home_controllers" xmlns:xacro="http://www.ros.org/wiki/xacro">
   <xacro:macro name="controllers" params="enable_gz:=False robot_name:=sobit_home">
+    <!-- Async hardware = separate read/write thread, decoupling serial/CAN I/O from
+         the control loop. Only meaningful on REAL hardware; gz_ros2_control is stepped
+         synchronously by the sim, so force sync (is_async=false) under Gazebo. -->
+    <xacro:property name="hw_is_async" value="${'false' if $(arg enable_gz) else 'true'}"/>
     <xacro:if value="${$(arg enable_mobile_base)}">
       <ros2_control name="dynamixel_control_lower" type="system">
@@ -121,9 +125,10 @@
     </xacro:if>
     <xacro:if value="${$(arg enable_body)}">
-      <!-- <ros2_control name="uirobot_control" type="system"> -->
-      <ros2_control name="uirobot_control" type="system" is_async="true">
-        <properties>
-          <async scheduling_policy="synchronized" thread_priority="79" affinity="[6]" print_warnings="true"/>
-        </properties>
+      <ros2_control name="uirobot_control" type="system" is_async="${hw_is_async}">
+        <xacro:unless value="${$(arg enable_gz)}">
+          <properties>
+            <async scheduling_policy="synchronized" thread_priority="79" affinity="[6]" print_warnings="true"/>
+          </properties>
+        </xacro:unless>
         <hardware>
           <xacro:if value="${$(arg enable_gz)}">

Commit message: [UPD]Adjust Goal Current.

File: sobit_home_description/urdf/controllers.urdf.xacro (robot description, xacro)
@@ -3,8 +3,4 @@
 <robot name="sobit_home_controllers" xmlns:xacro="http://www.ros.org/wiki/xacro">
   <xacro:macro name="controllers" params="enable_gz:=False robot_name:=sobit_home">
-    <!-- Async hardware = separate read/write thread, decoupling serial/CAN I/O from
-         the control loop. Only meaningful on REAL hardware; gz_ros2_control is stepped
-         synchronously by the sim, so force sync (is_async=false) under Gazebo. -->
-    <xacro:property name="hw_is_async" value="${'false' if $(arg enable_gz) else 'true'}"/>
     <xacro:if value="${$(arg enable_mobile_base)}">
       <ros2_control name="dynamixel_control_lower" type="system">
@@ -125,10 +121,9 @@
     </xacro:if>
     <xacro:if value="${$(arg enable_body)}">
-      <ros2_control name="uirobot_control" type="system" is_async="${hw_is_async}">
-        <xacro:unless value="${$(arg enable_gz)}">
-          <properties>
-            <async scheduling_policy="synchronized" thread_priority="79" affinity="[6]" print_warnings="true"/>
-          </properties>
-        </xacro:unless>
+      <!-- <ros2_control name="uirobot_control" type="system"> -->
+      <ros2_control name="uirobot_control" type="system" is_async="true">
+        <properties>
+          <async scheduling_policy="synchronized" thread_priority="79" affinity="[6]" print_warnings="true"/>
+        </properties>
         <hardware>
           <xacro:if value="${$(arg enable_gz)}">
@@ -679,5 +674,5 @@
         <param name="id">51</param>
         <param name="control_mode">6</param>
-        <param name="Goal_Current">100</param>
+        <param name="Goal_Current">150</param>
         <param name="interface">ttl</param>
         <param name="Return_Delay_Time">0</param>
@@ -724,5 +719,5 @@
         <param name="id">53</param>
         <param name="control_mode">6</param>
-        <param name="Goal_Current">50</param>
+        <param name="Goal_Current">75</param>
         <param name="interface">ttl</param>
         <param name="Return_Delay_Time">0</param>
@@ -760,5 +755,5 @@
         <param name="id">55</param>
         <param name="control_mode">6</param>
-        <param name="Goal_Current">50</param>
+        <param name="Goal_Current">75</param>
         <param name="interface">ttl</param>
         <param name="Return_Delay_Time">0</param>
@@ -796,5 +791,5 @@
         <param name="id">57</param>
         <param name="control_mode">6</param>
-        <param name="Goal_Current">50</param>
+        <param name="Goal_Current">75</param>
         <param name="interface">ttl</param>
         <param name="Return_Delay_Time">0</param>
@@ -816,5 +811,5 @@
         <param name="id">61</param>
         <param name="control_mode">6</param>
-        <param name="Goal_Current">100</param>
+        <param name="Goal_Current">150</param>
         <param name="interface">ttl</param>
         <param name="Return_Delay_Time">0</param>
@@ -861,5 +856,5 @@
         <param name="id">63</param>
         <param name="control_mode">6</param>
-        <param name="Goal_Current">50</param>
+        <param name="Goal_Current">75</param>
         <param name="interface">ttl</param>
         <param name="Return_Delay_Time">0</param>
@@ -897,5 +892,5 @@
         <param name="id">65</param>
         <param name="control_mode">6</param>
-        <param name="Goal_Current">50</param>
+        <param name="Goal_Current">75</param>
         <param name="interface">ttl</param>
         <param name="Return_Delay_Time">0</param>
@@ -933,5 +928,5 @@
         <param name="id">67</param>
         <param name="control_mode">6</param>
-        <param name="Goal_Current">50</param>
+        <param name="Goal_Current">75</param>
         <param name="interface">ttl</param>
         <param name="Return_Delay_Time">0</param>
