Commit message: [FIX] widen the finger closing limits and reconcile the pose files
The gripper's closing joints reach 120 deg on the assembled hardware, but the
URDF carried the CAD assumption of pi/2. Every grasp and fist pose therefore
commanded past the declared limit -- harmless while nothing enforced it, but the
joint-limit clamp added in the Phase 2 branch now corrects those values, which
would weaken the grasp.

Widen only the joints that actually overshoot, and only on the side they
overshoot: finger_c_ip, finger_l_dip and finger_r_dip take FINGER_CLOSE
(120 deg) on their closing bound and keep pi/6 on the opening bound. The other
five finger joints keep their CAD limits, since no pose has ever asked them for
more. The ros2_control command ranges are widened to match, so the two
descriptions stay in agreement.

Pose values reconciled with the limits:
  - two_fingers_grasp_pose finger_c_ip: 2.1 -> 2.0943, just inside 120 deg
  - thirteen values that were decimal roundings of pi/2 (1.58, 1.6) or pi/6
    (0.53, 0.54, 0.60) now use 1.5707 and 0.5235. These sit marginally inside
    the bound on purpose: 1.5708 is above pi/2 at full precision.
  - move_pose arm_left_wrist_tilt: -1.58 -> -1.57, matching the right arm's
    value in the same pose

All three pose files now report zero out-of-range entries, and all 35 joints
with a position command interface agree with their URDF limits.

Verified in Gazebo: 0 errors, 9 controllers active, and fist_pose,
two_fingers_grasp_pose, two_fingers_pick_pose, three_fingers_pick_pose and
move_pose all succeed with no clamp warnings. two_fingers_grasp_pose still
drives hand_left_finger_c_ip_joint to 2.0943, so the closing travel is
preserved rather than clamped away. The xacro expands with hands enabled,
disabled and mixed.

The 120 deg figure comes from the hardware owner, not from a measurement made
here; the collision model now assumes these three joints reach further than CAD
stated, which is worth confirming on the real gripper.

Co-Authored-By: Claude Opus 5 (1M context) <noreply@anthropic.com>

File: sobit_home_description/urdf/controllers.urdf.xacro (robot description, xacro)
@@ -643,4 +643,22 @@
       </xacro:unless>
       <command_interface name="position">
+        <param name="min">${-FINGER_CLOSE}</param>
+        <param name="max">${M_PI/6}</param>
+      </command_interface>
+      <state_interface name="position">
+        <param name="initial_value">0.0</param>
+      </state_interface>
+      <state_interface name="velocity"/>
+      <state_interface name="effort"/>
+    </joint>
+    <joint name="${prefix}_finger_c_mcp_joint">
+      <xacro:unless value="${$(arg enable_gz)}">
+        <param name="id">54</param>
+        <param name="control_mode">6</param>
+        <param name="Goal_Current">50</param>
+        <param name="interface">ttl</param>
+        <param name="Return_Delay_Time">0</param>
+      </xacro:unless>
+      <command_interface name="position">
         <param name="min">${-M_PI/2}</param>
         <param name="max">${M_PI/6}</param>
@@ -652,7 +670,25 @@
       <state_interface name="effort"/>
     </joint>
-    <joint name="${prefix}_finger_c_mcp_joint">
-      <xacro:unless value="${$(arg enable_gz)}">
-        <param name="id">54</param>
+    <joint name="${prefix}_finger_c_ip_joint">
+      <xacro:unless value="${$(arg enable_gz)}">
+        <param name="id">55</param>
+        <param name="control_mode">6</param>
+        <param name="Goal_Current">75</param>
+        <param name="interface">ttl</param>
+        <param name="Return_Delay_Time">0</param>
+      </xacro:unless>
+      <command_interface name="position">
+        <param name="min">${-M_PI/6}</param>
+        <param name="max">${FINGER_CLOSE}</param>
+      </command_interface>
+      <state_interface name="position">
+        <param name="initial_value">0.0</param>
+      </state_interface>
+      <state_interface name="velocity"/>
+      <state_interface name="effort"/>
+    </joint>
+    <joint name="${prefix}_finger_r_pip_joint">
+      <xacro:unless value="${$(arg enable_gz)}">
+        <param name="id">56</param>
         <param name="control_mode">6</param>
         <param name="Goal_Current">50</param>
@@ -670,7 +706,7 @@
       <state_interface name="effort"/>
     </joint>
-    <joint name="${prefix}_finger_c_ip_joint">
-      <xacro:unless value="${$(arg enable_gz)}">
-        <param name="id">55</param>
+    <joint name="${prefix}_finger_r_dip_joint">
+      <xacro:unless value="${$(arg enable_gz)}">
+        <param name="id">57</param>
         <param name="control_mode">6</param>
         <param name="Goal_Current">75</param>
@@ -680,41 +716,5 @@
       <command_interface name="position">
         <param name="min">${-M_PI/6}</param>
-        <param name="max">${M_PI/2}</param>
-      </command_interface>
-      <state_interface name="position">
-        <param name="initial_value">0.0</param>
-      </state_interface>
-      <state_interface name="velocity"/>
-      <state_interface name="effort"/>
-    </joint>
-    <joint name="${prefix}_finger_r_pip_joint">
-      <xacro:unless value="${$(arg enable_gz)}">
-        <param name="id">56</param>
-        <param name="control_mode">6</param>
-        <param name="Goal_Current">50</param>
-        <param name="interface">ttl</param>
-        <param name="Return_Delay_Time">0</param>
-      </xacro:unless>
-      <command_interface name="position">
-        <param name="min">${-M_PI/2}</param>
-        <param name="max">${M_PI/6}</param>
-      </command_interface>
-      <state_interface name="position">
-        <param name="initial_value">0.0</param>
-      </state_interface>
-      <state_interface name="velocity"/>
-      <state_interface name="effort"/>
-    </joint>
-    <joint name="${prefix}_finger_r_dip_joint">
-      <xacro:unless value="${$(arg enable_gz)}">
-        <param name="id">57</param>
-        <param name="control_mode">6</param>
-        <param name="Goal_Current">75</param>
-        <param name="interface">ttl</param>
-        <param name="Return_Delay_Time">0</param>
-      </xacro:unless>
-      <command_interface name="position">
-        <param name="min">${-M_PI/6}</param>
-        <param name="max">${M_PI/2}</param>
+        <param name="max">${FINGER_CLOSE}</param>
       </command_interface>
       <state_interface name="position">
@@ -780,4 +780,58 @@
       </xacro:unless>
       <command_interface name="position">
+        <param name="min">${-FINGER_CLOSE}</param>
+        <param name="max">${M_PI/6}</param>
+      </command_interface>
+      <state_interface name="position">
+        <param name="initial_value">0.0</param>
+      </state_interface>
+      <state_interface name="velocity"/>
+      <state_interface name="effort"/>
+    </joint>
+    <joint name="${prefix}_finger_c_mcp_joint">
+      <xacro:unless value="${$(arg enable_gz)}">
+        <param name="id">64</param>
+        <param name="control_mode">6</param>
+        <param name="Goal_Current">50</param>
+        <param name="interface">ttl</param>
+        <param name="Return_Delay_Time">0</param>
+      </xacro:unless>
+      <command_interface name="position">
+        <param name="min">${-M_PI/6}</param>
+        <param name="max">${M_PI/2}</param>
+      </command_interface>
+      <state_interface name="position">
+        <param name="initial_value">0.0</param>
+      </state_interface>
+      <state_interface name="velocity"/>
+      <state_interface name="effort"/>
+    </joint>
+    <joint name="${prefix}_finger_c_ip_joint">
+      <xacro:unless value="${$(arg enable_gz)}">
+        <param name="id">65</param>
+        <param name="control_mode">6</param>
+        <param name="Goal_Current">75</param>
+        <param name="interface">ttl</param>
+        <param name="Return_Delay_Time">0</param>
+      </xacro:unless>
+      <command_interface name="position">
+        <param name="min">${-FINGER_CLOSE}</param>
+        <param name="max">${M_PI/6}</param>
+      </command_interface>
+      <state_interface name="position">
+        <param name="initial_value">0.0</param>
+      </state_interface>
+      <state_interface name="velocity"/>
+      <state_interface name="effort"/>
+    </joint>
+    <joint name="${prefix}_finger_r_pip_joint">
+      <xacro:unless value="${$(arg enable_gz)}">
+        <param name="id">66</param>
+        <param name="control_mode">6</param>
+        <param name="Goal_Current">50</param>
+        <param name="interface">ttl</param>
+        <param name="Return_Delay_Time">0</param>
+      </xacro:unless>
+      <command_interface name="position">
         <param name="min">${-M_PI/2}</param>
         <param name="max">${M_PI/6}</param>
@@ -789,9 +843,9 @@
       <state_interface name="effort"/>
     </joint>
-    <joint name="${prefix}_finger_c_mcp_joint">
-      <xacro:unless value="${$(arg enable_gz)}">
-        <param name="id">64</param>
-        <param name="control_mode">6</param>
-        <param name="Goal_Current">50</param>
+    <joint name="${prefix}_finger_r_dip_joint">
+      <xacro:unless value="${$(arg enable_gz)}">
+        <param name="id">67</param>
+        <param name="control_mode">6</param>
+        <param name="Goal_Current">75</param>
         <param name="interface">ttl</param>
         <param name="Return_Delay_Time">0</param>
@@ -799,59 +853,5 @@
       <command_interface name="position">
         <param name="min">${-M_PI/6}</param>
-        <param name="max">${M_PI/2}</param>
-      </command_interface>
-      <state_interface name="position">
-        <param name="initial_value">0.0</param>
-      </state_interface>
-      <state_interface name="velocity"/>
-      <state_interface name="effort"/>
-    </joint>
-    <joint name="${prefix}_finger_c_ip_joint">
-      <xacro:unless value="${$(arg enable_gz)}">
-        <param name="id">65</param>
-        <param name="control_mode">6</param>
-        <param name="Goal_Current">75</param>
-        <param name="interface">ttl</param>
-        <param name="Return_Delay_Time">0</param>
-      </xacro:unless>
-      <command_interface name="position">
-        <param name="min">${-M_PI/2}</param>
-        <param name="max">${M_PI/6}</param>
-      </command_interface>
-      <state_interface name="position">
-        <param name="initial_value">0.0</param>
-      </state_interface>
-      <state_interface name="velocity"/>
-      <state_interface name="effort"/>
-    </joint>
-    <joint name="${prefix}_finger_r_pip_joint">
-      <xacro:unless value="${$(arg enable_gz)}">
-        <param name="id">66</param>
-        <param name="control_mode">6</param>
-        <param name="Goal_Current">50</param>
-        <param name="interface">ttl</param>
-        <param name="Return_Delay_Time">0</param>
-      </xacro:unless>
-      <command_interface name="position">
-        <param name="min">${-M_PI/2}</param>
-        <param name="max">${M_PI/6}</param>
-      </command_interface>
-      <state_interface name="position">
-        <param name="initial_value">0.0</param>
-      </state_interface>
-      <state_interface name="velocity"/>
-      <state_interface name="effort"/>
-    </joint>
-    <joint name="${prefix}_finger_r_dip_joint">
-      <xacro:unless value="${$(arg enable_gz)}">
-        <param name="id">67</param>
-        <param name="control_mode">6</param>
-        <param name="Goal_Current">75</param>
-        <param name="interface">ttl</param>
-        <param name="Return_Delay_Time">0</param>
-      </xacro:unless>
-      <command_interface name="position">
-        <param name="min">${-M_PI/6}</param>
-        <param name="max">${M_PI/2}</param>
+        <param name="max">${FINGER_CLOSE}</param>
       </command_interface>
       <state_interface name="position">

File: sobit_home_description/urdf/hand/hand.urdf.xacro (robot description, xacro)
@@ -3,4 +3,7 @@
        xmlns:xacro="http://ros.org/wiki/xacro" >
   <xacro:include filename="$(find sobit_home_description)/urdf/hand/hand.transmission.xacro" />
+  <!-- Closing travel measured on the assembled gripper: the c_ip and dip joints
+       reach 120 deg, past the pi/2 the CAD model assumed. -->
+  <xacro:property name="FINGER_CLOSE" value="${radians(120)}" />
   <xacro:macro name="hand" params="prefix_hand position prefix_finger parent" >
     <xacro:if value="${position == 'left'}">
@@ -99,5 +102,5 @@
       <origin xyz="0.0 ${y_sign * 0.050} 0.0" rpy="0.0 0.0 0.0" />
       <axis xyz="1.0 0.0 0.0 " />
-      <limit lower="${-M_PI/2}" upper="${M_PI/6}" effort="${0.52 * effort_ratio}" velocity="11.031179004" />
+      <limit lower="${-FINGER_CLOSE}" upper="${M_PI/6}" effort="${0.52 * effort_ratio}" velocity="11.031179004" />
     </joint>
     <link name="${prefix_hand}_${position}_${prefix_finger}_l_dip_link" >
@@ -188,5 +191,5 @@
       <origin xyz="0.0 ${y_sign * 0.050} 0.0" rpy="0.0 0.0 0.0" />
       <axis xyz="1.0 0.0 0.0 " />
-      <limit lower="${-M_PI/6}" upper="${M_PI/2}" effort="${0.52 * effort_ratio}" velocity="11.031179004" />
+      <limit lower="${-M_PI/6}" upper="${FINGER_CLOSE}" effort="${0.52 * effort_ratio}" velocity="11.031179004" />
     </joint>
     <link name="${prefix_hand}_${position}_${prefix_finger}_r_dip_link" >
@@ -258,8 +261,8 @@
       <axis xyz="0.0 0.0 1.0 " />
       <xacro:if value="${position == 'right'}">
-        <limit lower="${-M_PI/2}" upper="${M_PI/6}" effort="${0.52 * effort_ratio}" velocity="11.031" />
+        <limit lower="${-FINGER_CLOSE}" upper="${M_PI/6}" effort="${0.52 * effort_ratio}" velocity="11.031" />
       </xacro:if>
       <xacro:if value="${position == 'left'}">
-        <limit lower="${-M_PI/6}" upper="${M_PI/2}" effort="${0.52 * effort_ratio}" velocity="11.031" />
+        <limit lower="${-M_PI/6}" upper="${FINGER_CLOSE}" effort="${0.52 * effort_ratio}" velocity="11.031" />
       </xacro:if>
     </joint>
