Commit message: Restore hw_is_async property dropped by the jazzy-devel merge
The merge of jazzy-devel's Goal_Current adjustment (64835f8) in 2520b1d
silently dropped the hw_is_async xacro:property definition while leaving
its usage on uirobot_control's is_async attribute intact -- jazzy-devel
never had this property (it was only ever added on this branch, via
5f9a929), so the 3-way merge resolved that hunk by discarding it.

The result was a dangling ${hw_is_async} reference with nothing defining
it, which xacro cannot process. Restored the property and its original
comment verbatim; verified xacro expands the full robot description
cleanly again.

File: sobit_home_description/urdf/controllers.urdf.xacro (robot description, xacro)
@@ -3,4 +3,8 @@
 <robot name="sobit_home_controllers" xmlns:xacro="http://www.ros.org/wiki/xacro">
   <xacro:macro name="controllers" params="enable_gz:=False robot_name:=sobit_home">
+    <!-- Async hardware = separate read/write thread, decoupling serial/CAN I/O from
+         the control loop. Only meaningful on REAL hardware; gz_ros2_control is stepped
+         synchronously by the sim, so force sync (is_async=false) under Gazebo. -->
+    <xacro:property name="hw_is_async" value="${'false' if $(arg enable_gz) else 'true'}"/>
     <xacro:if value="${$(arg enable_mobile_base)}">
       <!-- <ros2_control name="dynamixel_control_lower" type="system"> -->

Commit message: Retune the swerve drive loop and add a cmd_vel watchdog
Drive loop (M3508 via rm_wheel_drive_controllers):
- Hoist the per-wheel gains into shared xacro properties and change them
  from kp 0.75 / ki 1.0 / kd 0.001 to kp 0.5 / ki 3.0 / kd 0.
- Expose velocity_i_decay_tau, velocity_lpf_hz and max_current per wheel.

Steering (Dynamixel): set Position_I_Gain to 100 on all four steer servos
to remove the load-dependent holding error (servo default is 0).

swerve_controller_main:
- Add a cmd_vel_timeout parameter (0.5 s) that forces STOP when no Twist
  has arrived, so a dead publisher cannot leave the base driving.
- Warn (throttled) when the steering gate discards a non-zero drive
  request, naming the worst steer joint and its error.

Add scripts/base_step_test.py, a bounded straight-line / pure-rotation
step test that logs odom, wheel commands and joint states for analysis.

File: sobit_home_description/urdf/controllers.urdf.xacro (robot description, xacro)
@@ -181,4 +181,11 @@
     </xacro:if>
   </xacro:macro>
+  <!-- Drive-loop tuning, shared by all four rm_wheel_drive_controllers joints -->
+  <xacro:property name="rm_drive_velocity_kp" value="0.5"/>
+  <xacro:property name="rm_drive_velocity_ki" value="3.0"/>
+  <xacro:property name="rm_drive_velocity_kd" value="0.0"/>
+  <xacro:property name="rm_drive_velocity_i_decay_tau" value="0.15"/>
+  <xacro:property name="rm_drive_velocity_lpf_hz" value="0.0"/>
+  <xacro:property name="rm_drive_max_current" value="10.0"/>
   <xacro:macro name="rm_wheel_drive_controllers"  params="prefix enable_gz:=False">
     <joint name="${prefix}_drive_f_l_joint">
@@ -186,7 +193,10 @@
       <param name="motor_type">m3508</param>
       <param name="invert_rotation">true</param>
-      <param name="velocity_kp">0.75</param>
-      <param name="velocity_ki">1.0</param>
-      <param name="velocity_kd">0.001</param>
+      <param name="velocity_kp">${rm_drive_velocity_kp}</param>
+      <param name="velocity_ki">${rm_drive_velocity_ki}</param>
+      <param name="velocity_kd">${rm_drive_velocity_kd}</param>
+      <param name="velocity_i_decay_tau">${rm_drive_velocity_i_decay_tau}</param>
+      <param name="velocity_lpf_hz">${rm_drive_velocity_lpf_hz}</param>
+      <param name="max_current">${rm_drive_max_current}</param>
       <command_interface name="velocity">
         <param name="min">-10</param>
@@ -202,7 +212,10 @@
       <param name="motor_type">m3508</param>
       <param name="invert_rotation">false</param>
-      <param name="velocity_kp">0.75</param>
-      <param name="velocity_ki">1.0</param>
-      <param name="velocity_kd">0.001</param>
+      <param name="velocity_kp">${rm_drive_velocity_kp}</param>
+      <param name="velocity_ki">${rm_drive_velocity_ki}</param>
+      <param name="velocity_kd">${rm_drive_velocity_kd}</param>
+      <param name="velocity_i_decay_tau">${rm_drive_velocity_i_decay_tau}</param>
+      <param name="velocity_lpf_hz">${rm_drive_velocity_lpf_hz}</param>
+      <param name="max_current">${rm_drive_max_current}</param>
       <command_interface name="velocity">
         <param name="min">-10</param>
@@ -218,7 +231,10 @@
       <param name="motor_type">m3508</param>
       <param name="invert_rotation">true</param>
-      <param name="velocity_kp">0.75</param>
-      <param name="velocity_ki">1.0</param>
-      <param name="velocity_kd">0.001</param>
+      <param name="velocity_kp">${rm_drive_velocity_kp}</param>
+      <param name="velocity_ki">${rm_drive_velocity_ki}</param>
+      <param name="velocity_kd">${rm_drive_velocity_kd}</param>
+      <param name="velocity_i_decay_tau">${rm_drive_velocity_i_decay_tau}</param>
+      <param name="velocity_lpf_hz">${rm_drive_velocity_lpf_hz}</param>
+      <param name="max_current">${rm_drive_max_current}</param>
       <command_interface name="velocity">
         <param name="min">-10</param>
@@ -234,7 +250,10 @@
       <param name="motor_type">m3508</param>
       <param name="invert_rotation">false</param>
-      <param name="velocity_kp">0.75</param>
-      <param name="velocity_ki">1.0</param>
-      <param name="velocity_kd">0.001</param>
+      <param name="velocity_kp">${rm_drive_velocity_kp}</param>
+      <param name="velocity_ki">${rm_drive_velocity_ki}</param>
+      <param name="velocity_kd">${rm_drive_velocity_kd}</param>
+      <param name="velocity_i_decay_tau">${rm_drive_velocity_i_decay_tau}</param>
+      <param name="velocity_lpf_hz">${rm_drive_velocity_lpf_hz}</param>
+      <param name="max_current">${rm_drive_max_current}</param>
       <command_interface name="velocity">
         <param name="min">-10</param>
@@ -247,4 +266,6 @@
     </joint>
   </xacro:macro>
+    <!-- Steer servo integral gain: removes the load-dependent holding error (servo default is 0) -->
+  <xacro:property name="dxl_steer_position_i_gain" value="100"/>
   <xacro:macro name="dxl_wheel_steer_controllers"  params="prefix enable_gz:=False">
     <joint name="${prefix}_steer_f_l_joint">
@@ -254,4 +275,5 @@
         <param name="interface">rs</param>
         <param name="Return_Delay_Time">0</param>
+        <param name="Position_I_Gain">${dxl_steer_position_i_gain}</param>
       </xacro:unless>
       <command_interface name="position">
@@ -271,4 +293,5 @@
         <param name="interface">rs</param>
         <param name="Return_Delay_Time">0</param>
+        <param name="Position_I_Gain">${dxl_steer_position_i_gain}</param>
       </xacro:unless>
       <command_interface name="position">
@@ -288,4 +311,5 @@
         <param name="interface">rs</param>
         <param name="Return_Delay_Time">0</param>
+        <param name="Position_I_Gain">${dxl_steer_position_i_gain}</param>
       </xacro:unless>
       <command_interface name="position">
@@ -305,4 +329,5 @@
         <param name="interface">rs</param>
         <param name="Return_Delay_Time">0</param>
+        <param name="Position_I_Gain">${dxl_steer_position_i_gain}</param>
       </xacro:unless>
       <command_interface name="position">
