Commit message: [ADD] body_joint

File: sobit_home_description/robots/sobit_home_robot.urdf.xacro (robot description, xacro)
@@ -9,5 +9,5 @@
   <xacro:include filename="$(find sobit_home_description)/urdf/base/base.urdf.xacro" />
   <xacro:include filename="$(find sobit_home_description)/urdf/body/plate.urdf.xacro" />
-  <xacro:include filename="$(find sobit_home_description)/urdf/body/cover.urdf.xacro" />
+  <xacro:include filename="$(find sobit_home_description)/urdf/body/body.urdf.xacro" />
   <xacro:include filename="$(find sobit_home_description)/urdf/back/back.urdf.xacro" />
   <xacro:include filename="$(find sobit_home_description)/urdf/wheel/wheel.urdf.xacro" />
@@ -92,5 +92,5 @@
     <xacro:plate prefix="plate" parent="base_link" />
     <xacro:wheel prefix="wheel" parent="plate_middle_link" />
-    <!-- <xacro:cover prefix="cover" parent="plate_top_link" /> -->
+    <xacro:body  prefix="body"  parent="plate_top_link" />
     <xacro:lidar prefix="lidar" parent="plate_middle_link" />
   </xacro:if>

File: sobit_home_description/urdf/body/body.urdf.xacro (robot description, xacro)
@@ -2,7 +2,7 @@
 <robot name="sobit_home"
        xmlns:xacro="http://ros.org/wiki/xacro" >
-  <xacro:macro name="cover" params="prefix parent" >
+  <xacro:macro name="body" params="prefix parent" >
     <joint name="${prefix}_joint" type="fixed" >
-      <origin xyz="0.179108 0.0 -0.034" rpy="0.0 0.0 0.0" />
+      <origin xyz="0.0 0.0 0.0" rpy="0.0 0.0 0.0" />
       <parent link="${parent}" />
       <child link="${prefix}_link" />
@@ -10,9 +10,9 @@
     <link name="${prefix}_link" >
       <visual>
-        <origin xyz="0.0 0.0 0.0" rpy="${M_PI/2} 0.0 ${M_PI/2}" />
+        <origin xyz="0.0 0.0 0.565" rpy="0.0 0.0 ${M_PI}" />
         <geometry>
-          <mesh filename="file://$(find sobit_home_description)/meshes/body/cover.stl" scale="0.001 0.001 0.001" />
+          <mesh filename="file://$(find sobit_home_description)/meshes/body/linear_actuator.stl" scale="0.001 0.001 0.001" />
         </geometry>
-        <material name="blue" />
+        <material name="grey" />
       </visual>
       <collision>

File: sobit_home_description/urdf/wheel/wheel.urdf.xacro (robot description, xacro)
@@ -38,4 +38,5 @@
       <child link="wheel_steer_${id}_link" />
       <axis xyz="0.0 0.0 1.0 " />
+      <limit effort="3.0" velocity="0.5" />
       <!-- <dynamics damping="0.2" friction="0" /> -->
     </joint>

Commit message: [ADD] mic&head_camera

File: sobit_home_description/robots/sobit_home_robot.urdf.xacro (robot description, xacro)
@@ -16,4 +16,5 @@
   <xacro:include filename="$(find sobit_home_description)/urdf/hand/hand.urdf.xacro" />
   <xacro:include filename="$(find sobit_home_description)/urdf/head/head.urdf.xacro" />
+  <xacro:include filename="$(find sobit_home_description)/urdf/sensor/camera_head.urdf.xacro" />
   <xacro:include filename="$(find sobit_home_description)/urdf/sensor/azure_camera.urdf.xacro" />
   <xacro:include filename="$(find sobit_home_description)/urdf/sensor/matrix.urdf.xacro" />
@@ -53,5 +54,6 @@
     <!-- <xacro:hand  prefix_hand="hand" prefix_finger="finger" parent="arm_wrist_tilt_link" /> -->
     <xacro:head  prefix="head"  parent="linear_actuator_link" />
-    <!-- <xacro:mic  prefix="mic"  parent="head_tilt_link" />  -->
+    <xacro:camera_head  prefix="head_camera"  parent="head_tilt_link" />
+    <xacro:mic  prefix="mic"  parent="head_tilt_link" />
   </xacro:if>
   <!-- enable_mb: true, enable_arm: true, enable_head: false -->

File: sobit_home_description/urdf/sensor/mic.urdf.xacro (robot description, xacro)
@@ -6,9 +6,9 @@
       <parent link="${parent}" />
       <child link="${prefix}_base_link" />
-      <origin xyz="0.0 0.0 0.5400" rpy="0.0 0.0 0.0" />
+      <origin xyz="-0.042 0.0 0.082" rpy="0.0 -${M_PI/9.0} 0.0" />
     </joint>
     <link name="${prefix}_base_link">
       <visual>
-        <origin xyz="0.0 0.0 0.0" rpy="${M_PI/2} 0.0 ${M_PI}" />
+        <origin xyz="0.0 0.0 0.0" rpy="0.0 0.0 ${M_PI/2.0}" />
         <geometry>
           <mesh filename="file://$(find sobit_home_description)/meshes/sensor/mic_base.stl" scale="0.001 0.001 0.001" />
@@ -35,9 +35,9 @@
       <parent link="${prefix}_base_link" />
       <child link="${prefix}_link" />
-      <origin xyz="0.0 -0.099 0.0240" rpy="0.0 0.0 0.0" />
+      <origin xyz="0.0 0.0 0.005" rpy="0.0 0.0 0.0" />
     </joint>
     <link name="${prefix}_link">
       <visual>
-        <origin xyz="0.0 0.0 0.0" rpy="${M_PI/2} 0.0 ${M_PI}" />
+        <origin xyz="0.0 0.0 0.0" rpy="0.0 0.0 ${M_PI/2.0}" />
         <geometry>
           <mesh filename="file://$(find sobit_home_description)/meshes/sensor/mic.stl" scale="0.001 0.001 0.001" />

Commit message: [ADD]  linear actuator controllers

File: sobit_home_description/robots/sobit_home_robot.urdf.xacro (robot description, xacro)
@@ -42,4 +42,6 @@
   <!-- <xacro:controllers_DxUpper name="joints_control_upper" enable_gz="$(arg enable_gz)" robot_name="$(arg robot_name)" /> -->
   <xacro:wheel_controllers name="wheel" enable_gz="$(arg enable_gz)" robot_name="$(arg robot_name)" />
+  <xacro:linear_actuator_controllers name="linear_actuator" enable_gz="$(arg enable_gz)" robot_name="$(arg robot_name)" />
+  <xacro:ros2_controllers enable_gz="$(arg enable_gz)" robot_name="$(arg robot_name)" />
   <!-- enable_mb: true, enable_arm: true, enable_head: true -->
   <xacro:if value="${$(arg enable_mb) and $(arg enable_arm) and $(arg enable_head)}">

File: sobit_home_description/urdf/controllers.urdf.xacro (robot description, xacro)
@@ -2,5 +2,5 @@
 <!-- SOBIT home (Dynamixel Control) -->
 <robot name="sobit_home_controllers" xmlns:xacro="http://www.ros.org/wiki/xacro">
-  <xacro:macro name="wheel_controllers" params="name enable_gz:=False robot_name:=sobit_pro">
+  <xacro:macro name="wheel_controllers" params="name enable_gz:=False robot_name:=sobit_home">
     <ros2_control name="${name}_steer_control" type="system">
       <hardware>
@@ -143,4 +143,37 @@
       </joint>
     </ros2_control>
+  </xacro:macro>
+  <xacro:macro name="linear_actuator_controllers" params="name enable_gz:=False robot_name:=sobit_home">
+    <ros2_control name="${name}_position_control" type="system">
+      <hardware>
+        <xacro:if value="${$(arg enable_gz)}">
+          <plugin>gz_ros2_control/GazeboSimSystem</plugin>
+        </xacro:if>
+        <xacro:unless value="${$(arg enable_gz)}">
+          <plugin>dynamixel_hardware/DynamixelHardware</plugin>
+          <param name="port_name">/dev/ttyUSB0</param>
+          <param name="baud_rate">1000000</param>
+        </xacro:unless>
+      </hardware>
+      <joint name="${name}_joint">
+        <xacro:unless value="${$(arg enable_gz)}">
+          <param name="id">20</param>
+          <param name="control_mode">3</param>
+          <param name="interface">rp</param>
+        </xacro:unless>
+        <command_interface name="position">
+          <param name="min">-0.4</param>
+          <param name="max">0.4</param>
+        </command_interface>
+        <!-- <command_interface name="velocity"/> -->
+        <state_interface name="position">
+          <param name="initial_value">0.0</param>
+        </state_interface>
+        <state_interface name="velocity"/>
+        <state_interface name="effort"/>
+      </joint>
+    </ros2_control>
+  </xacro:macro>
+  <xacro:macro name="ros2_controllers" params="enable_gz:=False robot_name:=sobit_home">
     <!-- Gazebo Sim ROS2 Control -->
     <xacro:if value="${$(arg enable_gz)}">
@@ -150,5 +183,5 @@
             <namespace>${robot_name}</namespace>
           </ros>
-          <parameters>$(find sobit_home_control)/config/gz_controllers.yaml</parameters>
+          <parameters>$(find ${robot_name}_control)/config/gz_controllers.yaml</parameters>
         </plugin>
       </gazebo>

Commit message: [UPD] head & arm ros control

File: sobit_home_description/robots/sobit_home_robot.urdf.xacro (robot description, xacro)
@@ -43,4 +43,6 @@
   <!-- <xacro:controllers_DxUpper name="joints_control_upper" enable_gz="$(arg enable_gz)" robot_name="$(arg robot_name)" /> -->
   <xacro:wheel_controllers name="wheel" enable_gz="$(arg enable_gz)" robot_name="$(arg robot_name)" />
+  <xacro:joint_controllers name="joint" enable_gz="$(arg enable_gz)" robot_name="$(arg robot_name)" />
+  <xacro:ros2_controllers enable_gz="$(arg enable_gz)" robot_name="$(arg robot_name)" />
   <!-- enable_mb: true, enable_arm: true, enable_head: true -->
   <xacro:if value="${$(arg enable_mb) and $(arg enable_arm) and $(arg enable_head)}">

File: sobit_home_description/urdf/body/body.urdf.xacro (robot description, xacro)
@@ -36,5 +36,5 @@
       <child link="linear_actuator_link" />
       <axis xyz="0.0 0.0 1.0" />
-      <limit lower="-0.4" upper="0.4" effort="50.0" velocity="0.1" />
+      <limit lower="-0.4" upper="0.4" effort="150.0" velocity="0.1" />
     </joint>
     <link name="linear_actuator_link" >

File: sobit_home_description/urdf/controllers.urdf.xacro (robot description, xacro)
@@ -2,5 +2,5 @@
 <!-- SOBIT home (Dynamixel Control) -->
 <robot name="sobit_home_controllers" xmlns:xacro="http://www.ros.org/wiki/xacro">
-  <xacro:macro name="wheel_controllers" params="name enable_gz:=False robot_name:=sobit_pro">
+  <xacro:macro name="wheel_controllers" params="name enable_gz:=False robot_name:=sobit_home">
     <ros2_control name="${name}_steer_control" type="system">
       <hardware>
@@ -143,4 +143,241 @@
       </joint>
     </ros2_control>
+  </xacro:macro>
+  <xacro:macro name="joint_controllers" params="name enable_gz:=False robot_name:=sobit_home">
+    <ros2_control name="${name}_position_control" type="system">
+      <hardware>
+        <xacro:if value="${$(arg enable_gz)}">
+          <plugin>gz_ros2_control/GazeboSimSystem</plugin>
+        </xacro:if>
+        <xacro:unless value="${$(arg enable_gz)}">
+          <plugin>dynamixel_hardware/DynamixelHardware</plugin>
+          <param name="port_name">/dev/ttyUSB0</param>
+          <param name="baud_rate">1000000</param>
+        </xacro:unless>
+      </hardware>
+      <joint name="arm_left_shoulder_tilt_joint">
+        <xacro:unless value="${$(arg enable_gz)}">
+          <param name="id">20</param>
+          <param name="control_mode">3</param>
+          <param name="interface">rp</param>
+        </xacro:unless>
+        <command_interface name="position">
+          <param name="min">-0.4</param>
+          <param name="max">0.4</param>
+        </command_interface>
+        <!-- <command_interface name="velocity"/> -->
+        <state_interface name="position">
+          <param name="initial_value">0.0</param>
+        </state_interface>
+        <state_interface name="velocity"/>
+        <state_interface name="effort"/>
+      </joint>
+      <joint name="arm_left_upper_roll_joint">
+        <xacro:unless value="${$(arg enable_gz)}">
+          <param name="id">21</param>
+          <param name="control_mode">3</param>
+          <param name="interface">rp</param>
+        </xacro:unless>
+        <command_interface name="position">
+          <param name="min">-0.4</param>
+          <param name="max">0.4</param>
+        </command_interface>
+        <!-- <command_interface name="velocity"/> -->
+        <state_interface name="position">
+          <param name="initial_value">0.0</param>
+        </state_interface>
+        <state_interface name="velocity"/>
+        <state_interface name="effort"/>
+      </joint>
+      <joint name="arm_left_upper_flex_joint">
+        <xacro:unless value="${$(arg enable_gz)}">
+          <param name="id">21</param>
+          <param name="control_mode">3</param>
+          <param name="interface">rp</param>
+        </xacro:unless>
+        <command_interface name="position">
+          <param name="min">-0.4</param>
+          <param name="max">0.4</param>
+        </command_interface>
+        <!-- <command_interface name="velocity"/> -->
+        <state_interface name="position">
+          <param name="initial_value">0.0</param>
+        </state_interface>
+        <state_interface name="velocity"/>
+        <state_interface name="effort"/>
+      </joint>
+      <joint name="arm_left_elbow_joint">
+        <xacro:unless value="${$(arg enable_gz)}">
+          <param name="id">21</param>
+          <param name="control_mode">3</param>
+          <param name="interface">rp</param>
+        </xacro:unless>
+        <command_interface name="position">
+          <param name="min">-0.4</param>
+          <param name="max">0.4</param>
+        </command_interface>
+        <!-- <command_interface name="velocity"/> -->
+        <state_interface name="position">
+          <param name="initial_value">0.0</param>
+        </state_interface>
+        <state_interface name="velocity"/>
+        <state_interface name="effort"/>
+      </joint>
+      <joint name="arm_left_wrist_joint">
+        <xacro:unless value="${$(arg enable_gz)}">
+          <param name="id">21</param>
+          <param name="control_mode">3</param>
+          <param name="interface">rp</param>
+        </xacro:unless>
+        <command_interface name="position">
+          <param name="min">-0.4</param>
+          <param name="max">0.4</param>
+        </command_interface>
+        <!-- <command_interface name="velocity"/> -->
+        <state_interface name="position">
+          <param name="initial_value">0.0</param>
+        </state_interface>
+        <state_interface name="velocity"/>
+        <state_interface name="effort"/>
+      </joint>
+      <joint name="arm_right_shoulder_tilt_joint">
+        <xacro:unless value="${$(arg enable_gz)}">
+          <param name="id">20</param>
+          <param name="control_mode">3</param>
+          <param name="interface">rp</param>
+        </xacro:unless>
+        <command_interface name="position">
+          <param name="min">-0.4</param>
+          <param name="max">0.4</param>
+        </command_interface>
+        <!-- <command_interface name="velocity"/> -->
+        <state_interface name="position">
+          <param name="initial_value">0.0</param>
+        </state_interface>
+        <state_interface name="velocity"/>
+        <state_interface name="effort"/>
+      </joint>
+      <joint name="arm_right_upper_roll_joint">
+        <xacro:unless value="${$(arg enable_gz)}">
+          <param name="id">21</param>
+          <param name="control_mode">3</param>
+          <param name="interface">rp</param>
+        </xacro:unless>
+        <command_interface name="position">
+          <param name="min">-0.4</param>
+          <param name="max">0.4</param>
+        </command_interface>
+        <!-- <command_interface name="velocity"/> -->
+        <state_interface name="position">
+          <param name="initial_value">0.0</param>
+        </state_interface>
+        <state_interface name="velocity"/>
+        <state_interface name="effort"/>
+      </joint>
+      <joint name="arm_right_upper_flex_joint">
+        <xacro:unless value="${$(arg enable_gz)}">
+          <param name="id">21</param>
+          <param name="control_mode">3</param>
+          <param name="interface">rp</param>
+        </xacro:unless>
+        <command_interface name="position">
+          <param name="min">-0.4</param>
+          <param name="max">0.4</param>
+        </command_interface>
+        <!-- <command_interface name="velocity"/> -->
+        <state_interface name="position">
+          <param name="initial_value">0.0</param>
+        </state_interface>
+        <state_interface name="velocity"/>
+        <state_interface name="effort"/>
+      </joint>
+      <joint name="arm_right_elbow_joint">
+        <xacro:unless value="${$(arg enable_gz)}">
+          <param name="id">21</param>
+          <param name="control_mode">3</param>
+          <param name="interface">rp</param>
+        </xacro:unless>
+        <command_interface name="position">
+          <param name="min">-0.4</param>
+          <param name="max">0.4</param>
+        </command_interface>
+        <!-- <command_interface name="velocity"/> -->
+        <state_interface name="position">
+          <param name="initial_value">0.0</param>
+        </state_interface>
+        <state_interface name="velocity"/>
+        <state_interface name="effort"/>
+      </joint>
+      <joint name="arm_right_wrist_joint">
+        <xacro:unless value="${$(arg enable_gz)}">
+          <param name="id">21</param>
+          <param name="control_mode">3</param>
+          <param name="interface">rp</param>
+        </xacro:unless>
+        <command_interface name="position">
+          <param name="min">-0.4</param>
+          <param name="max">0.4</param>
+        </command_interface>
+        <!-- <command_interface name="velocity"/> -->
+        <state_interface name="position">
+          <param name="initial_value">0.0</param>
+        </state_interface>
+        <state_interface name="velocity"/>
+        <state_interface name="effort"/>
+      </joint>
+      <joint name="head_pan_joint">
+        <xacro:unless value="${$(arg enable_gz)}">
+          <param name="id">21</param>
+          <param name="control_mode">3</param>
+          <param name="interface">rp</param>
+        </xacro:unless>
+        <command_interface name="position">
+          <param name="min">-0.4</param>
+          <param name="max">0.4</param>
+        </command_interface>
+        <!-- <command_interface name="velocity"/> -->
+        <state_interface name="position">
+          <param name="initial_value">0.0</param>
+        </state_interface>
+        <state_interface name="velocity"/>
+        <state_interface name="effort"/>
+      </joint>
+      <joint name="head_tilt_joint">
+        <xacro:unless value="${$(arg enable_gz)}">
+          <param name="id">21</param>
+          <param name="control_mode">3</param>
+          <param name="interface">rp</param>
+        </xacro:unless>
+        <command_interface name="position">
+          <param name="min">-0.4</param>
+          <param name="max">0.4</param>
+        </command_interface>
+        <!-- <command_interface name="velocity"/> -->
+        <state_interface name="position">
+          <param name="initial_value">0.0</param>
+        </state_interface>
+        <state_interface name="velocity"/>
+        <state_interface name="effort"/>
+      </joint>
+      <joint name="linear_actuator_joint">
+        <xacro:unless value="${$(arg enable_gz)}">
+          <param name="id">20</param>
+          <param name="control_mode">3</param>
+          <param name="interface">rp</param>
+        </xacro:unless>
+        <command_interface name="position">
+          <param name="min">-0.4</param>
+          <param name="max">0.4</param>
+        </command_interface>
+        <!-- <command_interface name="velocity"/> -->
+        <state_interface name="position">
+          <param name="initial_value">0.0</param>
+        </state_interface>
+        <state_interface name="velocity"/>
+        <state_interface name="effort"/>
+      </joint>
+    </ros2_control>
+  </xacro:macro>
+  <xacro:macro name="ros2_controllers" params="enable_gz:=False robot_name:=sobit_home">
     <!-- Gazebo Sim ROS2 Control -->
     <xacro:if value="${$(arg enable_gz)}">
@@ -150,5 +387,5 @@
             <namespace>${robot_name}</namespace>
           </ros>
-          <parameters>$(find sobit_home_control)/config/gz_controllers.yaml</parameters>
+          <parameters>$(find ${robot_name}_control)/config/gz_controllers.yaml</parameters>
         </plugin>
       </gazebo>
