Commit message: add hand parts

File: sobit_home_description/robots/sobit_home_robot.urdf.xacro (robot description, xacro)
@@ -56,8 +56,8 @@
   </xacro:if>
   <xacro:if value="${ $(arg enable_hand_left) }">
-    <xacro:hand  prefix_hand="hand" position="left"  prefix_finger="finger" parent="arm_wrist_tilt_link" />
+    <xacro:hand  prefix_hand="hand" position="left" prefix_finger="finger" parent="arm_left_wrist_roll_link" />
   </xacro:if>
   <xacro:if value="${ $(arg enable_hand_right) }">
-    <xacro:hand  prefix_hand="hand" position="right" prefix_finger="finger" parent="arm_wrist_tilt_link" />
+    <xacro:hand  prefix_hand="hand" position="right" prefix_finger="finger" parent="arm_right_wrist_roll_link" />
   </xacro:if>
   <xacro:if value="${ $(arg enable_head) }">

File: sobit_home_description/urdf/arm/arm.transmission.xacro (robot description, xacro)
@@ -7,5 +7,6 @@
     <xacro:SimpleTransmissionPosition joint="${prefix}_${position}_uppder_flex_joint"    reduction="1" />
     <xacro:SimpleTransmissionPosition joint="${prefix}_${position}_elbow_joint"          reduction="1" />
-    <xacro:SimpleTransmissionPosition joint="${prefix}_${position}_wrist_joint"          reduction="1" />
+    <xacro:SimpleTransmissionPosition joint="${prefix}_${position}_wrist_tilt_joint"     reduction="1" />
+    <xacro:SimpleTransmissionPosition joint="${prefix}_${position}_wrist_roll_joint"     reduction="1" />
   </xacro:macro>
 </robot>

File: sobit_home_description/urdf/arm/arm.urdf.xacro (robot description, xacro)
@@ -102,5 +102,5 @@
       </inertial>
     </link>
-    <!-- <joint name="${prefix}_${position}_upper_flex_joint" type="revolute" >
+    <joint name="${prefix}_${position}_upper_flex_joint" type="revolute" >
       <parent link="${prefix}_${position}_upper_roll_link" />
       <child link="${prefix}_${position}_upper_flex_link" />
@@ -160,12 +160,12 @@
       </inertial>
     </link>
-    <joint name="${prefix}_${position}_wrist_joint" type="revolute" >
+    <joint name="${prefix}_${position}_wrist_tilt_joint" type="revolute" >
       <parent link="${prefix}_${position}_elbow_link" />
-      <child link="${prefix}_${position}_wrist_link" />
+      <child link="${prefix}_${position}_wrist_tilt_link" />
       <origin xyz="0.0 0.0 -0.5" rpy="0.0 0.0 0.0" />
       <axis xyz="0.0 -1.0 0.0 " />
       <limit lower="${-M_PI/2}" upper="${M_PI/2}" effort="${10.6*2}" velocity="11.031179004" />
     </joint>
-    <link name="${prefix}_${position}_wrist_link" >
+    <link name="${prefix}_${position}_wrist_tilt_link" >
       <visual>
         <origin xyz="0.0 0.0 0.0" rpy="0.0 0.0 ${M_PI/2}" />
@@ -188,5 +188,35 @@
                  izz="${1/12*0.08*(0.1166**2+0.124**2)}" />
       </inertial>
-    </link> -->
+    </link>
+    <joint name="${prefix}_${position}_wrist_roll_joint" type="revolute" >
+      <parent link="${prefix}_${position}_wrist_tilt_link" />
+      <child link="${prefix}_${position}_wrist_roll_link" />
+      <origin xyz="0.0 0.0 -0.06648176" rpy="0.0 0.0 0.0" />
+      <axis xyz="0.0 0.0 1.0 " />
+      <limit lower="${-M_PI/2}" upper="${M_PI/2}" effort="${10.6*2}" velocity="11.031179004" />
+    </joint>
+    <link name="${prefix}_${position}_wrist_roll_link" >
+      <visual>
+        <origin xyz="0.0 0.0 0.0" rpy="0.0 ${M_PI} 0.0" />
+        <geometry>
+          <mesh filename="file://$(find sobit_home_description)/meshes/arm/arm_wrist_roll.stl" scale="0.001 0.001 0.001" />
+        </geometry>
+        <material name="grey" />
+      </visual>
+      <!-- 後でコメントアウト -->
+      <collision>
+        <origin xyz="${0.1166/2+0.0224} 0.0 0.0" rpy="0.0 0.0 0.0" />
+        <geometry>
+          <box size="0.1166 0.124 0.043" />
+        </geometry>
+      </collision>
+      <inertial>
+        <origin xyz="${0.1166/2+0.0224} 0.0 0.0" rpy="0.0 0.0 ${M_PI/2}" />
+        <mass value="0.08" />
+        <inertia ixx="${1/12*0.08*(0.1166**2+0.043**2)}" ixy="0.0" ixz="0.0"
+                 iyy="${1/12*0.08*(0.124**2 +0.043**2)}" iyz="0.0"
+                 izz="${1/12*0.08*(0.1166**2+0.124**2)}" />
+      </inertial>
+    </link>
     <xacro:arm_transmission prefix="${prefix}" position="${position}" />
   </xacro:macro>

File: sobit_home_description/urdf/controllers.urdf.xacro (robot description, xacro)
@@ -17,6 +17,6 @@
       <xacro:dx_arm_left_controllers    prefix="arm_left"   enable_gz="${$(arg enable_gz)}"/>
       <xacro:dx_arm_right_controllers   prefix="arm_right"  enable_gz="${$(arg enable_gz)}"/>
-      <!-- <xacro:dx_hand_left_controllers   prefix="hand_left"  enable_gz="${$(arg enable_gz)}"/> -->
-      <!-- <xacro:dx_hand_right_controllers  prefix="hand_right" enable_gz="${$(arg enable_gz)}"/> -->
+      <xacro:dx_hand_left_controllers   prefix="hand_left"  enable_gz="${$(arg enable_gz)}"/>
+      <xacro:dx_hand_right_controllers  prefix="hand_right" enable_gz="${$(arg enable_gz)}"/>
       <xacro:dx_wheel_steer_controllers prefix="wheel"      enable_gz="${$(arg enable_gz)}"/>
     </ros2_control>
@@ -285,7 +285,26 @@
       <state_interface name="effort"/>
     </joint>
-    <joint name="${prefix}_wrist_joint">
+<!-- rename joint : tsukada -->
+    <joint name="${prefix}_wrist_tilt_joint">
       <xacro:unless value="${$(arg enable_gz)}">
         <param name="id">35</param>
+        <param name="control_mode">0</param>
+        <param name="interface">rs</param>
+      </xacro:unless>
+      <command_interface name="position">
+        <param name="min">-1.570796327</param>
+        <param name="max">1.570796327</param>
+      </command_interface>
+      <!-- <command_interface name="velocity"/> -->
+      <state_interface name="position">
+        <param name="initial_value">0.0</param>
+      </state_interface>
+      <state_interface name="velocity"/>
+      <state_interface name="effort"/>
+    </joint>
+<!-- add joint : tsukada -->
+    <joint name="${prefix}_wrist_roll_joint">
+      <xacro:unless value="${$(arg enable_gz)}">
+        <param name="id">36</param>
         <param name="control_mode">0</param>
         <param name="interface">rs</param>
@@ -372,5 +391,6 @@
       <state_interface name="effort"/>
     </joint>
-    <joint name="${prefix}_wrist_joint">
+<!-- rename joint : tsukada -->
+    <joint name="${prefix}_wrist_tilt_joint">
       <xacro:unless value="${$(arg enable_gz)}">
         <param name="id">45</param>
@@ -389,7 +409,25 @@
       <state_interface name="effort"/>
     </joint>
+<!-- add joint : tsukada -->
+    <joint name="${prefix}_wrist_roll_joint">
+      <xacro:unless value="${$(arg enable_gz)}">
+        <param name="id">46</param>
+        <param name="control_mode">0</param>
+        <param name="interface">rs</param>
+      </xacro:unless>
+      <command_interface name="position">
+        <param name="min">-1.570796327</param>
+        <param name="max">1.570796327</param>
+      </command_interface>
+      <!-- <command_interface name="velocity"/> -->
+      <state_interface name="position">
+        <param name="initial_value">0.0</param>
+      </state_interface>
+      <state_interface name="velocity"/>
+      <state_interface name="effort"/>
+    </joint>
   </xacro:macro>
   <xacro:macro name="dx_hand_left_controllers"    params="prefix enable_gz:=False">
-    <joint name="${prefix}_finger_l_cmc_joint">
+    <joint name="${prefix}_finger_l_mcp_joint">
       <xacro:unless value="${$(arg enable_gz)}">
         <param name="id">50</param>
@@ -408,7 +446,111 @@
       <state_interface name="effort"/>
     </joint>
+    <joint name="${prefix}_finger_l_dip_joint">
+      <xacro:unless value="${$(arg enable_gz)}">
+        <param name="id">51</param>
+        <param name="control_mode">6</param>
+        <param name="interface">ttl</param>
+      </xacro:unless>
+      <command_interface name="position">
+        <param name="min">-1.570796327</param>
+        <param name="max">1.570796327</param>
+      </command_interface>
+      <!-- <command_interface name="velocity"/> -->
+      <state_interface name="position">
+        <param name="initial_value">0.0</param>
+      </state_interface>
+      <state_interface name="velocity"/>
+      <state_interface name="effort"/>
+    </joint>
+    <joint name="${prefix}_finger_l_pip_joint">
+      <xacro:unless value="${$(arg enable_gz)}">
+        <param name="id">52</param>
+        <param name="control_mode">6</param>
+        <param name="interface">ttl</param>
+      </xacro:unless>
+      <command_interface name="position">
+        <param name="min">-1.570796327</param>
+        <param name="max">1.570796327</param>
+      </command_interface>
+      <!-- <command_interface name="velocity"/> -->
+      <state_interface name="position">
+        <param name="initial_value">0.0</param>
+      </state_interface>
+      <state_interface name="velocity"/>
+      <state_interface name="effort"/>
+    </joint>
+    <joint name="${prefix}_finger_c_mcp_joint">
+      <xacro:unless value="${$(arg enable_gz)}">
+        <param name="id">53</param>
+        <param name="control_mode">6</param>
+        <param name="interface">ttl</param>
+      </xacro:unless>
+      <command_interface name="position">
+        <param name="min">-1.570796327</param>
+        <param name="max">1.570796327</param>
+      </command_interface>
+      <!-- <command_interface name="velocity"/> -->
+      <state_interface name="position">
+        <param name="initial_value">0.0</param>
+      </state_interface>
+      <state_interface name="velocity"/>
+      <state_interface name="effort"/>
+    </joint>
+    <joint name="${prefix}_finger_c_ip_joint">
+      <xacro:unless value="${$(arg enable_gz)}">
+        <param name="id">54</param>
+        <param name="control_mode">6</param>
+        <param name="interface">ttl</param>
+      </xacro:unless>
+      <command_interface name="position">
+        <param name="min">-1.570796327</param>
+        <param name="max">1.570796327</param>
+      </command_interface>
+      <!-- <command_interface name="velocity"/> -->
+      <state_interface name="position">
+        <param name="initial_value">0.0</param>
+      </state_interface>
+      <state_interface name="velocity"/>
+      <state_interface name="effort"/>
+    </joint>
+    <joint name="${prefix}_finger_r_dip_joint">
+      <xacro:unless value="${$(arg enable_gz)}">
+        <param name="id">55</param>
+        <param name="control_mode">6</param>
+        <param name="interface">ttl</param>
+      </xacro:unless>
+      <command_interface name="position">
+        <param name="min">-1.570796327</param>
+        <param name="max">1.570796327</param>
+      </command_interface>
+      <!-- <command_interface name="velocity"/> -->
+      <state_interface name="position">
+        <param name="initial_value">0.0</param>
+      </state_interface>
+      <state_interface name="velocity"/>
+      <state_interface name="effort"/>
+    </joint>
+      <joint name="${prefix}_finger_r_pip_joint">
+      <xacro:unless value="${$(arg enable_gz)}">
+        <param name="id">56</param>
+        <param name="control_mode">6</param>
+        <param name="interface">ttl</param>
+      </xacro:unless>
+      <command_interface name="position">
+        <param name="min">-1.570796327</param>
+        <param name="max">1.570796327</param>
+      </command_interface>
+      <!-- <command_interface name="velocity"/> -->
+      <state_interface name="position">
+        <param name="initial_value">0.0</param>
+      </state_interface>
+      <state_interface name="velocity"/>
+      <state_interface name="effort"/>
+    </joint>
+  </xacro:macro>
+  <xacro:macro name="dx_hand_right_controllers"   params="prefix enable_gz:=False">
     <joint name="${prefix}_finger_l_mcp_joint">
       <xacro:unless value="${$(arg enable_gz)}">
-        <param name="id">51</param>
+        <param name="id">60</param>
         <param name="control_mode">6</param>
         <param name="interface">ttl</param>
@@ -427,5 +569,22 @@
     <joint name="${prefix}_finger_l_dip_joint">
       <xacro:unless value="${$(arg enable_gz)}">
-        <param name="id">52</param>
+        <param name="id">61</param>
+        <param name="control_mode">6</param>
+        <param name="interface">ttl</param>
+      </xacro:unless>
+      <command_interface name="position">
+        <param name="min">-1.570796327</param>
+        <param name="max">1.570796327</param>
+      </command_interface>
+      <!-- <command_interface name="velocity"/> -->
+      <state_interface name="position">
+        <param name="initial_value">0.0</param>
+      </state_interface>
+      <state_interface name="velocity"/>
+      <state_interface name="effort"/>
+    </joint>
+    <joint name="${prefix}_finger_l_pip_joint">
+      <xacro:unless value="${$(arg enable_gz)}">
+        <param name="id">62</param>
         <param name="control_mode">6</param>
         <param name="interface">ttl</param>
@@ -444,39 +603,22 @@
     <joint name="${prefix}_finger_c_mcp_joint">
       <xacro:unless value="${$(arg enable_gz)}">
-        <param name="id">53</param>
-        <param name="control_mode">6</param>
-        <param name="interface">ttl</param>
-      </xacro:unless>
-      <command_interface name="position">
-        <param name="min">-1.570796327</param>
-        <param name="max">1.570796327</param>
-      </command_interface>
-      <!-- <command_interface name="velocity"/> -->
-      <state_interface name="position">
-        <param name="initial_value">0.0</param>
-      </state_interface>
-      <state_interface name="velocity"/>
-      <state_interface name="effort"/>
-    </joint>
-    <joint name="${prefix}_finger_c_dip_joint">
-      <xacro:unless value="${$(arg enable_gz)}">
-        <param name="id">54</param>
-        <param name="control_mode">6</param>
-        <param name="interface">ttl</param>
-      </xacro:unless>
-      <command_interface name="position">
-        <param name="min">-1.570796327</param>
-        <param name="max">1.570796327</param>
-      </command_interface>
-      <!-- <command_interface name="velocity"/> -->
-      <state_interface name="position">
-        <param name="initial_value">0.0</param>
-      </state_interface>
-      <state_interface name="velocity"/>
-      <state_interface name="effort"/>
-    </joint>
-    <joint name="${prefix}_finger_r_mcp_joint">
-      <xacro:unless value="${$(arg enable_gz)}">
-        <param name="id">55</param>
+        <param name="id">63</param>
+        <param name="control_mode">6</param>
+        <param name="interface">ttl</param>
+      </xacro:unless>
+      <command_interface name="position">
+        <param name="min">-1.570796327</param>
+        <param name="max">1.570796327</param>
+      </command_interface>
+      <!-- <command_interface name="velocity"/> -->
+      <state_interface name="position">
+        <param name="initial_value">0.0</param>
+      </state_interface>
+      <state_interface name="velocity"/>
+      <state_interface name="effort"/>
+    </joint>
+    <joint name="${prefix}_finger_c_ip_joint">
+      <xacro:unless value="${$(arg enable_gz)}">
+        <param name="id">64</param>
         <param name="control_mode">6</param>
         <param name="interface">ttl</param>
@@ -495,108 +637,4 @@
     <joint name="${prefix}_finger_r_dip_joint">
       <xacro:unless value="${$(arg enable_gz)}">
-        <param name="id">56</param>
-        <param name="control_mode">6</param>
-        <param name="interface">ttl</param>
-      </xacro:unless>
-      <command_interface name="position">
-        <param name="min">-1.570796327</param>
-        <param name="max">1.570796327</param>
-      </command_interface>
-      <!-- <command_interface name="velocity"/> -->
-      <state_interface name="position">
-        <param name="initial_value">0.0</param>
-      </state_interface>
-      <state_interface name="velocity"/>
-      <state_interface name="effort"/>
-    </joint>
-  </xacro:macro>
-  <xacro:macro name="dx_hand_right_controllers"   params="prefix enable_gz:=False">
-    <joint name="${prefix}_finger_l_cmc_joint">
-      <xacro:unless value="${$(arg enable_gz)}">
-        <param name="id">60</param>
-        <param name="control_mode">6</param>
-        <param name="interface">ttl</param>
-      </xacro:unless>
-      <command_interface name="position">
-        <param name="min">-1.570796327</param>
-        <param name="max">1.570796327</param>
-      </command_interface>
-      <!-- <command_interface name="velocity"/> -->
-      <state_interface name="position">
-        <param name="initial_value">0.0</param>
-      </state_interface>
-      <state_interface name="velocity"/>
-      <state_interface name="effort"/>
-    </joint>
-    <joint name="${prefix}_finger_l_mcp_joint">
-      <xacro:unless value="${$(arg enable_gz)}">
-        <param name="id">61</param>
-        <param name="control_mode">6</param>
-        <param name="interface">ttl</param>
-      </xacro:unless>
-      <command_interface name="position">
-        <param name="min">-1.570796327</param>
-        <param name="max">1.570796327</param>
-      </command_interface>
-      <!-- <command_interface name="velocity"/> -->
-      <state_interface name="position">
-        <param name="initial_value">0.0</param>
-      </state_interface>
-      <state_interface name="velocity"/>
-      <state_interface name="effort"/>
-    </joint>
-    <joint name="${prefix}_finger_l_dip_joint">
-      <xacro:unless value="${$(arg enable_gz)}">
-        <param name="id">62</param>
-        <param name="control_mode">6</param>
-        <param name="interface">ttl</param>
-      </xacro:unless>
-      <command_interface name="position">
-        <param name="min">-1.570796327</param>
-        <param name="max">1.570796327</param>
-      </command_interface>
-      <!-- <command_interface name="velocity"/> -->
-      <state_interface name="position">
-        <param name="initial_value">0.0</param>
-      </state_interface>
-      <state_interface name="velocity"/>
-      <state_interface name="effort"/>
-    </joint>
-    <joint name="${prefix}_finger_c_mcp_joint">
-      <xacro:unless value="${$(arg enable_gz)}">
-        <param name="id">63</param>
-        <param name="control_mode">6</param>
-        <param name="interface">ttl</param>
-      </xacro:unless>
-      <command_interface name="position">
-        <param name="min">-1.570796327</param>
-        <param name="max">1.570796327</param>
-      </command_interface>
-      <!-- <command_interface name="velocity"/> -->
-      <state_interface name="position">
-        <param name="initial_value">0.0</param>
-      </state_interface>
-      <state_interface name="velocity"/>
-      <state_interface name="effort"/>
-    </joint>
-    <joint name="${prefix}_finger_c_dip_joint">
-      <xacro:unless value="${$(arg enable_gz)}">
-        <param name="id">64</param>
-        <param name="control_mode">6</param>
-        <param name="interface">ttl</param>
-      </xacro:unless>
-      <command_interface name="position">
-        <param name="min">-1.570796327</param>
-        <param name="max">1.570796327</param>
-      </command_interface>
-      <!-- <command_interface name="velocity"/> -->
-      <state_interface name="position">
-        <param name="initial_value">0.0</param>
-      </state_interface>
-      <state_interface name="velocity"/>
-      <state_interface name="effort"/>
-    </joint>
-    <joint name="${prefix}_finger_r_mcp_joint">
-      <xacro:unless value="${$(arg enable_gz)}">
         <param name="id">65</param>
         <param name="control_mode">6</param>
@@ -614,5 +652,5 @@
       <state_interface name="effort"/>
     </joint>
-    <joint name="${prefix}_finger_r_dip_joint">
+    <joint name="${prefix}_finger_r_pip_joint">
       <xacro:unless value="${$(arg enable_gz)}">
         <param name="id">66</param>

File: sobit_home_description/urdf/hand/hand.transmission.xacro (robot description, xacro)
@@ -3,11 +3,11 @@
        xmlns:xacro="http://ros.org/wiki/xacro">
   <xacro:macro name="hand_transmission" params="prefix_hand position prefix_finger">
-    <xacro:SimpleTransmissionPosition joint="${prefix_hand}_${position}_mcp_joint"                     reduction="1" />
-    <xacro:SimpleTransmissionPosition joint="${prefix_hand}_${position}_${prefix_finger}_l_cmc_joint"  reduction="1" />
     <xacro:SimpleTransmissionPosition joint="${prefix_hand}_${position}_${prefix_finger}_l_mcp_joint"  reduction="1" />
-    <xacro:SimpleTransmissionPosition joint="${prefix_hand}_${position}_${prefix_finger}_c_cmc_joint"  reduction="1" />
+    <xacro:SimpleTransmissionPosition joint="${prefix_hand}_${position}_${prefix_finger}_l_pip_joint"  reduction="1" />
+    <xacro:SimpleTransmissionPosition joint="${prefix_hand}_${position}_${prefix_finger}_l_dip_joint"  reduction="1" />
     <xacro:SimpleTransmissionPosition joint="${prefix_hand}_${position}_${prefix_finger}_c_mcp_joint"  reduction="1" />
-    <xacro:SimpleTransmissionPosition joint="${prefix_hand}_${position}_${prefix_finger}_r_cmc_joint"  reduction="1" />
-    <xacro:SimpleTransmissionPosition joint="${prefix_hand}_${position}_${prefix_finger}_r_mcp_joint"  reduction="1" />
+    <xacro:SimpleTransmissionPosition joint="${prefix_hand}_${position}_${prefix_finger}_c_ip_joint"   reduction="1" />
+    <xacro:SimpleTransmissionPosition joint="${prefix_hand}_${position}_${prefix_finger}_r_pip_joint"  reduction="1" />
+    <xacro:SimpleTransmissionPosition joint="${prefix_hand}_${position}_${prefix_finger}_r_dip_joint"  reduction="1" />
   </xacro:macro>
 </robot>
