Commit message: add hand parts

File: sobit_home_description/urdf/hand/hand.urdf.xacro (robot description, xacro)
@@ -3,33 +3,283 @@
        xmlns:xacro="http://ros.org/wiki/xacro" >
   <xacro:include filename="$(find sobit_home_description)/urdf/hand/hand.transmission.xacro" />
-  <xacro:macro name="hand" params="prefix_hand position prefix_finger parent">
-    <joint name="${prefix_hand}_${position}_base_joint" type="fixed">
+  <xacro:macro name="hand" params="prefix_hand position prefix_finger parent" >
+    <xacro:if value="${position == 'left'}">
+      <xacro:property name="y_sign" value="1.0" />
+      <xacro:property name="yaw_rot" value="0.0" />
+        <xacro:property name="upper_roll_limit_lower" value="0" />
+        <xacro:property name="upper_roll_limit_upper" value="${M_PI}" />
+    </xacro:if>
+    <xacro:if value="${position == 'right'}">
+      <xacro:property name="y_sign" value="-1.0" />
+      <xacro:property name="yaw_rot" value="${M_PI}" />
+        <xacro:property name="upper_roll_limit_lower" value="${-M_PI}" />
+        <xacro:property name="upper_roll_limit_upper" value="0" />
+    </xacro:if>
+<!-- hand_base -->
+    <joint name="${prefix_hand}_${position}_cmc_joint" type="fixed" >
       <parent link="${parent}" />
-      <child link="${prefix_hand}_base_link" />
+      <child link="${prefix_hand}_${position}_cmc_link" />
       <origin xyz="0.0 0.0 0.0" rpy="0.0 0.0 0.0" />
     </joint>
-    <link name="${prefix_hand}_${position}_base_link">
-      <visual>
-        <origin xyz="0.0 0.0 0.0" rpy="${M_PI/2.0} 0.0 ${M_PI/2.0}" />
+    <link name="${prefix_hand}_${position}_cmc_link" >
+      <visual>
+        <origin xyz="0.0 0.0 0.0" rpy="${M_PI} 0.0 ${-M_PI/2}" />
         <geometry>
           <mesh filename="file://$(find sobit_home_description)/meshes/hand/hand_base.stl" scale="0.001 0.001 0.001" />
         </geometry>
-        <material name="black" />
-      </visual>
-      <collision>
-        <origin xyz="${0.0215+(0.08251-0.0215)/2} 0.0 ${(0.0415-0.033)/2}" rpy="0.0 0.0 0.0" />
-        <geometry>
-          <box size="0.06102 0.102 0.0745" />
-        </geometry>
-      </collision>
-      <inertial>
-        <origin xyz="${0.0215+(0.08251-0.0215)/2} 0.0 ${(0.0415-0.033)/2}" rpy="0.0 0.0 ${M_PI/2}" />
-        <mass value="0.08" />
-        <inertia ixx="${1/12*0.08*(0.06102**2+0.0745**2)}" ixy="0.0" ixz="0.0"
-                 iyy="${1/12*0.08*(0.102**2  +0.0745**2)}" iyz="0.0"
-                 izz="${1/12*0.08*(0.06102**2+0.102**2)}" />
-      </inertial>
-    </link>
-    <xacro:hand_transmission prefix_hand="${prefix_hand}" position="${position}" prefix_finger="${prefix_finger}" />
+        <material name="grey" />
+      </visual>
+      <collision>
+        <origin xyz="${0.140/2} 0.0 ${0.043/2}" rpy="0.0 0.0 0.0" />
+        <geometry>
+          <box size="0.140 0.156 0.043" />
+        </geometry>
+      </collision>
+      <inertial>
+        <origin xyz="${0.140/2} 0.0 ${0.043/2}" rpy="0.0 0.0 ${M_PI/2}" />
+        <mass value="0.08" />
+        <inertia ixx="${1/12*0.08*(0.140**2+0.043**2)}" ixy="0.0" ixz="0.0"
+                 iyy="${1/12*0.08*(0.156**2+0.043**2)}" iyz="0.0"
+                 izz="${1/12*0.08*(0.140**2+0.156**2)}" />
+      </inertial>
+    </link>
+<!-- l_finger -->
+    <joint name="${prefix_hand}_${position}_${prefix_finger}_l_mcp_joint" type="revolute" >
+      <parent link="${prefix_hand}_${position}_cmc_link" />
+      <child link="${prefix_hand}_${position}_${prefix_finger}_l_mcp_link" />
+      <origin xyz="-0.003249 0.024532 -0.046" rpy="0.0 0.0 0.0" />
+      <axis xyz="0.0 0.0 1.0 " />
+      <limit lower="${-M_PI/2}" upper="${M_PI/2}" effort="0.52" velocity="11.031179004" />
+    </joint>
+    <link name="${prefix_hand}_${position}_${prefix_finger}_l_mcp_link" >
+      <visual>
+        <origin xyz="0.0 0.0 0.0" rpy="${M_PI} 0.0 ${-(2*M_PI/15+M_PI/2)}" />
+        <geometry>
+          <mesh filename="file://$(find sobit_home_description)/meshes/hand/switching_gear.stl" scale="0.001 0.001 0.001" />
+        </geometry>
+        <material name="grey" />
+      </visual>
+      <collision>
+        <origin xyz="${0.140/2} 0.0 ${0.043/2}" rpy="0.0 0.0 0.0" />
+        <geometry>
+          <box size="0.140 0.156 0.043" />
+        </geometry>
+      </collision>
+      <inertial>
+        <origin xyz="${0.140/2} 0.0 ${0.043/2}" rpy="0.0 0.0 ${M_PI/2}" />
+        <mass value="0.08" />
+        <inertia ixx="${1/12*0.08*(0.140**2+0.043**2)}" ixy="0.0" ixz="0.0"
+                 iyy="${1/12*0.08*(0.156**2+0.043**2)}" iyz="0.0"
+                 izz="${1/12*0.08*(0.140**2+0.156**2)}" />
+      </inertial>
+    </link>
+    <joint name="${prefix_hand}_${position}_${prefix_finger}_l_pip_joint" type="revolute" >
+      <parent link="${prefix_hand}_${position}_${prefix_finger}_l_mcp_link" />
+      <child link="${prefix_hand}_${position}_${prefix_finger}_l_pip_link" />
+      <origin xyz="-0.02125 0.040125 -0.018575" rpy="0.0 0.0 0.0" />
+      <axis xyz="1.0 0.0 0.0 " />
+      <limit lower="${-M_PI/6}" upper="${M_PI/2}" effort="0.52" velocity="11.031179004" />
+    </joint>
+    <link name="${prefix_hand}_${position}_${prefix_finger}_l_pip_link" >
+      <visual>
+        <origin xyz="0.0 0.0 0.0" rpy="0.0 ${M_PI} ${M_PI/2}" />
+        <geometry>
+          <mesh filename="file://$(find sobit_home_description)/meshes/hand/middle_pharanx.stl" scale="0.001 0.001 0.001" />
+        </geometry>
+        <material name="grey" />
+      </visual>
+      <collision>
+        <origin xyz="${0.140/2} 0.0 ${0.043/2}" rpy="0.0 0.0 0.0" />
+        <geometry>
+          <box size="0.140 0.156 0.043" />
+        </geometry>
+      </collision>
+      <inertial>
+        <origin xyz="${0.140/2} 0.0 ${0.043/2}" rpy="0.0 0.0 ${M_PI/2}" />
+        <mass value="0.08" />
+        <inertia ixx="${1/12*0.08*(0.140**2+0.043**2)}" ixy="0.0" ixz="0.0"
+                 iyy="${1/12*0.08*(0.156**2+0.043**2)}" iyz="0.0"
+                 izz="${1/12*0.08*(0.140**2+0.156**2)}" />
+      </inertial>
+    </link>
+    <joint name="${prefix_hand}_${position}_${prefix_finger}_l_dip_joint" type="revolute" >
+      <parent link="${prefix_hand}_${position}_${prefix_finger}_l_pip_link" />
+      <child link="${prefix_hand}_${position}_${prefix_finger}_l_dip_link" />
+      <origin xyz="0.0 0.0 -0.050" rpy="0.0 0.0 0.0" />
+      <axis xyz="1.0 0.0 0.0 " />
+      <limit lower="${-M_PI/2}" upper="${M_PI/6}" effort="0.52" velocity="11.031179004" />
+    </joint>
+    <link name="${prefix_hand}_${position}_${prefix_finger}_l_dip_link" >
+      <visual>
+        <origin xyz="0.0 0.0 0.0" rpy="0.0 ${M_PI} ${M_PI/2}" />
+        <geometry>
+          <mesh filename="file://$(find sobit_home_description)/meshes/hand/distal_pharanx.stl" scale="0.001 0.001 0.001" />
+        </geometry>
+        <material name="blue" />
+      </visual>
+      <collision>
+        <origin xyz="${0.140/2} 0.0 ${0.043/2}" rpy="0.0 0.0 0.0" />
+        <geometry>
+          <box size="0.140 0.156 0.043" />
+        </geometry>
+      </collision>
+      <inertial>
+        <origin xyz="${0.140/2} 0.0 ${0.043/2}" rpy="0.0 0.0 ${M_PI/2}" />
+        <mass value="0.08" />
+        <inertia ixx="${1/12*0.08*(0.140**2+0.043**2)}" ixy="0.0" ixz="0.0"
+                 iyy="${1/12*0.08*(0.156**2+0.043**2)}" iyz="0.0"
+                 izz="${1/12*0.08*(0.140**2+0.156**2)}" />
+      </inertial>
+    </link>
+<!-- r_finger -->
+<!-- mimic part -->
+    <joint name="${prefix_hand}_${position}_${prefix_finger}_r_mcp_joint" type="revolute" >
+      <parent link="${prefix_hand}_${position}_cmc_link" />
+      <child link="${prefix_hand}_${position}_${prefix_finger}_r_mcp_link" />
+      <origin xyz="-0.003249 -0.024532 -0.046" rpy="0.0 0.0 0.0" />
+      <axis xyz="0.0 0.0 1.0 " />
+      <limit lower="${-M_PI/2}" upper="${M_PI/2}" effort="0.52" velocity="11.031179004" />
+      <mimic joint="${prefix_hand}_${position}_${prefix_finger}_l_mcp_joint" multiplier="-1.0" />
+    </joint>
+    <link name="${prefix_hand}_${position}_${prefix_finger}_r_mcp_link" >
+      <visual>
+        <origin xyz="0.0 0.0 -0.002006" rpy="${M_PI} 0.0 ${-M_PI/2}" />
+        <geometry>
+          <mesh filename="file://$(find sobit_home_description)/meshes/hand/switching_gear-m.stl" scale="0.001 0.001 0.001" />
+        </geometry>
+        <material name="grey" />
+      </visual>
+      <collision>
+        <origin xyz="${0.140/2} 0.0 ${0.043/2}" rpy="0.0 0.0 0.0" />
+        <geometry>
+          <box size="0.140 0.156 0.043" />
+        </geometry>
+      </collision>
+      <inertial>
+        <origin xyz="${0.140/2} 0.0 ${0.043/2}" rpy="0.0 0.0 ${M_PI/2}" />
+        <mass value="0.08" />
+        <inertia ixx="${1/12*0.08*(0.140**2+0.043**2)}" ixy="0.0" ixz="0.0"
+                 iyy="${1/12*0.08*(0.156**2+0.043**2)}" iyz="0.0"
+                 izz="${1/12*0.08*(0.140**2+0.156**2)}" />
+      </inertial>
+    </link>
+    <joint name="${prefix_hand}_${position}_${prefix_finger}_r_pip_joint" type="revolute" >
+      <parent link="${prefix_hand}_${position}_${prefix_finger}_r_mcp_link" />
+      <child link="${prefix_hand}_${position}_${prefix_finger}_r_pip_link" />
+      <origin xyz="-0.02125 -0.040125 -0.018575" rpy="0.0 0.0 0.0" />
+      <axis xyz="1.0 0.0 0.0 " />
+      <limit lower="${-M_PI/2}" upper="${M_PI/6}" effort="0.52" velocity="11.031179004" />
+    </joint>
+    <link name="${prefix_hand}_${position}_${prefix_finger}_r_pip_link" >
+      <visual>
+        <origin xyz="0.0 0.0 0.0" rpy="0.0 ${M_PI} ${-M_PI/2}" />
+        <geometry>
+          <mesh filename="file://$(find sobit_home_description)/meshes/hand/middle_pharanx-m.stl" scale="0.001 0.001 0.001" />
+        </geometry>
+        <material name="grey" />
+      </visual>
+      <collision>
+        <origin xyz="${0.140/2} 0.0 ${0.043/2}" rpy="0.0 0.0 0.0" />
+        <geometry>
+          <box size="0.140 0.156 0.043" />
+        </geometry>
+      </collision>
+      <inertial>
+        <origin xyz="${0.140/2} 0.0 ${0.043/2}" rpy="0.0 0.0 ${M_PI/2}" />
+        <mass value="0.08" />
+        <inertia ixx="${1/12*0.08*(0.140**2+0.043**2)}" ixy="0.0" ixz="0.0"
+                 iyy="${1/12*0.08*(0.156**2+0.043**2)}" iyz="0.0"
+                 izz="${1/12*0.08*(0.140**2+0.156**2)}" />
+      </inertial>
+    </link>
+    <joint name="${prefix_hand}_${position}_${prefix_finger}_r_dip_joint" type="revolute" >
+      <parent link="${prefix_hand}_${position}_${prefix_finger}_r_pip_link" />
+      <child link="${prefix_hand}_${position}_${prefix_finger}_r_dip_link" />
+      <origin xyz="0.0 0.0 -0.050" rpy="0.0 0.0 0.0" />
+      <axis xyz="1.0 0.0 0.0 " />
+      <limit lower="${-M_PI/6}" upper="${M_PI/2}" effort="0.52" velocity="11.031179004" />
+    </joint>
+    <link name="${prefix_hand}_${position}_${prefix_finger}_r_dip_link" >
+      <visual>
+        <origin xyz="0.0 0.0 0.0" rpy="0.0 ${M_PI} ${-M_PI/2}" />
+        <geometry>
+          <mesh filename="file://$(find sobit_home_description)/meshes/hand/distal_pharanx-m.stl" scale="0.001 0.001 0.001" />
+        </geometry>
+        <material name="green" />
+      </visual>
+      <collision>
+        <origin xyz="${0.140/2} 0.0 ${0.043/2}" rpy="0.0 0.0 0.0" />
+        <geometry>
+          <box size="0.140 0.156 0.043" />
+        </geometry>
+      </collision>
+      <inertial>
+        <origin xyz="${0.140/2} 0.0 ${0.043/2}" rpy="0.0 0.0 ${M_PI/2}" />
+        <mass value="0.08" />
+        <inertia ixx="${1/12*0.08*(0.140**2+0.043**2)}" ixy="0.0" ixz="0.0"
+                 iyy="${1/12*0.08*(0.156**2+0.043**2)}" iyz="0.0"
+                 izz="${1/12*0.08*(0.140**2+0.156**2)}" />
+      </inertial>
+    </link>
+<!-- c_finger-->
+    <joint name="${prefix_hand}_${position}_${prefix_finger}_c_mcp_joint" type="revolute" >
+      <parent link="${prefix_hand}_${position}_cmc_link" />
+      <child link="${prefix_hand}_${position}_${prefix_finger}_c_mcp_link" />
+      <origin xyz="0.036751 0.01435 -0.062" rpy="0.0 0.0 0.0" />
+      <axis xyz="0.0 1.0 0.0 " />
+      <limit lower="${-M_PI/2}" upper="${M_PI/6}" effort="0.52" velocity="11.031179004" />
+    </joint>
+    <link name="${prefix_hand}_${position}_${prefix_finger}_c_mcp_link" >
+      <visual>
+        <origin xyz="0.0 0.0 0.0" rpy="0.0 ${M_PI} ${M_PI}" />
+        <geometry>
+          <mesh filename="file://$(find sobit_home_description)/meshes/hand/thumb_middle_pharanx.stl" scale="0.001 0.001 0.001" />
+        </geometry>
+        <material name="grey" />
+      </visual>
+      <collision>
+        <origin xyz="${0.140/2} 0.0 ${0.043/2}" rpy="0.0 0.0 0.0" />
+        <geometry>
+          <box size="0.140 0.156 0.043" />
+        </geometry>
+      </collision>
+      <inertial>
+        <origin xyz="${0.140/2} 0.0 ${0.043/2}" rpy="0.0 0.0 ${M_PI/2}" />
+        <mass value="0.08" />
+        <inertia ixx="${1/12*0.08*(0.140**2+0.043**2)}" ixy="0.0" ixz="0.0"
+                 iyy="${1/12*0.08*(0.156**2+0.043**2)}" iyz="0.0"
+                 izz="${1/12*0.08*(0.140**2+0.156**2)}" />
+      </inertial>
+    </link>
+    <joint name="${prefix_hand}_${position}_${prefix_finger}_c_ip_joint" type="revolute" >
+      <parent link="${prefix_hand}_${position}_${prefix_finger}_c_mcp_link" />
+      <child link="${prefix_hand}_${position}_${prefix_finger}_c_ip_link" />
+      <origin xyz="0.0 0.0 -0.050" rpy="0.0 0.0 0.0" />
+      <axis xyz="0.0 1.0 0.0 " />
+      <limit lower="${-M_PI/6}" upper="${M_PI/2}" effort="0.52" velocity="11.031179004" />
+    </joint>
+    <link name="${prefix_hand}_${position}_${prefix_finger}_c_ip_link" >
+      <visual>
+        <origin xyz="0.0 0.0 0.0" rpy="0.0 ${M_PI} ${M_PI}" />
+        <geometry>
+          <mesh filename="file://$(find sobit_home_description)/meshes/hand/thumb_distal_pharanx.stl" scale="0.001 0.001 0.001" />
+        </geometry>
+        <material name="red" />
+      </visual>
+      <collision>
+        <origin xyz="${0.140/2} 0.0 ${0.043/2}" rpy="0.0 0.0 0.0" />
+        <geometry>
+          <box size="0.140 0.156 0.043" />
+        </geometry>
+      </collision>
+      <inertial>
+        <origin xyz="${0.140/2} 0.0 ${0.043/2}" rpy="0.0 0.0 ${M_PI/2}" />
+        <mass value="0.08" />
+        <inertia ixx="${1/12*0.08*(0.140**2+0.043**2)}" ixy="0.0" ixz="0.0"
+                 iyy="${1/12*0.08*(0.156**2+0.043**2)}" iyz="0.0"
+                 izz="${1/12*0.08*(0.140**2+0.156**2)}" />
+      </inertial>
+    </link>
+  <xacro:hand_transmission prefix_hand="${prefix_hand}" position="${position}" prefix_finger="${prefix_finger}"/>
   </xacro:macro>
 </robot>

File: sobit_home_description/urdf/sensor/mic.urdf.xacro (robot description, xacro)
@@ -41,5 +41,5 @@
         <origin xyz="0.0 0.0 0.0" rpy="0.0 0.0 ${M_PI/2.0}" />
         <geometry>
-          <mesh filename="file://$(find sobit_home_description)/meshes/sensor/mic.stl" scale="0.001 0.001 0.001" />
+          <mesh filename="file://$(find sobit_home_description)/meshes/sensor/mic_base.stl" scale="0.001 0.001 0.001" />
         </geometry>
         <material name="black" />

Commit message: [FIX] prefix name

File: sobit_home_description/robots/sobit_home_robot.urdf.xacro (robot description, xacro)
@@ -65,5 +65,5 @@
     <xacro:head  prefix="head"  parent="body_lift_link" />
     <!-- <xacro:mic   prefix="mic"   parent="head_tilt_link" />  -->
-    <xacro:camera_head  prefix="head_camera"  parent="head_tilt_link" />
+    <xacro:camera_head  prefix="head"  parent="head_tilt_link" />
   </xacro:if>
   <!-- Add Actuators Controllers -->

File: sobit_home_description/urdf/gazebo.urdf.xacro (robot description, xacro)
@@ -7,5 +7,5 @@
       <gazebo reference="head_camera_color_optical_frame">
         <sensor name="head_camera_color" type="camera">
-          <pose>0 0 ${0.0175/2} ${M_PI/2} -${M_PI/2} 0 </pose>
+          <pose>0 0 0 ${M_PI/2} -${M_PI/2} 0 </pose>
           <ignition_frame_id>${robot_name}/head_camera_color_optical_frame</ignition_frame_id>
           <!-- <gz_frame_id>${robot_name}/head_camera_color_optical_frame</gz_frame_id> -->
@@ -13,5 +13,5 @@
           <always_on>1</always_on>
           <visualize>true</visualize>
-          <update_rate>1</update_rate>
+          <update_rate>50</update_rate>
           <camera name="head_camera_color">
             <horizontal_fov>1.21126</horizontal_fov>
@@ -39,5 +39,5 @@
       <gazebo reference="head_camera_depth_optical_frame">
         <sensor name="head_camera_depth" type="depth">
-          <pose>0 0 ${0.0175/2} ${M_PI/2} -${M_PI/2} 0 </pose>
+          <pose>0 0 0 ${M_PI/2} -${M_PI/2} 0 </pose>
           <ignition_frame_id>${robot_name}/head_camera_depth_optical_frame</ignition_frame_id>
           <!-- <gz_frame_id>${robot_name}/head_camera_depth_optical_frame</gz_frame_id> -->
@@ -45,5 +45,5 @@
           <always_on>1</always_on>
           <visualize>true</visualize>
-          <update_rate>1</update_rate>
+          <update_rate>50</update_rate>
           <camera name="head_camera_depth">
             <horizontal_fov>1.48702</horizontal_fov>

File: sobit_home_description/urdf/sensor/camera_head.urdf.xacro (robot description, xacro)
@@ -4,11 +4,11 @@
   <xacro:include filename="$(find orbbec_description)/urdf/gemini_336.urdf.xacro" />
   <xacro:macro name="camera_head" params="prefix parent">
-    <joint name="${prefix}_base_joint" type="fixed">
+    <joint name="${prefix}_camera_base_joint" type="fixed">
       <parent link="${parent}" />
-      <child link="${prefix}_base_link" />
+      <child link="${prefix}_camera_base_link" />
       <origin xyz="0.0398 0.0 0.074" rpy="0.0 0.0 0.0" />
     </joint>
-    <link name="${prefix}_base_link"/>
-    <xacro:gemini_336 parent="${prefix}_base_link" tf_prefix="${prefix}_">
+    <link name="${prefix}_camera_base_link"/>
+    <xacro:gemini_336 parent="${prefix}_camera_base_link" tf_prefix="${prefix}_">
       <origin xyz="0.01 0 -0.0125" rpy="0 0 0"/>
     </xacro:gemini_336>

Commit message: [UPD] allow toggle off body

File: sobit_home_description/robots/sobit_home_robot.urdf.xacro (robot description, xacro)
@@ -50,4 +50,12 @@
     <xacro:body  prefix="body"  parent="plate_top_link" />
   </xacro:if>
+  <xacro:unless value="${ $(arg enable_body) }">
+    <joint name="body_joint" type="fixed" >
+      <origin xyz="0.11275 0.0 0.565" rpy="0.0 0.0 0.0" />
+      <parent link="plate_top_link" />
+      <child link="body_lift_link" />
+    </joint>
+    <link name="body_lift_link" />
+  </xacro:unless>
   <xacro:if value="${ $(arg enable_arm_left) }">
     <xacro:arm   prefix="arm"   position="left"  parent="body_lift_link" />

Commit message: [UPD] allow no mobile base launch

File: sobit_home_description/robots/sobit_home_robot.urdf.xacro (robot description, xacro)
@@ -45,4 +45,13 @@
     <xacro:lidar prefix="lidar" parent="plate_middle_link" robot_name="$(arg robot_name)" />
   </xacro:if>
+  <xacro:unless value="${ $(arg enable_mobile_base) }">
+    <xacro:base/>
+    <joint name="plate_top_joint" type="fixed" >
+      <origin xyz="0.0 0.0 0.371058" rpy="0.0 0.0 0.0" />
+      <parent link="base_link" />
+      <child link="plate_top_link" />
+    </joint>
+    <link name="plate_top_link" />
+  </xacro:unless>
   <xacro:if value="${ $(arg enable_body) }">
     <xacro:body  prefix="body"  parent="plate_top_link" />

Commit message: [UPD] allow hand without arm

File: sobit_home_description/robots/sobit_home_robot.urdf.xacro (robot description, xacro)
@@ -68,7 +68,23 @@
     <xacro:arm   prefix="arm"   position="left"  parent="body_lift_link" />
   </xacro:if>
+  <xacro:unless value="${ $(arg enable_arm_left) }">
+    <joint name="arm_left_wrist_roll_joint" type="fixed" >
+      <origin xyz="0.0 1.17790032 0.0" rpy="0.0 0.0 0.0" />
+      <parent link="body_lift_link" />
+      <child link="arm_left_wrist_roll_link" />
+    </joint>
+    <link name="arm_left_wrist_roll_link" />
+  </xacro:unless>
   <xacro:if value="${ $(arg enable_arm_right) }">
     <xacro:arm   prefix="arm"   position="right" parent="body_lift_link" />
   </xacro:if>
+  <xacro:unless value="${ $(arg enable_arm_right) }">
+    <joint name="arm_right_wrist_roll_joint" type="fixed" >
+      <origin xyz="0.0 -1.17790032 0.0" rpy="0.0 0.0 0.0" />
+      <parent link="body_lift_link" />
+      <child link="arm_right_wrist_roll_link" />
+    </joint>
+    <link name="arm_right_wrist_roll_link" />
+  </xacro:unless>
   <xacro:if value="${ $(arg enable_hand_left) }">
     <xacro:hand  prefix_hand="hand" position="left" prefix_finger="finger" parent="arm_left_wrist_roll_link" />
