Commit message: [FIX] multiple dxl series are not supported in dynamixel_hardware. separate port

File: sobit_home_description/robots/sobit_home_robot.urdf.xacro (robot description, xacro)
@@ -40,6 +40,7 @@
   <xacro:arg name="enable_head"         default="True" />
   <!-- DXL Ports -->
-  <xacro:arg name="dxl_lower_body_port"  default="/dev/ttyUSB0" />
-  <xacro:arg name="dxl_upper_body_port"  default="/dev/ttyUSB1" />
+  <xacro:arg name="dxl_x_lower_body_port"  default="/dev/ttyUSB0" />
+  <xacro:arg name="dxl_x_upper_body_port"  default="/dev/ttyUSB1" />
+  <xacro:arg name="dxl_p_upper_body_port"  default="/dev/ttyUSB2" />
   <xacro:if value="${ $(arg enable_mobile_base) }">
     <xacro:base/>

File: sobit_home_description/urdf/controllers.urdf.xacro (robot description, xacro)
@@ -10,11 +10,11 @@
           </xacro:if>
           <xacro:unless value="${$(arg enable_gz)}">
-            <xacro:property name="dxl_lower_body_port" value="$(arg dxl_lower_body_port)"/>
+            <xacro:property name="dxl_x_lower_body_port" value="$(arg dxl_x_lower_body_port)"/>
             <plugin>dynamixel_hardware/DynamixelHardware</plugin>
-            <param name="port_name">${dxl_lower_body_port}</param>
+            <param name="port_name">${dxl_x_lower_body_port}</param>
             <param name="baud_rate">1000000</param>
           </xacro:unless>
         </hardware>
-          <xacro:dx_wheel_steer_controllers prefix="wheel"      enable_gz="${$(arg enable_gz)}"/>
+          <xacro:dxl_wheel_steer_controllers prefix="wheel"      enable_gz="${$(arg enable_gz)}"/>
       </ros2_control>
     </xacro:if>
@@ -26,24 +26,45 @@
           </xacro:if>
           <xacro:unless value="${$(arg enable_gz)}">
-            <xacro:property name="dxl_upper_body_port" value="$(arg dxl_upper_body_port)"/>
+            <xacro:property name="dxl_x_upper_body_port" value="$(arg dxl_x_upper_body_port)"/>
             <plugin>dynamixel_hardware/DynamixelHardware</plugin>
-            <param name="port_name">${dxl_upper_body_port}</param>
+            <param name="port_name">${dxl_x_upper_body_port}</param>
             <param name="baud_rate">1000000</param>
           </xacro:unless>
         </hardware>
         <xacro:if value="${$(arg enable_head)}">
-          <xacro:dx_head_controllers        prefix="head"       enable_gz="${$(arg enable_gz)}"/>
+          <xacro:dxl_head_controllers        prefix="head"       enable_gz="${$(arg enable_gz)}"/>
         </xacro:if>
         <xacro:if value="${$(arg enable_arm_left)}">
-          <xacro:dx_arm_left_controllers    prefix="arm_left"   enable_gz="${$(arg enable_gz)}"/>
+          <xacro:dxl_arm_left_controllers    prefix="arm_left"   enable_gz="${$(arg enable_gz)}"/>
         </xacro:if>
         <xacro:if value="${$(arg enable_arm_right)}">
-          <xacro:dx_arm_right_controllers   prefix="arm_right"  enable_gz="${$(arg enable_gz)}"/>
+          <xacro:dxl_arm_right_controllers   prefix="arm_right"  enable_gz="${$(arg enable_gz)}"/>
         </xacro:if>
         <xacro:if value="${$(arg enable_hand_left)}">
-          <xacro:dx_hand_left_controllers   prefix="hand_left"  enable_gz="${$(arg enable_gz)}"/>
+          <xacro:dxl_hand_left_controllers   prefix="hand_left"  enable_gz="${$(arg enable_gz)}"/>
         </xacro:if>
         <xacro:if value="${$(arg enable_hand_right)}">
-          <xacro:dx_hand_right_controllers  prefix="hand_right" enable_gz="${$(arg enable_gz)}"/>
+          <xacro:dxl_hand_right_controllers  prefix="hand_right" enable_gz="${$(arg enable_gz)}"/>
+        </xacro:if>
+      </ros2_control>
+    </xacro:if>
+    <xacro:if value="${$(arg enable_arm_left) + $(arg enable_arm_right)}">
+      <ros2_control name="dynamixel_pro_upper" type="system">
+        <hardware>
+          <xacro:if value="${$(arg enable_gz)}">
+            <plugin>gz_ros2_control/GazeboSimSystem</plugin>
+          </xacro:if>
+          <xacro:unless value="${$(arg enable_gz)}">
+            <xacro:property name="dxl_p_upper_body_port" value="$(arg dxl_p_upper_body_port)"/>
+            <plugin>dynamixel_hardware/DynamixelHardware</plugin>
+            <param name="port_name">${dxl_p_upper_body_port}</param>
+            <param name="baud_rate">1000000</param>
+          </xacro:unless>
+        </hardware>
+        <xacro:if value="${$(arg enable_arm_left)}">
+          <xacro:dxl_pro_arm_left_controllers    prefix="arm_left"   enable_gz="${$(arg enable_gz)}"/>
+        </xacro:if>
+        <xacro:if value="${$(arg enable_arm_right)}">
+          <xacro:dxl_pro_arm_right_controllers   prefix="arm_right"  enable_gz="${$(arg enable_gz)}"/>
         </xacro:if>
       </ros2_control>
@@ -158,5 +179,5 @@
     </joint>
   </xacro:macro>
-  <xacro:macro name="dx_wheel_steer_controllers"  params="prefix enable_gz:=False">
+  <xacro:macro name="dxl_wheel_steer_controllers"  params="prefix enable_gz:=False">
     <joint name="${prefix}_steer_f_l_joint">
       <xacro:unless value="${$(arg enable_gz)}">
@@ -228,5 +249,5 @@
     </joint>
   </xacro:macro>
-  <xacro:macro name="dx_head_controllers"         params="prefix enable_gz:=False">
+  <xacro:macro name="dxl_head_controllers"         params="prefix enable_gz:=False">
     <joint name="head_pan_joint">
       <xacro:unless value="${$(arg enable_gz)}">
@@ -264,5 +285,5 @@
     </joint>
   </xacro:macro>
-  <xacro:macro name="dx_arm_left_controllers"     params="prefix enable_gz:=False">
+  <xacro:macro name="dxl_pro_arm_left_controllers"     params="prefix enable_gz:=False">
     <joint name="${prefix}_shoulder_tilt_joint">
       <xacro:unless value="${$(arg enable_gz)}">
@@ -282,4 +303,25 @@
       <state_interface name="effort"/>
     </joint>
+  </xacro:macro>
+  <xacro:macro name="dxl_pro_arm_right_controllers"    params="prefix enable_gz:=False">
+    <joint name="${prefix}_shoulder_tilt_joint">
+      <xacro:unless value="${$(arg enable_gz)}">
+        <param name="id">41</param>
+        <param name="control_mode">0</param>
+        <param name="interface">rs</param>
+      </xacro:unless>
+      <command_interface name="position">
+        <param name="min">-${M_PI/2}</param>
+        <param name="max">${M_PI/2}</param>
+      </command_interface>
+      <!-- <command_interface name="velocity"/> -->
+      <state_interface name="position">
+        <param name="initial_value">0.0</param>
+      </state_interface>
+      <state_interface name="velocity"/>
+      <state_interface name="effort"/>
+    </joint>
+  </xacro:macro>
+  <xacro:macro name="dxl_arm_left_controllers"     params="prefix enable_gz:=False">
     <joint name="${prefix}_upper_roll_joint">
       <xacro:unless value="${$(arg enable_gz)}">
@@ -333,5 +375,4 @@
       <state_interface name="effort"/>
     </joint>
-<!-- rename joint : tsukada -->
     <joint name="${prefix}_wrist_tilt_joint">
       <xacro:unless value="${$(arg enable_gz)}">
@@ -351,5 +392,4 @@
       <state_interface name="effort"/>
     </joint>
-<!-- add joint : tsukada -->
     <joint name="${prefix}_wrist_roll_joint">
       <xacro:unless value="${$(arg enable_gz)}">
@@ -370,22 +410,5 @@
     </joint>
   </xacro:macro>
-  <xacro:macro name="dx_arm_right_controllers"    params="prefix enable_gz:=False">
-    <joint name="${prefix}_shoulder_tilt_joint">
-      <xacro:unless value="${$(arg enable_gz)}">
-        <param name="id">41</param>
-        <param name="control_mode">0</param>
-        <param name="interface">rs</param>
-      </xacro:unless>
-      <command_interface name="position">
-        <param name="min">-${M_PI/2}</param>
-        <param name="max">${M_PI/2}</param>
-      </command_interface>
-      <!-- <command_interface name="velocity"/> -->
-      <state_interface name="position">
-        <param name="initial_value">0.0</param>
-      </state_interface>
-      <state_interface name="velocity"/>
-      <state_interface name="effort"/>
-    </joint>
+  <xacro:macro name="dxl_arm_right_controllers"    params="prefix enable_gz:=False">
     <joint name="${prefix}_upper_roll_joint">
       <xacro:unless value="${$(arg enable_gz)}">
@@ -439,5 +462,4 @@
       <state_interface name="effort"/>
     </joint>
-<!-- rename joint : tsukada -->
     <joint name="${prefix}_wrist_tilt_joint">
       <xacro:unless value="${$(arg enable_gz)}">
@@ -457,5 +479,4 @@
       <state_interface name="effort"/>
     </joint>
-<!-- add joint : tsukada -->
     <joint name="${prefix}_wrist_roll_joint">
       <xacro:unless value="${$(arg enable_gz)}">
@@ -476,5 +497,5 @@
     </joint>
   </xacro:macro>
-  <xacro:macro name="dx_hand_left_controllers"    params="prefix enable_gz:=False">
+  <xacro:macro name="dxl_hand_left_controllers"    params="prefix enable_gz:=False">
     <joint name="${prefix}_finger_l_mcp_joint">
       <xacro:unless value="${$(arg enable_gz)}">
@@ -596,5 +617,5 @@
       <state_interface name="effort"/>
     </joint>
-      <joint name="${prefix}_finger_r_dip_joint">
+    <joint name="${prefix}_finger_r_dip_joint">
       <xacro:unless value="${$(arg enable_gz)}">
         <param name="id">56</param>
@@ -615,5 +636,5 @@
     </joint>
   </xacro:macro>
-  <xacro:macro name="dx_hand_right_controllers"   params="prefix enable_gz:=False">
+  <xacro:macro name="dxl_hand_right_controllers"   params="prefix enable_gz:=False">
     <joint name="${prefix}_finger_l_mcp_joint">
       <xacro:unless value="${$(arg enable_gz)}">

Commit message: [UPD] Head & Mic URDF

File: sobit_home_description/robots/sobit_home_robot.urdf.xacro (robot description, xacro)
@@ -15,5 +15,5 @@
   <xacro:include filename="$(find sobit_home_description)/urdf/head/head.urdf.xacro" />
   <xacro:include filename="$(find sobit_home_description)/urdf/sensor/camera_head.urdf.xacro" />
-  <!-- <xacro:include filename="$(find sobit_home_description)/urdf/sensor/mic.urdf.xacro" /> -->
+  <xacro:include filename="$(find sobit_home_description)/urdf/sensor/mic.urdf.xacro" />
   <xacro:include filename="$(find sobit_home_description)/urdf/sensor/lidar.urdf.xacro" />
   <!-- <xacro:include filename="$(find sobit_home_description)/urdf/sensor/realsense_d405.urdf.xacro" /> -->
@@ -99,5 +99,5 @@
   <xacro:if value="${ $(arg enable_head) }">
     <xacro:head  prefix="head"  parent="body_lift_link" />
-    <!-- <xacro:mic   prefix="mic"   parent="head_tilt_link" />  -->
+    <xacro:mic   prefix="mic"   parent="head_tilt_link" />
     <xacro:camera_head  prefix="head"  parent="head_tilt_link" />
   </xacro:if>

File: sobit_home_description/urdf/head/head.urdf.xacro (robot description, xacro)
@@ -40,5 +40,5 @@
     <link name="${prefix}_pan_link">
       <visual>
-        <origin xyz="0.0 0.0 -0.0272" rpy="0.0 0.0 ${M_PI/2.0}" />
+        <origin xyz="0.0 0.0 0.0" rpy="0.0 0.0 ${M_PI/2.0}" />
         <geometry>
           <mesh filename="file://$(find sobit_home_description)/meshes/head/neck.stl" scale="0.001 0.001 0.001" />
@@ -75,4 +75,25 @@
         <material name="black" />
       </visual>
+      <visual>
+        <origin xyz="0.0 0.0 0.0" rpy="0.0 0.0 ${M_PI/2.0}" />
+        <geometry>
+          <mesh filename="file://$(find sobit_home_description)/meshes/head/ear.dae"/>
+        </geometry>
+        <!-- <material name="blue" /> -->
+      </visual>
+      <visual>
+        <origin xyz="0.07815 0.05 0.0" rpy="0.0 0.0 ${M_PI/2.0}" />
+        <geometry>
+          <mesh filename="file://$(find sobit_home_description)/meshes/head/eye.dae"/>
+        </geometry>
+        <!-- <material name="blue" /> -->
+      </visual>
+      <visual>
+        <origin xyz="0.07815 -0.05 0.0" rpy="0.0 0.0 ${M_PI/2.0}" />
+        <geometry>
+          <mesh filename="file://$(find sobit_home_description)/meshes/head/eye.dae"/>
+        </geometry>
+        <!-- <material name="blue" /> -->
+      </visual>
       <collision>
         <origin xyz="-0.01 0.0 0.00943" rpy="0.0 0.0 0.0" />

File: sobit_home_description/urdf/sensor/mic.urdf.xacro (robot description, xacro)
@@ -35,5 +35,5 @@
       <parent link="${prefix}_base_link" />
       <child link="${prefix}_link" />
-      <origin xyz="0.0 0.0 0.005" rpy="0.0 0.0 0.0" />
+      <origin xyz="0.0 0.0 0.0" rpy="0.0 0.0 0.0" />
     </joint>
     <link name="${prefix}_link">
@@ -41,7 +41,14 @@
         <origin xyz="0.0 0.0 0.0" rpy="0.0 0.0 ${M_PI/2.0}" />
         <geometry>
-          <mesh filename="file://$(find sobit_home_description)/meshes/sensor/mic_base.stl" scale="0.001 0.001 0.001" />
+          <mesh filename="file://$(find sobit_home_description)/meshes/sensor/mic_rode.stl" scale="0.001 0.001 0.001" />
         </geometry>
         <material name="black" />
+      </visual>
+      <visual>
+        <origin xyz="0.0 0.0 0.0" rpy="0.0 0.0 ${M_PI/2.0}" />
+        <geometry>
+          <mesh filename="file://$(find sobit_home_description)/meshes/sensor/mic_mount.dae" />
+        </geometry>
+        <!-- <material name="black" /> -->
       </visual>
       <!-- <collision>

Commit message: fix: body joint position when enable body False

File: sobit_home_description/robots/sobit_home_robot.urdf.xacro (robot description, xacro)
@@ -63,5 +63,5 @@
   <xacro:unless value="${ $(arg enable_body) }">
     <joint name="body_joint" type="fixed" >
-      <origin xyz="0.11275 0.0 0.565" rpy="0.0 0.0 0.0" />
+      <origin xyz="-0.1702 0.0 0.3169" rpy="0.0 0.0 0.0" />
       <parent link="plate_top_link" />
       <child link="body_lift_link" />

Commit message: [ADD] lidar_merged_laser frame to SOBIT HOME robot description

File: sobit_home_description/robots/sobit_home_robot.urdf.xacro (robot description, xacro)
@@ -45,4 +45,10 @@
   <xacro:if value="${ $(arg enable_mobile_base) }">
     <xacro:base/>
+    <joint name="lidar_merged_joint" type="fixed">
+      <origin xyz="0.0 0.0 0.185" rpy="0.0 0.0 0.0" />
+      <parent link="base_footprint" />
+      <child link="lidar_merged_laser" />
+    </joint>
+    <link name="lidar_merged_laser" />
     <xacro:plate prefix="plate" parent="base_link" />
     <xacro:wheel prefix="wheel" parent="plate_middle_link" />
@@ -51,4 +57,10 @@
   <xacro:unless value="${ $(arg enable_mobile_base) }">
     <xacro:base/>
+    <joint name="lidar_merged_joint" type="fixed">
+      <origin xyz="0.0 0.0 0.185" rpy="0.0 0.0 0.0" />
+      <parent link="base_footprint" />
+      <child link="lidar_merged_laser" />
+    </joint>
+    <link name="lidar_merged_laser" />
     <joint name="plate_top_joint" type="fixed" >
       <origin xyz="0.0 0.0 0.371058" rpy="0.0 0.0 0.0" />

Commit message: Add config for body lift joint

File: sobit_home_description/robots/sobit_home_robot.urdf.xacro (robot description, xacro)
@@ -43,4 +43,6 @@
   <xacro:arg name="dxl_x_upper_body_port"  default="/dev/ttyUSB1" />
   <xacro:arg name="dxl_p_upper_body_port"  default="/dev/ttyUSB2" />
+  <!-- Uirobot Motors Ports -->
+  <xacro:arg name="um_body_port" default="/dev/ttyUSB3" />
   <xacro:if value="${ $(arg enable_mobile_base) }">
     <xacro:base/>

File: sobit_home_description/urdf/controllers.urdf.xacro (robot description, xacro)
@@ -91,12 +91,12 @@
             <plugin>gz_ros2_control/GazeboSimSystem</plugin>
           </xacro:if>
-          <!-- TODO - Develop IAI controller -->
-          <!-- <xacro:unless value="${$(arg enable_gz)}">
-            <plugin>iai_hardware/IaiHardware</plugin>
-            <param name="port_name">/dev/ttyUSB1</param>
-            <param name="baud_rate">115200</param>
-          </xacro:unless> -->
+          <xacro:unless value="${$(arg enable_gz)}">
+            <xacro:property name="um_body_port" value="$(arg um_body_port)"/>
+            <plugin>uirobot_hardware/UirobotHardware</plugin>
+            <param name="port_name">${um_body_port}</param>
+            <param name="baud_rate">57600</param>
+          </xacro:unless>
         </hardware>
-        <xacro:iai_body_controllers prefix="body" enable_gz="${$(arg enable_gz)}"/>
+        <xacro:uirobot_control prefix="body" enable_gz="${$(arg enable_gz)}"/>
       </ros2_control>
     </xacro:if>
@@ -803,12 +803,10 @@
     </joint>
   </xacro:macro>
-  <xacro:macro name="iai_body_controllers"        params="prefix enable_gz:=False">
+  <xacro:macro name="uirobot_control" params="prefix enable_gz:=False">
     <joint name="${prefix}_lift_joint">
-      <!-- TODO - Develop IAI controller -->
-      <!-- <xacro:unless value="${$(arg enable_gz)}">
-        <param name="id">1</param>
-        <param name="control_mode">0</param>
-        <param name="interface">rs</param>
-      </xacro:unless> -->
+      <xacro:unless value="${$(arg enable_gz)}">
+        <param name="id">5</param>
+        <param name="gear_ratio">${200*M_PI}</param>
+      </xacro:unless>
       <command_interface name="position">
         <param name="min">0.0</param>
