Commit message: [UPD] param name, add hand cam

File: sobit_home_description/robots/sobit_home_robot.urdf.xacro (robot description, xacro)
@@ -17,4 +17,5 @@
   <xacro:include filename="$(find sobit_home_description)/urdf/sensor/mic.urdf.xacro" />
   <xacro:include filename="$(find sobit_home_description)/urdf/sensor/lidar.urdf.xacro" />
+  <xacro:include filename="$(find sobit_home_description)/urdf/sensor/camera_hand.urdf.xacro" />
   <!-- <xacro:include filename="$(find sobit_home_description)/urdf/sensor/realsense_d405.urdf.xacro" /> -->
   <xacro:include filename="$(find urg_node)/urdf/hokuyo_ust.urdf.xacro" />
@@ -25,10 +26,8 @@
   <xacro:arg name="robot_name" default="sobit_home" />
   <xacro:arg name="enable_gz"                       default="True" />
-  <xacro:arg name="enable_gz_head_cam_color"        default="True" />
-  <xacro:arg name="enable_gz_head_cam_depth"        default="True" />
-  <xacro:arg name="enable_gz_hand_left_cam_color"   default="False" />
-  <xacro:arg name="enable_gz_hand_left_cam_depth"   default="False" />
-  <xacro:arg name="enable_gz_hand_right_cam_color"  default="False" />
-  <xacro:arg name="enable_gz_hand_right_cam_depth"  default="False" />
+  <xacro:arg name="enable_head_cam_color"        default="True" />
+  <xacro:arg name="enable_head_cam_depth"        default="True" />
+  <xacro:arg name="enable_hand_left_cam_color"   default="True" />
+  <xacro:arg name="enable_hand_right_cam_color"  default="True" />
   <!-- Activate Components -->
   <xacro:arg name="enable_mobile_base"  default="True" />
@@ -83,4 +82,7 @@
   <xacro:if value="${ $(arg enable_arm_left) }">
     <xacro:arm   prefix="arm"   position="left"  parent="body_lift_link" />
+    <xacro:camera_hand prefix="hand_left" parent="arm_left_wrist_roll_link">
+      <origin xyz="0.03475112 0.0305 -0.017" rpy="0.0 0.970255199812 0.0"/>
+    </xacro:camera_hand>
   </xacro:if>
   <xacro:unless value="${ $(arg enable_arm_left) }">
@@ -94,4 +96,7 @@
   <xacro:if value="${ $(arg enable_arm_right) }">
     <xacro:arm   prefix="arm"   position="right" parent="body_lift_link" />
+    <xacro:camera_hand prefix="hand_right" parent="arm_right_wrist_roll_link">
+      <origin xyz="-0.00174888 -0.0305 -0.042" rpy="${M_PI} 0.970255199812 0.0"/>
+    </xacro:camera_hand>
   </xacro:if>
   <xacro:unless value="${ $(arg enable_arm_right) }">
@@ -119,10 +124,8 @@
   <xacro:if value="${$(arg enable_gz)}">
     <xacro:gazebo_sensors robot_name="$(arg robot_name)"
-      enable_gz_head_cam_color="$(arg enable_gz_head_cam_color)"
-      enable_gz_head_cam_depth="$(arg enable_gz_head_cam_depth)"
-      enable_gz_hand_left_cam_color="$(arg enable_gz_hand_left_cam_color)"
-      enable_gz_hand_left_cam_depth="$(arg enable_gz_hand_left_cam_depth)"
-      enable_gz_hand_right_cam_color="$(arg enable_gz_hand_right_cam_color)"
-      enable_gz_hand_right_cam_depth="$(arg enable_gz_hand_right_cam_depth)"
+      enable_head_cam_color="$(arg enable_head_cam_color)"
+      enable_head_cam_depth="$(arg enable_head_cam_depth)"
+      enable_hand_left_cam_color="$(arg enable_hand_left_cam_color)"
+      enable_hand_right_cam_color="$(arg enable_hand_right_cam_color)"
     />
   </xacro:if>

File: sobit_home_description/urdf/gazebo.urdf.xacro (robot description, xacro)
@@ -2,7 +2,7 @@
 <!-- SOBIT HOME (Gazebo) -->
 <robot name="sobit_home_gazebo" xmlns:xacro="http://ros.org/wiki/xacro">
-  <xacro:macro name="gazebo_sensors" params="robot_name enable_gz_head_cam_color:=True enable_gz_head_cam_depth:=True enable_gz_hand_left_cam_color:=True enable_gz_hand_left_cam_depth:=True enable_gz_hand_right_cam_color:=True enable_gz_hand_right_cam_depth:=True">
+  <xacro:macro name="gazebo_sensors" params="robot_name enable_head_cam_color:=True enable_head_cam_depth:=True enable_hand_left_cam_color:=True enable_hand_right_cam_color:=True">
     <!-- Sensor - Head Camera (Color) -->
-    <xacro:if value="${enable_gz_head_cam_color}">
+    <xacro:if value="${enable_head_cam_color}">
       <gazebo reference="head_camera_color_optical_frame">
         <sensor name="head_camera_color" type="camera">
@@ -36,5 +36,5 @@
     </xacro:if>
     <!-- Sensor - Head Camera (Depth) -->
-    <xacro:if value="${enable_gz_head_cam_depth}">
+    <xacro:if value="${enable_head_cam_depth}">
       <gazebo reference="head_camera_depth_optical_frame">
         <sensor name="head_camera_depth" type="depth_camera">
@@ -66,63 +66,54 @@
       </gazebo>
     </xacro:if>
-    <!-- Sensor - Hand Left Camera (Color) -->
-    <xacro:if value="${enable_gz_hand_left_cam_color}">
-      <gazebo reference="hand_camera_color_optical_frame">
-        <sensor name="hand_camera_color" type="camera">
-          <pose>0 0 ${0.0175/2} ${M_PI/2} -${M_PI/2} 0 </pose>
-          <!-- <ignition_frame_id>${robot_name}/hand_camera_color_optical_frame</ignition_frame_id> -->
-          <gz_frame_id>${robot_name}/hand_camera_color_optical_frame</gz_frame_id>
-          <topic>${robot_name}/hand_camera/color</topic>
+    <!-- Sensor - Wrist Left Camera (ELP-USBGS1200P01-H120, Color) -->
+    <!-- AR0234 Global Shutter, HFOV 126 deg (2.19911 rad), 1920x1200 @ 90fps -->
+    <xacro:if value="${enable_hand_left_cam_color}">
+      <gazebo reference="hand_left_camera_optical_frame">
+        <sensor name="hand_left_camera_color" type="camera">
+          <pose>0 0 0 ${M_PI/2} -${M_PI/2} ${M_PI}</pose>
+          <gz_frame_id>${robot_name}/hand_left_camera_optical_frame</gz_frame_id>
+          <topic>${robot_name}/hand_left_camera/color</topic>
           <always_on>1</always_on>
           <visualize>true</visualize>
           <update_rate>1</update_rate>
-          <camera name="hand_camera_color">
-            <horizontal_fov>1.21126</horizontal_fov>
+          <camera name="hand_left_camera_color">
+            <!-- ELP-USBGS1200P01-H120: HFOV 126 deg -->
+            <horizontal_fov>2.19911</horizontal_fov>
             <image>
-              <width>640</width>
-              <height>480</height>
+              <width>1920</width>
+              <height>1200</height>
               <format>RGB_INT8</format>
             </image>
             <clip>
-              <near>0.1</near>
-              <far>10</far>
+              <near>0.01</near>
+              <!-- <far>10</far> -->
             </clip>
-            <!-- TODO - adjust noise -->
-            <!-- <noise>
-              <type>gaussian</type>
-              <mean>0</mean>
-              <stddev>0.007</stddev>
-            </noise> -->
           </camera>
         </sensor>
       </gazebo>
     </xacro:if>
-    <!-- Sensor - Hand Left Camera (Depth) -->
-    <xacro:if value="${enable_gz_hand_left_cam_depth}">
-      <gazebo reference="hand_camera_depth_optical_frame">
-        <sensor name="hand_camera_depth" type="depth">
-          <pose>0 0 ${0.0175/2} ${M_PI/2} -${M_PI/2} 0 </pose>
-          <!-- <ignition_frame_id>${robot_name}/hand_camera_depth_optical_frame</ignition_frame_id> -->
-          <gz_frame_id>${robot_name}/hand_camera_depth_optical_frame</gz_frame_id>
-          <topic>${robot_name}/hand_camera/depth</topic>
+    <!-- Sensor - Wrist Right Camera (ELP-USBGS1200P01-H120, Color) -->
+    <!-- AR0234 Global Shutter, HFOV 126 deg (2.19911 rad), 1920x1200 @ 90fps -->
+    <xacro:if value="${enable_hand_right_cam_color}">
+      <gazebo reference="hand_right_camera_optical_frame">
+        <sensor name="hand_right_camera_color" type="camera">
+          <pose>0 0 0 ${M_PI/2} -${M_PI/2} ${M_PI}</pose>
+          <gz_frame_id>${robot_name}/hand_right_camera_optical_frame</gz_frame_id>
+          <topic>${robot_name}/hand_right_camera/color</topic>
           <always_on>1</always_on>
           <visualize>true</visualize>
           <update_rate>1</update_rate>
-          <camera name="head_camera_depth">
-            <horizontal_fov>1.48702</horizontal_fov>
+          <camera name="hand_right_camera_color">
+            <!-- ELP-USBGS1200P01-H120: HFOV 126 deg -->
+            <horizontal_fov>2.19911</horizontal_fov>
             <image>
-              <width>1280</width>
-              <height>720</height>
+              <width>1920</width>
+              <height>1200</height>
+              <format>RGB_INT8</format>
             </image>
             <clip>
-              <near>0.1</near>
-              <far>10</far>
+              <near>0.01</near>
+              <!-- <far>10</far> -->
             </clip>
-            <!-- TODO - adjust noise -->
-            <!-- <noise>
-              <type>gaussian</type>
-              <mean>0</mean>
-              <stddev>0.1</stddev>
-            </noise> -->
           </camera>
         </sensor>

Commit message: [FEAT] split hand usb

File: sobit_home_description/robots/sobit_home_robot.urdf.xacro (robot description, xacro)
@@ -44,6 +44,7 @@
   <xacro:arg name="dxl_x_upper_body_port"  default="/dev/ttyUSB1" />
   <xacro:arg name="dxl_p_upper_body_port"  default="/dev/ttyUSB2" />
+  <xacro:arg name="dxl_x_hand_port"        default="/dev/ttyUSB3" />
   <!-- Uirobot Body Lift Gateway Port -->
-  <xacro:arg name="um_body_port" default="/dev/ttyUSB3" />
+  <xacro:arg name="um_body_port" default="/dev/ttyUSB4" />
   <xacro:arg name="um_body_id" default="5" />
   <xacro:if value="${ $(arg enable_mobile_base) }">

File: sobit_home_description/urdf/controllers.urdf.xacro (robot description, xacro)
@@ -22,5 +22,5 @@
       </ros2_control>
     </xacro:if>
-    <xacro:if value="${$(arg enable_head) + $(arg enable_arm_left) + $(arg enable_arm_right) + $(arg enable_hand_left) + $(arg enable_hand_right)}">
+    <xacro:if value="${$(arg enable_head) + $(arg enable_arm_left) + $(arg enable_arm_right)}">
       <ros2_control name="dynamixel_upper" type="system" is_async="true">
         <properties>
@@ -47,4 +47,22 @@
           <xacro:dxl_arm_right_controllers   prefix="arm_right"  enable_gz="${$(arg enable_gz)}"/>
         </xacro:if>
+      </ros2_control>
+    </xacro:if>
+    <xacro:if value="${$(arg enable_hand_left) + $(arg enable_hand_right)}">
+      <ros2_control name="dynamixel_hand" type="system" is_async="true">
+        <properties>
+          <async scheduling_policy="synchronized" thread_priority="79" affinity="[5]" print_warnings="true"/>
+        </properties>
+        <hardware>
+          <xacro:if value="${$(arg enable_gz)}">
+            <plugin>gz_ros2_control/GazeboSimSystem</plugin>
+          </xacro:if>
+          <xacro:unless value="${$(arg enable_gz)}">
+            <xacro:property name="dxl_x_hand_port" value="$(arg dxl_x_hand_port)"/>
+            <plugin>dynamixel_hardware/DynamixelHardware</plugin>
+            <param name="port_name">${dxl_x_hand_port}</param>
+            <param name="baud_rate">4000000</param>
+          </xacro:unless>
+        </hardware>
         <xacro:if value="${$(arg enable_hand_left)}">
           <xacro:dxl_hand_left_controllers   prefix="hand_left"  enable_gz="${$(arg enable_gz)}"/>

Commit message: [UPD] Update arm limitation, adjust port settings and update Dynamixel settings.

File: sobit_home_description/robots/sobit_home_robot.urdf.xacro (robot description, xacro)
@@ -41,10 +41,12 @@
   <xacro:arg name="enable_dxl_pro"      default="True" />
   <!-- DXL Ports -->
-  <xacro:arg name="dxl_x_lower_body_port"  default="/dev/ttyUSB0" />
-  <xacro:arg name="dxl_x_upper_body_port"  default="/dev/ttyUSB1" />
+  <xacro:arg name="dxl_x_lower_body_port"  default="/dev/ttyUSB1" />
+  <xacro:arg name="dxl_x_upper_body_port"  default="/dev/ttyUSB3" />
   <xacro:arg name="dxl_p_upper_body_port"  default="/dev/ttyUSB2" />
-  <xacro:arg name="dxl_x_hand_port"        default="/dev/ttyUSB3" />
+  <xacro:arg name="dxl_x_hand_port"        default="/dev/ttyUSB4" />
+  <!-- <xacro:arg name="dxl_x_hand_port"        default="/dev/ttyUSB3" /> -->
   <!-- Uirobot Body Lift Gateway Port -->
-  <xacro:arg name="um_body_port" default="/dev/ttyUSB4" />
+  <!-- <xacro:arg name="um_body_port" default="/dev/ttyUSB4" /> -->
+  <xacro:arg name="um_body_port" default="/dev/ttyUSB0" />
   <xacro:arg name="um_body_id" default="5" />
   <xacro:if value="${ $(arg enable_mobile_base) }">

File: sobit_home_description/urdf/arm/arm.urdf.xacro (robot description, xacro)
@@ -126,5 +126,5 @@
       <origin xyz="-0.0510 ${y_sign * 0.1135} 0.0" rpy="0.0 0.0 0.0" />
       <axis xyz="0.0 -1.0 0.0" />
-      <limit lower="${-M_PI/2}" upper="${M_PI/2}" effort="${10.6 * effort_ratio}" velocity="3.14" />
+      <limit lower="${-M_PI}" upper="0" effort="${10.6 * effort_ratio}" velocity="3.14" />
     </joint>
     <link name="${prefix}_${position}_upper_flex_link" >

File: sobit_home_description/urdf/controllers.urdf.xacro (robot description, xacro)
@@ -130,5 +130,5 @@
             <plugin>uirobot_hardware/UirobotHardware</plugin>
             <param name="port_name">${um_body_port}</param>
-            <param name="baud_rate">57600</param>
+            <param name="baud_rate">115200</param>
             <param name="toggle_torque_on_configure">false</param>
             <param name="enable_torque_before_motion">false</param>
@@ -329,4 +329,5 @@
         <param name="interface">rs</param>
         <param name="Return_Delay_Time">0</param>
+        <param name="Drive_Mode">1</param>
       </xacro:unless>
       <command_interface name="position">
@@ -367,4 +368,5 @@
         <param name="interface">rs</param>
         <param name="Return_Delay_Time">0</param>
+        <param name="drive_mode">1</param>
       </xacro:unless>
       <command_interface name="position">
@@ -399,4 +401,5 @@
         <param name="interface">rs</param>
         <param name="Return_Delay_Time">0</param>
+        <param name="Drive_Mode">1</param>
       </xacro:unless>
       <command_interface name="position">
@@ -412,5 +415,5 @@
     <joint name="${prefix}_upper_flex_sub_joint">
       <param name="mimic">${prefix}_upper_flex_joint</param>
-      <param name="multiplier">-1</param>
+      <param name="multiplier">1</param>
       <xacro:unless value="${$(arg enable_gz)}">
         <param name="id">35</param>
@@ -431,4 +434,5 @@
         <param name="interface">rs</param>
         <param name="Return_Delay_Time">0</param>
+        <param name="Drive_Mode">1</param>
       </xacro:unless>
       <command_interface name="position">
@@ -463,4 +467,5 @@
         <param name="interface">rs</param>
         <param name="Return_Delay_Time">0</param>
+        <param name="Drive_Mode">1</param>
       </xacro:unless>
       <command_interface name="position">
@@ -480,4 +485,5 @@
         <param name="interface">rs</param>
         <param name="Return_Delay_Time">0</param>
+        <param name="Drive_Mode">1</param>
       </xacro:unless>
       <command_interface name="position">
@@ -497,4 +503,5 @@
         <param name="interface">rs</param>
         <param name="Return_Delay_Time">0</param>
+        <param name="Drive_Mode">1</param>
       </xacro:unless>
       <command_interface name="position">
@@ -550,6 +557,6 @@
       </xacro:unless>
       <command_interface name="position">
-        <param name="min">-${M_PI/2}</param>
-        <param name="max">${M_PI/2}</param>
+        <param name="min">-${M_PI}</param>
+        <param name="max">0</param>
       </command_interface>
       <state_interface name="position">
@@ -561,5 +568,5 @@
     <joint name="${prefix}_upper_flex_sub_joint">
       <param name="mimic">${prefix}_upper_flex_joint</param>
-      <param name="multiplier">-1</param>
+      <param name="multiplier">1</param>
       <xacro:unless value="${$(arg enable_gz)}">
         <param name="id">45</param>
@@ -661,7 +668,7 @@
     <joint name="${prefix}_finger_l_mcp_joint">
       <xacro:unless value="${$(arg enable_gz)}">
-        <param name="id">50</param>
-        <param name="control_mode">6</param>
-        <param name="Goal_Current">300</param>
+        <param name="id">51</param>
+        <param name="control_mode">6</param>
+        <param name="Goal_Current">100</param>
         <param name="interface">ttl</param>
         <param name="Return_Delay_Time">0</param>
@@ -688,7 +695,7 @@
     <joint name="${prefix}_finger_l_pip_joint">
       <xacro:unless value="${$(arg enable_gz)}">
-        <param name="id">51</param>
-        <param name="control_mode">6</param>
-        <param name="Goal_Current">150</param>
+        <param name="id">52</param>
+        <param name="control_mode">6</param>
+        <param name="Goal_Current">50</param>
         <param name="interface">ttl</param>
         <param name="Return_Delay_Time">0</param>
@@ -706,7 +713,7 @@
     <joint name="${prefix}_finger_l_dip_joint">
       <xacro:unless value="${$(arg enable_gz)}">
-        <param name="id">52</param>
-        <param name="control_mode">6</param>
-        <param name="Goal_Current">100</param>
+        <param name="id">53</param>
+        <param name="control_mode">6</param>
+        <param name="Goal_Current">55</param>
         <param name="interface">ttl</param>
         <param name="Return_Delay_Time">0</param>
@@ -724,7 +731,7 @@
     <joint name="${prefix}_finger_c_mcp_joint">
       <xacro:unless value="${$(arg enable_gz)}">
-        <param name="id">53</param>
-        <param name="control_mode">6</param>
-        <param name="Goal_Current">225</param>
+        <param name="id">54</param>
+        <param name="control_mode">6</param>
+        <param name="Goal_Current">50</param>
         <param name="interface">ttl</param>
         <param name="Return_Delay_Time">0</param>
@@ -742,7 +749,7 @@
     <joint name="${prefix}_finger_c_ip_joint">
       <xacro:unless value="${$(arg enable_gz)}">
-        <param name="id">54</param>
-        <param name="control_mode">6</param>
-        <param name="Goal_Current">150</param>
+        <param name="id">55</param>
+        <param name="control_mode">6</param>
+        <param name="Goal_Current">55</param>
         <param name="interface">ttl</param>
         <param name="Return_Delay_Time">0</param>
@@ -760,7 +767,7 @@
     <joint name="${prefix}_finger_r_pip_joint">
       <xacro:unless value="${$(arg enable_gz)}">
-        <param name="id">55</param>
-        <param name="control_mode">6</param>
-        <param name="Goal_Current">150</param>
+        <param name="id">56</param>
+        <param name="control_mode">6</param>
+        <param name="Goal_Current">50</param>
         <param name="interface">ttl</param>
         <param name="Return_Delay_Time">0</param>
@@ -778,7 +785,7 @@
     <joint name="${prefix}_finger_r_dip_joint">
       <xacro:unless value="${$(arg enable_gz)}">
-        <param name="id">56</param>
-        <param name="control_mode">6</param>
-        <param name="Goal_Current">100</param>
+        <param name="id">57</param>
+        <param name="control_mode">6</param>
+        <param name="Goal_Current">55</param>
         <param name="interface">ttl</param>
         <param name="Return_Delay_Time">0</param>
@@ -798,7 +805,7 @@
     <joint name="${prefix}_finger_l_mcp_joint">
       <xacro:unless value="${$(arg enable_gz)}">
-        <param name="id">60</param>
-        <param name="control_mode">6</param>
-        <param name="Goal_Current">300</param>
+        <param name="id">61</param>
+        <param name="control_mode">6</param>
+        <param name="Goal_Current">100</param>
         <param name="interface">ttl</param>
         <param name="Return_Delay_Time">0</param>
@@ -825,7 +832,7 @@
     <joint name="${prefix}_finger_l_pip_joint">
       <xacro:unless value="${$(arg enable_gz)}">
-        <param name="id">61</param>
-        <param name="control_mode">6</param>
-        <param name="Goal_Current">200</param>
+        <param name="id">62</param>
+        <param name="control_mode">6</param>
+        <param name="Goal_Current">50</param>
         <param name="interface">ttl</param>
         <param name="Return_Delay_Time">0</param>
@@ -843,7 +850,7 @@
     <joint name="${prefix}_finger_l_dip_joint">
       <xacro:unless value="${$(arg enable_gz)}">
-        <param name="id">62</param>
-        <param name="control_mode">6</param>
-        <param name="Goal_Current">50</param>
+        <param name="id">63</param>
+        <param name="control_mode">6</param>
+        <param name="Goal_Current">55</param>
         <param name="interface">ttl</param>
         <param name="Return_Delay_Time">0</param>
@@ -861,5 +868,5 @@
     <joint name="${prefix}_finger_c_mcp_joint">
       <xacro:unless value="${$(arg enable_gz)}">
-        <param name="id">63</param>
+        <param name="id">64</param>
         <param name="control_mode">6</param>
         <param name="Goal_Current">50</param>
@@ -879,7 +886,7 @@
     <joint name="${prefix}_finger_c_ip_joint">
       <xacro:unless value="${$(arg enable_gz)}">
-        <param name="id">64</param>
-        <param name="control_mode">6</param>
-        <param name="Goal_Current">50</param>
+        <param name="id">65</param>
+        <param name="control_mode">6</param>
+        <param name="Goal_Current">55</param>
         <param name="interface">ttl</param>
         <param name="Return_Delay_Time">0</param>
@@ -897,5 +904,5 @@
     <joint name="${prefix}_finger_r_pip_joint">
       <xacro:unless value="${$(arg enable_gz)}">
-        <param name="id">65</param>
+        <param name="id">66</param>
         <param name="control_mode">6</param>
         <param name="Goal_Current">50</param>
@@ -915,7 +922,7 @@
     <joint name="${prefix}_finger_r_dip_joint">
       <xacro:unless value="${$(arg enable_gz)}">
-        <param name="id">66</param>
-        <param name="control_mode">6</param>
-        <param name="Goal_Current">50</param>
+        <param name="id">67</param>
+        <param name="control_mode">6</param>
+        <param name="Goal_Current">55</param>
         <param name="interface">ttl</param>
         <param name="Return_Delay_Time">0</param>
@@ -938,7 +945,8 @@
         <param name="gear_ratio">${200*M_PI}</param>
         <param name="position_kp">0.7</param>
-        <param name="stop_threshold">0.005</param>
+        <param name="stop_threshold">0.00005</param>
         <param name="min_velocity">0.01</param> <!-- [m/s], 1 cm in 1 s is smooth; slower tends to stall -->
-        <param name="max_velocity">0.025</param> <!-- [m/s] -->
+        <param name="max_velocity">0.03</param> <!-- [m/s] -->
+        <param name="mode">JOG</param>
       </xacro:unless>
       <command_interface name="position">
@@ -946,4 +954,5 @@
         <param name="max">0.6</param>
       </command_interface>
+      <!-- <command_interface name="velocity"/> -->
       <state_interface name="position">
         <param name="initial_value">0.50</param>
