Commit message: [FEAT] toogle enable_tf_prefix as param

File: sobit_home_description/robots/sobit_home_robot.urdf.xacro (robot description, xacro)
@@ -25,4 +25,5 @@
   <!-- Add variables -->
   <xacro:arg name="robot_name" default="sobit_home" />
+  <xacro:arg name="enable_tf_prefix" default="False" />
   <xacro:arg name="enable_gz"                       default="True" />
   <xacro:arg name="enable_head_cam_color"        default="True" />
@@ -58,5 +59,5 @@
     <xacro:plate prefix="plate" parent="base_link" />
     <xacro:wheel prefix="wheel" parent="plate_middle_link" />
-    <xacro:lidar prefix="lidar" parent="plate_middle_link" robot_name="$(arg robot_name)" />
+    <xacro:lidar prefix="lidar" parent="plate_middle_link" robot_name="$(arg robot_name)" enable_tf_prefix="$(arg enable_tf_prefix)" />
   </xacro:if>
   <xacro:unless value="${ $(arg enable_mobile_base) }">

File: sobit_home_description/urdf/sensor/lidar.urdf.xacro (robot description, xacro)
@@ -2,5 +2,5 @@
 <robot name="sobit_home"
        xmlns:xacro="http://ros.org/wiki/xacro">
-  <xacro:macro name="lidar_edge" params="prefix parent robot_name stand_x stand_y stand_z hokuyo_x hokuyo_y hokuyo_z yaw">
+  <xacro:macro name="lidar_edge" params="prefix parent robot_name enable_tf_prefix:=False stand_x stand_y stand_z hokuyo_x hokuyo_y hokuyo_z yaw">
     <joint name="${prefix}_base_joint" type="fixed">
       <parent link="${parent}" />
@@ -30,11 +30,11 @@
       </inertial>
     </link>
-    <xacro:hokuyo_ust_mount prefix="${prefix}" parent="${prefix}_base_link" topic="${prefix}/scan" model="ust-20" robot_name="${robot_name}">
+    <xacro:hokuyo_ust_mount prefix="${prefix}" parent="${prefix}_base_link" topic="${prefix}/scan" model="ust-20" robot_name="${robot_name}" enable_tf_prefix="${enable_tf_prefix}">
       <origin xyz="${hokuyo_x} ${hokuyo_y} ${hokuyo_z}" rpy="0.0 0.0 0.0" />
     </xacro:hokuyo_ust_mount>
   </xacro:macro>
-  <xacro:macro name="lidar" params="parent prefix robot_name">
-    <xacro:lidar_edge prefix="${prefix}_front" parent="${parent}" robot_name="${robot_name}" stand_x= " 0.2357767" stand_y=" 0.2357767" stand_z="0.01" hokuyo_x="0.06914214" hokuyo_y="0.0" hokuyo_z="-0.142" yaw="${M_PI-M_PI/4}"/>
-    <xacro:lidar_edge prefix="${prefix}_back"  parent="${parent}" robot_name="${robot_name}" stand_x= "-0.2357767" stand_y="-0.2357767" stand_z="0.01" hokuyo_x="0.06914214" hokuyo_y="0.0" hokuyo_z="-0.142" yaw="${-M_PI/4}"/>
+  <xacro:macro name="lidar" params="parent prefix robot_name enable_tf_prefix:=False">
+    <xacro:lidar_edge prefix="${prefix}_front" parent="${parent}" robot_name="${robot_name}" enable_tf_prefix="${enable_tf_prefix}" stand_x= " 0.2357767" stand_y=" 0.2357767" stand_z="0.01" hokuyo_x="0.06914214" hokuyo_y="0.0" hokuyo_z="-0.142" yaw="${M_PI-M_PI/4}"/>
+    <xacro:lidar_edge prefix="${prefix}_back"  parent="${parent}" robot_name="${robot_name}" enable_tf_prefix="${enable_tf_prefix}" stand_x= "-0.2357767" stand_y="-0.2357767" stand_z="0.01" hokuyo_x="0.06914214" hokuyo_y="0.0" hokuyo_z="-0.142" yaw="${-M_PI/4}"/>
   </xacro:macro>
 </robot>
