Commit message: Accept either case for enable_gz
${...} evaluates a Python literal, so only True and False parsed and the
lowercase spelling a launch file accepts failed outright against xacro.
The argument is normalized once into a gz_on property, which every test
then reads, so true, True and 1 all work.

Co-Authored-By: Claude Opus 5 (1M context) <noreply@anthropic.com>

File: sobit_home_description/robots/sobit_home_robot.urdf.xacro (robot description, xacro)
@@ -44,4 +44,6 @@
   <xacro:arg name="enable_head"         default="True" />
   <xacro:arg name="enable_dxl_pro"      default="True" />
+  <!-- ${...} evaluates a Python literal, where only True/False parse. -->
+  <xacro:property name="gz_on" value="${'$(arg enable_gz)'.lower() in ('true', '1')}" />
   <!-- DXL Ports -->
   <xacro:arg name="dxl_x_lower_body_port"  default="/dev/ttyUSB1" />
@@ -131,7 +133,7 @@
   </xacro:if>
   <!-- Add Actuators Controllers -->
-  <xacro:controllers enable_gz="$(arg enable_gz)" robot_name="$(arg robot_name)" />
+  <xacro:controllers enable_gz="${gz_on}" robot_name="$(arg robot_name)" />
   <!-- Add Gazebo plugins -->
-  <xacro:if value="${$(arg enable_gz)}">
+  <xacro:if value="${gz_on}">
     <xacro:gazebo_sensors robot_name="$(arg robot_name)"
       head_cam_type="$(arg head_cam_type)"

File: sobit_home_description/urdf/controllers.urdf.xacro (robot description, xacro)
@@ -5,5 +5,5 @@
     <!-- Async hardware = separate read/write thread, decoupling I/O from the control
          loop. Real hardware only - gz_ros2_control steps sync, so force sync under Gazebo. -->
-    <xacro:property name="hw_is_async" value="${'false' if $(arg enable_gz) else 'true'}"/>
+    <xacro:property name="hw_is_async" value="${'false' if gz_on else 'true'}"/>
     <xacro:if value="${$(arg enable_mobile_base)}">
       <!-- rw_rate 100 Hz on real hardware: this 4-servo bus nearly keeps up with a
@@ -11,5 +11,5 @@
       <ros2_control name="dynamixel_control_lower" type="system" is_async="${hw_is_async}"
                     rw_rate="100">
-        <xacro:unless value="${$(arg enable_gz)}">
+        <xacro:unless value="${gz_on}">
           <properties>
             <async scheduling_policy="synchronized" thread_priority="79" affinity="[7]" print_warnings="true"/>
@@ -17,8 +17,8 @@
         </xacro:unless>
         <hardware>
-          <xacro:if value="${$(arg enable_gz)}">
+          <xacro:if value="${gz_on}">
             <plugin>gz_ros2_control/GazeboSimSystem</plugin>
           </xacro:if>
-          <xacro:unless value="${$(arg enable_gz)}">
+          <xacro:unless value="${gz_on}">
             <xacro:property name="dxl_x_lower_body_port" value="$(arg dxl_x_lower_body_port)"/>
             <plugin>dynamixel_hardware/DynamixelHardware</plugin>
@@ -27,5 +27,5 @@
           </xacro:unless>
         </hardware>
-          <xacro:dxl_wheel_steer_controllers prefix="wheel"      enable_gz="${$(arg enable_gz)}"/>
+          <xacro:dxl_wheel_steer_controllers prefix="wheel"      enable_gz="${gz_on}"/>
       </ros2_control>
     </xacro:if>
@@ -35,5 +35,5 @@
       <ros2_control name="dynamixel_upper" type="system" is_async="${hw_is_async}"
                     rw_rate="100">
-        <xacro:unless value="${$(arg enable_gz)}">
+        <xacro:unless value="${gz_on}">
           <properties>
             <async scheduling_policy="synchronized" thread_priority="79" affinity="[2]" print_warnings="true"/>
@@ -41,8 +41,8 @@
         </xacro:unless>
         <hardware>
-          <xacro:if value="${$(arg enable_gz)}">
+          <xacro:if value="${gz_on}">
             <plugin>gz_ros2_control/GazeboSimSystem</plugin>
           </xacro:if>
-          <xacro:unless value="${$(arg enable_gz)}">
+          <xacro:unless value="${gz_on}">
             <xacro:property name="dxl_x_upper_body_port" value="$(arg dxl_x_upper_body_port)"/>
             <plugin>dynamixel_hardware/DynamixelHardware</plugin>
@@ -52,11 +52,11 @@
         </hardware>
         <xacro:if value="${$(arg enable_head)}">
-          <xacro:dxl_head_controllers        prefix="head"       enable_gz="${$(arg enable_gz)}"/>
+          <xacro:dxl_head_controllers        prefix="head"       enable_gz="${gz_on}"/>
         </xacro:if>
         <xacro:if value="${$(arg enable_arm_left)}">
-          <xacro:dxl_arm_left_controllers    prefix="arm_left"   enable_gz="${$(arg enable_gz)}"/>
+          <xacro:dxl_arm_left_controllers    prefix="arm_left"   enable_gz="${gz_on}"/>
         </xacro:if>
         <xacro:if value="${$(arg enable_arm_right)}">
-          <xacro:dxl_arm_right_controllers   prefix="arm_right"  enable_gz="${$(arg enable_gz)}"/>
+          <xacro:dxl_arm_right_controllers   prefix="arm_right"  enable_gz="${gz_on}"/>
         </xacro:if>
       </ros2_control>
@@ -67,5 +67,5 @@
       <ros2_control name="dynamixel_hand" type="system" is_async="${hw_is_async}"
                     rw_rate="100">
-        <xacro:unless value="${$(arg enable_gz)}">
+        <xacro:unless value="${gz_on}">
           <properties>
             <async scheduling_policy="synchronized" thread_priority="79" affinity="[5]" print_warnings="true"/>
@@ -73,8 +73,8 @@
         </xacro:unless>
         <hardware>
-          <xacro:if value="${$(arg enable_gz)}">
+          <xacro:if value="${gz_on}">
             <plugin>gz_ros2_control/GazeboSimSystem</plugin>
           </xacro:if>
-          <xacro:unless value="${$(arg enable_gz)}">
+          <xacro:unless value="${gz_on}">
             <xacro:property name="dxl_x_hand_port" value="$(arg dxl_x_hand_port)"/>
             <plugin>dynamixel_hardware/DynamixelHardware</plugin>
@@ -84,8 +84,8 @@
         </hardware>
         <xacro:if value="${$(arg enable_hand_left)}">
-          <xacro:dxl_hand_left_controllers   prefix="hand_left"  enable_gz="${$(arg enable_gz)}"/>
+          <xacro:dxl_hand_left_controllers   prefix="hand_left"  enable_gz="${gz_on}"/>
         </xacro:if>
         <xacro:if value="${$(arg enable_hand_right)}">
-          <xacro:dxl_hand_right_controllers  prefix="hand_right" enable_gz="${$(arg enable_gz)}"/>
+          <xacro:dxl_hand_right_controllers  prefix="hand_right" enable_gz="${gz_on}"/>
         </xacro:if>
       </ros2_control>
@@ -96,5 +96,5 @@
       <ros2_control name="dynamixel_pro_upper" type="system" is_async="${hw_is_async}"
                     rw_rate="50">
-        <xacro:unless value="${$(arg enable_gz)}">
+        <xacro:unless value="${gz_on}">
           <properties>
             <async scheduling_policy="synchronized" thread_priority="79" affinity="[3]" print_warnings="true"/>
@@ -102,8 +102,8 @@
         </xacro:unless>
         <hardware>
-          <xacro:if value="${$(arg enable_gz)}">
+          <xacro:if value="${gz_on}">
             <plugin>gz_ros2_control/GazeboSimSystem</plugin>
           </xacro:if>
-          <xacro:unless value="${$(arg enable_gz)}">
+          <xacro:unless value="${gz_on}">
             <xacro:property name="dxl_p_upper_body_port" value="$(arg dxl_p_upper_body_port)"/>
             <plugin>dynamixel_hardware/DynamixelHardware</plugin>
@@ -113,8 +113,8 @@
         </hardware>
         <xacro:if value="${$(arg enable_arm_left)}">
-          <xacro:dxl_pro_arm_left_controllers    prefix="arm_left"   enable_gz="${$(arg enable_gz)}"/>
+          <xacro:dxl_pro_arm_left_controllers    prefix="arm_left"   enable_gz="${gz_on}"/>
         </xacro:if>
         <xacro:if value="${$(arg enable_arm_right)}">
-          <xacro:dxl_pro_arm_right_controllers   prefix="arm_right"  enable_gz="${$(arg enable_gz)}"/>
+          <xacro:dxl_pro_arm_right_controllers   prefix="arm_right"  enable_gz="${gz_on}"/>
         </xacro:if>
       </ros2_control>
@@ -125,5 +125,5 @@
       <ros2_control name="robomaster_control" type="system" is_async="${hw_is_async}"
                     rw_rate="100">
-        <xacro:unless value="${$(arg enable_gz)}">
+        <xacro:unless value="${gz_on}">
           <properties>
             <async scheduling_policy="synchronized" thread_priority="79" affinity="[4]" print_warnings="true"/>
@@ -131,8 +131,8 @@
         </xacro:unless>
         <hardware>
-          <xacro:if value="${$(arg enable_gz)}">
+          <xacro:if value="${gz_on}">
             <plugin>gz_ros2_control/GazeboSimSystem</plugin>
           </xacro:if>
-          <xacro:unless value="${$(arg enable_gz)}">
+          <xacro:unless value="${gz_on}">
             <plugin>rm_motors_hw/RmMotorsSystemHardware</plugin>
             <param name="can_interface">$(arg can_interface)</param>
@@ -140,5 +140,5 @@
           </xacro:unless>
         </hardware>
-        <xacro:rm_wheel_drive_controllers prefix="wheel" enable_gz="${$(arg enable_gz)}"/>
+        <xacro:rm_wheel_drive_controllers prefix="wheel" enable_gz="${gz_on}"/>
       </ros2_control>
     </xacro:if>
@@ -148,5 +148,5 @@
       <ros2_control name="uirobot_control" type="system" is_async="${hw_is_async}"
                     rw_rate="20">
-        <xacro:unless value="${$(arg enable_gz)}">
+        <xacro:unless value="${gz_on}">
           <properties>
             <async scheduling_policy="synchronized" thread_priority="79" affinity="[6]" print_warnings="true"/>
@@ -154,8 +154,8 @@
         </xacro:unless>
         <hardware>
-          <xacro:if value="${$(arg enable_gz)}">
+          <xacro:if value="${gz_on}">
             <plugin>gz_ros2_control/GazeboSimSystem</plugin>
           </xacro:if>
-          <xacro:unless value="${$(arg enable_gz)}">
+          <xacro:unless value="${gz_on}">
             <xacro:property name="um_body_port" value="$(arg um_body_port)"/>
             <plugin>uirobot_hardware/UirobotHardware</plugin>
@@ -166,9 +166,9 @@
           </xacro:unless>
         </hardware>
-        <xacro:uirobot_control prefix="body" enable_gz="${$(arg enable_gz)}"/>
+        <xacro:uirobot_control prefix="body" enable_gz="${gz_on}"/>
       </ros2_control>
     </xacro:if>
     <!-- Gazebo Sim ROS2 Control -->
-    <xacro:if value="${$(arg enable_gz)}">
+    <xacro:if value="${gz_on}">
       <gazebo>
         <plugin filename="gz_ros2_control-system" name="gz_ros2_control::GazeboSimROS2ControlPlugin">
@@ -249,5 +249,5 @@
   <xacro:macro name="dxl_wheel_steer_controllers"  params="prefix enable_gz:=False">
     <joint name="${prefix}_steer_f_l_joint">
-      <xacro:unless value="${$(arg enable_gz)}">
+      <xacro:unless value="${gz_on}">
         <param name="id">11</param>
         <param name="control_mode">0</param>
@@ -266,5 +266,5 @@
     </joint>
     <joint name="${prefix}_steer_f_r_joint">
-      <xacro:unless value="${$(arg enable_gz)}">
+      <xacro:unless value="${gz_on}">
         <param name="id">12</param>
         <param name="control_mode">0</param>
@@ -283,5 +283,5 @@
     </joint>
     <joint name="${prefix}_steer_b_l_joint">
-      <xacro:unless value="${$(arg enable_gz)}">
+      <xacro:unless value="${gz_on}">
         <param name="id">13</param>
         <param name="control_mode">0</param>
@@ -300,5 +300,5 @@
     </joint>
     <joint name="${prefix}_steer_b_r_joint">
-      <xacro:unless value="${$(arg enable_gz)}">
+      <xacro:unless value="${gz_on}">
         <param name="id">14</param>
         <param name="control_mode">0</param>
@@ -319,5 +319,5 @@
   <xacro:macro name="dxl_head_controllers"         params="prefix enable_gz:=False">
     <joint name="head_pan_joint">
-      <xacro:unless value="${$(arg enable_gz)}">
+      <xacro:unless value="${gz_on}">
         <param name="id">21</param>
         <param name="control_mode">0</param>
@@ -336,5 +336,5 @@
     </joint>
     <joint name="head_tilt_joint">
-      <xacro:unless value="${$(arg enable_gz)}">
+      <xacro:unless value="${gz_on}">
         <param name="id">22</param>
         <param name="control_mode">0</param>
@@ -355,5 +355,5 @@
   <xacro:macro name="dxl_pro_arm_left_controllers"     params="prefix enable_gz:=False">
     <joint name="${prefix}_shoulder_tilt_joint">
-      <xacro:unless value="${$(arg enable_gz)}">
+      <xacro:unless value="${gz_on}">
         <param name="id">31</param>
         <param name="control_mode">0</param>
@@ -375,5 +375,5 @@
   <xacro:macro name="dxl_pro_arm_right_controllers"    params="prefix enable_gz:=False">
     <joint name="${prefix}_shoulder_tilt_joint">
-      <xacro:unless value="${$(arg enable_gz)}">
+      <xacro:unless value="${gz_on}">
         <param name="id">41</param>
         <param name="control_mode">0</param>
@@ -394,5 +394,5 @@
   <xacro:macro name="dxl_arm_left_controllers"     params="prefix enable_gz:=False">
     <joint name="${prefix}_upper_roll_joint">
-      <xacro:unless value="${$(arg enable_gz)}">
+      <xacro:unless value="${gz_on}">
         <param name="id">32</param>
         <param name="control_mode">0</param>
@@ -412,5 +412,5 @@
     </joint>
     <joint name="${prefix}_upper_flex_joint">
-      <xacro:unless value="${$(arg enable_gz)}">
+      <xacro:unless value="${gz_on}">
         <param name="id">34</param>
         <param name="control_mode">0</param>
@@ -430,5 +430,5 @@
     </joint>
     <joint name="${prefix}_elbow_joint">
-      <xacro:unless value="${$(arg enable_gz)}">
+      <xacro:unless value="${gz_on}">
         <param name="id">36</param>
         <param name="control_mode">0</param>
@@ -448,5 +448,5 @@
     </joint>
     <joint name="${prefix}_lower_flex_joint">
-      <xacro:unless value="${$(arg enable_gz)}">
+      <xacro:unless value="${gz_on}">
         <param name="id">38</param>
         <param name="control_mode">0</param>
@@ -466,5 +466,5 @@
     </joint>
     <joint name="${prefix}_wrist_tilt_joint">
-      <xacro:unless value="${$(arg enable_gz)}">
+      <xacro:unless value="${gz_on}">
         <param name="id">39</param>
         <param name="control_mode">0</param>
@@ -484,5 +484,5 @@
     </joint>
     <joint name="${prefix}_wrist_roll_joint">
-      <xacro:unless value="${$(arg enable_gz)}">
+      <xacro:unless value="${gz_on}">
         <param name="id">40</param>
         <param name="control_mode">0</param>
@@ -504,5 +504,5 @@
   <xacro:macro name="dxl_arm_right_controllers"     params="prefix enable_gz:=False">
     <joint name="${prefix}_upper_roll_joint">
-      <xacro:unless value="${$(arg enable_gz)}">
+      <xacro:unless value="${gz_on}">
         <param name="id">42</param>
         <param name="control_mode">0</param>
@@ -521,5 +521,5 @@
     </joint>
     <joint name="${prefix}_upper_flex_joint">
-      <xacro:unless value="${$(arg enable_gz)}">
+      <xacro:unless value="${gz_on}">
         <param name="id">44</param>
         <param name="control_mode">0</param>
@@ -538,5 +538,5 @@
     </joint>
     <joint name="${prefix}_elbow_joint">
-      <xacro:unless value="${$(arg enable_gz)}">
+      <xacro:unless value="${gz_on}">
         <param name="id">46</param>
         <param name="control_mode">0</param>
@@ -555,5 +555,5 @@
     </joint>
     <joint name="${prefix}_lower_flex_joint">
-      <xacro:unless value="${$(arg enable_gz)}">
+      <xacro:unless value="${gz_on}">
         <param name="id">48</param>
         <param name="control_mode">0</param>
@@ -572,5 +572,5 @@
     </joint>
     <joint name="${prefix}_wrist_tilt_joint">
-      <xacro:unless value="${$(arg enable_gz)}">
+      <xacro:unless value="${gz_on}">
         <param name="id">49</param>
         <param name="control_mode">0</param>
@@ -589,5 +589,5 @@
     </joint>
     <joint name="${prefix}_wrist_roll_joint">
-      <xacro:unless value="${$(arg enable_gz)}">
+      <xacro:unless value="${gz_on}">
         <param name="id">50</param>
         <param name="control_mode">0</param>
@@ -608,5 +608,5 @@
   <xacro:macro name="dxl_hand_left_controllers"    params="prefix enable_gz:=False">
     <joint name="${prefix}_finger_l_mcp_joint">
-      <xacro:unless value="${$(arg enable_gz)}">
+      <xacro:unless value="${gz_on}">
         <param name="id">51</param>
         <param name="control_mode">6</param>
@@ -625,5 +625,5 @@
       <state_interface name="effort"/>
     </joint>
-    <xacro:if value="${$(arg enable_gz)}">
+    <xacro:if value="${gz_on}">
       <joint name="${prefix}_finger_r_mcp_joint">
         <state_interface name="position">
@@ -635,5 +635,5 @@
     </xacro:if>
     <joint name="${prefix}_finger_l_pip_joint">
-      <xacro:unless value="${$(arg enable_gz)}">
+      <xacro:unless value="${gz_on}">
         <param name="id">52</param>
         <param name="control_mode">6</param>
@@ -653,5 +653,5 @@
     </joint>
     <joint name="${prefix}_finger_l_dip_joint">
-      <xacro:unless value="${$(arg enable_gz)}">
+      <xacro:unless value="${gz_on}">
         <param name="id">53</param>
         <param name="control_mode">6</param>
@@ -671,5 +671,5 @@
     </joint>
     <joint name="${prefix}_finger_c_mcp_joint">
-      <xacro:unless value="${$(arg enable_gz)}">
+      <xacro:unless value="${gz_on}">
         <param name="id">54</param>
         <param name="control_mode">6</param>
@@ -689,5 +689,5 @@
     </joint>
     <joint name="${prefix}_finger_c_ip_joint">
-      <xacro:unless value="${$(arg enable_gz)}">
+      <xacro:unless value="${gz_on}">
         <param name="id">55</param>
         <param name="control_mode">6</param>
@@ -707,5 +707,5 @@
     </joint>
     <joint name="${prefix}_finger_r_pip_joint">
-      <xacro:unless value="${$(arg enable_gz)}">
+      <xacro:unless value="${gz_on}">
         <param name="id">56</param>
         <param name="control_mode">6</param>
@@ -725,5 +725,5 @@
     </joint>
     <joint name="${prefix}_finger_r_dip_joint">
-      <xacro:unless value="${$(arg enable_gz)}">
+      <xacro:unless value="${gz_on}">
         <param name="id">57</param>
         <param name="control_mode">6</param>
@@ -745,5 +745,5 @@
   <xacro:macro name="dxl_hand_right_controllers"   params="prefix enable_gz:=False">
     <joint name="${prefix}_finger_l_mcp_joint">
-      <xacro:unless value="${$(arg enable_gz)}">
+      <xacro:unless value="${gz_on}">
         <param name="id">61</param>
         <param name="control_mode">6</param>
@@ -762,5 +762,5 @@
       <state_interface name="effort"/>
     </joint>
-    <xacro:if value="${$(arg enable_gz)}">
+    <xacro:if value="${gz_on}">
       <joint name="${prefix}_finger_r_mcp_joint">
         <state_interface name="position">
@@ -772,5 +772,5 @@
     </xacro:if>
     <joint name="${prefix}_finger_l_pip_joint">
-      <xacro:unless value="${$(arg enable_gz)}">
+      <xacro:unless value="${gz_on}">
         <param name="id">62</param>
         <param name="control_mode">6</param>
@@ -790,5 +790,5 @@
     </joint>
     <joint name="${prefix}_finger_l_dip_joint">
-      <xacro:unless value="${$(arg enable_gz)}">
+      <xacro:unless value="${gz_on}">
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