Commit message: Keep the end effector frames when a hand is disabled
The EE frames lived in the hand macro, so disabling a hand removed
hand_*_end_effector_link and broke the SRDF arm groups and teleop.
They now hang off arm_*_wrist_roll_link in the robot xacro, which
exists for every arm/hand combination.

File: sobit_home_description/robots/sobit_home_robot.urdf.xacro (robot description, xacro)
@@ -127,4 +127,15 @@
     <xacro:hand  prefix_hand="hand" position="right" prefix_finger="finger" parent="arm_right_wrist_roll_link" />
   </xacro:if>
+  <!-- EE frames: wrist_roll_link exists (real or stub) for every arm/hand combination. -->
+  <xacro:macro name="end_effector" params="position y_sign">
+    <joint name="hand_${position}_end_effector_joint" type="fixed">
+      <origin xyz="0.0 ${y_sign*0.13} 0.0" rpy="${y_sign * M_PI/2} 0.0 ${y_sign * M_PI/2}"/>
+      <parent link="arm_${position}_wrist_roll_link"/>
+      <child link="hand_${position}_end_effector_link"/>
+    </joint>
+    <link name="hand_${position}_end_effector_link"/>
+  </xacro:macro>
+  <xacro:end_effector position="left"  y_sign="1.0" />
+  <xacro:end_effector position="right" y_sign="-1.0" />
   <xacro:if value="${ $(arg enable_head) }">
     <xacro:head  prefix="head"  parent="body_lift_link" />

File: sobit_home_description/urdf/hand/hand.urdf.xacro (robot description, xacro)
@@ -291,27 +291,4 @@
       </inertial>
     </link>
-    <!-- Joint: End Effector -->
-    <joint name="${prefix_hand}_${position}_end_effector_joint" type="fixed">
-      <origin xyz="0.0 ${y_sign*0.13} 0.0" rpy="${y_sign * M_PI/2} 0.0 ${y_sign * M_PI/2}"/>
-      <parent link="${parent}"/>
-      <child link="${prefix_hand}_${position}_end_effector_link"/>
-    </joint>
-    <!-- Link: End Effector -->
-    <link name="${prefix_hand}_${position}_end_effector_link">
-      <!-- <visual>
-        <origin xyz="0.0 0.0 0.0" rpy="0 0 0"/>
-        <geometry>
-          <box size="0.01 0.01 0.01" />
-        </geometry>
-        <material name="red"/>
-      </visual> -->
-      <!-- <inertial>
-        <origin xyz="0.0 0.0 0.0" rpy="0 0 0"/>
-        <mass value="0.0001" />
-        <inertia  ixx="${1/12*0.0001*(0.01**2+0.01**2)}" ixy="0.0" ixz="0.0"
-                  iyy="${1/12*0.0001*(0.01**2+0.01**2)}" iyz="0.0"
-                  izz="${1/12*0.0001*(0.01**2+0.01**2)}" />
-      </inertial> -->
-    </link>
   <xacro:hand_transmission prefix_hand="${prefix_hand}" position="${position}" prefix_finger="${prefix_finger}"/>
   </xacro:macro>

Commit message: [ADD] description: MuJoCo mode, one MujocoSystem ros2_control block
enable_mujoco / mujoco_model / mujoco_headless; the six hardware blocks move
into hardware_controllers, the sim guards become sim_on (gz or mujoco), the
RM temperature state interface is left out under MuJoCo. Real and Gazebo
renders are byte-identical.

File: sobit_home_description/robots/sobit_home_robot.urdf.xacro (robot description, xacro)
@@ -30,4 +30,8 @@
   <xacro:arg name="enable_tf_prefix" default="False" />
   <xacro:arg name="enable_gz"                       default="True" />
+  <!-- MuJoCo (mujoco_ros2_control) supersedes enable_gz; mujoco_model = absolute scene.xml -->
+  <xacro:arg name="enable_mujoco"                   default="False" />
+  <xacro:arg name="mujoco_model"                    default="" />
+  <xacro:arg name="mujoco_headless"                 default="false" />
   <xacro:arg name="enable_head_cam_color"        default="True" />
   <xacro:arg name="enable_head_cam_depth"        default="True" />
@@ -45,5 +49,8 @@
   <xacro:arg name="enable_dxl_pro"      default="True" />
   <!-- ${...} evaluates a Python literal, where only True/False parse. -->
-  <xacro:property name="gz_on" value="${'$(arg enable_gz)'.lower() in ('true', '1')}" />
+  <xacro:property name="mujoco_on" value="${'$(arg enable_mujoco)'.lower() in ('true', '1')}" />
+  <xacro:property name="gz_on" value="${'$(arg enable_gz)'.lower() in ('true', '1') and not mujoco_on}" />
+  <!-- Any simulator: no real hardware params, sync hardware -->
+  <xacro:property name="sim_on" value="${gz_on or mujoco_on}" />
   <!-- DXL Ports -->
   <xacro:arg name="dxl_x_lower_body_port"  default="/dev/ttyUSB1" />
@@ -144,5 +151,5 @@
   </xacro:if>
   <!-- Add Actuators Controllers -->
-  <xacro:controllers enable_gz="${gz_on}" robot_name="$(arg robot_name)" />
+  <xacro:controllers enable_gz="${gz_on}" enable_mujoco="${mujoco_on}" robot_name="$(arg robot_name)" />
   <!-- Add Gazebo plugins -->
   <xacro:if value="${gz_on}">

File: sobit_home_description/urdf/controllers.urdf.xacro (robot description, xacro)
@@ -2,5 +2,14 @@
 <!-- SOBIT HOME (Controllers) -->
 <robot name="sobit_home_controllers" xmlns:xacro="http://www.ros.org/wiki/xacro">
-  <xacro:macro name="controllers" params="enable_gz:=False robot_name:=sobit_home">
+  <xacro:macro name="controllers" params="enable_gz:=False enable_mujoco:=False robot_name:=sobit_home">
+    <xacro:if value="${mujoco_on}">
+      <xacro:mujoco_controllers robot_name="${robot_name}"/>
+    </xacro:if>
+    <xacro:unless value="${mujoco_on}">
+      <xacro:hardware_controllers/>
+    </xacro:unless>
+  </xacro:macro>
+  <!-- Per-bus hardware (real) or GazeboSimSystem blocks; MuJoCo replaces all of them -->
+  <xacro:macro name="hardware_controllers">
     <!-- Async hardware = separate read/write thread, decoupling I/O from the control
          loop. Real hardware only - gz_ros2_control steps sync, so force sync under Gazebo. -->
@@ -181,4 +190,47 @@
     </xacro:if>
   </xacro:macro>
+  <!-- MuJoCo: ONE system block, since each block would start its own MuJoCo instance.
+       Joints map to the MJCF actuators of the same name; sensors live in mujoco_plugins.yaml. -->
+  <xacro:macro name="mujoco_controllers" params="robot_name:=sobit_home">
+    <ros2_control name="MujocoSystem" type="system" is_async="false">
+      <hardware>
+        <plugin>mujoco_ros2_control/MujocoSystemInterface</plugin>
+        <param name="mujoco_model">$(arg mujoco_model)</param>
+        <param name="headless">$(arg mujoco_headless)</param>
+        <param name="initial_keyframe">home</param>
+      </hardware>
+      <xacro:if value="${$(arg enable_mobile_base)}">
+        <xacro:dxl_wheel_steer_controllers   prefix="wheel"/>
+        <xacro:if value="${$(arg enable_rm_motors)}">
+          <xacro:rm_wheel_drive_controllers  prefix="wheel"/>
+        </xacro:if>
+      </xacro:if>
+      <xacro:if value="${$(arg enable_head)}">
+        <xacro:dxl_head_controllers          prefix="head"/>
+      </xacro:if>
+      <xacro:if value="${$(arg enable_arm_left)}">
+        <xacro:if value="${$(arg enable_dxl_pro)}">
+          <xacro:dxl_pro_arm_left_controllers  prefix="arm_left"/>
+        </xacro:if>
+        <xacro:dxl_arm_left_controllers      prefix="arm_left"/>
+      </xacro:if>
+      <xacro:if value="${$(arg enable_arm_right)}">
+        <xacro:if value="${$(arg enable_dxl_pro)}">
+          <xacro:dxl_pro_arm_right_controllers prefix="arm_right"/>
+        </xacro:if>
+        <xacro:dxl_arm_right_controllers     prefix="arm_right"/>
+      </xacro:if>
+      <xacro:if value="${$(arg enable_hand_left)}">
+        <xacro:dxl_hand_left_controllers     prefix="hand_left"/>
+      </xacro:if>
+      <xacro:if value="${$(arg enable_hand_right)}">
+        <xacro:dxl_hand_right_controllers    prefix="hand_right"/>
+      </xacro:if>
+      <xacro:if value="${$(arg enable_body)}">
+        <xacro:uirobot_control               prefix="body"/>
+      </xacro:if>
+    </ros2_control>
+  </xacro:macro>
+  <!-- temperature is RM-motor only; MuJoCo exports position/velocity/effort and rejects extra interfaces -->
   <xacro:macro name="rm_wheel_drive_controllers"  params="prefix enable_gz:=False">
     <joint name="${prefix}_drive_f_l_joint">
@@ -196,5 +248,7 @@
       <state_interface name="velocity"/>
       <state_interface name="effort"/>
-      <state_interface name="temperature"/>
+      <xacro:unless value="${mujoco_on}">
+        <state_interface name="temperature"/>
+      </xacro:unless>
     </joint>
     <joint name="${prefix}_drive_f_r_joint">
@@ -212,5 +266,7 @@
       <state_interface name="velocity"/>
       <state_interface name="effort"/>
-      <state_interface name="temperature"/>
+      <xacro:unless value="${mujoco_on}">
+        <state_interface name="temperature"/>
+      </xacro:unless>
     </joint>
     <joint name="${prefix}_drive_b_l_joint">
@@ -228,5 +284,7 @@
       <state_interface name="velocity"/>
       <state_interface name="effort"/>
-      <state_interface name="temperature"/>
+      <xacro:unless value="${mujoco_on}">
+        <state_interface name="temperature"/>
+      </xacro:unless>
     </joint>
     <joint name="${prefix}_drive_b_r_joint">
@@ -244,10 +302,12 @@
       <state_interface name="velocity"/>
       <state_interface name="effort"/>
-      <state_interface name="temperature"/>
+      <xacro:unless value="${mujoco_on}">
+        <state_interface name="temperature"/>
+      </xacro:unless>
     </joint>
   </xacro:macro>
   <xacro:macro name="dxl_wheel_steer_controllers"  params="prefix enable_gz:=False">
     <joint name="${prefix}_steer_f_l_joint">
-      <xacro:unless value="${gz_on}">
+      <xacro:unless value="${sim_on}">
         <param name="id">11</param>
         <param name="control_mode">0</param>
@@ -266,5 +326,5 @@
     </joint>
     <joint name="${prefix}_steer_f_r_joint">
-      <xacro:unless value="${gz_on}">
+      <xacro:unless value="${sim_on}">
         <param name="id">12</param>
         <param name="control_mode">0</param>
@@ -283,5 +343,5 @@
     </joint>
     <joint name="${prefix}_steer_b_l_joint">
-      <xacro:unless value="${gz_on}">
+      <xacro:unless value="${sim_on}">
         <param name="id">13</param>
         <param name="control_mode">0</param>
@@ -300,5 +360,5 @@
     </joint>
     <joint name="${prefix}_steer_b_r_joint">
-      <xacro:unless value="${gz_on}">
+      <xacro:unless value="${sim_on}">
         <param name="id">14</param>
         <param name="control_mode">0</param>
@@ -319,5 +379,5 @@
   <xacro:macro name="dxl_head_controllers"         params="prefix enable_gz:=False">
     <joint name="head_pan_joint">
-      <xacro:unless value="${gz_on}">
+      <xacro:unless value="${sim_on}">
         <param name="id">21</param>
         <param name="control_mode">0</param>
@@ -336,5 +396,5 @@
     </joint>
     <joint name="head_tilt_joint">
-      <xacro:unless value="${gz_on}">
+      <xacro:unless value="${sim_on}">
         <param name="id">22</param>
         <param name="control_mode">0</param>
@@ -355,5 +415,5 @@
   <xacro:macro name="dxl_pro_arm_left_controllers"     params="prefix enable_gz:=False">
     <joint name="${prefix}_shoulder_tilt_joint">
-      <xacro:unless value="${gz_on}">
+      <xacro:unless value="${sim_on}">
         <param name="id">31</param>
         <param name="control_mode">0</param>
@@ -375,5 +435,5 @@
   <xacro:macro name="dxl_pro_arm_right_controllers"    params="prefix enable_gz:=False">
     <joint name="${prefix}_shoulder_tilt_joint">
-      <xacro:unless value="${gz_on}">
+      <xacro:unless value="${sim_on}">
         <param name="id">41</param>
         <param name="control_mode">0</param>
@@ -394,5 +454,5 @@
   <xacro:macro name="dxl_arm_left_controllers"     params="prefix enable_gz:=False">
     <joint name="${prefix}_upper_roll_joint">
-      <xacro:unless value="${gz_on}">
+      <xacro:unless value="${sim_on}">
         <param name="id">32</param>
         <param name="control_mode">0</param>
@@ -412,5 +472,5 @@
     </joint>
     <joint name="${prefix}_upper_flex_joint">
-      <xacro:unless value="${gz_on}">
+      <xacro:unless value="${sim_on}">
         <param name="id">34</param>
         <param name="control_mode">0</param>
@@ -430,5 +490,5 @@
     </joint>
     <joint name="${prefix}_elbow_joint">
-      <xacro:unless value="${gz_on}">
+      <xacro:unless value="${sim_on}">
         <param name="id">36</param>
         <param name="control_mode">0</param>
@@ -448,5 +508,5 @@
     </joint>
     <joint name="${prefix}_lower_flex_joint">
-      <xacro:unless value="${gz_on}">
+      <xacro:unless value="${sim_on}">
         <param name="id">38</param>
         <param name="control_mode">0</param>
@@ -466,5 +526,5 @@
     </joint>
     <joint name="${prefix}_wrist_tilt_joint">
-      <xacro:unless value="${gz_on}">
+      <xacro:unless value="${sim_on}">
         <param name="id">39</param>
         <param name="control_mode">0</param>
@@ -484,5 +544,5 @@
     </joint>
     <joint name="${prefix}_wrist_roll_joint">
-      <xacro:unless value="${gz_on}">
+      <xacro:unless value="${sim_on}">
         <param name="id">40</param>
         <param name="control_mode">0</param>
@@ -504,5 +564,5 @@
   <xacro:macro name="dxl_arm_right_controllers"     params="prefix enable_gz:=False">
     <joint name="${prefix}_upper_roll_joint">
-      <xacro:unless value="${gz_on}">
+      <xacro:unless value="${sim_on}">
         <param name="id">42</param>
         <param name="control_mode">0</param>
@@ -521,5 +581,5 @@
     </joint>
     <joint name="${prefix}_upper_flex_joint">
-      <xacro:unless value="${gz_on}">
+      <xacro:unless value="${sim_on}">
         <param name="id">44</param>
         <param name="control_mode">0</param>
@@ -538,5 +598,5 @@
     </joint>
     <joint name="${prefix}_elbow_joint">
-      <xacro:unless value="${gz_on}">
+      <xacro:unless value="${sim_on}">
         <param name="id">46</param>
         <param name="control_mode">0</param>
@@ -555,5 +615,5 @@
     </joint>
     <joint name="${prefix}_lower_flex_joint">
-      <xacro:unless value="${gz_on}">
+      <xacro:unless value="${sim_on}">
         <param name="id">48</param>
         <param name="control_mode">0</param>
@@ -572,5 +632,5 @@
     </joint>
     <joint name="${prefix}_wrist_tilt_joint">
-      <xacro:unless value="${gz_on}">
+      <xacro:unless value="${sim_on}">
         <param name="id">49</param>
         <param name="control_mode">0</param>
@@ -589,5 +649,5 @@
     </joint>
     <joint name="${prefix}_wrist_roll_joint">
-      <xacro:unless value="${gz_on}">
+      <xacro:unless value="${sim_on}">
         <param name="id">50</param>
         <param name="control_mode">0</param>
@@ -608,5 +668,5 @@
   <xacro:macro name="dxl_hand_left_controllers"    params="prefix enable_gz:=False">
     <joint name="${prefix}_finger_l_mcp_joint">
-      <xacro:unless value="${gz_on}">
+      <xacro:unless value="${sim_on}">
         <param name="id">51</param>
         <param name="control_mode">6</param>
@@ -625,5 +685,5 @@
       <state_interface name="effort"/>
     </joint>
-    <xacro:if value="${gz_on}">
+    <xacro:if value="${sim_on}">
       <joint name="${prefix}_finger_r_mcp_joint">
         <state_interface name="position">
@@ -635,5 +695,5 @@
     </xacro:if>
     <joint name="${prefix}_finger_l_pip_joint">
-      <xacro:unless value="${gz_on}">
+      <xacro:unless value="${sim_on}">
         <param name="id">52</param>
         <param name="control_mode">6</param>
@@ -653,5 +713,5 @@
     </joint>
     <joint name="${prefix}_finger_l_dip_joint">
-      <xacro:unless value="${gz_on}">
+      <xacro:unless value="${sim_on}">
         <param name="id">53</param>
         <param name="control_mode">6</param>
@@ -671,5 +731,5 @@
     </joint>
     <joint name="${prefix}_finger_c_mcp_joint">
-      <xacro:unless value="${gz_on}">
+      <xacro:unless value="${sim_on}">
         <param name="id">54</param>
         <param name="control_mode">6</param>
@@ -689,5 +749,5 @@
     </joint>
     <joint name="${prefix}_finger_c_ip_joint">
-      <xacro:unless value="${gz_on}">
+      <xacro:unless value="${sim_on}">
         <param name="id">55</param>
         <param name="control_mode">6</param>
@@ -707,5 +767,5 @@
     </joint>
     <joint name="${prefix}_finger_r_pip_joint">
-      <xacro:unless value="${gz_on}">
+      <xacro:unless value="${sim_on}">
         <param name="id">56</param>
         <param name="control_mode">6</param>
@@ -725,5 +785,5 @@
     </joint>
     <joint name="${prefix}_finger_r_dip_joint">
-      <xacro:unless value="${gz_on}">
+      <xacro:unless value="${sim_on}">
         <param name="id">57</param>
         <param name="control_mode">6</param>
@@ -745,5 +805,5 @@
   <xacro:macro name="dxl_hand_right_controllers"   params="prefix enable_gz:=False">
     <joint name="${prefix}_finger_l_mcp_joint">
-      <xacro:unless value="${gz_on}">
+      <xacro:unless value="${sim_on}">
         <param name="id">61</param>
         <param name="control_mode">6</param>
@@ -762,5 +822,5 @@
       <state_interface name="effort"/>
     </joint>
-    <xacro:if value="${gz_on}">
+    <xacro:if value="${sim_on}">
       <joint name="${prefix}_finger_r_mcp_joint">
         <state_interface name="position">
@@ -772,5 +832,5 @@
     </xacro:if>
     <joint name="${prefix}_finger_l_pip_joint">
-      <xacro:unless value="${gz_on}">
+      <xacro:unless value="${sim_on}">
         <param name="id">62</param>
         <param name="control_mode">6</param>
@@ -790,5 +850,5 @@
     </joint>
     <joint name="${prefix}_finger_l_dip_joint">
-      <xacro:unless value="${gz_on}">
+      <xacro:unless value="${sim_on}">
         <param name="id">63</param>
         <param name="control_mode">6</param>
@@ -808,5 +868,5 @@
     </joint>
     <joint name="${prefix}_finger_c_mcp_joint">
-      <xacro:unless value="${gz_on}">
+      <xacro:unless value="${sim_on}">
         <param name="id">64</param>
         <param name="control_mode">6</param>
@@ -826,5 +886,5 @@
     </joint>
     <joint name="${prefix}_finger_c_ip_joint">
-      <xacro:unless value="${gz_on}">
+      <xacro:unless value="${sim_on}">
         <param name="id">65</param>
         <param name="control_mode">6</param>
@@ -844,5 +904,5 @@
     </joint>
     <joint name="${prefix}_finger_r_pip_joint">
-      <xacro:unless value="${gz_on}">
+      <xacro:unless value="${sim_on}">
         <param name="id">66</param>
         <param name="control_mode">6</param>
@@ -862,5 +922,5 @@
     </joint>
     <joint name="${prefix}_finger_r_dip_joint">
-      <xacro:unless value="${gz_on}">
+      <xacro:unless value="${sim_on}">
         <param name="id">67</param>
         <param name="control_mode">6</param>
@@ -882,5 +942,5 @@
   <xacro:macro name="uirobot_control" params="prefix enable_gz:=False">
     <joint name="${prefix}_lift_joint">
-      <xacro:unless value="${gz_on}">
+      <xacro:unless value="${sim_on}">
         <param name="id">$(arg um_body_id)</param>
         <param name="gear_ratio">${200*M_PI}</param>
