Commit message: Regenerate sobit_home_robot.urdf from the fixed xacro tree
Reflects the restored hw_is_async property (8286265) and the fast-forward
onto origin/fix/bringup-camera-can-lidar (pose lists, joint action server
changes). Mesh URIs use package:// instead of the baked-in absolute
install-space paths xacro's $(find) substitution produces, so the file
resolves correctly regardless of which machine generated it.

File: sobit_home_description/robots/sobit_home_robot.urdf (robot description, URDF)
Before this commit: robot sobit_home, 92 links, 91 joints
Links:
- removed link arm_left_elbow_sub_link
- removed link arm_left_upper_flex_sub_link
- removed link arm_left_upper_roll_sub_link
- removed link arm_right_elbow_sub_link
- removed link arm_right_upper_flex_sub_link
- removed link arm_right_upper_roll_sub_link
- link arm_left_base_link: geometry collision box size=0.054 0.124 0.054; visual mesh filename=package://sobit_home_description/meshes/arm/arm_scapula.stl scale=0.001 0.001 0.001
- link arm_left_elbow_link: geometry collision cylinder length=0.12 radius=0.055; visual mesh filename=package://sobit_home_description/meshes/arm/arm_elbow.stl scale=0.001 0.001 0.001
- link arm_left_lower_flex_link: geometry collision cylinder length=0.300 radius=0.042; visual mesh filename=package://sobit_home_description/meshes/arm/arm_lower_botto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 scale=0.001 0.001 0.001
- link arm_left_shoulder_tilt_link: geometry collision cylinder length=0.100 radius=0.089; visual mesh filename=package://sobit_home_description/meshes/arm/arm_shoulder.stl scale=0.001 0.001 0.001
- link arm_left_upper_flex_link: geometry collision cylinder length=0.170 radius=0.03; visual mesh filename=package://sobit_home_description/meshes/arm/arm_upper_flex.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 scale=0.001 0.001 0.001
- link arm_left_upper_roll_link: geometry collision cylinder length=0.1285 radius=0.071; visual mesh filename=package://sobit_home_description/meshes/arm/arm_upper_roll.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 scale=0.001 0.001 0.001
- link arm_left_wrist_roll_link: geometry collision box size=0.108 0.0826 0.0645; visual mesh filename=package://sobit_home_description/meshes/arm/arm_wrist_roll.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 scale=0.001 0.001 0.001
- link arm_left_wrist_tilt_link: geometry collision cylinder length=0.0453 radius=0.04; visual mesh filename=package://sobit_home_description/meshes/arm/arm_wrist_tilt.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 scale=0.001 0.001 0.001
- link arm_right_base_link: geometry collision box size=0.054 0.124 0.054; visual mesh filename=package://sobit_home_description/meshes/arm/arm_scapula.stl scale=0.001 0.001 0.001
- link arm_right_elbow_link: geometry collision cylinder length=0.12 radius=0.055; visual mesh filename=package://sobit_home_description/meshes/arm/arm_elbow.stl scale=0.001 0.001 0.001
- link arm_right_lower_flex_link: geometry collision cylinder length=0.300 radius=0.042; visual mesh filename=package://sobit_home_description/meshes/arm/arm_lower_botto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 scale=0.001 0.001 0.001
- link arm_right_shoulder_tilt_link: geometry collision cylinder length=0.100 radius=0.089; visual mesh filename=package://sobit_home_description/meshes/arm/arm_shoulder.stl scale=0.001 0.001 0.001
- link arm_right_upper_flex_link: geometry collision cylinder length=0.170 radius=0.03; visual mesh filename=package://sobit_home_description/meshes/arm/arm_upper_flex.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 scale=0.001 0.001 0.001
- link arm_right_upper_roll_link: geometry collision cylinder length=0.1285 radius=0.071; visual mesh filename=package://sobit_home_description/meshes/arm/arm_upper_roll.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 scale=0.001 0.001 0.001
- link arm_right_wrist_roll_link: geometry collision box size=0.108 0.0826 0.0645; visual mesh filename=package://sobit_home_description/meshes/arm/arm_wrist_roll.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 scale=0.001 0.001 0.001
- link arm_right_wrist_tilt_link: geometry collision cylinder length=0.0453 radius=0.04; visual mesh filename=package://sobit_home_description/meshes/arm/arm_wrist_tilt.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 scale=0.001 0.001 0.001
- link body_lift_link: geometry collision box size=0.15 0.35 0.15; visual mesh filename=package://sobit_home_description/meshes/body/body_cover.dae
- link body_link: geometry collision box size=0.13 0.13 1.05; visual mesh filename=package://sobit_home_description/meshes/body/lift_w_cover.s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
- link hand_left_camera_base_link: geometry collision box size=0.05 0.05 0.05; visual mesh filename=package://sobit_home_description/meshes/sensor/hand_cam_bas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 scale=0.001 0.001 0.001
- link hand_left_camera_link: geometry collision box size=0.05 0.05 0.05; visual mesh filename=package://sobit_home_description/meshes/sensor/cam_elp.stl scale=0.001 0.001 0.001
- link hand_left_cmc_link: geometry visual mesh filename=package://sobit_home_description/meshes/hand/hand_base.stl scale=0.001 0.001 0.001
- link hand_left_finger_c_ip_link: geometry collision box size=0.022 0.031 0.0334; visual mesh filename=package://sobit_home_description/meshes/hand/thumb_distal_p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 scale=0.001 0.001 0.001
- link hand_left_finger_c_mcp_link: geometry collision box size=0.022 0.031 0.034; visual mesh filename=package://sobit_home_description/meshes/hand/thumb_middle_p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 scale=0.001 0.001 0.001
- link hand_left_finger_l_dip_link: geometry collision box size=0.022 0.031 0.035; visual mesh filename=package://sobit_home_description/meshes/hand/distal_pharanx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 scale=0.001 0.001 0.001
- link hand_left_finger_l_mcp_link: geometry visual mesh filename=package://sobit_home_description/meshes/hand/switching_gear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 scale=0.001 0.001 0.001
- link hand_left_finger_l_pip_link: geometry collision box size=0.022 0.031 0.030; visual mesh filename=package://sobit_home_description/meshes/hand/middle_pharanx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 scale=0.001 0.001 0.001
- link hand_left_finger_r_dip_link: geometry collision box size=0.022 0.031 0.035; visual mesh filename=package://sobit_home_description/meshes/hand/distal_pharanx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 scale=0.001 0.001 0.001
- link hand_left_finger_r_mcp_link: geometry visual mesh filename=package://sobit_home_description/meshes/hand/switching_gear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 scale=0.001 0.001 0.001
- link hand_left_finger_r_pip_link: geometry collision box size=0.022 0.031 0.030; visual mesh filename=package://sobit_home_description/meshes/hand/middle_pharanx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 scale=0.001 0.001 0.001
- link hand_right_camera_base_link: geometry collision box size=0.05 0.05 0.05; visual mesh filename=package://sobit_home_description/meshes/sensor/hand_cam_bas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 scale=0.001 0.001 0.001
- link hand_right_camera_link: geometry collision box size=0.05 0.05 0.05; visual mesh filename=package://sobit_home_description/meshes/sensor/cam_elp.stl scale=0.001 0.001 0.001
- link hand_right_cmc_link: geometry visual mesh filename=package://sobit_home_description/meshes/hand/hand_base.stl scale=0.001 0.001 0.001
- link hand_right_finger_c_ip_link: geometry collision box size=0.022 0.031 0.0334; visual mesh filename=package://sobit_home_description/meshes/hand/thumb_distal_p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 scale=0.001 0.001 0.001
- link hand_right_finger_c_mcp_link: geometry collision box size=0.022 0.031 0.034; visual mesh filename=package://sobit_home_description/meshes/hand/thumb_middle_p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 scale=0.001 0.001 0.001
- link hand_right_finger_l_dip_link: geometry collision box size=0.022 0.031 0.035; visual mesh filename=package://sobit_home_description/meshes/hand/distal_pharanx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 scale=0.001 0.001 0.001
- link hand_right_finger_l_mcp_link: geometry visual mesh filename=package://sobit_home_description/meshes/hand/switching_gear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 scale=0.001 0.001 0.001
- link hand_right_finger_l_pip_link: geometry collision box size=0.022 0.031 0.030; visual mesh filename=package://sobit_home_description/meshes/hand/middle_pharanx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 scale=0.001 0.001 0.001
- link hand_right_finger_r_dip_link: geometry collision box size=0.022 0.031 0.035; visual mesh filename=package://sobit_home_description/meshes/hand/distal_pharanx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 scale=0.001 0.001 0.001
- link hand_right_finger_r_mcp_link: geometry visual mesh filename=package://sobit_home_description/meshes/hand/switching_gear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 scale=0.001 0.001 0.001
- link hand_right_finger_r_pip_link: geometry collision box size=0.022 0.031 0.030; visual mesh filename=package://sobit_home_description/meshes/hand/middle_pharanx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 scale=0.001 0.001 0.001
- link head_base_link: geometry collision box size=0.15 0.125 0.01; visual mesh filename=package://sobit_home_description/meshes/head/neck_base.stl scale=0.001 0.001 0.001
- link head_camera_color_screw_frame: geometry visual mesh filename=package://orbbec_description/meshes/gemini335L_336L/camera_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
- link head_camera_link: geometry visual mesh filename=package://orbbec_description/meshes/gemini335L_336L/base_li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
- link head_pan_link: geometry collision cylinder length=0.0092 radius=0.0325; visual mesh filename=package://sobit_home_description/meshes/head/neck.stl scale=0.001 0.001 0.001
- link head_tilt_link: geometry collision box size=0.155 0.278 0.2; visual mesh filename=package://sobit_home_description/meshes/head/ear.dae
- link lidar_back_base_link: geometry collision box size=0.0941 0.05 0.158; visual mesh filename=package://sobit_home_description/meshes/sensor/lidar_stand_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 scale=0.001 0.001 0.001
- link lidar_back_laser_mount: geometry visual mesh filename=package://urg_node/meshes/hokuyo_ust.stl
- link lidar_front_base_link: geometry collision box size=0.0941 0.05 0.158; visual mesh filename=package://sobit_home_description/meshes/sensor/lidar_stand_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 scale=0.001 0.001 0.001
- link lidar_front_laser_mount: geometry visual mesh filename=package://urg_node/meshes/hokuyo_ust.stl
- link mic_base_link: geometry visual mesh filename=package://sobit_home_description/meshes/sensor/mic_base.stl scale=0.001 0.001 0.001
- link mic_link: geometry visual mesh filename=package://sobit_home_description/meshes/sensor/mic_mount.dae; visual mesh filename=package://sobit_home_description/meshes/sensor/mic_rode.stl scale=0.001 0.001 0.001
- link plate_bottom_link: geometry collision box size=0.47 0.19 0.20; visual mesh filename=package://sobit_home_description/meshes/body/mobile_platfor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 scale=0.001 0.001 0.001
- link plate_cover_link: geometry collision box size=0.01 0.575 0.470; collision box size=0.01 0.575 0.470
- link plate_middle_link: geometry collision box size=0.47 0.47 0.02; visual mesh filename=package://sobit_home_description/meshes/body/mobile_platfor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 scale=0.001 0.001 0.001
- link plate_top_link: geometry collision box size=0.47 0.47 0.02; visual mesh filename=package://sobit_home_description/meshes/body/mobile_platfor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 scale=0.001 0.001 0.001
- link wheel_drive_b_l_link: geometry collision cylinder length=0.035 radius=0.075; visual mesh filename=package://sobit_home_description/meshes/wheel/wheel_drive.s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 scale=0.001 0.001 0.001
- link wheel_drive_b_r_link: geometry collision cylinder length=0.035 radius=0.075; visual mesh filename=package://sobit_home_description/meshes/wheel/wheel_drive.s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 scale=0.001 0.001 0.001
- link wheel_drive_f_l_link: geometry collision cylinder length=0.035 radius=0.075; visual mesh filename=package://sobit_home_description/meshes/wheel/wheel_drive.s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 scale=0.001 0.001 0.001
- link wheel_drive_f_r_link: geometry collision cylinder length=0.035 radius=0.075; visual mesh filename=package://sobit_home_description/meshes/wheel/wheel_drive.s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 scale=0.001 0.001 0.001
- link wheel_steer_b_l_link: geometry collision box size=0.1 0.1 0.06185; visual mesh filename=package://sobit_home_description/meshes/wheel/wheel_steer.s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 scale=0.001 0.001 0.001
- link wheel_steer_b_r_link: geometry collision box size=0.1 0.1 0.06185; visual mesh filename=package://sobit_home_description/meshes/wheel/wheel_steer.s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 scale=0.001 0.001 0.001
- link wheel_steer_base_b_l_link: geometry collision cylinder length=0.0797 radius=0.075; visual mesh filename=package://sobit_home_description/meshes/wheel/wheel_base.stl scale=0.001 0.001 0.001
- link wheel_steer_base_b_r_link: geometry collision cylinder length=0.0797 radius=0.075; visual mesh filename=package://sobit_home_description/meshes/wheel/wheel_base.stl scale=0.001 0.001 0.001
- link wheel_steer_base_f_l_link: geometry collision cylinder length=0.0797 radius=0.075; visual mesh filename=package://sobit_home_description/meshes/wheel/wheel_base.stl scale=0.001 0.001 0.001
- link wheel_steer_base_f_r_link: geometry collision cylinder length=0.0797 radius=0.075; visual mesh filename=package://sobit_home_description/meshes/wheel/wheel_base.stl scale=0.001 0.001 0.001
- link wheel_steer_f_l_link: geometry collision box size=0.1 0.1 0.06185; visual mesh filename=package://sobit_home_description/meshes/wheel/wheel_steer.s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 scale=0.001 0.001 0.001
- link wheel_steer_f_r_link: geometry collision box size=0.1 0.1 0.06185; visual mesh filename=package://sobit_home_description/meshes/wheel/wheel_steer.s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 scale=0.001 0.001 0.001
Joints:
- removed joint arm_left_elbow_sub_joint
- removed joint arm_left_upper_flex_sub_joint
- removed joint arm_left_upper_roll_sub_joint
- removed joint arm_right_elbow_sub_joint
- removed joint arm_right_upper_flex_sub_joint
- removed joint arm_right_upper_roll_sub_joint

Commit message: [FIX] parent the plate cover to plate_middle_link, not the massless base_footprint
Isaac Sim's importer anchors fixed joints hanging off massless frames to the
world, which split the cover into a second articulation root. World pose is
unchanged (0.496258 = 0.271358 + 0.2249). The tracked URDF is edited in place
because it is not a regeneration of the current xacro.

File: sobit_home_description/robots/sobit_home_robot.urdf (robot description, URDF)
Before this commit: robot sobit_home, 86 links, 85 joints
Joints:
- joint plate_cover_joint: origin xyz=0.0 0.0 0.49625800000000003 rpy=0.0 0.0 0.0 -> xyz=0.0 0.0 0.22490000000000004 rpy=0.0 0.0 0.0; parent base_footprint -> plate_middle_link

File: sobit_home_description/urdf/body/plate.urdf.xacro (robot description, xacro)
@@ -84,7 +84,9 @@
       </inertial>
     </link>
+    <!-- Parent is the middle plate (a massive link), not base_footprint: Isaac Sim pins
+         fixed joints hanging off massless frames to the world. Same world pose. -->
     <joint name="${prefix}_cover_joint" type="fixed">
-      <origin xyz="0.0 0.0 ${0.421258 + 0.15/2}" rpy="0.0 0.0 0.0" />
-      <parent link="base_footprint" />
+      <origin xyz="0.0 0.0 ${0.421258 + 0.15/2 - 0.271358}" rpy="0.0 0.0 0.0" />
+      <parent link="${prefix}_middle_link" />
       <child link="${prefix}_cover_link" />
     </joint>
